File: NumPad-MUSB/NumPad.brd (EAGLE design)
At the start: 99.7 x 121.9 mm, 141 parts, among them IC1 MEGA8-AI, J1 J, J10 J, J11 J, J2 J, J3 J, J4 J, J5 J, J6 J, J7 J, J8 J, J9 J

Commit message: add led.c
Parts:
- removed C1, C2, C3: (no value), rcl:C0805
- removed ISP1: (no value), con-lstb:MA03-2
- removed J1, J10, J11, J3, J4, J5, J6, J7, J8, J9: J, detali:R1206W
- removed JA87, JB87, SJ1: (no value), detali:SJ
- removed Q1: (no value), crystal:HC49/S
- removed S87: Num, cherrymx:CHERRY-MX-4P
- added IC2: 74AC00N, 74xx-eu:DIL14
- added R2, R3: (no value), rcl:R0805
- added S1: (no value), switch-omron:B3F-31XX
- added SV1: (no value), con-lstb:MA08-1
- IC1: value MEGA8-AI -> 74AC138N; device atmel:TQFP32-08 -> 74xx-eu:DIL16
- moved IC1 78.1 mm to (67.9, 135.9), flipped to the top, turned to 0 degrees
- moved R1 73.2 mm to (40.6, 135.3), turned to 270 degrees
- moved J2 66.5 mm to (-3.17, 129.5)
- moved D108 26.7 mm to (53.3, 32.7), turned to 0 degrees
- moved JB107 26.2 mm to (82.5, 47.0), turned to 90 degrees
- moved D87 24.7 mm to (25.6, 126.8), turned to 0 degrees
- moved D107 22.3 mm to (69.2, 22.2), turned to 0 degrees
- moved D89 14.7 mm to (45.1, 125.1), turned to 90 degrees
- moved D110 14.6 mm to (64.1, 18.4)
- moved D109 14.5 mm to (58.4, 14.0), turned to 0 degrees
- moved JA92 9.25 mm to (9.53, 94.0), turned to 0 degrees
- moved D96 8.98 mm to (26.0, 81.9), turned to 90 degrees
- moved D100 8.90 mm to (33.3, 51.6)
- moved JA100 8.26 mm to (9.53, 55.9), turned to 0 degrees
- moved JA104 8.25 mm to (9.53, 36.8), turned to 0 degrees
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Connections:
- removed net AVCC: IC1.18
- removed net MISO: IC1.16, ISP1.1
- removed net MOSI: IC1.15, ISP1.4
- removed net N$15: D96.C, J2.1, J3.2
- removed net N$17: D109.C, J4.2
- removed net N$18: D105.C, J4.1, J5.2
- removed net N$19: D101.C, J5.1, J6.2
- removed net N$20: D97.C, J6.1, J7.2
- removed net N$21: D88.C, D93.C, J7.1, J8.2
- removed net N$23: D106.C, D110.C, J9.2
- removed net N$24: D98.C, J10.1, J11.2
- removed net N$270: JB87.2, S87.SW1
- removed net N$272: JA87.1, S87.SW2
- removed net N$3: IC1.1, JA103.2, JA104.2, JA105.2, JA106.2
- removed net N$338: C1.2, IC1.7, Q1.2
- removed net N$339: C2.2, IC1.8, Q1.1
- removed net N$4: IC1.32, JA100.2, JA101.2, JA102.2, JA99.2
- removed net N$5: IC1.31, JA95.2, JA96.2, JA97.2, JA98.2
- removed net RESET: ISP1.5, SJ1.1
- new net N$11: IC2.8
- new net N$33: D87.C, D89.C, D90.C, IC1.15
- new net N$34: D101.C, D91.C, D96.C, IC1.12
- new net N$35: D100.C, D105.C, D95.C, IC1.11
- new net N$36: D103.C, D106.C, D108.C, IC1.9
- net +5V: now also IC1.16, IC2.14, R2.2, R3.2; no longer C3.1, IC1.4, ISP1.2
- net GND: now also IC1.4, IC1.8, IC2.7; no longer C1.1, C2.1, C3.2, IC1.21, IC1.3, ISP1.6
- net N$1: now also D92.C, D97.C, D98.C, IC1.13; no longer IC1.2, JA108.2, JA109.2, JA110.2, JB107.1
- net N$10: now also IC1.1; no longer IC1.17
- net N$12: now also IC2.6; no longer D104.C, D108.C, J1.2
- net N$13: now also IC2.3; no longer D87.C, D92.C, IC1.27, J3.1
- net N$14: now also IC2.1, IC2.2, JA100.2, JA104.2, JA108.2, JA109.2, JA88.2, JA92.2, JA96.2, R1.1, S1.2; no longer IC1.28, J8.1
- net N$16: now also D88.C, D93.C, IC1.14; no longer D89.C, IC1.25, J11.1
- net N$22: now also IC2.10, IC2.9, JA103.2, JA90.2, JA91.2, JA94.2, JA95.2, JA98.2, JA99.2, JB107.1, R3.1; no longer D102.C, J10.2, J9.1
- net N$268: now also S1.1; no longer JB87.1
- net N$6: now also IC1.3; no longer IC1.30, JA91.2, JA92.2, JA93.2, JA94.2
- net N$7: now also IC2.4, IC2.5, JA101.2, JA102.2, JA105.2, JA106.2, JA110.2, JA93.2, JA97.2, R2.1; no longer IC1.26, JA87.2, JA88.2, JA90.2
- net N$8: now also IC1.2; no longer D100.C, J1.1, J2.2
- net N$9: now also D102.C, D104.C, D99.C, IC1.10; no longer IC1.29, R1.1, SJ1.2
- net SCK: now also D109.C, D110.C, IC1.7; no longer D103.C, D90.C, D91.C, D95.C, D99.C, IC1.24, ISP1.3
Routing:
- net N$1: track 147.0 -> 0.00 mm
- net N$3: track 140.4 -> 0.00 mm
- net N$14: track 28.1 -> 150.5 mm
- net N$4: track 116.9 -> 0.00 mm
- net N$16: track 147.1 -> 33.5 mm
- net N$7: track 65.5 -> 166.9 mm
- net N$5: track 100.3 -> 0.00 mm
- net SCK: track 231.3 -> 139.5 mm
- net N$22: track 17.8 -> 107.8 mm
- net N$6: track 81.2 -> 0.00 mm
- net N$13: track 51.7 -> 0.00 mm
- net N$36: track 0.00 -> 36.6 mm
- net N$21: track 35.8 -> 0.00 mm
- net N$24: track 30.4 -> 0.00 mm
- net N$331: track 11.5 -> 37.8 mm
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Other:
- board size 99.7 x 121.9 mm -> 95.4 x 133.4 mm

Commit message: pcb np
Parts:
- removed IC2: 74AC00N, 74xx-eu:DIL14
- removed U$87: (no value), kbmx:18X18
- added IC3: 74HC10N, detali:DIL14
- added J1, J10, J11, J12, J13, J14, J15, J16, J17, J3, J4, J5, J6, J7, J8, J9: J, detali:R1206W
- added LED1: (no value), detali:LED5MM
- added R4, R5: (no value), rcl:R1206W
- IC1: value 74AC138N -> 74HC138N; device 74xx-eu:DIL16 -> detali:DIL16
- R1, R2, R3: device rcl:R0805 -> rcl:R1206W
- S1: device switch-omron:B3F-31XX -> detali:B3F-31XX
- SV1: device con-lstb:MA08-1 -> detali:MA09-1
- moved J2 87.7 mm to (46.4, 57.1), turned to 90 degrees
- moved R1 33.7 mm to (6.99, 134.9), turned to 90 degrees
- moved SV1 33.4 mm to (49.8, 141.3)
- moved R3 33.0 mm to (14.6, 141.8), turned to 0 degrees
- moved D107 29.2 mm to (70.5, 51.4), turned to 315 degrees
- moved D104 21.8 mm to (47.6, 47.0), turned to 0 degrees
- moved R2 21.0 mm to (12.1, 134.3), turned to 0 degrees
- moved D96 17.3 mm to (27.9, 64.8), turned to 0 degrees
- moved D87 16.9 mm to (40.3, 135.1)
- moved D92 16.7 mm to (28.3, 84.1), turned to 0 degrees
- moved S1 16.5 mm to (32.4, 136.8)
- moved D99 11.5 mm to (70.5, 71.4), turned to 180 degrees
- moved D102 7.24 mm to (58.4, 52.1), turned to 0 degrees
- moved IC1 6.16 mm to (74.0, 134.6), turned to 195 degrees
- moved JB92 5.85 mm to (21.0, 92.1), turned to 270 degrees
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Connections:
- new net COLN1: IC3.12, SV1.2
- new net COLN2: IC3.6, J15.1
- new net COLN3: IC3.8, SV1.3
- new net N$15: J5.2, J6.1
- new net N$17: IC3.10, IC3.11, IC3.9, J14.1, R3.1
- new net N$18: IC1.7, J10.1
- new net N$19: J10.2, J9.1
- new net N$20: J11.1, J12.1
- new net N$21: J12.2, J13.1
- new net N$23: IC1.9, J13.2
- new net N$24: IC1.6, R4.2
- new net N$26: J14.2, J8.1
- new net N$27: LED1.A, R5.2
- new net N$28: J16.2, SV1.5
- new net N$29: J15.2, J16.1
- new net N$3: D107.C, JB107.1
- new net N$30: J17.2, SV1.4
- new net N$31: J17.1, R5.1
- new net N$4: J1.2, J3.1
- new net N$5: J1.1, J2.2
- net +5V: now also IC3.14, R4.1, SV1.9; no longer IC1.6, IC2.14
- net GND: now also IC3.7, LED1.K, SV1.1; no longer IC2.7
- net N$1: now also J11.2; no longer IC1.13
- net N$10: now also IC1.3, SV1.6; no longer IC1.1
- net N$11: now also IC1.13, J4.2; no longer IC2.8
- net N$12: now also D101.C, D96.C, J5.1; no longer IC2.6
- net N$13: now also J6.2, J7.1; no longer IC2.3
- net N$14: now also IC3.1, IC3.13, IC3.2; no longer IC2.1, IC2.2
- net N$16: now also J9.2; no longer IC1.14
- net N$2: now also D100.C, D105.C, J2.1; no longer D107.A, JA107.2
- net N$22: now also D107.A, J8.2; no longer IC2.10, IC2.9, JB107.1, R3.1
- net N$33: now also IC1.10; no longer IC1.15
- net N$34: now also IC1.11, J7.2; no longer D101.C, D96.C, IC1.12
- net N$35: now also IC1.12, J3.2; no longer D100.C, D105.C, IC1.11
- net N$36: now also IC1.14; no longer IC1.9
- net N$6: now also IC1.1, SV1.8; no longer IC1.3
- net N$7: now also IC3.3, IC3.4, IC3.5; no longer IC2.4, IC2.5
- net N$8: now also SV1.7
- net N$9: now also J4.1; no longer IC1.10
- net SCK: now also IC1.15, JA107.2; no longer D107.C, IC1.7
Routing:
- net N$25: track 0.00 -> 120.0 mm
- net +5V: track 0.00 -> 111.5 mm
- net N$36: track 36.6 -> 130.4 mm
- net N$11: track 0.00 -> 78.3 mm
- net GND: track 12.7 -> 77.0 mm
- net N$1: track 0.00 -> 59.0 mm
- net N$35: track 13.9 -> 61.3 mm
- net N$26: track 0.00 -> 44.8 mm
- net N$34: track 0.00 -> 39.1 mm
- net N$12: track 0.00 -> 38.4 mm
- net N$9: track 0.00 -> 37.5 mm
- net COLN1: track 0.00 -> 36.7 mm
- net N$60: track 0.00 -> 34.7 mm
- net N$10: track 0.00 -> 30.0 mm
- net N$8: track 0.00 -> 28.9 mm
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Other:
- board size 95.4 x 133.4 mm -> 85.1 x 137.2 mm

Commit message: num src
Parts:
- added C1: (no value), rcl:C1206
- S1: value (none) -> NumLock
- moved R4 1.27 mm to (72.4, 134.9)
Connections:
- net +5V: now also C1.1
- net GND: now also C1.2
Routing:
- net N$25: track 120.0 -> 0.00 mm
- net +5V: track 111.5 -> 126.1 mm
- net GND: track 77.0 -> 79.6 mm
- net N$24: track 5.23 -> 3.96 mm
Changed lines of the file:
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@@
 <setting verticaltext="up"/>
 </settings>
-<grid distance="12.5" unitdist="mil" unit="mil" style="lines" multiple="1" display="yes" altdistance="0.025" altunitdist="inch" altunit="inch"/>
+<grid distance="25" unitdist="mil" unit="mil" style="lines" multiple="1" display="yes" altdistance="0.025" altunitdist="inch" altunit="inch"/>
 <layers>
 <layer number="1" name="Top" color="4" fill="1" visible="yes" active="yes"/>
@@
 <wire x1="88.265" y1="146.05" x2="88.265" y2="8.89" width="0.2" layer="20"/>
 <wire x1="3.175" y1="146.05" x2="3.175" y2="8.89" width="0.2" layer="20"/>
-<dimension x1="59.69" y1="151.13" x2="78.74" y2="151.13" x3="69.215" y3="163.83" layer="1" dtype="horizontal"/>
-<dimension x1="89.535" y1="145.7325" x2="89.8525" y2="125.73" x3="100.965" y3="135.73125" layer="1" dtype="vertical"/>
+<dimension x1="3.175" y1="147.955" x2="88.265" y2="151.13" x3="45.72" y3="163.83" layer="1" dtype="horizontal"/>
+<dimension x1="89.535" y1="146.05" x2="90.4875" y2="8.89" x3="100.965" y3="77.47" layer="1" dtype="vertical"/>
 <circle x="64.77" y="32.385" radius="3" width="0.254" layer="20"/>
 <circle x="64.77" y="108.585" radius="3" width="0.254" layer="20"/>
@@
 <element name="J2" library="detali" package="R1206W" value="J" x="46.355" y="57.15" rot="MR90"/>
 <element name="IC1" library="detali" package="DIL16" value="74HC138N" x="73.9775" y="134.62" rot="R195"/>
-<element name="S1" library="detali" package="B3F-31XX" value="" x="32.385" y="136.8425" rot="R180">
+<element name="S1" library="detali" package="B3F-31XX" value="NumLock" x="32.385" y="136.8425" rot="R180">
 <attribute name="OC_NEWARK" value="36M3582" x="32.385" y="136.8425" size="1.778" layer="27" rot="R180" display="off"/>
 <attribute name="MPN" value="B3F-3100" x="32.385" y="136.8425" size="1.778" layer="27" rot="R180" display="off"/>
@@
 <element name="J12" library="detali" package="R1206W" value="J" x="47.0535" y="126.8095" rot="MR90"/>
 <element name="J13" library="detali" package="R1206W" value="J" x="52.3875" y="130.81" rot="MR180"/>
-<element name="R4" library="rcl" package="R1206W" value="" x="73.66" y="134.9375" rot="MR0"/>
+<element name="R4" library="rcl" package="R1206W" value="" x="72.39" y="134.9375" rot="MR0"/>
 <element name="LED1" library="detali" package="LED5MM" value="" x="36.195" y="131.445" rot="R180"/>
 <element name="R5" library="rcl" package="R1206W" value="" x="41.275" y="131.445" rot="MR0"/>
@@
 <element name="J16" library="detali" package="R1206W" value="J" x="48.26" y="136.525" rot="MR90"/>
 <element name="J17" library="detali" package="R1206W" value="J" x="45.72" y="136.525" rot="MR90"/>
+<element name="C1" library="rcl" package="C1206" value="" x="62.23" y="133.0325" rot="MR90"/>
 </elements>
 <signals>
@@
 <contactref element="D96" pad="A"/>
 <contactref element="JB96" pad="1"/>
-<wire x1="26.24" y1="64.77" x2="22.86" y2="68.15" width="0.6096" layer="16"/>
-<wire x1="22.86" y1="68.15" x2="22.86" y2="70.358" width="0.6096" layer="16"/>
-<wire x1="22.86" y1="70.358" x2="20.955" y2="72.263" width="0.6096" layer="16"/>
+<wire x1="26.24" y1="64.77" x2="22.5425" y2="68.4675" width="0.6096" layer="16"/>
+<wire x1="22.5425" y1="68.4675" x2="22.5425" y2="70.358" width="0.6096" layer="16"/>
+<wire x1="22.5425" y1="70.358" x2="20.955" y2="72.263" width="0.6096" layer="16"/>
 </signal>
 <signal name="N$296">
@@
 <wire x1="69.5325" y1="140.97" x2="64.51359375" y2="139.7" width="0.6096" layer="1"/>
 <wire x1="64.51359375" y1="139.7" x2="63.87859375" y2="138.1125" width="0.6096" layer="1"/>
+<contactref element="C1" pad="2"/>
+<wire x1="62.23" y1="134.4325" x2="64.40431875" y2="135.999275" width="0.6096" layer="16"/>
 </signal>
 <signal name="+5V">
@@
 <wire x1="84.1375" y1="141.9225" x2="84.1375" y2="136.05004375" width="0.6096" layer="16"/>
 <wire x1="84.1375" y1="136.05004375" x2="83.550678125" y2="133.240721875" width="0.6096" layer="16"/>
-<wire x1="75.159" y1="134.9375" x2="83.550678125" y2="134.9375" width="0.6096" layer="16"/>
+<wire x1="73.889" y1="134.9375" x2="83.550678125" y2="134.9375" width="0.6096" layer="16"/>
 <wire x1="83.550678125" y1="134.9375" x2="83.550678125" y2="133.240721875" width="0.6096" layer="16"/>
 <wire x1="17.144696875" y1="144.5096125" x2="12.4296125" y2="144.5096125" width="0.6096" layer="16"/>
@@
 <wire x1="9.525" y1="141.605" x2="9.525" y2="138.43" width="0.6096" layer="16"/>
 <wire x1="13.106" y1="141.76375" x2="11.1125" y2="143.1925" width="0.6096" layer="16"/>
+<contactref element="C1" pad="1"/>
+<wire x1="62.23" y1="131.6325" x2="66.545" y2="131.6325" width="0.6096" layer="16"/>
+<wire x1="66.545" y1="131.6325" x2="68.2625" y2="133.0325" width="0.6096" layer="16"/>
+<wire x1="68.2625" y1="133.0325" x2="71.755" y2="133.0325" width="0.6096" layer="16"/>
+<wire x1="71.755" y1="133.0325" x2="73.66" y2="133.6675" width="0.6096" layer="16"/>
+<wire x1="73.66" y1="133.6675" x2="73.889" y2="134.9375" width="0.6096" layer="16"/>
 </signal>
 <signal name="N$14">
@@
 <contactref element="IC3" pad="6"/>
 <wire x1="22.225" y1="130.81" x2="23.1775" y2="127.635" width="0.6096" layer="16"/>
-<wire x1="23.1775" y1="127.635" x2="37.465" y2="127.635" width="0.6096" layer="16"/>
+<wire x1="23.1775" y1="127.635" x2="38.1885" y2="127.635" width="0.6096" layer="16"/>
 <contactref element="J15" pad="1"/>
-<wire x1="37.465" y1="127.635" x2="38.1885" y2="127.635" width="0.4064" layer="16"/>
-<wire x1="38.1885" y1="127.635" x2="39.776" y2="129.2225" width="0.4064" layer="16"/>
+<wire x1="38.1885" y1="127.635" x2="39.776" y2="129.2225" width="0.6096" layer="16"/>
 </signal>
 <signal name="COLN1">
@@
 <contactref element="IC1" pad="6"/>
 <contactref element="R4" pad="2"/>
-<wire x1="72.161" y1="134.9375" x2="69.311221875" y2="134.9375" width="0.6096" layer="16"/>
+<wire x1="70.891" y1="134.9375" x2="69.311221875" y2="134.9375" width="0.6096" layer="16"/>
 <wire x1="69.311221875" y1="134.9375" x2="69.311221875" y2="137.314075" width="0.6096" layer="16"/>
 </signal>
@@
 <wire x1="53.975" y1="135.89" x2="52.3875" y2="141.2875" width="0.4064" layer="16"/>
 </signal>
-<signal name="N$25">
-<wire x1="-13.6525" y1="149.225" x2="106.3625" y2="149.225" width="0.4064" layer="1"/>
-</signal>
 <signal name="N$27">

Commit message: edit map
Parts:
- added C2: (no value), rcl:C1206
- added D1, D2: LL4148, detali:SOD80C
- 3D2: value 74HC10N -> К155ЛА4
- moved R1 7.31 mm to (6.67, 127.6), turned to 0 degrees
- renumbered IC1 to 3D1, IC3 to 3D2
Connections:
- new net N$38: D1.A, D2.C
- new net N$39: 3D2.14, C2.1, D1.C
- net +5V: now also D2.A; no longer 3D2.14
- net GND: now also C2.2
Routing:
- net GND: track 79.6 -> 92.1 mm
- net +5V: track 126.1 -> 137.7 mm
- net N$39: track 0.00 -> 9.34 mm
- net N$38: track 0.00 -> 3.54 mm

Commit message: err
Parts:
- added U$1: (no value), kbmx:18X18
- S107B: device cherrymx:CHERRY-MX -> cherrymx:CHERRY-MX-4P
- moved JB90 38.9 mm to (78.7, 151.1), turned to 90 degrees
- moved R1 38.4 mm to (21.3, 163.2)
- moved D2 38.1 mm to (21.6, 166.4), turned to 180 degrees
- moved JA109 37.4 mm to (45.1, 49.5), turned to 0 degrees
- moved D90 37.0 mm to (77.5, 156.5)
- moved D1 35.9 mm to (21.3, 169.5)
- moved JA110 35.5 mm to (64.1, 50.2)
- moved JB91 35.2 mm to (90.8, 144.1)
- moved D88 35.2 mm to (49.8, 140.3)
- moved D93 35.2 mm to (58.4, 134.0)
- moved J11 35.2 mm to (60.6, 134.3)
- moved J12 35.2 mm to (62.3, 158.6)
- moved J6 35.2 mm to (62.9, 134.3)
- moved J8 35.2 mm to (64.4, 158.6)
- moved J9 35.2 mm to (60.2, 158.6)
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Routing:
- net SCK: track 168.1 -> 177.6 mm
- net N$277: track 9.16 -> 3.20 mm
- net +5V: track 137.7 -> 132.5 mm
- net N$319: track 34.4 -> 39.6 mm
- net N$278: track 3.05 -> 6.36 mm
- net N$11: track 78.3 -> 81.5 mm
- net N$36: track 130.4 -> 132.6 mm
- net N$35: track 61.3 -> 59.3 mm
- net N$317: track 3.50 -> 5.43 mm
- net N$33: track 42.7 -> 40.9 mm
- net N$14: track 176.8 -> 178.4 mm
- net N$3: track 11.8 -> 13.0 mm
- net N$34: track 39.1 -> 38.1 mm
- net N$7: track 190.9 -> 189.9 mm
- net COLN3: track 24.6 -> 23.7 mm
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Other:
- board size 85.1 x 137.2 mm -> 88.3 x 140.3 mm

Commit message: 16-07-28
Parts:
- added U$10, U$11, U$12, U$13, U$14, U$15, U$16, U$17, U$18, U$19, U$20, U$21, U$22, U$23, U$24, U$3, U$4, U$5, U$6, U$7, U$8, U$9: (no value), kbmxco:KEY
- added U$2, U$25: (no value), kbmxco:NUMENTER
- added U$26: (no value), kbmxco:SIZE132
- SV1: device detali:MA09-1 -> detali:FE09
- moved D109 1.71 mm to (74.3, 47.3)
- moved JB99 1.27 mm to (92.1, 105.4), turned to 180 degrees
- moved C1 1.14 mm to (78.1, 163.8), turned to 75 degrees
Routing:
- net N$11: track 81.5 -> 78.2 mm
- net N$319: track 39.6 -> 36.7 mm
- net +5V: track 132.5 -> 134.2 mm
- net N$35: track 59.3 -> 57.7 mm
- net N$8: track 28.7 -> 30.1 mm
- net N$36: track 132.6 -> 134.0 mm
- net N$333: track 14.9 -> 16.2 mm
- net N$10: track 29.8 -> 31.1 mm
- net N$6: track 27.8 -> 29.0 mm
- net N$5: track 27.6 -> 28.7 mm
- net N$304: track 6.52 -> 5.52 mm
- net SCK: track 177.6 -> 176.6 mm
- net N$34: track 38.1 -> 37.1 mm
- net N$24: track 3.96 -> 2.99 mm
- net N$18: track 15.5 -> 16.4 mm
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Other:
- board size 88.3 x 140.3 mm -> 107.2 x 166.4 mm

Commit message: upd
Parts:
- removed U$25: (no value), kbmxco:NUMENTER
- moved 3D1 24.8 mm to (90.8, 141.6)
- moved 3D2 24.8 mm to (34.0, 141.6)
- moved C1 24.8 mm to (79.7, 139.1)
- moved C2 24.8 mm to (31.4, 149.5)
- moved D87 24.8 mm to (57.2, 142.0)
- moved D88 24.8 mm to (51.4, 115.6)
- moved D90 24.8 mm to (79.1, 131.8)
- moved D93 24.8 mm to (60.0, 109.2)
- moved J11 24.8 mm to (62.2, 109.5)
- moved J12 24.8 mm to (63.9, 133.8)
- moved J13 24.8 mm to (69.2, 137.8)
- moved J16 24.8 mm to (65.1, 143.5)
- moved J17 24.8 mm to (62.5, 143.5)
- moved J6 24.8 mm to (64.5, 109.5)
- moved J8 24.8 mm to (66.0, 133.8)
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Routing:
- net GND: track 91.7 -> 97.0 mm, vias 0 -> 3
- net N$39: track 8.78 -> 9.31 mm
Other:
- board size 107.2 x 166.4 mm -> 88.9 x 142.9 mm

Commit message: + stab reserv
Parts:
- moved D110 5.65 mm to (79.7, 23.8)
- moved D109 1.85 mm to (74.3, 21.6)
- moved JA91 0.90 mm to (84.8, 121.0)
- moved JB110 0.45 mm to (79.4, 27.0), turned to 270 degrees
- moved JA95 0.45 mm to (85.1, 101.3)
- moved D98 0.32 mm to (79.7, 90.5)
- moved J3 0.32 mm to (87.9, 96.8)
Routing:
- net SCK: track 176.6 -> 186.6 mm
- net N$333: track 16.2 -> 14.1 mm
- net N$335: track 1.98 -> 2.78 mm
- net N$282: track 2.43 -> 3.19 mm
