File: NumPad-MUSB/NumPad.brd (EAGLE design)
At the start: 88.9 x 142.9 mm, 174 parts, among them J1 J, J10 J, J11 J, J12 J, J13 J, J14 J, J15 J, J16 J, J17 J, J2 J, J3 J, J4 J, J5 J, J6 J, J7 J, J8 J, J9 J

Commit message: f np1
Parts:
- moved D2 8.58 mm to (27.9, 148.9)
- moved R3 6.70 mm to (38.1, 149.4), turned to 180 degrees
- moved JA105 1.59 mm to (47.3, 45.4)
- moved R1 1.35 mm to (23.8, 140.0), turned to 90 degrees
- moved D1 0.95 mm to (23.8, 145.4), turned to 270 degrees
- moved JB88 0.64 mm to (41.6, 121.9)
- moved J14 0.32 mm to (36.2, 141.6)
- moved 3D2 0.32 mm to (34.0, 141.3)
- moved J15 0.32 mm to (58.1, 136.5)
- moved R2 0.32 mm to (28.9, 141.0)
- moved R5 0.32 mm to (58.1, 138.7)
Routing:
- net +5V: track 134.3 -> 136.4 mm
- net COLN1: track 35.9 -> 37.8 mm
- net N$39: track 9.31 -> 10.7 mm
- net N$33: track 40.9 -> 42.3 mm
- net N$7: track 189.9 -> 188.7 mm
- net SCK: track 186.6 -> 185.4 mm
- net N$36: track 133.7 -> 132.8 mm
- net N$1: track 58.9 -> 59.6 mm
- net N$304: track 5.52 -> 4.81 mm
- net N$12: track 38.4 -> 39.1 mm
- net N$18: track 16.1 -> 16.7 mm
- net N$26: track 45.6 -> 45.1 mm
- net N$17: track 12.6 -> 12.1 mm
- added copper zone on layer 1, net GND
- added copper zone on layer 1, net N$39
Other:
- board text added: "1"
- board text added: "1176-16"
- board text added: "9"

Commit message: move
Parts:
- R1, R2, R3: value (none) -> 10k
- moved D93 0.45 mm to (59.7, 109.5)
