File: NumPad-MUSB/NumPad.sch (EAGLE design)
At the start: 102 parts, among them IC1 74AC138N, IC2 74AC00N, J2 J

Commit message: pcb np
Parts:
- removed IC2: 74AC00N, 74xx-eu:74AC00N
- added IC3: 74HC10N, detali:74HC10N
- added J1, J10, J11, J12, J13, J14, J15, J16, J17, J3, J4, J5, J6, J7, J8, J9: J, detali:J
- added LED1: (no value), detali:LED5MM
- added R4, R5: (no value), rcl:R-EU_R1206W
- IC1: value 74AC138N -> 74HC138N; device 74xx-eu:74AC138N -> detali:74HC138N
- R1, R2, R3: device rcl:R-EU_R0805 -> rcl:R-EU_R1206W
- S1: device switch-omron:31-XX -> detali:31-XX
- SV1: device con-lstb:MA08-1 -> detali:MA09-1
Connections:
- new net COLN1: IC3A.O, SV1.2
- new net COLN2: IC3B.O, J15.P$1
- new net COLN3: IC3C.O, SV1.3
- new net N$15: J5.P$2, J6.P$1
- new net N$17: IC3C.I0, IC3C.I1, IC3C.I2, J14.P$1, R3.1
- new net N$18: IC1A.Y7, J10.P$1
- new net N$19: J10.P$2, J9.P$1
- new net N$20: J11.P$1, J12.P$1
- new net N$21: J12.P$2, J13.P$1
- new net N$23: IC1A.Y6, J13.P$2
- new net N$24: IC1A.G1, R4.2
- new net N$26: J14.P$2, J8.P$1
- new net N$27: LED1.A, R5.2
- new net N$28: J16.P$2, SV1.5
- new net N$29: J15.P$2, J16.P$1
- new net N$3: D107.C, JB107.1
- new net N$30: J17.P$2, SV1.4
- new net N$31: J17.P$1, R5.1
- new net N$4: J1.P$2, J3.P$1
- new net N$5: J1.P$1, J2.P$2
- net +5V: now also IC3P.VCC, R4.1, SV1.9; no longer IC1A.G1, IC2P.VCC
- net GND: now also IC3P.GND, LED1.C, SV1.1; no longer IC2P.GND
- net N$1: now also J11.P$2; no longer IC1A.Y2
- net N$10: now also IC1A.C, SV1.6; no longer IC1A.A
- net N$11: now also IC1A.Y2, J4.P$2; no longer IC2C.O
- net N$12: now also D101.C, D96.C, J5.P$1; no longer IC2B.O
- net N$13: now also J6.P$2, J7.P$1; no longer IC2A.O
- net N$14: now also IC3A.I0, IC3A.I1, IC3A.I2; no longer IC2A.I0, IC2A.I1
- net N$16: now also J9.P$2; no longer IC1A.Y1
- net N$2: now also D100.C, D105.C, J2.P$1; no longer D107.A, JA107.2
- net N$22: now also D107.A, J8.P$2; no longer IC2C.I0, IC2C.I1, JB107.1, R3.1
- net N$33: now also IC1A.Y5; no longer IC1A.Y0
- net N$34: now also IC1A.Y4, J7.P$2; no longer D101.C, D96.C, IC1A.Y3
- net N$35: now also IC1A.Y3, J3.P$2; no longer D100.C, D105.C, IC1A.Y4
- net N$36: now also IC1A.Y1; no longer IC1A.Y6
- net N$6: now also IC1A.A, SV1.8; no longer IC1A.C
- net N$7: now also IC3B.I0, IC3B.I1, IC3B.I2; no longer IC2B.I0, IC2B.I1
- net N$8: now also SV1.7
- net N$9: now also J4.P$1; no longer IC1A.Y5
- net SCK: now also IC1A.Y0, JA107.2; no longer D107.C, IC1A.Y7
Other:
- moved on the sheet: D100, D102, D103, D104, D105, D106, D107, D108, D109, D110, D95, D99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

Commit message: num src
Parts:
- added C1: (no value), rcl:C-EUC1206
- S1: value (none) -> NumLock
Connections:
- net +5V: now also C1.1
- net GND: now also C1.2
Other:
- moved on the sheet: IC1P, IC3P
Changed lines of the file:
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@@
 <part name="P+1" library="supply1" deviceset="+5V" device=""/>
 <part name="GND1" library="supply1" deviceset="GND" device=""/>
-<part name="S1" library="detali" deviceset="31-XX" device=""/>
+<part name="S1" library="detali" deviceset="31-XX" device="" value="NumLock"/>
 <part name="R1" library="rcl" deviceset="R-EU_" device="R1206W"/>
 <part name="R2" library="rcl" deviceset="R-EU_" device="R1206W"/>
@@
 <part name="J16" library="detali" deviceset="J" device=""/>
 <part name="J17" library="detali" deviceset="J" device=""/>
+<part name="C1" library="rcl" deviceset="C-EU" device="C1206"/>
 </parts>
 <sheets>
@@
 <attribute name="VALUE" x="185.42" y="256.54" size="1.778" layer="96" rot="R180"/>
 </instance>
-<instance part="IC1" gate="P" x="317.5" y="170.18"/>
-<instance part="P+3" gate="1" x="320.04" y="185.42" smashed="yes">
-<attribute name="VALUE" x="325.12" y="187.96" size="1.778" layer="96" rot="R180"/>
-</instance>
-<instance part="GND2" gate="1" x="320.04" y="154.94"/>
+<instance part="IC1" gate="P" x="-7.62" y="127"/>
+<instance part="P+3" gate="1" x="-5.08" y="142.24" smashed="yes">
+<attribute name="VALUE" x="0" y="144.78" size="1.778" layer="96" rot="R180"/>
+</instance>
+<instance part="GND2" gate="1" x="-5.08" y="111.76"/>
 <instance part="SV1" gate="1" x="-10.16" y="195.58" smashed="yes">
 <attribute name="VALUE" x="-11.43" y="180.34" size="1.778" layer="96"/>
@@
 <instance part="IC3" gate="B" x="248.92" y="231.14"/>
 <instance part="IC3" gate="C" x="332.74" y="231.14"/>
-<instance part="IC3" gate="P" x="325.12" y="170.18"/>
+<instance part="IC3" gate="P" x="0" y="127"/>
 <instance part="J1" gate="G$1" x="157.48" y="152.4" smashed="yes">
 <attribute name="NAME" x="160.02" y="153.67" size="1.27" layer="95" rot="R180"/>
@@
 <attribute name="NAME" x="35.56" y="163.83" size="1.27" layer="95" rot="R180"/>
 </instance>
+<instance part="C1" gate="G$1" x="7.62" y="129.54"/>
 </instances>
 <busses>
@@
 <segment>
 <pinref part="IC1" gate="P" pin="GND"/>
-<wire x1="317.5" y1="162.56" x2="317.5" y2="160.02" width="0.1524" layer="91"/>
-<wire x1="317.5" y1="160.02" x2="320.04" y2="160.02" width="0.1524" layer="91"/>
-<wire x1="320.04" y1="160.02" x2="325.12" y2="160.02" width="0.1524" layer="91"/>
-<wire x1="325.12" y1="160.02" x2="325.12" y2="162.56" width="0.1524" layer="91"/>
-<junction x="320.04" y="160.02"/>
+<wire x1="-7.62" y1="119.38" x2="-7.62" y2="116.84" width="0.1524" layer="91"/>
+<wire x1="-7.62" y1="116.84" x2="-5.08" y2="116.84" width="0.1524" layer="91"/>
+<wire x1="-5.08" y1="116.84" x2="0" y2="116.84" width="0.1524" layer="91"/>
+<wire x1="0" y1="116.84" x2="0" y2="119.38" width="0.1524" layer="91"/>
+<junction x="-5.08" y="116.84"/>
 <pinref part="GND2" gate="1" pin="GND"/>
-<wire x1="320.04" y1="160.02" x2="320.04" y2="157.48" width="0.1524" layer="91"/>
+<wire x1="-5.08" y1="116.84" x2="-5.08" y2="114.3" width="0.1524" layer="91"/>
 <pinref part="IC3" gate="P" pin="GND"/>
+<wire x1="0" y1="116.84" x2="7.62" y2="116.84" width="0.1524" layer="91"/>
+<pinref part="C1" gate="G$1" pin="2"/>
+<wire x1="7.62" y1="116.84" x2="7.62" y2="124.46" width="0.1524" layer="91"/>
+<junction x="0" y="116.84"/>
 </segment>
 <segment>
@@
 <segment>
 <pinref part="IC1" gate="P" pin="VCC"/>
-<wire x1="317.5" y1="177.8" x2="317.5" y2="180.34" width="0.1524" layer="91"/>
-<wire x1="317.5" y1="180.34" x2="320.04" y2="180.34" width="0.1524" layer="91"/>
-<wire x1="320.04" y1="180.34" x2="325.12" y2="180.34" width="0.1524" layer="91"/>
-<wire x1="325.12" y1="180.34" x2="325.12" y2="177.8" width="0.1524" layer="91"/>
-<junction x="320.04" y="180.34"/>
+<wire x1="-7.62" y1="134.62" x2="-7.62" y2="137.16" width="0.1524" layer="91"/>
+<wire x1="-7.62" y1="137.16" x2="-5.08" y2="137.16" width="0.1524" layer="91"/>
+<wire x1="-5.08" y1="137.16" x2="0" y2="137.16" width="0.1524" layer="91"/>
+<wire x1="0" y1="137.16" x2="0" y2="134.62" width="0.1524" layer="91"/>
+<junction x="-5.08" y="137.16"/>
 <pinref part="P+3" gate="1" pin="+5V"/>
-<wire x1="320.04" y1="182.88" x2="320.04" y2="180.34" width="0.1524" layer="91"/>
+<wire x1="-5.08" y1="139.7" x2="-5.08" y2="137.16" width="0.1524" layer="91"/>
 <pinref part="IC3" gate="P" pin="VCC"/>
-</segment>
-<segment>
+<wire x1="0" y1="137.16" x2="7.62" y2="137.16" width="0.1524" layer="91"/>
+<pinref part="C1" gate="G$1" pin="1"/>
+<wire x1="7.62" y1="137.16" x2="7.62" y2="132.08" width="0.1524" layer="91"/>
+<junction x="0" y="137.16"/>
+</segment>
+<segment>

Commit message: edit map
Parts:
- removed IC1: 74HC138N, detali:74HC138N
- removed IC3: 74HC10N, detali:74HC10N
- added 3D1: 74HC138N, detali:74HC138N
- added 3D2: К155ЛА4, detali:74HC10N
- added C2: (no value), rcl:C-EUC1206
- added D1, D2: LL4148, detali:LL4148
Connections:
- new net N$38: D1.A, D2.C
- new net N$39: 3D2P.VCC, C2.1, D1.C
- net +5V: now also 3D1P.VCC, D2.A; no longer IC1P.VCC, IC3P.VCC
- net COLN1: now also 3D2A.O; no longer IC3A.O
- net COLN2: now also 3D2B.O; no longer IC3B.O
- net COLN3: now also 3D2C.O; no longer IC3C.O
- net GND: now also 3D1A.G2A, 3D1A.G2B, 3D1P.GND, 3D2P.GND, C2.2; no longer IC1A.G2A, IC1A.G2B, IC1P.GND, IC3P.GND
- net N$10: now also 3D1A.C; no longer IC1A.C
- net N$11: now also 3D1A.Y2; no longer IC1A.Y2
- net N$14: now also 3D2A.I0, 3D2A.I1, 3D2A.I2; no longer IC3A.I0, IC3A.I1, IC3A.I2
- net N$17: now also 3D2C.I0, 3D2C.I1, 3D2C.I2; no longer IC3C.I0, IC3C.I1, IC3C.I2
- net N$18: now also 3D1A.Y7; no longer IC1A.Y7
- net N$23: now also 3D1A.Y6; no longer IC1A.Y6
- net N$24: now also 3D1A.G1; no longer IC1A.G1
- net N$33: now also 3D1A.Y5; no longer IC1A.Y5
- net N$34: now also 3D1A.Y4; no longer IC1A.Y4
- net N$35: now also 3D1A.Y3; no longer IC1A.Y3
- net N$36: now also 3D1A.Y1; no longer IC1A.Y1
- net N$6: now also 3D1A.A; no longer IC1A.A
- net N$7: now also 3D2B.I0, 3D2B.I1, 3D2B.I2; no longer IC3B.I0, IC3B.I1, IC3B.I2
- net N$8: now also 3D1A.B; no longer IC1A.B
- net SCK: now also 3D1A.Y0; no longer IC1A.Y0
Other:
- moved on the sheet: C1, D100, D101, D102, D103, D104, D105, D106, D107, D108, D109, D110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

Commit message: err
Parts:
- S107B: device cherrymx:CHERRY-MX -> cherrymx:CHERRY-MX-4P
Connections:
- net N$319: now also S107BG$1.PIN-1; no longer S107B.PIN-1
- net N$51: now also S107BG$1.PIN-2; no longer S107B.PIN-2
Changed lines of the file:
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@@
 <grid distance="100" unitdist="mil" unit="mil" style="lines" multiple="1" display="yes" altdistance="0.01" altunitdist="inch" altunit="inch"/>
 <layers>
-<layer number="1" name="Top" color="4" fill="1" visible="yes" active="no"/>
-<layer number="2" name="Route2" color="1" fill="3" visible="yes" active="no"/>
-<layer number="3" name="Route3" color="4" fill="3" visible="yes" active="no"/>
-<layer number="4" name="Route4" color="1" fill="4" visible="yes" active="no"/>
-<layer number="5" name="Route5" color="4" fill="4" visible="yes" active="no"/>
-<layer number="6" name="Route6" color="1" fill="8" visible="yes" active="no"/>
-<layer number="7" name="Route7" color="4" fill="8" visible="yes" active="no"/>
-<layer number="8" name="Route8" color="1" fill="2" visible="yes" active="no"/>
-<layer number="9" name="Route9" color="4" fill="2" visible="yes" active="no"/>
-<layer number="10" name="Route10" color="1" fill="7" visible="yes" active="no"/>
-<layer number="11" name="Route11" color="4" fill="7" visible="yes" active="no"/>
-<layer number="12" name="Route12" color="1" fill="5" visible="yes" active="no"/>
-<layer number="13" name="Route13" color="4" fill="5" visible="yes" active="no"/>
-<layer number="14" name="Route14" color="1" fill="6" visible="yes" active="no"/>
-<layer number="15" name="Route15" color="4" fill="6" visible="yes" active="no"/>
-<layer number="16" name="Bottom" color="1" fill="1" visible="yes" active="no"/>
-<layer number="17" name="Pads" color="2" fill="1" visible="yes" active="no"/>
-<layer number="18" name="Vias" color="2" fill="1" visible="yes" active="no"/>
-<layer number="19" name="Unrouted" color="6" fill="1" visible="yes" active="no"/>
-<layer number="20" name="Dimension" color="15" fill="1" visible="yes" active="no"/>
-<layer number="21" name="tPlace" color="7" fill="1" visible="yes" active="no"/>
-<layer number="22" name="bPlace" color="7" fill="1" visible="yes" active="no"/>
-<layer number="23" name="tOrigins" color="15" fill="1" visible="yes" active="no"/>
-<layer number="24" name="bOrigins" color="15" fill="1" visible="yes" active="no"/>
-<layer number="25" name="tNames" color="7" fill="1" visible="yes" active="no"/>
-<layer number="26" name="bNames" color="7" fill="1" visible="yes" active="no"/>
-<layer number="27" name="tValues" color="7" fill="1" visible="yes" active="no"/>
-<layer number="28" name="bValues" color="7" fill="1" visible="yes" active="no"/>
+<layer number="1" name="Top" color="4" fill="1" visible="no" active="no"/>
+<layer number="2" name="Route2" color="1" fill="3" visible="no" active="no"/>
+<layer number="3" name="Route3" color="4" fill="3" visible="no" active="no"/>
+<layer number="4" name="Route4" color="1" fill="4" visible="no" active="no"/>
+<layer number="5" name="Route5" color="4" fill="4" visible="no" active="no"/>
+<layer number="6" name="Route6" color="1" fill="8" visible="no" active="no"/>
+<layer number="7" name="Route7" color="4" fill="8" visible="no" active="no"/>
+<layer number="8" name="Route8" color="1" fill="2" visible="no" active="no"/>
+<layer number="9" name="Route9" color="4" fill="2" visible="no" active="no"/>
+<layer number="10" name="Route10" color="1" fill="7" visible="no" active="no"/>
+<layer number="11" name="Route11" color="4" fill="7" visible="no" active="no"/>
+<layer number="12" name="Route12" color="1" fill="5" visible="no" active="no"/>
+<layer number="13" name="Route13" color="4" fill="5" visible="no" active="no"/>
+<layer number="14" name="Route14" color="1" fill="6" visible="no" active="no"/>
+<layer number="15" name="Route15" color="4" fill="6" visible="no" active="no"/>
+<layer number="16" name="Bottom" color="1" fill="1" visible="no" active="no"/>
+<layer number="17" name="Pads" color="2" fill="1" visible="no" active="no"/>
+<layer number="18" name="Vias" color="2" fill="1" visible="no" active="no"/>
+<layer number="19" name="Unrouted" color="6" fill="1" visible="no" active="no"/>
+<layer number="20" name="Dimension" color="15" fill="1" visible="no" active="no"/>
+<layer number="21" name="tPlace" color="7" fill="1" visible="no" active="no"/>
+<layer number="22" name="bPlace" color="7" fill="1" visible="no" active="no"/>
+<layer number="23" name="tOrigins" color="15" fill="1" visible="no" active="no"/>
+<layer number="24" name="bOrigins" color="15" fill="1" visible="no" active="no"/>
+<layer number="25" name="tNames" color="7" fill="1" visible="no" active="no"/>
+<layer number="26" name="bNames" color="7" fill="1" visible="no" active="no"/>
+<layer number="27" name="tValues" color="7" fill="1" visible="no" active="no"/>
+<layer number="28" name="bValues" color="7" fill="1" visible="no" active="no"/>
 <layer number="29" name="tStop" color="7" fill="3" visible="no" active="no"/>
 <layer number="30" name="bStop" color="7" fill="6" visible="no" active="no"/>
@@
 <layer number="35" name="tGlue" color="7" fill="4" visible="no" active="no"/>
 <layer number="36" name="bGlue" color="7" fill="5" visible="no" active="no"/>
-<layer number="37" name="tTest" color="7" fill="1" visible="yes" active="no"/>
-<layer number="38" name="bTest" color="7" fill="1" visible="yes" active="no"/>
+<layer number="37" name="tTest" color="7" fill="1" visible="no" active="no"/>
+<layer number="38" name="bTest" color="7" fill="1" visible="no" active="no"/>
 <layer number="39" name="tKeepout" color="4" fill="11" visible="no" active="no"/>
 <layer number="40" name="bKeepout" color="1" fill="11" visible="no" active="no"/>
@@
 <layer number="44" name="Drills" color="7" fill="1" visible="no" active="no"/>
 <layer number="45" name="Holes" color="7" fill="1" visible="no" active="no"/>
-<layer number="46" name="Milling" color="3" fill="1" visible="yes" active="no"/>
-<layer number="47" name="Measures" color="7" fill="1" visible="yes" active="no"/>
-<layer number="48" name="Document" color="7" fill="1" visible="yes" active="no"/>
-<layer number="49" name="Reference" color="7" fill="1" visible="yes" active="no"/>
-<layer number="50" name="dxf" color="7" fill="1" visible="yes" active="no"/>
-<layer number="51" name="tDocu" color="7" fill="1" visible="yes" active="no"/>
-<layer number="52" name="bDocu" color="7" fill="1" visible="yes" active="no"/>
-<layer number="53" name="tGND_GNDA" color="7" fill="9" visible="yes" active="no"/>
-<layer number="54" name="bGND_GNDA" color="1" fill="9" visible="yes" active="no"/>
-<layer number="56" name="wert" color="7" fill="1" visible="yes" active="no"/>
-<layer number="57" name="tCAD" color="7" fill="1" visible="yes" active="no"/>
+<layer number="46" name="Milling" color="3" fill="1" visible="no" active="no"/>
+<layer number="47" name="Measures" color="7" fill="1" visible="no" active="no"/>
+<layer number="48" name="Document" color="7" fill="1" visible="no" active="no"/>
+<layer number="49" name="Reference" color="7" fill="1" visible="no" active="no"/>
+<layer number="50" name="dxf" color="7" fill="1" visible="no" active="no"/>
+<layer number="51" name="tDocu" color="7" fill="1" visible="no" active="no"/>
+<layer number="52" name="bDocu" color="7" fill="1" visible="no" active="no"/>
+<layer number="53" name="tGND_GNDA" color="7" fill="9" visible="no" active="no"/>
+<layer number="54" name="bGND_GNDA" color="1" fill="9" visible="no" active="no"/>
+<layer number="56" name="wert" color="7" fill="1" visible="no" active="no"/>
+<layer number="57" name="tCAD" color="7" fill="1" visible="no" active="no"/>
 <layer number="90" name="Modules" color="5" fill="1" visible="yes" active="yes"/>
 <layer number="91" name="Nets" color="2" fill="1" visible="yes" active="yes"/>
@@
 <part name="S109" library="cherrymx" deviceset="CHERRY-MX-4P" device="" value="00"/>
 <part name="S110" library="cherrymx" deviceset="CHERRY-MX-4P" device="" value="."/>
-<part name="S107B" library="cherrymx" deviceset="CHERRY-MX" device="" value="NumEnter"/>
+<part name="S107B" library="cherrymx" deviceset="CHERRY-MX-4P" device="" value="NumEnter"/>
 <part name="JA88" library="detali" deviceset="SJ" device=""/>
 <part name="JB88" library="detali" deviceset="SJ" device=""/>

Commit message: 16-07-28
Parts:
- SV1: device detali:MA09-1 -> detali:FE09-1
Changed lines of the file:
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@@
 <part name="P+3" library="supply1" deviceset="+5V" device=""/>
 <part name="GND2" library="supply1" deviceset="GND" device=""/>
-<part name="SV1" library="detali" deviceset="MA09-1" device=""/>
+<part name="SV1" library="detali" deviceset="FE09-1" device=""/>
 <part name="3D2" library="detali" deviceset="74*10" device="N" technology="HC" value="К155ЛА4"/>
 <part name="J1" library="detali" deviceset="J" device=""/>
@@
 </instance>
 <instance part="GND2" gate="1" x="76.2" y="40.64"/>
-<instance part="SV1" gate="1" x="30.48" y="119.38" smashed="yes">
+<instance part="SV1" gate="G$1" x="30.48" y="119.38" smashed="yes">
 <attribute name="VALUE" x="29.21" y="104.14" size="1.778" layer="96"/>
 <attribute name="NAME" x="29.21" y="132.842" size="1.778" layer="95"/>
@@
 </segment>
 <segment>
-<pinref part="SV1" gate="1" pin="1"/>
+<pinref part="SV1" gate="G$1" pin="1"/>
 <wire x1="38.1" y1="109.22" x2="40.64" y2="109.22" width="0.1524" layer="91"/>
 <pinref part="GND3" gate="1" pin="GND"/>
@@
 <wire x1="78.74" y1="114.3" x2="81.28" y2="114.3" width="0.1524" layer="91"/>
 <wire x1="78.74" y1="114.3" x2="78.74" y2="129.54" width="0.1524" layer="91"/>
-<pinref part="SV1" gate="1" pin="9"/>
+<pinref part="SV1" gate="G$1" pin="9"/>
 <wire x1="38.1" y1="129.54" x2="78.74" y2="129.54" width="0.1524" layer="91"/>
 <junction x="78.74" y="114.3"/>
@@
 </segment>
 <segment>
-<pinref part="SV1" gate="1" pin="3"/>
+<pinref part="SV1" gate="G$1" pin="3"/>
 <wire x1="38.1" y1="114.3" x2="48.26" y2="114.3" width="0.1524" layer="91"/>
 <label x="40.64" y="114.3" size="1.778" layer="95"/>
@@
 </segment>
 <segment>
-<pinref part="SV1" gate="1" pin="2"/>
+<pinref part="SV1" gate="G$1" pin="2"/>
 <wire x1="38.1" y1="111.76" x2="48.26" y2="111.76" width="0.1524" layer="91"/>
 <label x="40.64" y="111.76" size="1.778" layer="95"/>
@@
 <net name="N$6" class="0">
 <segment>
-<pinref part="SV1" gate="1" pin="8"/>
+<pinref part="SV1" gate="G$1" pin="8"/>
 <pinref part="3D1" gate="A" pin="A"/>
 <wire x1="38.1" y1="127" x2="93.98" y2="127" width="0.1524" layer="91"/>
@@
 <segment>
 <pinref part="3D1" gate="A" pin="B"/>
-<pinref part="SV1" gate="1" pin="7"/>
+<pinref part="SV1" gate="G$1" pin="7"/>
 <wire x1="93.98" y1="124.46" x2="38.1" y2="124.46" width="0.1524" layer="91"/>
 </segment>
@@
 <segment>
 <pinref part="3D1" gate="A" pin="C"/>
-<pinref part="SV1" gate="1" pin="6"/>
+<pinref part="SV1" gate="G$1" pin="6"/>
 <wire x1="93.98" y1="121.92" x2="38.1" y2="121.92" width="0.1524" layer="91"/>
 </segment>
@@
 <segment>
 <pinref part="J16" gate="G$1" pin="P$2"/>
-<pinref part="SV1" gate="1" pin="5"/>
+<pinref part="SV1" gate="G$1" pin="5"/>
 <wire x1="40.64" y1="119.38" x2="38.1" y2="119.38" width="0.1524" layer="91"/>
 </segment>
@@
 <net name="N$30" class="0">
 <segment>
-<pinref part="SV1" gate="1" pin="4"/>
+<pinref part="SV1" gate="G$1" pin="4"/>
 <wire x1="38.1" y1="116.84" x2="55.88" y2="116.84" width="0.1524" layer="91"/>
 <pinref part="J17" gate="G$1" pin="P$2"/>

Commit message: move
Parts:
- R1, R2, R3: value (none) -> 10k
Changed lines of the file:
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@@
 <part name="GND1" library="supply1" deviceset="GND" device=""/>
 <part name="S1" library="detali" deviceset="31-XX" device="" value="NumLock"/>
-<part name="R1" library="rcl" deviceset="R-EU_" device="R1206W"/>
-<part name="R2" library="rcl" deviceset="R-EU_" device="R1206W"/>
-<part name="R3" library="rcl" deviceset="R-EU_" device="R1206W"/>
+<part name="R1" library="rcl" deviceset="R-EU_" device="R1206W" value="10k"/>
+<part name="R2" library="rcl" deviceset="R-EU_" device="R1206W" value="10k"/>
+<part name="R3" library="rcl" deviceset="R-EU_" device="R1206W" value="10k"/>
 <part name="P+2" library="supply1" deviceset="+5V" device=""/>
 <part name="P+3" library="supply1" deviceset="+5V" device=""/>
