File: Keyboard_pro/Keyboard.brd (EAGLE design)
At the start: 492.8 x 141 mm, 588 parts, among them IC1 MEGA8-AI

Commit message: move
Other:
- board size 492.8 x 141 mm -> 496.6 x 154.9 mm
Changed lines of the file:
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@@
 <wire x1="363.22" y1="139.7" x2="363.22" y2="8.89" width="0.2" layer="20"/>
 <dimension x1="210.185" y1="151.13" x2="372.11" y2="144.145" x3="291.1475" y3="157.48" layer="1" dtype="horizontal"/>
+<wire x1="8.89" y1="20.32" x2="30.48" y2="-0.635" width="0.4064" layer="20"/>
+<wire x1="381.635" y1="31.75" x2="361.315" y2="-5.08" width="0.4064" layer="20"/>
 </plain>
 <attributes>
