File: PCB/Keyboard_pro/Keyboard.brd (EAGLE design)
At the start: 479.1 x 340.4 mm, 762 parts, among them IC1 MEGA8-AI, J1 J, J10 J, J11 J, J12 J, J13 J, J14 J, J15 J, J16 J, J17 J, J2 J, J3 J, J4 J, J5 J, J6 J, J7 J, J8 J, J9 J

Commit message: get all vil
Parts:
- removed 2S1: (no value), con-lsta:FE10
- removed 2S2, 2S3: (no value), con-lsta:FE08
- removed 2S4: (no value), con-lsta:FE05-1
- removed U$113: (no value), kbmx:18X28
- removed U$165: (no value), kbmxco:SIZE132
- added 2D1: 74HC138N, detali2:DIL16
- added 2D2: 74ALS04N, detali2:DIL14
- added C3, C4: 100n, rcl:C0805
- added D137, D138, D139, D67B: LL4148, detali:SOD80C
- added J18, J19, J20, J21, J22, J23, J24, J25, J26, J27, J28, J29, J30, J31, J32, J33, J34, J35, J36, J37, J38, J39, J40, J41, J42, J43, J44, J45, J46, J47, J48, J49, J50, J51, J52, J53, J54, J55, J56, J57, J58, J59, J60, J61, J62, J63, J64, J65, J66: (no value), detali2:R1206W
- added JA134, JA67B, JA67B1, JB134, JB67B1: (no value), detali:SJ
- added S67C1: FN2, cherrymx:CHERRY-MX-4P
- added SV4: CON_KB_B, detali2:FE12
- added U$213: (no value), kbmx:18X42
- added U$214, U$216, U$217: (no value), kbmx:18X28
- added U$215: (no value), kbmx:18X18
- S47, S48, S49, S50, S51, S52, S53, S54, S55, S56, S57, S58, S59, S60, S61, S62, S63, S64, S65, S66, S67C, S68, S69, S70, S71, S72, S73, S74, S74A, S75, S76, S77, S78, S79, S80, S81, S82, S85, S86: device cherrymx:CHERRY-MX -> cherrymx:CHERRY-MX-4P
- S67: value | -> |d; device cherrymx:CHERRY-MX -> cherrymx:CHERRY-MX-4P
- S67B: value | -> |u
- S83: value Mouse2(Menu) -> FN3; device cherrymx:CHERRY-MX -> cherrymx:CHERRY-MX-4P
- S84: value Alt -> R_Alt; device cherrymx:CHERRY-MX -> cherrymx:CHERRY-MX-4P
- moved R3 424.4 mm to (360.4, 109.2), turned to 270 degrees
- moved D67 64.5 mm to (317.2, 45.7), turned to 180 degrees
- moved JB67 61.1 mm to (321.0, 39.4), turned to 180 degrees
- moved U$118 55.1 mm to (379.4, -4.45)
- moved JA67 53.4 mm to (335.6, 40.6), turned to 180 degrees
- moved D74 38.3 mm to (317.2, 64.1), turned to 180 degrees
- moved D59 34.3 mm to (318.5, 102.6), turned to 180 degrees
- moved D68 32.2 mm to (233.0, 34.3)
- moved D47 30.0 mm to (223.8, 85.1)
- moved JA82 26.5 mm to (223.8, 18.4)
- moved JA48 25.1 mm to (222.6, 127.3), turned to 270 degrees
- moved D60 25.0 mm to (235.3, 53.3)
- moved D83 23.7 mm to (295.6, 16.8), turned to 270 degrees
- moved D86 23.4 mm to (363.9, 17.1)
- moved JA75 23.0 mm to (206.7, 37.5)
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Connections:
- removed net 2A1: JA61.2
- removed net 2A2: 2S3.2, JA47.2, JA60.2
- removed net 2A3: JA69.2
- removed net 2A4: 2S3.4, JA68.2, JA82.2
- removed net 2A5: JA76.2
- removed net 2A6: 2S3.6, JA75.2, JA83.2
- removed net 2A7: 2S3.7, JA48.2
- removed net 2A8: 2S3.8, JA53.2, JA54.2
- removed net 2B0: 2S1.1, D53.C
- removed net 2B1: 2S1.2, D54.C
- removed net 2B10: 2S2.1, D82.C
- removed net 2B4: 2S1.5, D60.C, D61.C, D68.C, D69.C, D75.C, D76.C
- removed net 2B6: 2S1.7, D47.C, D48.C, D83.C
- removed net GND_K2: R3.1
- new net +3VD: 2D2.14, C4.1, D138.C
- new net 1: D49.C, D50.C, D52.C, D56.C, D64B.C, J57.1
- new net 2: D51.C, D58.C, D59.C, J18.2, J24.2
- new net 2I: 2D1.14, D48.C, J66.1
- new net 2J: D55.C, J24.1
- new net 3: D47.C, D54.C, D57.C, D63.C, J19.2
- new net 3J: D66.C, D67B.C, J20.1, J59.1
- new net 4: D65.C, D74.C, J21.1, J62.1
- new net 4J: D64.C, D71.C, J21.2, J25.2
- new net 4J2: D53.C, D61.C, J25.1
- new net 5: D67.C, D73.C, J22.1, J60.1
- new net 5J: D60.C, D62.C, D69.C, D72.C, J22.2
- new net 6: D79.C, D80.C, D81.C, J26.2, J65.1
- new net 6J2: D70.C, J26.1, J27.2
- new net 6J3: D68.C, J27.1
- new net 7: 2D1.13, D84.C, D85.C, J23.1
- new net 7J: D75.C, D76.C, D78.C, J23.2
- new net 8: 2D1.12, D86.C, J58.2
- new net 8J: D137.C, D77.C, D82.C, D83.C, J58.1
- new net D1: J41.2, SV4.10
- new net D2: J42.2, SV4.9
- new net D3: J43.2, SV4.8
- new net G3: J28.2, JA62.2, JA63.2, JA71.2
- new net G4: J47.2, JA134.2, JA50.2, JA51.2, JA57.2, JA64.2, JA72.2, JA78.2, JA79.2
- new net G5: J33.2, JA52.2, JA58.2, JA65.2, JA66.2, JA73.2, JA80.2, JA83.2, JA84.2
- new net G6: J30.2, JA59.2, JA67.2, JA67B.2, JA67B1.2, JA74B.2, JA81.2, JA85.2, JA86.2, JB74.1
- new net N$171: D67B.A, JB67B1.1
- new net N$179: JB57.2, S57.SW2
- new net N$249: J19.1, J20.2
- new net N$257: JB62.2, S62.SW2
- new net N$480: JA62.1, S62.SW1
- new net N$483: 2D1.6, R3.2
- new net N$484: JB76.2, S76.SW2
- new net N$485: JA76.1, S76.SW1
- new net N$486: 2D2.6, SV4.7
- new net N$487: 2D2.4, SV4.6
- new net N$488: 2D2.2, SV4.5
- new net N$489: 2D2.12, J35.2
- new net N$490: 2D2.8, J40.2
- new net N$491: J28.1, J29.2
- new net N$492: 2D2.3, J29.1
- new net N$493: J30.1, J31.2
- new net N$494: 2D2.13, J31.1
- new net N$495: J32.2, J33.1
- new net N$496: 2D2.11, J32.1
- new net N$497: 2D2.1, J34.1
- new net N$498: J35.1, SV4.4
- new net N$499: J36.1, SV4.3
- new net N$500: J36.2, J37.1
- new net N$501: 2D2.10, J37.2
- new net N$502: J38.1, SV4.2
- new net N$503: J38.2, J39.1
- new net N$504: J39.2, J40.1
- new net N$505: D138.A, D139.C
- new net N$506: J41.1, J44.2
- new net N$507: J42.1, J45.2
- new net N$508: J43.1, J46.2
- new net N$509: 2D2.5, J47.1
- new net N$510: J44.1, J48.2
- new net N$511: J45.1, J49.2
- new net N$512: J46.1, J50.2
- new net N$513: J50.1, J51.2
- new net N$514: J48.1, J52.2
- new net N$515: J49.1, J53.2
- new net N$516: J51.1, J54.2
- new net N$517: J53.1, J55.2
- new net N$518: J52.1, J56.2
- new net N$519: 2D1.1, J54.1
- new net N$520: 2D1.2, J55.1
- new net N$521: 2D1.3, J56.1
- new net N$522: 2D1.15, J57.2
- new net N$525: 2D1.7, J59.2
- new net N$526: J61.1, J62.2
- new net N$527: 2D1.11, J61.2
- new net N$528: J60.2, J63.1
- new net N$529: J64.1, J65.2
- new net N$530: 2D1.9, J64.2
- new net N$531: 2D1.10, J63.2
- new net N$532: J18.1, J66.2
- net +5V: now also 2D1.16, C3.1, D139.A, R3.1, SV4.11
- net G1: now also 2D2.9, JA47.2, JA48.2, JA49.2, JA53.2, JA60.2, JA68.2, JA75.2, JA82.2
- net G2: now also J34.2, JA54.2, JA55.2, JA56.2, JA61.2, JA69.2, JA70.2, JA76.2, JA77.2
- net GND: now also 2D1.4, 2D1.5, 2D1.8, 2D2.7, C3.2, C4.2, SV4.1
- net N$152: now also JB74B.2, S74.SW2; no longer R3.2
- net N$161: now also JB67B1.2, S67B.SW1, S67C.SW2; no longer JB76.2, S76.SW1
- net N$162: now also JA134.1, S67C1.SW1; no longer JB83.2, S83.SW1
- net N$165: now also JB134.2, S67C1.SW2; no longer JB62.2, S62.SW1
- net N$168: now also D137.A, JB134.1; no longer JB84.2, S84.SW1
- net N$169: now also S50.SW2; no longer S50.SW1
- net N$172: now also S78.SW2; no longer S78.SW1
- net N$173: now also S85.SW2; no longer S85.SW1
- net N$175: now also JB83.2, S83.SW2; no longer JB57.2, S57.SW1
- net N$176: now also JB73.2, S73.SW2; no longer JB64.2, S64.SW1
- net N$177: now also JA73.1, S73.SW1; no longer JB72.2, S72.SW1
- net N$178: now also S79.SW2; no longer S79.SW1
- net N$180: now also S58.SW2; no longer S58.SW1
- net N$181: now also S65.SW2; no longer S65.SW1
- net N$182: now also JA80.1; no longer JB80.2
- net N$183: now also S59.SW2; no longer S59.SW1
- net N$185: now also S67.SW2; no longer S67.SW1, S67B.SW1, S67C.SW2
- net N$186: now also S81.SW2; no longer S81.SW1
- net N$225: now also JA74.2; no longer JB74.1
- net N$238: now also JA57.1, S57.SW1; no longer JA76.1, S76.SW2
- net N$239: now also S83.SW1; no longer S83.SW2
- net N$242: now also JA64.1, S64.SW1; no longer JA62.1, S62.SW2
- net N$245: now also JB80.2, S80.SW2; no longer JA84.1, S84.SW2
- net N$246: now also S50.SW1; no longer S50.SW2
- net N$250: now also S78.SW1; no longer S78.SW2
- net N$251: now also S85.SW1; no longer S85.SW2
- net N$253: now also JB64.2, S64.SW2; no longer JA57.1, S57.SW2
- net N$254: now also JB72.2, S72.SW2; no longer JA64.1, S64.SW2
- net N$255: now also S72.SW1; no longer S72.SW2
- net N$256: now also S79.SW1; no longer S79.SW2
- net N$259: now also JA65.1, S65.SW1; no longer JA58.1, S58.SW2
- net N$260: now also JA58.1, S58.SW1; no longer JA65.1, S65.SW2
- net N$261: now also JB84.2, S84.SW2; no longer JA73.1, S73.SW2
- net N$262: now also JA84.1, S84.SW1; no longer JA80.1, S80.SW2
- net N$263: now also S81.SW1; no longer S81.SW2
- net N$264: now also S67.SW1; no longer S67.SW2, S67B.SW2, S67C.SW1
- net N$265: now also S59.SW1; no longer S59.SW2
- net N$267: now also S74.SW1; no longer S74.SW2
- net N$70: now also JA67B1.1, S67B.SW2; no longer JB74B.2, S74.SW1
- net N$89: now also JA67B.1, S67C.SW1; no longer JB73.2, S73.SW1
Routing:
- net G6: track 0.00 -> 213.0 mm
- net 7: track 0.00 -> 209.9 mm
- net GND: track 96.7 -> 306.2 mm
- net G1: track 22.3 -> 221.3 mm
- net +5V: track 136.4 -> 324.5 mm
- net G5: track 0.00 -> 173.2 mm
- net G4: track 0.00 -> 168.9 mm
- net 2I: track 0.00 -> 165.0 mm
- net G2: track 0.00 -> 138.3 mm
- net 1: track 0.00 -> 135.7 mm
- net 8J: track 0.00 -> 133.5 mm
- net 8: track 0.00 -> 120.3 mm
- net N$493: track 0.00 -> 96.2 mm
- net 5J: track 0.00 -> 93.2 mm
- net N$530: track 0.00 -> 90.5 mm
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Other:
- board size 479.1 x 340.4 mm -> 479.1 x 335.9 mm
- board text added: "1177-16"
