File: PCB/Keyboard_pro/Keyboard.sch (EAGLE design)
At the start: 597 parts, among them IC1 MEGA8-AI, J1 J, J10 J, J11 J, J12 J, J13 J, J14 J, J15 J, J16 J, J17 J, J2 J, J3 J, J4 J, J5 J, J6 J, J7 J, J8 J, J9 J

Commit message: get all vil
Parts:
- removed 2S1: (no value), con-lsta:FE10-1
- removed 2S2, 2S3: (no value), con-lsta:FE08-1
- removed 2S4: (no value), con-lsta:FE05-1
- added 2D1: 74HC138N, detali2:74AC138N
- added 2D2: 74ALS04N, detali2:74ALS04N
- added C3, C4: 100n, rcl:C-EUC0805
- added D137, D138, D139, D67B: LL4148, detali:LL4148
- added J18, J19, J20, J21, J22, J23, J24, J25, J26, J27, J28, J29, J30, J31, J32, J33, J34, J35, J36, J37, J38, J39, J40, J41, J42, J43, J44, J45, J46, J47, J48, J49, J50, J51, J52, J53, J54, J55, J56, J57, J58, J59, J60, J61, J62, J63, J64, J65, J66: J, detali2:J
- added JA134, JA67B, JA67B1, JB134, JB67B1: (no value), detali:SJ
- added S67C1: FN2, cherrymx:CHERRY-MX-4P
- added SV4: CON_KB_B, detali2:FE12-1
- S47, S48, S49, S50, S51, S52, S53, S54, S55, S56, S57, S58, S59, S60, S61, S62, S63, S64, S65, S66, S67C, S68, S69, S70, S71, S72, S73, S74, S74A, S75, S76, S77, S78, S79, S80, S81, S82, S85, S86: device cherrymx:CHERRY-MX -> cherrymx:CHERRY-MX-4P
- S67: value | -> |d; device cherrymx:CHERRY-MX -> cherrymx:CHERRY-MX-4P
- S67B: value | -> |u
- S83: value Mouse2(Menu) -> FN3; device cherrymx:CHERRY-MX -> cherrymx:CHERRY-MX-4P
- S84: value Alt -> R_Alt; device cherrymx:CHERRY-MX -> cherrymx:CHERRY-MX-4P
Connections:
- removed net 2A1: JA61.2
- removed net 2A2: 2S3.2, JA47.2, JA60.2
- removed net 2A3: JA69.2
- removed net 2A4: 2S3.4, JA68.2, JA82.2
- removed net 2A5: JA76.2
- removed net 2A6: 2S3.6, JA75.2, JA83.2
- removed net 2A7: 2S3.7, JA48.2
- removed net 2A8: 2S3.8, JA53.2, JA54.2
- removed net 2B0: 2S1.1, D53.C
- removed net 2B1: 2S1.2, D54.C
- removed net 2B10: 2S2.1, D82.C
- removed net 2B4: 2S1.5, D60.C, D61.C, D68.C, D69.C, D75.C, D76.C
- removed net 2B6: 2S1.7, D47.C, D48.C, D83.C
- removed net GND_K2: R3.1
- new net +3VD: 2D2P.VCC, C4.1, D138.C
- new net 1: D49.C, D50.C, D52.C, D56.C, D64B.C, J57.P$1
- new net 2: D51.C, D58.C, D59.C, J18.P$2, J24.P$2
- new net 2I: 2D1A.Y1, D48.C, J66.P$1
- new net 2J: D55.C, J24.P$1
- new net 3: D47.C, D54.C, D57.C, D63.C, J19.P$2
- new net 3J: D66.C, D67B.C, J20.P$1, J59.P$1
- new net 4: D65.C, D74.C, J21.P$1, J62.P$1
- new net 4J: D64.C, D71.C, J21.P$2, J25.P$2
- new net 4J2: D53.C, D61.C, J25.P$1
- new net 5: D67.C, D73.C, J22.P$1, J60.P$1
- new net 5J: D60.C, D62.C, D69.C, D72.C, J22.P$2
- new net 6: D79.C, D80.C, D81.C, J26.P$2, J65.P$1
- new net 6J2: D70.C, J26.P$1, J27.P$2
- new net 6J3: D68.C, J27.P$1
- new net 7: 2D1A.Y2, D84.C, D85.C, J23.P$1
- new net 7J: D75.C, D76.C, D78.C, J23.P$2
- new net 8: 2D1A.Y3, D86.C, J58.P$2
- new net 8J: D137.C, D77.C, D82.C, D83.C, J58.P$1
- new net D1: J41.P$2, SV4.10
- new net D2: J42.P$2, SV4.9
- new net D3: J43.P$2, SV4.8
- new net G3: J28.P$2, JA62.2, JA63.2, JA71.2
- new net G4: J47.P$2, JA134.2, JA50.2, JA51.2, JA57.2, JA64.2, JA72.2, JA78.2, JA79.2
- new net G5: J33.P$2, JA52.2, JA58.2, JA65.2, JA66.2, JA73.2, JA80.2, JA83.2, JA84.2
- new net G6: J30.P$2, JA59.2, JA67.2, JA67B.2, JA67B1.2, JA74B.2, JA81.2, JA85.2, JA86.2, JB74.1
- new net N$480: JA62.1, S62G$1.PIN-1
- new net N$481: JB71.2, S71G$1.PIN-1
- new net N$482: JA71.1, S71G$1.PIN-2
- new net N$483: 2D1A.G1, R3.2
- new net N$484: JB76.2, S76G$1.PIN-2
- new net N$485: JA76.1, S76G$1.PIN-1
- new net N$486: 2D2C.O, SV4.7
- new net N$487: 2D2B.O, SV4.6
- new net N$488: 2D2A.O, SV4.5
- new net N$489: 2D2F.O, J35.P$2
- new net N$490: 2D2D.O, J40.P$2
- new net N$491: J28.P$1, J29.P$2
- new net N$492: 2D2B.I, J29.P$1
- new net N$493: J30.P$1, J31.P$2
- new net N$494: 2D2F.I, J31.P$1
- new net N$495: J32.P$2, J33.P$1
- new net N$496: 2D2E.I, J32.P$1
- new net N$497: 2D2A.I, J34.P$1
- new net N$498: J35.P$1, SV4.4
- new net N$499: J36.P$1, SV4.3
- new net N$500: J36.P$2, J37.P$1
- new net N$501: 2D2E.O, J37.P$2
- new net N$502: J38.P$1, SV4.2
- new net N$503: J38.P$2, J39.P$1
- new net N$504: J39.P$2, J40.P$1
- new net N$505: D138.A, D139.C
- new net N$506: J41.P$1, J44.P$2
- new net N$507: J42.P$1, J45.P$2
- new net N$508: J43.P$1, J46.P$2
- new net N$509: 2D2C.I, J47.P$1
- new net N$510: J44.P$1, J48.P$2
- new net N$511: J45.P$1, J49.P$2
- new net N$512: J46.P$1, J50.P$2
- new net N$513: J50.P$1, J51.P$2
- new net N$514: J48.P$1, J52.P$2
- new net N$515: J49.P$1, J53.P$2
- new net N$516: J51.P$1, J54.P$2
- new net N$517: J53.P$1, J55.P$2
- new net N$518: J52.P$1, J56.P$2
- new net N$519: 2D1A.A, J54.P$1
- new net N$520: 2D1A.B, J55.P$1
- new net N$521: 2D1A.C, J56.P$1
- new net N$522: 2D1A.Y0, J57.P$2
- new net N$523: JB86.2, S86G$1.PIN-1
- new net N$524: JA86.1, S86G$1.PIN-2
- new net N$525: 2D1A.Y7, J59.P$2
- new net N$526: J61.P$1, J62.P$2
- new net N$527: 2D1A.Y4, J61.P$2
- new net N$528: J60.P$2, J63.P$1
- new net N$529: J64.P$1, J65.P$2
- new net N$530: 2D1A.Y6, J64.P$2
- new net N$531: 2D1A.Y5, J63.P$2
- new net N$532: J18.P$1, J66.P$2
- net +5V: now also 2D1P.VCC, C3.1, D139.A, R3.1, SV4.11
- net G1: now also 2D2D.I, JA47.2, JA48.2, JA49.2, JA53.2, JA60.2, JA68.2, JA75.2, JA82.2
- net G2: now also J34.P$2, JA54.2, JA55.2, JA56.2, JA61.2, JA69.2, JA70.2, JA76.2, JA77.2
- net GND: now also 2D1A.G2A, 2D1A.G2B, 2D1P.GND, 2D2P.GND, C3.2, C4.2, SV4.1
- net N$112: now also S47G$1.PIN-1; no longer S47.PIN-1
- net N$127: now also S53G$1.PIN-1; no longer S53.PIN-1
- net N$152: now also JB74B.2, S74G$1.PIN-2; no longer R3.2
- net N$153: now also S60G$1.PIN-1; no longer S60.PIN-1
- net N$154: now also S68G$1.PIN-1; no longer S68.PIN-1
- net N$155: now also S75G$1.PIN-1; no longer S75.PIN-1
- net N$156: now also S82G$1.PIN-1; no longer S82.PIN-1
- net N$157: now also S48G$1.PIN-1; no longer S48.PIN-1
- net N$158: now also S54G$1.PIN-1; no longer S54.PIN-1
- net N$159: now also S61G$1.PIN-1; no longer S61.PIN-1
- net N$160: now also S69G$1.PIN-1; no longer S69.PIN-1
- net N$161: now also JB67B1.2, S67B.PIN-1, S67CG$1.PIN-2; no longer JB76.2, S76.PIN-1
- net N$162: now also JA134.1, S67C1G$1.PIN-1; no longer JB83.2, S83.PIN-1
- net N$163: now also S49G$1.PIN-1; no longer S49.PIN-1
- net N$164: now also S55G$1.PIN-1; no longer S55.PIN-1
- net N$165: now also JB134.2, S67C1G$1.PIN-2; no longer JB62.2, S62.PIN-1
- net N$166: now also S70G$1.PIN-1; no longer S70.PIN-1
- net N$167: now also S77G$1.PIN-1; no longer S77.PIN-1
- net N$168: now also D137.A, JB134.1; no longer JB84.2, S84.PIN-1
- net N$169: now also S50G$1.PIN-2; no longer S50.PIN-1
- net N$170: now also S56G$1.PIN-1; no longer S56.PIN-1
- net N$171: now also D67B.A, JB67B1.1; no longer JB71.2, S71.PIN-1
- net N$172: now also S78G$1.PIN-2; no longer S78.PIN-1
- net N$173: now also S85G$1.PIN-2; no longer S85.PIN-1
- net N$174: now also S51G$1.PIN-1; no longer S51.PIN-1
- net N$175: now also JB83.2, S83G$1.PIN-2; no longer JB57.2, S57.PIN-1
- net N$176: now also JB73.2, S73G$1.PIN-2; no longer JB64.2, S64.PIN-1
- net N$177: now also JA73.1, S73G$1.PIN-1; no longer JB72.2, S72.PIN-1
- net N$178: now also S79G$1.PIN-2; no longer S79.PIN-1
- net N$179: now also JB57.2, S57G$1.PIN-2; no longer JB86.2, S86.PIN-1
- net N$180: now also S58G$1.PIN-2; no longer S58.PIN-1
- net N$181: now also S65G$1.PIN-2; no longer S65.PIN-1
- net N$182: now also JA80.1, S80G$1.PIN-1; no longer JB80.2, S80.PIN-1
- net N$183: now also S59G$1.PIN-2; no longer S59.PIN-1
- net N$184: now also S66G$1.PIN-1; no longer S66.PIN-1
- net N$185: now also S67G$1.PIN-2; no longer S67.PIN-1, S67B.PIN-1, S67C.PIN-2
- net N$186: now also S81G$1.PIN-2; no longer S81.PIN-1
- net N$225: now also JA74.2; no longer JB74.1
- net N$227: now also S66G$1.PIN-2; no longer S66.PIN-2
- net N$228: now also S47G$1.PIN-2; no longer S47.PIN-2
- net N$229: now also S53G$1.PIN-2; no longer S53.PIN-2
- net N$230: now also S60G$1.PIN-2; no longer S60.PIN-2
- net N$231: now also S68G$1.PIN-2; no longer S68.PIN-2
- net N$232: now also S75G$1.PIN-2; no longer S75.PIN-2
- net N$233: now also S82G$1.PIN-2; no longer S82.PIN-2
- net N$234: now also S48G$1.PIN-2; no longer S48.PIN-2
- net N$235: now also S54G$1.PIN-2; no longer S54.PIN-2
- net N$236: now also S61G$1.PIN-2; no longer S61.PIN-2
- net N$237: now also S69G$1.PIN-2; no longer S69.PIN-2
- net N$238: now also JA57.1, S57G$1.PIN-1; no longer JA76.1, S76.PIN-2
- net N$239: now also S83G$1.PIN-1; no longer S83.PIN-2
- net N$240: now also S49G$1.PIN-2; no longer S49.PIN-2
- net N$241: now also S55G$1.PIN-2; no longer S55.PIN-2
- net N$242: now also JA64.1, S64G$1.PIN-1; no longer JA62.1, S62.PIN-2
- net N$243: now also S70G$1.PIN-2; no longer S70.PIN-2
- net N$244: now also S77G$1.PIN-2; no longer S77.PIN-2
- net N$245: now also JB80.2, S80G$1.PIN-2; no longer JA84.1, S84.PIN-2
- net N$246: now also S50G$1.PIN-1; no longer S50.PIN-2
- net N$247: now also S56G$1.PIN-2; no longer S56.PIN-2
- net N$248: now also S63G$1.PIN-2; no longer S63.PIN-2
- net N$249: now also J19.P$1, J20.P$2; no longer JA71.1, S71.PIN-2
- net N$250: now also S78G$1.PIN-1; no longer S78.PIN-2
- net N$251: now also S85G$1.PIN-1; no longer S85.PIN-2
- net N$252: now also S51G$1.PIN-2; no longer S51.PIN-2
- net N$253: now also JB64.2, S64G$1.PIN-2; no longer JA57.1, S57.PIN-2
- net N$254: now also JB72.2, S72G$1.PIN-2; no longer JA64.1, S64.PIN-2
- net N$255: now also S72G$1.PIN-1; no longer S72.PIN-2
- net N$256: now also S79G$1.PIN-1; no longer S79.PIN-2
- net N$257: now also JB62.2, S62G$1.PIN-2; no longer JA86.1, S86.PIN-2
- net N$258: now also S52G$1.PIN-2; no longer S52.PIN-2
- net N$259: now also JA65.1, S65G$1.PIN-1; no longer JA58.1, S58.PIN-2
- net N$260: now also JA58.1, S58G$1.PIN-1; no longer JA65.1, S65.PIN-2
- net N$261: now also JB84.2, S84G$1.PIN-2; no longer JA73.1, S73.PIN-2
- net N$262: now also JA84.1, S84G$1.PIN-1; no longer JA80.1, S80.PIN-2
- net N$263: now also S81G$1.PIN-1; no longer S81.PIN-2
- net N$264: now also S67G$1.PIN-1; no longer S67.PIN-2, S67B.PIN-2, S67C.PIN-1
- net N$265: now also S59G$1.PIN-1; no longer S59.PIN-2
- net N$267: now also S74G$1.PIN-1; no longer S74.PIN-2
- net N$70: now also JA67B1.1, S67B.PIN-2; no longer JB74B.2, S74.PIN-1
- net N$71: now also S52G$1.PIN-1; no longer S52.PIN-1
- net N$84: now also S63G$1.PIN-1; no longer S63.PIN-1
- net N$89: now also JA67B.1, S67CG$1.PIN-1; no longer JB73.2, S73.PIN-1
- net N$94: now also S74AG$1.PIN-1; no longer S74A.PIN-1
- net N$97: now also S74AG$1.PIN-2; no longer S74A.PIN-2
Other:
- note added: "d1"
- note added: "d2"
- note added: "d3"
- note added: "gnd"
- note added: "kbb1"
- note added: "kbb2"
- note added: "kbb3"
- note added: "kbb4"
- note added: "kbb5"
- note added: "kbb6"
- note added: "vcc"
