File: PCB/NumPad-MUSB/NumPad.brd (EAGLE design)
At the start: 88.9 x 142.9 mm, 174 parts, among them J1 J, J10 J, J11 J, J12 J, J13 J, J14 J, J15 J, J16 J, J17 J, J2 J, J3 J, J4 J, J5 J, J6 J, J7 J, J8 J, J9 J

Commit message: fix b
Parts:
- moved J14 0.45 mm to (35.9, 141.3)
Changed lines of the file:
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@@
 </element>
 <element name="R2" library="rcl" package="R1206W" value="10k" x="28.8925" y="140.97" smashed="yes" rot="MR0">
-<attribute name="NAME" x="33.3375" y="140.0175" size="1.27" layer="26" rot="MR0"/>
+<attribute name="NAME" x="33.9725" y="140.0175" size="1.27" layer="26" rot="MR0"/>
 <attribute name="VALUE" x="30.7975" y="138.43" size="1.27" layer="28" rot="MR0"/>
 </element>
@@
 <element name="LED1" library="detali" package="LED5MM" value="" x="53.0225" y="138.43" rot="R180"/>
 <element name="R5" library="rcl" package="R1206W" value="" x="58.1025" y="138.7475" rot="MR0"/>
-<element name="J14" library="detali" package="R1206W" value="J" x="36.195" y="141.605" rot="MR225"/>
+<element name="J14" library="detali" package="R1206W" value="J" x="35.8775" y="141.2875" smashed="yes" rot="MR225">
+<attribute name="NAME" x="38.0774375" y="143.0065125" size="1.27" layer="26" rot="MR225"/>
+<attribute name="VALUE" x="36.326515625" y="144.4305875" size="1.27" layer="28" rot="MR225"/>
+</element>
 <element name="J15" library="detali" package="R1206W" value="J" x="58.1025" y="136.525" smashed="yes" rot="MR180">
 <attribute name="NAME" x="52.07" y="136.8425" size="1.27" layer="26" rot="MR180"/>
@@
 </element>
 <element name="C1" library="rcl" package="C1206" value="" x="79.6925" y="139.065" rot="MR75"/>
-<element name="D1" library="detali" package="SOD80C" value="LL4148" x="23.8125" y="145.415" rot="R270"/>
-<element name="D2" library="detali" package="SOD80C" value="LL4148" x="27.94" y="148.9075" rot="R180"/>
+<element name="D1" library="detali" package="SOD80C" value="LL4148" x="23.8125" y="145.415" smashed="yes" rot="R270">
+<attribute name="NAME" x="21.1455" y="144.2085" size="1.27" layer="26" rot="MR90"/>
+<attribute name="VALUE" x="21.3995" y="142.621" size="1.27" layer="28" rot="MR90"/>
+</element>
+<element name="D2" library="detali" package="SOD80C" value="LL4148" x="27.94" y="148.9075" smashed="yes" rot="R180">
+<attribute name="NAME" x="26.416" y="151.5745" size="1.27" layer="26" rot="MR180"/>
+<attribute name="VALUE" x="25.146" y="151.3205" size="1.27" layer="28" rot="MR180"/>
+</element>
 <element name="C2" library="rcl" package="C1206" value="" x="31.4325" y="149.5425"/>
 <element name="U$1" library="kbmx" package="18X18" value="" x="89.8525" y="31.115" smashed="yes"/>
@@
 <contactref element="J14" pad="1"/>
 <contactref element="R3" pad="1"/>
-<wire x1="35.13505" y1="142.66495" x2="33.9725" y2="145.0975" width="1.016" layer="16"/>
+<wire x1="34.81755" y1="142.34745" x2="33.9725" y2="145.0975" width="1.016" layer="16"/>
 <wire x1="33.9725" y1="145.0975" x2="36.5125" y2="145.0975" width="1.016" layer="16"/>
 <wire x1="36.5125" y1="145.0975" x2="39.0525" y2="145.0975" width="1.016" layer="16"/>
@@
 <wire x1="49.8475" y1="139.7" x2="46.0375" y2="139.7" width="1.016" layer="16"/>
 <wire x1="46.0375" y1="139.7" x2="43.287453125" y2="140.862546875" width="1.016" layer="16"/>
-<wire x1="43.287453125" y1="140.862546875" x2="37.254953125" y2="140.545046875" width="0.8128" layer="16"/>
+<wire x1="43.287453125" y1="140.862546875" x2="36.937453125" y2="140.227546875" width="0.8128" layer="16"/>
 <wire x1="67.31" y1="143.51" x2="69.215" y2="141.605" width="0.8128" layer="16"/>
 <wire x1="65.9765" y1="135.2935" x2="67.9835" y2="135.2935" width="0.8128" layer="16"/>

Commit message: pcb b
Parts:
- moved JB93 2.88 mm to (54.9, 99.7)
- moved JA93 1.71 mm to (46.7, 102.6)
- moved D92 1.27 mm to (45.1, 89.9)
- moved J5 0.64 mm to (64.5, 90.2)
Routing:
- net N$288: track 8.75 -> 11.2 mm
- net N$1: track 59.6 -> 61.4 mm
- net N$287: track 3.50 -> 5.22 mm
- net N$286: track 2.41 -> 3.44 mm
- net N$284: track 9.62 -> 10.5 mm
- net N$12: track 39.1 -> 38.5 mm
- net N$15: track 17.5 -> 18.0 mm
Other:
- outline, holes or cut-outs redrawn
