File: PCB/keyBoard_A_GPad/keyBoard_B.brd (EAGLE design)
At the start: 488.3 x 207 mm, 427 parts, among them IC1 74HC04N, IC2 LMV358IDGKR, J1 J, J10 J, J11 J, J12 J, J13 J, J14 J, J15 J, J16 J, J17 J, J18 J, J19 J, J2 J, J20 J, J21 J, J22 J, J23 J, J24 J, J25 J, J26 J, J27 J, J28 J, J29 J, J3 J, J30 J, J31 J, J32 J, J33 J, J34 J, J35 J, J36 J, J37 J, J38 J, J39 J, J4 J, J40 J, J41 J, J42 J, J43 J, J44 J, J45 J, J47 USB MICRO, J5 J, J6 J, J7 J, J8 J, J9 J, Y1 16MHz KX-7, Y2 16MHz KX-7

Commit message: fix b
Parts:
- moved C15 254.0 mm to (185.7, -418.5)
- moved C22 254.0 mm to (157.2, -407.0)
- moved C3 254.0 mm to (187.6, -418.5)
- moved C4 254.0 mm to (173.0, -435.6)
- moved C6 254.0 mm to (191.5, -435.6)
- moved C8 254.0 mm to (147.0, -416.6)
- moved IC2 254.0 mm to (155.3, -410.8)
- moved ICSP 254.0 mm to (211.9, -416.6)
- moved J47 254.0 mm to (135.8, -407.0)
- moved L1 254.0 mm to (189.5, -418.5)
- moved R4 254.0 mm to (182.6, -419.7)
- moved RESET 254.0 mm to (140.7, -395.7)
- moved RN1 254.0 mm to (164.8, -426.7)
- moved RN3 254.0 mm to (147.0, -407.7)
- moved Y1 254.0 mm to (183.2, -416.6)
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Other:
- board size 488.3 x 207 mm -> 488.3 x 222.2 mm

Commit message: pcb b
Parts:
- removed S37A, S37B: L Shift, cherrymx:CHERRY-MX
- removed U$114: (no value), kbmx:18X33
- removed U$115: (no value), kbmx:18X28
- added R10, R11, R12, R13, R14, R15: (no value), rcl:M0805
- S37: device cherrymx:CHERRY-MX -> cherrymx:CHERRY-MX-4P
- S44: value Alt -> F1
- S45: value F1 -> L_Alt
- U$22: device kbmx:18X42 -> kbmx:18X37
- moved D37 24.8 mm to (88.9, -325.1), turned to 90 degrees
- moved JB37 18.5 mm to (81.9, -333.4), turned to 0 degrees
- moved JA37 14.5 mm to (67.9, -334.6), turned to 0 degrees
- moved D48 4.14 mm to (2.86, -332.7), turned to 0 degrees
- moved S37 2.54 mm to (74.3, -330.8), turned to 180 degrees
- moved U$22 2.54 mm to (74.3, -330.8)
- moved C18 1.35 mm to (17.1, -338.1), turned to 90 degrees
- moved D12 0.90 mm to (68.9, -340.0)
Connections:
- removed net N$107: S37A.SW1, S37B.SW1
- removed net N$274: S37A.SW2, S37B.SW2
- net +5V: now also R10.1, R11.1, R12.1, R13.1, R14.1, R15.1
- net L1: now also R10.2
- net L4: now also R13.2
- net L5: now also R14.2
- net L6: now also R15.2
- net N$150: now also R11.2
- net N$193: now also R12.2
Routing:
- net N$56: track 14.8 -> 5.21 mm
- net 4J3: track 56.6 -> 50.9 mm
- net N$273: track 4.32 -> 0.00 mm
- net 3J3: track 42.5 -> 38.6 mm
- net N$62: track 3.05 -> 0.00 mm
- net N$274: track 2.54 -> 0.00 mm
- net N$107: track 2.54 -> 0.00 mm
- net GND: track 299.8 -> 301.7 mm
- net L5: track 178.1 -> 177.4 mm
