File: PCB/keyBoard_A_GPad/keyBoard_B.sch (EAGLE design)
At the start: 285 parts, among them IC1 74HC04N, IC2 LMV358IDGKR, J1 J, J10 J, J11 J, J12 J, J13 J, J14 J, J15 J, J16 J, J17 J, J18 J, J19 J, J2 J, J20 J, J21 J, J22 J, J23 J, J24 J, J25 J, J26 J, J27 J, J28 J, J29 J, J3 J, J30 J, J31 J, J32 J, J33 J, J34 J, J35 J, J36 J, J37 J, J38 J, J39 J, J4 J, J40 J, J41 J, J42 J, J43 J, J44 J, J45 J, J47 USB MICRO, J5 J, J6 J, J7 J, J8 J, J9 J, Y1 16MHz KX-7, Y2 16MHz KX-7

Commit message: pcb b
Parts:
- removed S37A, S37B: L Shift, cherrymx:CHERRY-MX
- added R10, R11, R12, R13, R14, R15: (no value), rcl:R-EU_M0805
- S37: device cherrymx:CHERRY-MX -> cherrymx:CHERRY-MX-4P
- S44: value Alt -> F1
- S45: value F1 -> L_Alt
Connections:
- removed net N$107: S37A.PIN-1, S37B.PIN-1
- removed net N$274: S37A.PIN-2, S37B.PIN-2
- net +5V: now also R10.1, R11.1, R12.1, R13.1, R14.1, R15.1
- net L1: now also R10.2
- net L4: now also R13.2
- net L5: now also R14.2
- net L6: now also R15.2
- net N$150: now also R11.2
- net N$193: now also R12.2
- net N$273: now also S37G$1.PIN-2; no longer S37.PIN-2
- net N$62: now also S37G$1.PIN-1; no longer S37.PIN-1
Changed lines of the file:
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@@
 <part name="S35" library="cherrymx" deviceset="CHERRY-MX-4P" device="" value="F"/>
 <part name="S36" library="cherrymx" deviceset="CHERRY-MX-4P" device="" value="G"/>
-<part name="S37" library="cherrymx" deviceset="CHERRY-MX" device="" value="L Shift"/>
+<part name="S37" library="cherrymx" deviceset="CHERRY-MX-4P" device="" value="L Shift"/>
 <part name="S38" library="cherrymx" deviceset="CHERRY-MX-4P" device="" value="Z"/>
 <part name="S39" library="cherrymx" deviceset="CHERRY-MX-4P" device="" value="X"/>
@@
 <part name="S42" library="cherrymx" deviceset="CHERRY-MX-4P" device="" value="B"/>
 <part name="S43" library="cherrymx" deviceset="CHERRY-MX-4P" device="" value="Caps Lock"/>
-<part name="S44" library="cherrymx" deviceset="CHERRY-MX-4P" device="" value="Alt"/>
-<part name="S45" library="cherrymx" deviceset="CHERRY-MX-4P" device="" value="F1"/>
+<part name="S44" library="cherrymx" deviceset="CHERRY-MX-4P" device="" value="F1"/>
+<part name="S45" library="cherrymx" deviceset="CHERRY-MX-4P" device="" value="L_Alt"/>
 <part name="S46" library="cherrymx" deviceset="CHERRY-MX-4P" device="" value="Space"/>
 <part name="JB1" library="detali" deviceset="SJ" device=""/>
@@
 <part name="D45" library="detali" deviceset="LL4148" device=""/>
 <part name="D46" library="detali" deviceset="LL4148" device=""/>
-<part name="S37A" library="cherrymx" deviceset="CHERRY-MX" device="" value="L Shift"/>
-<part name="S37B" library="cherrymx" deviceset="CHERRY-MX" device="" value="L Shift"/>
 <part name="ICSP" library="SmartPrj" deviceset="PINHD-2X3" device="" value="ICSP"/>
 <part name="P+4" library="supply1" deviceset="+5V" device=""/>
@@
 <part name="R3" library="rcl" deviceset="R-EU_" device="R1206W"/>
 <part name="R9" library="rcl" deviceset="R-EU_" device="R1206W"/>
+<part name="R10" library="rcl" deviceset="R-EU_" device="M0805"/>
+<part name="R11" library="rcl" deviceset="R-EU_" device="M0805"/>
+<part name="R12" library="rcl" deviceset="R-EU_" device="M0805"/>
+<part name="R13" library="rcl" deviceset="R-EU_" device="M0805"/>
+<part name="R14" library="rcl" deviceset="R-EU_" device="M0805"/>
+<part name="R15" library="rcl" deviceset="R-EU_" device="M0805"/>
+<part name="P+13" library="supply1" deviceset="+5V" device=""/>
 </parts>
 <sheets>
@@
 <instance part="D45" gate="G$1" x="165.1" y="142.24"/>
 <instance part="D46" gate="G$1" x="165.1" y="132.08"/>
-<instance part="S37A" gate="G$1" x="124.46" y="195.58"/>
-<instance part="S37B" gate="G$1" x="124.46" y="203.2"/>
 <instance part="1D0" gate="G$1" x="538.48" y="314.96"/>
 <instance part="1D1" gate="A" x="101.6" y="320.04"/>
@@
 <instance part="R3" gate="G$1" x="297.18" y="198.12"/>
 <instance part="R9" gate="G$1" x="297.18" y="187.96"/>
+<instance part="R10" gate="G$1" x="254" y="332.74"/>
+<instance part="R11" gate="G$1" x="254" y="322.58"/>
+<instance part="R12" gate="G$1" x="254" y="309.88"/>
+<instance part="R13" gate="G$1" x="254" y="297.18"/>
+<instance part="R14" gate="G$1" x="254" y="284.48"/>
+<instance part="R15" gate="G$1" x="254" y="271.78"/>
+<instance part="P+13" gate="1" x="246.38" y="337.82" smashed="yes">
+<attribute name="VALUE" x="248.92" y="340.36" size="1.778" layer="96" rot="R180"/>
+</instance>
 </instances>
 <busses>
@@
 <pinref part="JA37" gate="1" pin="1"/>
 <wire x1="134.62" y1="182.88" x2="137.16" y2="182.88" width="0.1524" layer="91"/>
-</segment>
-</net>
-<net name="N$107" class="0">
-<segment>
-<pinref part="S37B" gate="G$1" pin="PIN-1"/>
-<wire x1="119.38" y1="203.2" x2="116.84" y2="203.2" width="0.1524" layer="91"/>
-<wire x1="116.84" y1="203.2" x2="116.84" y2="195.58" width="0.1524" layer="91"/>
-<pinref part="S37A" gate="G$1" pin="PIN-1"/>
-<wire x1="116.84" y1="195.58" x2="119.38" y2="195.58" width="0.1524" layer="91"/>
-</segment>
-</net>
-<net name="N$274" class="0">
-<segment>
-<pinref part="S37A" gate="G$1" pin="PIN-2"/>
-<wire x1="129.54" y1="195.58" x2="132.08" y2="195.58" width="0.1524" layer="91"/>
-<wire x1="132.08" y1="195.58" x2="132.08" y2="203.2" width="0.1524" layer="91"/>
-<pinref part="S37B" gate="G$1" pin="PIN-2"/>
-<wire x1="132.08" y1="203.2" x2="129.54" y2="203.2" width="0.1524" layer="91"/>
 </segment>
 </net>
@@
 <wire x1="279.4" y1="187.96" x2="279.4" y2="198.12" width="0.1524" layer="91"/>
 <junction x="279.4" y="198.12"/>
+</segment>
+<segment>
+<pinref part="R10" gate="G$1" pin="1"/>
+<wire x1="248.92" y1="332.74" x2="246.38" y2="332.74" width="0.1524" layer="91"/>
+<wire x1="246.38" y1="332.74" x2="246.38" y2="322.58" width="0.1524" layer="91"/>
+<pinref part="R11" gate="G$1" pin="1"/>
+<wire x1="246.38" y1="322.58" x2="248.92" y2="322.58" width="0.1524" layer="91"/>
+<wire x1="246.38" y1="322.58" x2="246.38" y2="309.88" width="0.1524" layer="91"/>
+<pinref part="R12" gate="G$1" pin="1"/>
+<wire x1="246.38" y1="309.88" x2="248.92" y2="309.88" width="0.1524" layer="91"/>
+<wire x1="246.38" y1="309.88" x2="246.38" y2="297.18" width="0.1524" layer="91"/>
+<pinref part="R13" gate="G$1" pin="1"/>
+<wire x1="246.38" y1="297.18" x2="248.92" y2="297.18" width="0.1524" layer="91"/>
+<wire x1="246.38" y1="297.18" x2="246.38" y2="284.48" width="0.1524" layer="91"/>
+<pinref part="R14" gate="G$1" pin="1"/>
+<wire x1="246.38" y1="284.48" x2="248.92" y2="284.48" width="0.1524" layer="91"/>
+<wire x1="246.38" y1="284.48" x2="246.38" y2="271.78" width="0.1524" layer="91"/>
+<pinref part="R15" gate="G$1" pin="1"/>
+<wire x1="246.38" y1="271.78" x2="248.92" y2="271.78" width="0.1524" layer="91"/>
+<pinref part="P+13" gate="1" pin="+5V"/>
+<wire x1="246.38" y1="335.28" x2="246.38" y2="332.74" width="0.1524" layer="91"/>
+<junction x="246.38" y="332.74"/>
+<junction x="246.38" y="322.58"/>
+<junction x="246.38" y="309.88"/>
+<junction x="246.38" y="297.18"/>
+<junction x="246.38" y="284.48"/>
 </segment>
 </net>
@@
 <wire x1="266.7" y1="335.28" x2="292.1" y2="335.28" width="0.1524" layer="91"/>
 <label x="266.7" y="335.28" size="1.778" layer="95"/>
+</segment>
+<segment>
+<pinref part="R10" gate="G$1" pin="2"/>
+<wire x1="266.7" y1="332.74" x2="259.08" y2="332.74" width="0.1524" layer="91"/>
+<label x="261.62" y="332.74" size="1.778" layer="95"/>
 </segment>
 </net>
@@
 <label x="269.24" y="297.18" size="1.778" layer="95"/>
 </segment>
+<segment>
+<pinref part="R13" gate="G$1" pin="2"/>
+<wire x1="266.7" y1="297.18" x2="259.08" y2="297.18" width="0.1524" layer="91"/>
+<label x="261.62" y="297.18" size="1.778" layer="95"/>
+</segment>
 </net>
 <net name="L5" class="0">
@@
 <wire x1="266.7" y1="284.48" x2="292.1" y2="284.48" width="0.1524" layer="91"/>
 <label x="269.24" y="284.48" size="1.778" layer="95"/>
+</segment>
+<segment>
+<pinref part="R14" gate="G$1" pin="2"/>
+<wire x1="266.7" y1="284.48" x2="259.08" y2="284.48" width="0.1524" layer="91"/>
+<label x="261.62" y="284.48" size="1.778" layer="95"/>
 </segment>
 </net>
@@
 <label x="269.24" y="271.78" size="1.778" layer="95"/>
 </segment>
+<segment>
+<pinref part="R15" gate="G$1" pin="2"/>
+<wire x1="266.7" y1="271.78" x2="259.08" y2="271.78" width="0.1524" layer="91"/>
+<label x="261.62" y="271.78" size="1.778" layer="95"/>
+</segment>
 </net>
 <net name="N$60" class="0">
@@
 <wire x1="279.4" y1="322.58" x2="281.94" y2="322.58" width="0.1524" layer="91"/>
 </segment>
+<segment>
+<pinref part="R11" gate="G$1" pin="2"/>
+<wire x1="266.7" y1="322.58" x2="259.08" y2="322.58" width="0.1524" layer="91"/>
+<label x="261.62" y="322.58" size="1.778" layer="95"/>
+</segment>
 </net>
 <net name="N$193" class="0">
@@
 <wire x1="281.94" y1="309.88" x2="292.1" y2="309.88" width="0.1524" layer="91"/>
 </segment>
-</net>
+<segment>
+<pinref part="R12" gate="G$1" pin="2"/>
+<wire x1="266.7" y1="309.88" x2="259.08" y2="309.88" width="0.1524" layer="91"/>
+<label x="261.62" y="309.88" size="1.778" layer="95"/>
+</segment>
+</net>
