File: PCB/keyBoard_A_GPad/keyBoard_A.brd (EAGLE design)
At the start: 386.7 x 253 mm, 625 parts, among them IC1 74HC04N, IC2 LMV358IDGKR, J1 J, J10 J, J11 J, J12 J, J13 J, J14 J, J15 J, J16 J, J17 J, J18 J, J19 J, J2 J, J20 J, J21 J, J22 J, J23 J, J24 J, J25 J, J26 J, J27 J, J28 J, J29 J, J3 J, J30 J, J31 J, J32 J, J33 J, J34 J, J35 J, J36 J, J37 J, J38 J, J39 J, J4 J, J40 J, J41 J, J42 J, J43 J, J44 J, J45 J, J47 USB MICRO, J5 J, J6 J, J7 J, J8 J, J9 J, Y1 16MHz KX-7, Y3 16MHz KX-7

Commit message: pcb b > ab .2
Parts:
- removed J84, J85, J86: (no value), detali2:R1206W
- removed U$116: (no value), kbmx:18X18
- added U$81: (no value), kbmx:18X18
- moved J83 57.8 mm to (324.5, -273.1), turned to 270 degrees
- moved 2D1 26.8 mm to (321.9, -254.6), turned to 275 degrees
- moved C19 26.5 mm to (320.7, -248.0)
- moved R16 26.3 mm to (321.0, -256.2)
- moved D69 22.6 mm to (331.2, -302.6)
- moved J88 16.7 mm to (325.4, -278.1)
- moved JA59 13.1 mm to (339.1, -279.4), turned to 180 degrees
- moved D64B 8.64 mm to (330.2, -242.6)
- moved J46 7.63 mm to (303.2, -255.0)
- moved J80 7.63 mm to (303.2, -257.2)
- moved J81 7.63 mm to (303.2, -261.6)
- moved J82 7.63 mm to (303.2, -259.4)
- moved JA74B 7.13 mm to (341.0, -253.4), turned to 90 degrees
- moved J94 6.03 mm to (308.9, -337.5)
- moved D83 6.03 mm to (308.9, -335.0)
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Connections:
- net N$401 renamed B5J4
- removed net N$392: 2D1.1, J83.1
- removed net N$393: 2D1.2, J84.1
- removed net N$394: 2D1.3, J85.1
- removed net N$395: 2D1.15, J86.2
- removed net N$398: 2D1.7, J88.2
- removed net N$404: 2D1.10, J92.2
- new net B5J5: 2D1.10, D69.C, J92.2
- new net N$117: 2D1.7, J83.2
- new net N$197: J83.1, J88.2
- net B1: now also 2D1.15; no longer J86.1
- net B5: no longer D69.C
- net N$388: now also 2D1.1; no longer J83.2
- net N$389: now also 2D1.2; no longer J84.2
- net N$391: now also 2D1.3; no longer J85.2
Routing:
- net B5J5: track 0.00 -> 64.5 mm
- net N$404: track 58.6 -> 0.00 mm
- net +5V_B: track 192.7 -> 134.7 mm
- net GND_B: track 180.8 -> 140.4 mm
- net 2I: track 167.9 -> 133.2 mm
- net N$395: track 18.0 -> 0.00 mm
- net N$389: track 0.00 -> 15.9 mm
- net B3J: track 71.2 -> 55.4 mm
- net N$388: track 0.00 -> 15.3 mm
- net B1: track 137.4 -> 123.2 mm
- net N$391: track 0.00 -> 14.2 mm
- net N$117: track 0.00 -> 12.9 mm
- net N$403: track 82.4 -> 94.5 mm
- net G6: track 166.8 -> 175.8 mm
- net N$398: track 8.77 -> 0.00 mm
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Other:
- board size 386.7 x 253 mm -> 358.8 x 253 mm
