File: PCB/keyBoard_B/keyBoard_B.brd (EAGLE design)
At the start: 494 x 340.4 mm, 762 parts, among them IC1 MEGA8-AI, J1 J, J10 J, J11 J, J12 J, J13 J, J14 J, J15 J, J16 J, J17 J, J2 J, J3 J, J4 J, J5 J, J6 J, J7 J, J8 J, J9 J

Commit message: move +m2
Parts:
- removed D100, D101, D102, D103, D104, D105, D106, D107, D108, D109, D110, D87, D88, D89, D90, D91, D92, D93, D94, D95, D96, D97, D98, D99: LL4148, detali:SOD80C
- removed HL4: (no value), led:RGB2X5
- removed IC1: MEGA8-AI, atmel:TQFP32-08
- removed JA100, JA101, JA102, JA103, JA104, JA105, JA106, JA107, JA108, JA109, JA110, JA87, JA88, JA89, JA90, JA91, JA92, JA93, JA94, JA95, JA96, JA97, JA98, JA99, JB100, JB101, JB102, JB103, JB104, JB105, JB106, JB107, JB108, JB109, JB110, JB87, JB88, JB89, JB90, JB91, JB92, JB93, JB94, JB95, JB96, JB97, JB98, JB99: (no value), detali:SJ
- removed S100: 4, cherrymx:CHERRY-MX-4P
- removed S101: 5, cherrymx:CHERRY-MX-4P
- removed S102: 6, cherrymx:CHERRY-MX-4P
- removed S103: +, cherrymx:CHERRY-MX-4P
- removed S104: 1, cherrymx:CHERRY-MX-4P
- removed S105: 2, cherrymx:CHERRY-MX-4P
- removed S106: 3, cherrymx:CHERRY-MX-4P
- removed S107: NumEnter, cherrymx:CHERRY-MX-4P
- removed S107B: NumEnter, cherrymx:CHERRY-MX
- removed S108: 0, cherrymx:CHERRY-MX-4P
- removed S109: 00, cherrymx:CHERRY-MX-4P
- removed S110: ., cherrymx:CHERRY-MX-4P
- removed S67B: |, cherrymx:CHERRY-MX
- removed S74B: Enter, cherrymx:CHERRY-MX
- removed S87: Num, cherrymx:CHERRY-MX-4P
- removed S88: D, cherrymx:CHERRY-MX-4P
- removed S89: E, cherrymx:CHERRY-MX-4P
- removed S90: F, cherrymx:CHERRY-MX-4P
- removed S91: /, cherrymx:CHERRY-MX-4P
- removed S92: A, cherrymx:CHERRY-MX-4P
- removed S93: B, cherrymx:CHERRY-MX-4P
- removed S94: C, cherrymx:CHERRY-MX-4P
- removed S95: *, cherrymx:CHERRY-MX-4P
- removed S96: 7, cherrymx:CHERRY-MX-4P
- removed S97: 8, cherrymx:CHERRY-MX-4P
- removed S98: 9, cherrymx:CHERRY-MX-4P
- removed S99: -, cherrymx:CHERRY-MX-4P
- removed SV2: (no value), con-lsta:FE06
- removed SV3: (no value), con-lsta:FE07
- removed U$100, U$101, U$102, U$103, U$104, U$105, U$106, U$107, U$108, U$109, U$110, U$87, U$88, U$89, U$90, U$91, U$92, U$93, U$94, U$95, U$96, U$97, U$98, U$99: (no value), kbmx:18X18
- removed U$111: (no value), kbmx:37X18
- removed U$113: (no value), kbmx:18X28
- added 3D3: 74AC138N, detali2:DIL16
- added JA67B, JB67B: (no value), detali:SJ
- S47, S48, S49, S50, S51, S52, S53, S54, S55, S56, S57, S58, S59, S60, S61, S62, S63, S64, S65, S66, S67, S67C, S68, S69, S70, S71, S72, S73, S74, S74A, S75, S76, S77, S78, S79, S80, S81, S82, S83, S84, S85, S86: device cherrymx:CHERRY-MX -> cherrymx:CHERRY-MX-4P
- moved R3 169.5 mm to (17.1, 169.5)
- moved JA67 61.1 mm to (325.1, 40.0), turned to 270 degrees
- moved D67 41.6 mm to (328.9, 67.9), turned to 180 degrees
- moved JB67 38.8 mm to (330.2, 60.3), turned to 90 degrees
- moved D81 31.3 mm to (365.8, 36.2), turned to 90 degrees
- moved D64B 25.3 mm to (368.3, 119.4)
- moved D84 24.0 mm to (317.5, 10.8)
- moved JB83 22.2 mm to (288.3, 14.0), turned to 270 degrees
- moved D86 22.2 mm to (367.7, 27.3)
- moved JB85 18.9 mm to (340.4, 21.0)
- moved JB84 18.9 mm to (311.8, 14.6), turned to 270 degrees
- moved JA52 17.8 mm to (314.3, 121.3)
- moved JB86 16.5 mm to (363.2, 24.1)
- moved D85 15.9 mm to (340.4, 27.3), turned to 90 degrees
- moved JB65 15.9 mm to (323.2, 76.2)
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Connections:
- removed net 3A1: JA103.2, JA89.2, JA96.2, JA97.2, JA98.2, SV2.1
- removed net 3A2: JA100.2, JA101.2, JA102.2, SV2.2
- removed net 3A3: JA104.2, JA105.2, JA106.2, JA107.2, JA88.2, JA90.2, JA92.2, SV2.3
- removed net 3A4: JA108.2, JA110.2, SV2.4
- removed net 3A5: JA87.2, JA91.2, JA94.2, JA95.2, SV2.5
- removed net 3A6: JA93.2, JA99.2, SV2.6
- removed net 3B0: D92.C, SV3.1
- removed net 3B10: D100.C, D104.C, D87.C, D96.C, SV3.7
- removed net 3B2: D88.C, D89.C, D94.C, SV3.2
- removed net 3B3: D90.C, D93.C, SV3.3
- removed net 3B7: D103.C, D107.C, SV3.4
- removed net 3B8: D102.C, D106.C, D110.C, D95.C, D98.C, D99.C, SV3.5
- removed net 3B9: D101.C, D105.C, D108.C, D91.C, D97.C, SV3.6
- removed net AVCC: IC1.18
- removed net N$269: D88.A, JB88.1
- removed net N$270: JB87.2, S87.SW1
- removed net N$271: JB88.2, S88.SW1
- removed net N$272: JA87.1, S87.SW2
- removed net N$273: JA88.1, S88.SW2
- removed net N$274: D89.A, JB89.1
- removed net N$275: JB89.2, S89.SW1
- removed net N$276: JA89.1, S89.SW2
- removed net N$277: D90.A, JB90.1
- removed net N$278: JB90.2, S90.SW1
- removed net N$279: JA90.1, S90.SW2
- removed net N$280: D91.A, JB91.1
- removed net N$281: JB91.2, S91.SW1
- removed net N$282: JA91.1, S91.SW2
- removed net N$283: JB92.2, S92.SW1
- removed net N$284: D92.A, JB92.1
- removed net N$285: JA92.1, S92.SW2
- removed net N$286: JA93.1, S93.SW2
- removed net N$287: JB93.2, S93.SW1
- removed net N$288: D93.A, JB93.1
- removed net N$289: D94.A, JB94.1
- removed net N$290: JB94.2, S94.SW1
- removed net N$291: JA94.1, S94.SW2
- removed net N$292: D95.A, JB95.1
- removed net N$293: JB95.2, S95.SW1
- removed net N$294: JA95.1, S95.SW2
- removed net N$295: D96.A, JB96.1
- removed net N$296: JB96.2, S96.SW1
- removed net N$297: JA96.1, S96.SW2
- removed net N$298: JB97.2, S97.SW1
- removed net N$299: JA97.1, S97.SW2
- removed net N$300: D97.A, JB97.1
- removed net N$301: D98.A, JB98.1
- removed net N$302: JB98.2, S98.SW1
- removed net N$303: JA98.1, S98.SW2
- removed net N$304: D99.A, JB99.1
- removed net N$305: JB99.2, S99.SW1
- removed net N$306: JA99.1, S99.SW2
- removed net N$307: D100.A, JB100.1
- removed net N$308: JB100.2, S100.SW1
- removed net N$309: JA100.1, S100.SW2
- removed net N$310: JB101.2, S101.SW1
- removed net N$311: D101.A, JB101.1
- removed net N$312: JA101.1, S101.SW2
- removed net N$313: D102.A, JB102.1
- removed net N$314: JB102.2, S102.SW1
- removed net N$315: JA102.1, S102.SW2
- removed net N$316: D103.A, JB103.1
- removed net N$317: JB103.2, S103.SW1
- removed net N$318: JA103.1, S103.SW2
- removed net N$319: JB107.2, S107.SW1, S107B.SW1
- removed net N$320: JB104.2, S104.SW1
- removed net N$321: JA104.1, S104.SW2
- removed net N$322: JB105.2, S105.SW1
- removed net N$323: D105.A, JB105.1
- removed net N$324: JA105.1, S105.SW2
- removed net N$325: D106.A, JB106.1
- removed net N$326: JB106.2, S106.SW1
- removed net N$327: JA106.1, S106.SW2
- removed net N$328: D107.A, JB107.1
- removed net N$329: JB108.2, S108.SW1
- removed net N$330: JA108.1, S108.SW2
- removed net N$331: D108.A, JB108.1
- removed net N$332: JB109.2, S109.SW1
- removed net N$333: D109.A, JB109.1
- removed net N$334: JA109.1, S109.SW2
- removed net N$335: D110.A, JB110.1
- removed net N$336: JB110.2, S110.SW1
- removed net N$337: JA110.1, S110.SW2
- net GND: now also 3D3.8; no longer IC1.21, IC1.3, IC1.5
- net N$185: no longer S67B.SW1, S67C.SW2
- net N$224: now also JB67B.1
- net N$264: no longer S67B.SW2, S67C.SW1
- net N$268: now also JA67.2, JA67B.2; no longer D87.A, JB87.1
- net N$51: now also JB67B.2, S67C.SW2; no longer JA107.1, S107.SW2, S107B.SW2
- net N$60: now also JA67B.1, S67C.SW1; no longer D104.A, JB104.1
- net N$94: no longer S74B.SW1
- net N$97: no longer S74B.SW2
- net VCC: now also 3D3.16; no longer IC1.4, IC1.6
Routing:
- net 3A4: track 209.3 -> 0.00 mm
- net 3A3: track 184.2 -> 0.00 mm
- net 3B8: track 180.5 -> 0.00 mm
- net 3A5: track 146.4 -> 0.00 mm
- net 3B10: track 140.9 -> 0.00 mm
- net 3B2: track 61.9 -> 0.00 mm
- net 3A1: track 60.5 -> 0.00 mm
- net 3B0: track 47.0 -> 0.00 mm
- net 3B9: track 45.2 -> 0.00 mm
- net 3A2: track 38.1 -> 0.00 mm
- net N$289: track 23.8 -> 0.00 mm
- net N$335: track 22.4 -> 0.00 mm
- net 3B7: track 17.2 -> 0.00 mm
- net N$319: track 17.1 -> 0.00 mm
- net N$295: track 14.4 -> 0.00 mm
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Other:
- board size 494 x 340.4 mm -> 485.8 x 154.9 mm

Commit message: .
Parts:
- removed 2S1: (no value), con-lsta:FE10
- removed 2S2, 2S3: (no value), con-lsta:FE08
- removed 2S4: (no value), con-lsta:FE05-1
- removed R3: 1k, rcl:R0805
- added S67C1: |, cherrymx:CHERRY-MX-4P
- added U$87: (no value), kbmx:18X42
- added U$88: CHERRY-MX, cherrymx:CHERRY-MX
- added U$89: (no value), kbmx:18X28
- added U$90: (no value), kbmx:18X18
- added U$91: (no value), kbmx:18X23
- U$14: device kbmx:18X18 -> kbmx:18X28
- moved U$14 276.3 mm to (358.1, 41.9), turned to 0 degrees
- moved U$112 75.0 mm to (341.0, -14.0)
- moved U$118 59.2 mm to (386.1, -5.08)
- moved S67C 45.0 mm to (396.2, 92.7)
- moved D83 27.3 mm to (297.8, 12.7), turned to 180 degrees
- moved JA86 14.5 mm to (360.0, 14.0)
- moved JA85 14.2 mm to (338.5, 15.2)
- moved JA83 12.8 mm to (288.9, 17.8)
- moved JB83 11.7 mm to (299.7, 16.5)
- moved JA67B 11.7 mm to (372.1, 55.9)
- moved S83 11.4 mm to (294.6, 22.9)
- moved S84 11.4 mm to (318.8, 22.9)
- moved S86 11.4 mm to (364.5, 22.9)
- moved U$83 11.4 mm to (363.2, 24.1)
- moved U$85 11.4 mm to (318.8, 22.9)
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Connections:
- removed net 2A2: 2S3.2, JA47.2, JA60.2
- removed net 2A4: 2S3.4, JA68.2, JA82.2
- removed net 2B0: 2S1.1, D53.C
- removed net 2B1: 2S1.2, D54.C
- removed net 2B10: 2S2.1, D82.C
- removed net 2B4: 2S1.5, D60.C, D61.C, D68.C, D69.C, D75.C, D76.C
- removed net 2B6: 2S1.7, D47.C, D48.C, D83.C
- removed net GND_K2: R3.1
- removed net N$152: R3.2
- net 2A6: no longer 2S3.6, JA75.2
- net 2A7: no longer 2S3.7
- net 2A8: no longer 2S3.8, JA53.2
- net N$94: now also U$88.SW1
- net N$97: now also U$88.SW2
Routing:
- net B10: track 243.7 -> 50.7 mm
- net A2: track 241.1 -> 164.1 mm
- net N$56: track 61.0 -> 0.00 mm
- net B11: track 79.6 -> 31.7 mm
- net B7: track 76.2 -> 37.6 mm
- net A6: track 37.5 -> 0.00 mm
- net B1: track 157.6 -> 141.0 mm
- net N$28: track 12.4 -> 0.00 mm
- net N$36: track 12.0 -> 0.00 mm
- net N$37: track 11.3 -> 0.00 mm
- net N$146: track 9.04 -> 0.00 mm
- net N$62: track 6.20 -> 0.00 mm
- net N$31: track 5.16 -> 0.00 mm
- net B9: track 48.5 -> 43.4 mm
- net N$23: track 5.08 -> 0.00 mm
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Other:
- board size 485.8 x 154.9 mm -> 485.8 x 150.5 mm

Commit message: arc
Parts:
- added IC1: 74ALS04N, detali2:DIL14
- added S67C2: FN1, cherrymx:CHERRY-MX-4P
- S67C1: value | -> FN2
- moved 3D3 55.9 mm to (252.7, 112.4)
- moved U$88 48.3 mm to (394.3, 61.0)
- moved U$89 13.0 mm to (393.7, 105.4)
- moved S67C 11.5 mm to (395.0, 81.3)
- moved JB83 5.24 mm to (304.8, 17.8)
- moved JA83 2.54 mm to (286.4, 17.8)
- moved S74A 2.54 mm to (346.1, 61.0)
- moved U$29 1.80 mm to (127.0, 78.7)
- moved U$23 1.80 mm to (127.0, 59.7)
- moved U$4 1.80 mm to (25.4, 88.9)
- moved U$26 1.80 mm to (165.1, 62.2)
- moved U$32 1.80 mm to (165.1, 81.3)
- moved U$35 1.80 mm to (127.0, 97.8)
- moved U$38 1.80 mm to (165.1, 100.3)
- moved U$42 1.80 mm to (165.1, 127.0)
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Connections:
- net GND: now also IC1.7
- net VCC: now also IC1.14
Routing:
- net A4: track 240.5 -> 0.00 mm
- net B3: track 207.1 -> 0.00 mm
- net A2: track 164.1 -> 0.00 mm
- net A7: track 147.5 -> 0.00 mm, vias 2 -> 0
- net A8: track 141.0 -> 0.00 mm
- net B1: track 141.0 -> 0.00 mm
- net B14: track 132.5 -> 0.00 mm, vias 2 -> 0
- net B4: track 130.9 -> 0.00 mm
- net B5: track 119.5 -> 0.00 mm
- net B2: track 111.2 -> 0.00 mm
- net B0: track 101.2 -> 0.00 mm
- net B6: track 66.2 -> 0.00 mm
- net A3: track 57.5 -> 0.00 mm
- net A5: track 57.1 -> 0.00 mm
- net N$120: track 51.5 -> 0.00 mm
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
Commit message: get all vil
Parts:
- removed 1S1, 1S1O: (no value), con-lsta:FE10
- removed 1S2, 1S2O, 1S3, 1S3O: (no value), con-lsta:FE08
- removed 1S4, 1S4O: (no value), con-lsta:FE05-1
- removed 3D1: 74HC138N, detali:DIL16
- removed 3D2: К155ЛА4, detali:DIL14
- removed 3D3: 74AC138N, detali2:DIL16
- removed D10, D11, D111, D112, D113, D114, D115, D116, D117, D118, D119, D12, D120, D121, D122, D123, D124, D125, D126, D127, D128, D129, D13, D130, D131, D132, D133, D134, D135, D136, D14, D15, D16, D17, D18, D19, D20, D21, D22, D23, D24, D25, D26, D27, D28, D29, D3, D30, D31, D32, D33, D34, D35, D36, D37, D38, D39, D4, D40, D41, D42, D43, D44, D45, D46, D5, D6, D7, D8, D9: LL4148, detali:SOD80C
- removed HL1, HL2, HL3: (no value), led:RGB2X5
- removed IC1: 74ALS04N, detali2:DIL14
- removed J13: J, detali:R1206W
- removed JA1, JA10, JA11, JA12, JA2, JA3, JA4, JA5, JA6, JA7, JA8, JA9, JB10, JB11, JB12, JB13, JB14, JB15, JB16, JB17, JB2, JB4, JB5, JB6, JB7, JB8, JB9: (no value), jumper:SJ
- removed JA111, JA112, JA113, JA114, JA115, JA116, JA117, JA118, JA119, JA120, JA121, JA122, JA123, JA124, JA125, JA126, JA127, JA128, JA129, JA13, JA130, JA131, JA132, JA133, JA14, JA15, JA16, JA17, JA18, JA19, JA20, JA21, JA22, JA23, JA24, JA25, JA26, JA27, JA28, JA29, JA30, JA31, JA32, JA33, JA34, JA35, JA36, JA37, JA38, JA39, JA40, JA41, JA42, JA43, JA44, JA45, JA46, JB1, JB111, JB112, JB113, JB114, JB115, JB116, JB117, JB118, JB119, JB120, JB121, JB122, JB123, JB124, JB125, JB126, JB127, JB128, JB129, JB130, JB131, JB132, JB133, JB18, JB19, JB20, JB21, JB22, JB23, JB24, JB25, JB26, JB27, JB28, JB29, JB3, JB30, JB31, JB32, JB33, JB34, JB35, JB36, JB37, JB38, JB39, JB40, JB41, JB42, JB43, JB44, JB45, JB46, JB67B: (no value), detali:SJ
- removed LED1: (no value), detali:LED5MM
- removed R1, R2: 1k, rcl:R1206W
- removed R4, R5, R6: 10k, rcl:R1206W
- removed R7, R8: (no value), rcl:R1206W
- removed S1: Scroll Lock, cherrymx:CHERRY-MX-LED
- removed S10: Left, cherrymx:CHERRY-MX
- removed S107B1, S130: NumEnter, cherrymx:CHERRY-MX-4P
- removed S11: Down, cherrymx:CHERRY-MX
- removed S111: D, cherrymx:CHERRY-MX-4P
- removed S112: E, cherrymx:CHERRY-MX-4P
- removed S113: F, cherrymx:CHERRY-MX-4P
- removed S114: /, cherrymx:CHERRY-MX-4P
- removed S115: A, cherrymx:CHERRY-MX-4P
- removed S116: B, cherrymx:CHERRY-MX-4P
- removed S117: C, cherrymx:CHERRY-MX-4P
- removed S118: *, cherrymx:CHERRY-MX-4P
- removed S119: 7, cherrymx:CHERRY-MX-4P
- removed S12: Right, cherrymx:CHERRY-MX
- removed S120: 8, cherrymx:CHERRY-MX-4P
- removed S121: 9, cherrymx:CHERRY-MX-4P
- removed S122: -, cherrymx:CHERRY-MX-4P
- removed S123: 4, cherrymx:CHERRY-MX-4P
- removed S124: 5, cherrymx:CHERRY-MX-4P
- removed S125: 6, cherrymx:CHERRY-MX-4P
- removed S126: +, cherrymx:CHERRY-MX-4P
- removed S127: 1, cherrymx:CHERRY-MX-4P
- removed S128: 2, cherrymx:CHERRY-MX-4P
- removed S129: 3, cherrymx:CHERRY-MX-4P
- removed S13: F1, cherrymx:CHERRY-MX
- removed S131: 0, cherrymx:CHERRY-MX-4P
- removed S132: 00, cherrymx:CHERRY-MX-4P
- removed S133: ., cherrymx:CHERRY-MX-4P
- removed S134: NumLock, detali:B3F-31XX
- removed S14: F2, cherrymx:CHERRY-MX
- removed S15: F3, cherrymx:CHERRY-MX
- removed S16: F4, cherrymx:CHERRY-MX
- removed S17: F5, cherrymx:CHERRY-MX
- removed S18: F6, cherrymx:CHERRY-MX
- removed S19: 1, cherrymx:CHERRY-MX
- removed S2: ESC, cherrymx:CHERRY-MX-LED
- removed S20: 2, cherrymx:CHERRY-MX
- removed S21: 3, cherrymx:CHERRY-MX
- removed S22: 4, cherrymx:CHERRY-MX
- removed S23: 5, cherrymx:CHERRY-MX
- removed S24: 6, cherrymx:CHERRY-MX
- removed S25: TAB, cherrymx:CHERRY-MX
- removed S26: Q, cherrymx:CHERRY-MX
- removed S27: W, cherrymx:CHERRY-MX@1
- removed S28: E, cherrymx:CHERRY-MX
- removed S29: R, cherrymx:CHERRY-MX
- removed S3: Ins, cherrymx:CHERRY-MX-LED
- removed S30: T, cherrymx:CHERRY-MX
- removed S31: LCtrl, cherrymx:CHERRY-MX
- removed S32: A, cherrymx:CHERRY-MX
- removed S33: S, cherrymx:CHERRY-MX
- removed S34: D, cherrymx:CHERRY-MX
- removed S35: F, cherrymx:CHERRY-MX
- removed S36: G, cherrymx:CHERRY-MX
- removed S37, S37B, S37B1: L Shift, cherrymx:CHERRY-MX
- removed S38: Z, cherrymx:CHERRY-MX
- removed S39: X, cherrymx:CHERRY-MX
- removed S4: Pause, cherrymx:CHERRY-MX@1
- removed S40: C, cherrymx:CHERRY-MX
- removed S41: V, cherrymx:CHERRY-MX
- removed S42: B, cherrymx:CHERRY-MX
- removed S43: Caps Lock, cherrymx:CHERRY-MX-LED
- removed S44: Alt, cherrymx:CHERRY-MX
- removed S45: Menu(Win), cherrymx:CHERRY-MX
- removed S46: Space, cherrymx:CHERRY-MX
- removed S5: Home, cherrymx:CHERRY-MX
- removed S6: P Up, cherrymx:CHERRY-MX
- removed S67C2: FN1, cherrymx:CHERRY-MX-4P
- removed S7: End, cherrymx:CHERRY-MX
- removed S8: P Dn, cherrymx:CHERRY-MX
- removed S9: Up, cherrymx:CHERRY-MX
- removed U$10, U$11, U$118, U$119, U$12, U$120, U$121, U$122, U$123, U$124, U$125, U$126, U$127, U$128, U$129, U$13, U$130, U$131, U$132, U$133, U$134, U$135, U$136, U$137, U$138, U$139, U$141, U$18, U$19, U$2, U$20, U$21, U$23, U$24, U$25, U$26, U$27, U$29, U$3, U$30, U$31, U$32, U$33, U$35, U$36, U$37, U$38, U$39, U$4, U$40, U$41, U$42, U$43, U$44, U$45, U$46, U$5, U$6, U$7, U$8, U$81, U$82, U$9: (no value), kbmx:18X18
- removed U$114, U$28: (no value), kbmx:18X33
- removed U$115, U$34, U$89: (no value), kbmx:18X28
- removed U$140: (no value), kbmx:37X18
- removed U$142, U$143, U$144, U$145, U$146, U$147, U$148, U$150, U$151, U$152, U$153, U$154, U$155, U$156, U$157, U$158, U$159, U$160, U$161, U$162, U$163, U$164: (no value), kbmxco:KEY
- removed U$149: (no value), kbmxco:NUMENTER
- removed U$15, U$16, U$91: (no value), kbmx:18X23
- removed U$17: (no value), kbmx:18X52
- removed U$22: (no value), kbmx:18X42
- removed U$88: CHERRY-MX, cherrymx:CHERRY-MX
- added 2D1: 74HC138N, detali2:DIL16
- added 2D2: 74HC04N, detali2:DIL14
- added D67B, D87: LL4148, detali:SOD80C
- added J18, J19, J21, J22, J23, J24, J25, J26, J27, J28, J29, J30, J31, J32, J33, J34, J35, J36, J37, J38, J39, J40, J41, J42, J43, J44, J46, J48, J49, J50, J51, J52, J53: (no value), detali2:R1206W
- added JA67B1, JA87, JB67B1, JB87: (no value), detali:SJ
- added R3: 1k, rcl:R0805
- added S67B: |u, cherrymx:CHERRY-MX
- added S74B: Enter, cherrymx:CHERRY-MX
- added U$92: (no value), kbmx:18X28
- C1: value (none) -> 100n; device rcl:C1206 -> rcl:C0805
- C2: value (none) -> 100n
- J1, J10, J11, J12, J14, J15, J16, J17, J2, J3, J4, J5, J6, J7, J8, J9: value J -> (none); device detali:R1206W -> detali2:R1206W
- S67: value | -> |d
- S83: value Mouse2(Menu) -> FN3
- S84: value Alt -> R_Alt
- SV1: value (none) -> CON_KB_B; device detali:FE09 -> detali2:FE12
- U$1: device kbmx:18X18 -> kbmxco:SIZE132
- moved SV1 426.5 mm to (28.6, 115.6)
- moved J16 403.7 mm to (51.1, 95.9), flipped to the top
- moved J11 390.1 mm to (60.6, 76.5), flipped to the top, turned to 180 degrees
- moved J15 381.7 mm to (66.4, 87.9), flipped to the top, turned to 90 degrees
- moved J9 381.4 mm to (80.3, 30.8), flipped to the top, turned to 0 degrees
- moved J14 381.2 mm to (55.9, 35.2), flipped to the top, turned to 180 degrees
- moved J3 376.9 mm to (98.7, 94.3), flipped to the top, turned to 0 degrees
- moved C2 375.6 mm to (44.5, 116.5), turned to 270 degrees
- moved J12 373.6 mm to (88.9, 37.1), flipped to the top
- moved J1 372.3 mm to (99.4, 114.9), flipped to the top, turned to 0 degrees
- moved J4 358.4 mm to (117.2, 94.3), flipped to the top, turned to 0 degrees
- moved J10 354.6 mm to (103.2, 107.3), flipped to the top, turned to 180 degrees
- moved J6 352.2 mm to (104.0, 49.2), flipped to the top, turned to 0 degrees
- moved J5 349.3 mm to (103.2, 68.9), flipped to the top, turned to 0 degrees
- moved J7 340.9 mm to (135.3, 133.3), flipped to the top, turned to 90 degrees
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Connections:
- removed net +5V_K1: 1S4.4, R1.1, R2.1
- removed net 2A1: JA61.2
- removed net 2A3: JA69.2
- removed net 2A5: JA76.2
- removed net 2A6: JA83.2
- removed net 2A7: JA48.2
- removed net 2A8: JA54.2
- removed net A1: 1S3.1, JA1.2, JA26.2, JA28.2, JA29.2
- removed net A2: 1S3.2, 1S3O.2, JA15.2, JA25.2, JA30.2, JA37.2, JA43.2, JA45.2
- removed net A3: 1S3.3, JA27.2, JA32.2, JA33.2, JA34.2, JA35.2
- removed net A4: 1S3.4, JA16.2, JA18.2, JA2.2, JA36.2, JA44.2, JA46.2, JA9.2
- removed net A5: 1S3.5, JA38.2, JA39.2, JA40.2, JA41.2
- removed net A6: 1S3.6, JA10.2, JA11.2, JA12.2, JA42.2
- removed net A7: 1S3.7, D24.A, JA13.2, JA14.2, JA23.2, JA3.2, JA31.2, JA5.2, JA6.2
- removed net A8: 1S3.8, JA17.2, JA19.2, JA20.2, JA21.2, JA22.2, JA4.2, JA7.2, JA8.2
- removed net B0: 1S1.1, D2.C, D25.C, D26.C, D32.C, D38.C
- removed net B1: 1S1.2, D13.C, D33.C, D39.C, D43.C, HL1.4, HL2.4
- removed net B10: 1S2.1, D11.C, D46.C
- removed net B11: 1S2.2, D37.C
- removed net B12: 1S2.3
- removed net B13: 1S2.4, D22.C
- removed net B14: 1S2.5, D1.C, D27.C, D4.C, D44.C
- removed net B15: 1S2.6, D17.C, D31.C
- removed net B16: 1S2.7, D45.C
- removed net B17: 1S2.8
- removed net B2: 1S1.3, D14.C, D15.C, D16.C, D28.C, D34.C, D40.C, HL3.4
- removed net B3: 1S1.4, D23.C, D29.C, D30.C, D35.C, D36.C, D41.C, D42.C
- removed net B4: 1S1.5, D19.C, JA24.2
- removed net B5: 1S1.6, D18.C, D20.C
- removed net B6: 1S1.7, 1S2O.5, D21.C
- removed net B7: 1S1.8, D10.C, D5.C, D7.C, D9.C
- removed net B8: 1S1.9, D6.C, D8.C
- removed net B9: 1S1.10, D12.C, D3.C
- removed net COLN1: 3D2.12, SV1.2
- removed net COLN2: 3D2.6, J15.1
- removed net COLN3: 3D2.8, SV1.3
- removed net GND_K1: 1S4.5
- removed net K1: HL1.2, HL3.2
- removed net LED_CAPS: 1S4.3, S43.LED2
- removed net LED_NUM: 1S4.1
- removed net LED_SCR: 1S4.2, S1.LED2
- removed net N$100: JA30.1, S30.SW2
- removed net N$101: JA31.1, S31.SW2
- removed net N$102: JA32.1, S32.SW2
- removed net N$103: JA33.1, S33.SW2
- removed net N$104: JA34.1, S34.SW2
- removed net N$105: JA35.1, S35.SW2
- removed net N$106: JA36.1, S36.SW2
- removed net N$107: JA37.1, S37.SW2, S37B.SW2, S37B1.SW2
- removed net N$108: JA38.1, S38.SW2
- removed net N$109: JA39.1, S39.SW2
- removed net N$110: JA40.1, S40.SW2
- removed net N$111: JA41.1, S41.SW2
- removed net N$113: JA43.1, S43.SW2
- removed net N$114: JA45.1, S45.SW2
- removed net N$115: JA46.1, S46.SW2
- removed net N$116: JA19.1, S19.SW2
- removed net N$117: JA44.1, S44.SW2
- removed net N$118: JA21.1, S21.SW2
- removed net N$119: JA16.1, S16.SW2
- removed net N$120: D17.A, JB17.1
- removed net N$121: D18.A, JB18.1
- removed net N$122: D19.A, JB19.1
- removed net N$123: D20.A, JB20.1
- removed net N$124: D21.A, JB21.1
- removed net N$125: D22.A, JB22.1
- removed net N$126: D23.A, JB23.1
- removed net N$128: D25.A, JB25.1
- removed net N$129: D26.A, JB26.1
- removed net N$130: D27.A, JB27.1
- removed net N$131: D28.A, JB28.1
- removed net N$132: D29.A, JB29.1
- removed net N$133: D30.A, JB30.1
- removed net N$134: D31.A, JB31.1
- removed net N$135: D32.A, JB32.1
- removed net N$136: D33.A, JB33.1
- removed net N$137: D34.A, JB34.1
- removed net N$138: D35.A, JB35.1
- removed net N$139: D36.A, JB36.1
- removed net N$140: D37.A, JB37.1
- removed net N$141: D38.A, JB38.1
- removed net N$142: D39.A, JB39.1
- removed net N$143: D40.A, JB40.1
- removed net N$144: D41.A, JB41.1
- removed net N$145: D42.A, JB42.1
- removed net N$146: D43.A, JB43.1
- removed net N$147: D44.A, JB44.1
- removed net N$148: D45.A, JB45.1
- removed net N$149: D46.A, JB46.1
- removed net N$150: R1.2, S1.LED1
- removed net N$151: R2.2, S43.LED1
- removed net N$28 (its old number): JA10.1, S10.SW2
- removed net N$29 (its old number): JA1.1, S1.SW2
- removed net N$30: D9.A, JB9.1
- removed net N$31: D11.A, JB11.1
- removed net N$338: D112.A, S134.1
- removed net N$339: JA111.1, S111.SW2
- removed net N$340: D113.A, JB112.1
- removed net N$341: JB112.2, S112.SW1
- removed net N$342: JA112.1, S112.SW2
- removed net N$343: D111.A, JB111.1
- removed net N$344: JB111.2, S111.SW1
- removed net N$345: D114.A, JB113.1
- removed net N$346: JB113.2, S113.SW1
- removed net N$347: JA113.1, S113.SW2
- removed net N$348: D115.A, JB114.1
- removed net N$349: JB114.2, S114.SW1
- removed net N$350: JA114.1, S114.SW2
- removed net N$351: JB115.2, S115.SW1
- removed net N$352: D116.A, JB115.1
- removed net N$353: JA115.1, S115.SW2
- removed net N$354: JA116.1, S116.SW2
- removed net N$355: JB116.2, S116.SW1
- removed net N$356: D117.A, JB116.1
- removed net N$357: D118.A, JB117.1
- removed net N$358: JB117.2, S117.SW1
- removed net N$359: JA117.1, S117.SW2
- removed net N$360: D119.A, JB118.1
- removed net N$361: JB118.2, S118.SW1
- removed net N$362: JA118.1, S118.SW2
- removed net N$363: D120.A, JB119.1
- removed net N$364: JB119.2, S119.SW1
- removed net N$365: JA119.1, S119.SW2
- removed net N$366: JB120.2, S120.SW1
- removed net N$367: JA120.1, S120.SW2
- removed net N$368: D121.A, JB120.1
- removed net N$369: D122.A, JB121.1
- removed net N$370: JB121.2, S121.SW1
- removed net N$371: JA121.1, S121.SW2
- removed net N$372: D123.A, JB122.1
- removed net N$373: JB122.2, S122.SW1
- removed net N$374: JA122.1, S122.SW2
- removed net N$375: D124.A, JB123.1
- removed net N$376: JB123.2, S123.SW1
- removed net N$377: JA123.1, S123.SW2
- removed net N$378: JB124.2, S124.SW1
- removed net N$379: D125.A, JB124.1
- removed net N$38: JA14.1, S14.SW2
- removed net N$380: JA124.1, S124.SW2
- removed net N$381: D126.A, JB125.1
- removed net N$382: JB125.2, S125.SW1
- removed net N$383: JA125.1, S125.SW2
- removed net N$384: D127.A, JB126.1
- removed net N$385: JB126.2, S126.SW1
- removed net N$386: JA126.1, S126.SW2
- removed net N$387: JB130.2, S107B1.SW1, S130.SW1
- removed net N$388: JA130.1, S107B1.SW2, S130.SW2
- removed net N$389: D128.A, JB127.1
- removed net N$390: JB127.2, S127.SW1
- removed net N$391: JA127.1, S127.SW2
- removed net N$392: JB128.2, S128.SW1
- removed net N$393: D129.A, JB128.1
- removed net N$394: JA128.1, S128.SW2
- removed net N$395: D130.A, JB129.1
- removed net N$396: JB129.2, S129.SW1
- removed net N$397: JA129.1, S129.SW2
- removed net N$398: JB131.2, S131.SW1
- removed net N$399: JA131.1, S131.SW2
- removed net N$40: JA13.1, S13.SW2
- removed net N$400: D132.A, JB131.1
- removed net N$401: JB132.2, S132.SW1
- removed net N$402: D133.A, JB132.1
- removed net N$403: JA132.1, S132.SW2
- removed net N$404: D134.A, JB133.1
- removed net N$405: JB133.2, S133.SW1
- removed net N$406: JA133.1, S133.SW2
- removed net N$407: 3D2.3, 3D2.4, 3D2.5, JA112.2, JA116.2, JA120.2, JA124.2, JA125.2, JA128.2, JA129.2, JA133.2, R5.1
- removed net N$408: D111.C, D117.C, D118.C, J9.2
- removed net N$409: D123.C, D126.C, D128.C, J4.1
- removed net N$41: D14.A, JB14.1
- removed net N$410: 3D2.1, 3D2.13, 3D2.2, JA111.2, JA115.2, JA119.2, JA123.2, JA127.2, JA131.2, JA132.2, R4.1, S134.2
- removed net N$411: 3D1.10, D112.C, D113.C, D114.C
- removed net N$412: 3D1.11, D115.C, J7.2
- removed net N$413: 3D1.12, D119.C, J3.2
- removed net N$414: 3D1.14, D127.C, D130.C, D132.C
- removed net N$415: D116.C, D121.C, D122.C, J11.2
- removed net N$416: D131.A, J8.2, JA113.2, JA114.2, JA117.2, JA118.2, JA121.2, JA122.2, JA126.2
- removed net N$417: D131.C, JB130.1
- removed net N$418: D124.C, D129.C, J2.1
- removed net N$419: J1.1, J2.2
- removed net N$42: JB42.2, S42.SW2
- removed net N$420: J1.2, J3.1
- removed net N$421: 3D1.13, J4.2
- removed net N$422: D120.C, D125.C, J5.1
- removed net N$423: J6.2, J7.1
- removed net N$424: J5.2, J6.1
- removed net N$425: 3D2.10, 3D2.11, 3D2.9, J14.1, R6.1
- removed net N$426: 3D1.7, J10.1
- removed net N$427: J10.2, J9.1
- removed net N$428: J11.1, J12.1
- removed net N$429: J12.2, J13.1
- removed net N$43: JA42.1, S42.SW1
- removed net N$430: 3D1.9, J13.2
- removed net N$431: 3D1.6, R7.2
- removed net N$432: 3D1.1, SV1.8
- removed net N$433: 3D1.2, SV1.7
- removed net N$434: 3D1.3, SV1.6
- removed net N$435: LED1.A, R8.2
- removed net N$436: J14.2, J8.1
- removed net N$437: J15.2, J16.1
- removed net N$438: J16.2, SV1.5
- removed net N$439: J17.2, SV1.4
- removed net N$44: JB27.2, S27.SW1
- removed net N$440: J17.1, R8.1
- removed net N$441: D135.A, D136.C
- removed net N$442: 3D2.14, C2.1, D135.C
- removed net N$45: JA27.1, S27.SW2
- removed net N$46: JB17.2, S17.SW2
- removed net N$47: JA17.1, S17.SW1
- removed net N$48: D24.C, JB24.1
- removed net N$49: JB24.2, S24.SW2
- removed net N$50: JA24.1, S24.SW1
- removed net N$51 (its old number): JB67B.2, S67C.SW2
- removed net N$52: D4.A, JB4.1
- removed net N$53: D6.A, JB6.1
- removed net N$54: D8.A, JB8.1
- removed net N$56: D12.A, JB12.1
- removed net N$57: D13.A, JB13.1
- removed net N$58: JB19.2, S19.SW1
- removed net N$59: JB25.2, S25.SW1
- removed net N$61: JB31.2, S31.SW1
- removed net N$62: JB37.2, S37.SW1, S37B.SW1, S37B1.SW1
- removed net N$63: JB43.2, S43.SW1
- removed net N$64: JB26.2, S26.SW1
- removed net N$65: JB44.2, S44.SW1
- removed net N$66: JB18.2, S18.SW1
- removed net N$68: JB30.2, S30.SW1
- removed net N$69: JB36.2, S36.SW1
- removed net N$72: JB23.2, S23.SW1
- removed net N$73: JB29.2, S29.SW1
- removed net N$74: JB35.2, S35.SW1
- removed net N$75: JB41.2, S41.SW1
- removed net N$76: JB16.2, S16.SW1
- removed net N$77: JB22.2, S22.SW1
- removed net N$78: JB28.2, S28.SW1
- removed net N$79: JB34.2, S34.SW1
- removed net N$80: JB40.2, S40.SW1
- removed net N$81: JB46.2, S46.SW1
- removed net N$82: JB15.2, S15.SW1
- removed net N$83: JB21.2, S21.SW1
- removed net N$85: JB33.2, S33.SW1
- removed net N$86: JB39.2, S39.SW1
- removed net N$87: JB45.2, S45.SW1
- removed net N$88: JA15.1, S15.SW2
- removed net N$9: JB6.2, S6.SW1
- removed net N$90: JA18.1, S18.SW2
- removed net N$91: JA20.1, S20.SW2
- removed net N$92: JA22.1, S22.SW2
- removed net N$93: JA23.1, S23.SW2
- removed net N$95: JA25.1, S25.SW2
- removed net N$96: JA26.1, S26.SW2
- removed net N$98: JA28.1, S28.SW2
- removed net N$99: JA29.1, S29.SW2
- removed net R1: HL1.1, HL2.1
- removed net R2: HL3.1
- removed net SCK: 3D1.15, D133.C, D134.C, JA130.2
- removed net VCC: 3D3.16, IC1.14
- new net +3VD: 2D2.14, C2.1, D1.C
- new net 1: D49.C, D50.C, D52.C, D56.C, D64B.C, J44.1
- new net 2: D51.C, D58.C, D59.C, J10.2, J2.2
- new net 2I: 2D1.14, D48.C, J7.1
- new net 2J: D55.C, J10.1
- new net 3: D47.C, D54.C, D57.C, D63.C, J3.2
- new net 3J: D66.C, D67B.C, J4.1, J46.1
- new net 4: D65.C, D74.C, J5.1, J50.1
- new net 4J: D64.C, D71.C, J11.2, J5.2
- new net 4J2: D53.C, D61.C, J11.1
- new net 5: D67.C, D73.C, J48.1, J6.1
- new net 5J: D60.C, D62.C, D69.C, D72.C, J6.2
- new net 6: D79.C, D80.C, D81.C, J12.2, J53.1
- new net 6J2: D70.C, J12.1, J14.2
- new net 6J3: D68.C, J14.1
- new net 7: 2D1.13, D84.C, D85.C, J9.1
- new net 7J: D75.C, D76.C, D78.C, J9.2
- new net 8: 2D1.12, D86.C, J8.2
- new net 8J: D77.C, D82.C, D83.C, D87.C, J8.1
- new net D1: J29.2, SV1.10
- new net D2: J30.2, SV1.9
- new net D3: J31.2, SV1.8
- new net G3: J15.2, JA62.2, JA63.2, JA71.2
- new net G4: J34.2, JA50.2, JA51.2, JA57.2, JA64.2, JA72.2, JA78.2, JA79.2, JA87.2
- new net G5: J21.2, JA52.2, JA58.2, JA65.2, JA66.2, JA73.2, JA80.2, JA83.2, JA84.2
- new net G6: J17.2, JA59.2, JA67.2, JA67B.2, JA67B1.2, JA74B.2, JA81.2, JA85.2, JA86.2, JB74.1
- new net N$152: J17.1, J18.2
- new net N$269: J3.1, J4.2
- new net N$270: 2D2.2, SV1.5
- new net N$271: JB67B1.2, S67B.SW1, S67C.SW2
- new net N$275: 2D2.12, J23.2
- new net N$277: 2D1.6, R3.2
- new net N$281: 2D2.8, J28.2
- new net N$282: D67B.A, JB67B1.1
- new net N$285: J15.1, J16.2
- new net N$286: JA87.1, S67C1.SW1
- new net N$287: JB87.2, S67C1.SW2
- new net N$288: D87.A, JB87.1
- new net N$289: 2D2.3, J16.1
- new net N$290: 2D2.13, J18.1
- new net N$293: J19.2, J21.1
- new net N$294: 2D2.11, J19.1
- new net N$60: JA67B1.1, S67B.SW2
- new net N$67: 2D2.6, SV1.7
- net +5V: now also 2D1.16, D2.A, R3.1, SV1.11; no longer 3D1.16, D136.A, R4.2, R5.2, R6.2, R7.1, SV1.9
- net G1: now also 2D2.9, JA47.2, JA48.2, JA49.2, JA53.2, JA60.2, JA68.2, JA75.2, JA82.2; no longer HL1.3, HL2.3
- net G2: now also J22.2, JA54.2, JA55.2, JA56.2, JA61.2, JA69.2, JA70.2, JA76.2, JA77.2; no longer HL3.3
- net GND: now also 2D1.4, 2D1.5, 2D1.8, 2D2.7; no longer 3D1.4, 3D1.5, 3D1.8, 3D2.7, 3D3.8, IC1.7, LED1.K
- net N$1: now also 2D2.1, J22.1; no longer D15.A, JB15.1
- net N$10: now also D1.A, D2.C; no longer JA6.1, S6.SW2
- net N$11: now also J1.2, J29.1; no longer JA8.1, S8.SW2
- net N$12: now also J30.1, J32.2; no longer JB8.2, S8.SW1
- net N$13: now also J31.1, J33.2; no longer JB10.2, S10.SW1
- net N$14: now also J1.1, J35.2; no longer JB1.2, S1.SW1
- net N$15: now also J32.1, J36.2; no longer D2.A, JB2.1
- net N$16: now also J33.1, J37.2; no longer JB2.2, S2.SW2
- net N$161: now also S76.SW2; no longer S76.SW1
- net N$162: now also S83.SW2; no longer S83.SW1
- net N$165: now also S62.SW2; no longer S62.SW1
- net N$168: now also JA73.1, S73.SW1; no longer JB84.2, S84.SW1
- net N$169: now also S50.SW2; no longer S50.SW1
- net N$17: now also 2D2.5, J34.1; no longer JA2.1, S2.SW1
- net N$172: now also S78.SW2; no longer S78.SW1
- net N$173: now also S85.SW2; no longer S85.SW1
- net N$175: now also S57.SW2; no longer S57.SW1
- net N$176: now also JA57.1, S57.SW1; no longer JB64.2, S64.SW1
- net N$177: now also JA64.1, S64.SW1; no longer JB72.2, S72.SW1
- net N$178: now also S79.SW2; no longer S79.SW1
- net N$18: now also J37.1, J38.2; no longer D16.A, JB16.1
- net N$180: now also S58.SW2; no longer S58.SW1
- net N$181: now also S65.SW2; no longer S65.SW1
- net N$182: now also JA80.1; no longer JB80.2
- net N$183: now also S59.SW2; no longer S59.SW1
- net N$185: now also S67.SW2; no longer S67.SW1
- net N$186: now also S81.SW2; no longer S81.SW1
- net N$19: now also J36.1, J40.2; no longer JB3.2, S3.SW1
- net N$2: now also J23.1, SV1.4; no longer JB4.2, S4.SW1
- net N$20: now also J35.1, J39.2; no longer JB5.2, S5.SW1
- net N$21: now also J38.1, J41.2; no longer JB7.2, S7.SW1
- net N$22: now also J40.1, J42.2; no longer JB9.2, S9.SW1
- net N$224: no longer JB67B.1
- net N$225: now also JA74.2; no longer JB74.1
- net N$23: now also J39.1, J43.2; no longer JB11.2, S11.SW1
- net N$238: now also S76.SW1; no longer S76.SW2
- net N$239: now also S83.SW1; no longer S83.SW2
- net N$24: now also 2D1.1, J41.1; no longer D3.A, JB3.1
- net N$242: now also S62.SW1; no longer S62.SW2
- net N$245: now also JB80.2, S80.SW2; no longer JA84.1, S84.SW2
- net N$246: now also S50.SW1; no longer S50.SW2
- net N$25: now also 2D1.2, J42.1; no longer JB12.2, S12.SW1
- net N$250: now also S78.SW1; no longer S78.SW2
- net N$251: now also S85.SW1; no longer S85.SW2
- net N$253: now also JB64.2, S64.SW2; no longer JA57.1, S57.SW2
- net N$254: now also JB72.2, S72.SW2; no longer JA64.1, S64.SW2
- net N$255: now also S72.SW1; no longer S72.SW2
- net N$256: now also S79.SW1; no longer S79.SW2
- net N$259: now also JA65.1, S65.SW1; no longer JA58.1, S58.SW2
- net N$26: now also 2D1.3, J43.1; no longer D5.A, JB5.1
- net N$260: now also JA58.1, S58.SW1; no longer JA65.1, S65.SW2
- net N$261: now also JB84.2, S84.SW2; no longer JA73.1, S73.SW2
- net N$262: now also JA84.1, S84.SW1; no longer JA80.1, S80.SW2
- net N$263: now also S81.SW1; no longer S81.SW2
- net N$264: now also S67.SW1; no longer S67.SW2
- net N$265: now also S59.SW1; no longer S59.SW2
- net N$267: now also S74.SW1; no longer S74.SW2
- net N$268: now also 2D2.4, SV1.6; no longer JA67.2, JA67B.2
- net N$27: now also 2D1.15, J44.2; no longer D7.A, JB7.1
- net N$3: now also 2D2.10, J25.2; no longer D1.A, JB1.1
- net N$32: now also 2D1.7, J46.2; no longer JA3.1, S3.SW2
- net N$33: now also J48.2, J51.1; no longer JA5.1, S5.SW2
- net N$34: now also 2D1.9, J52.2; no longer JA7.1, S7.SW2
- net N$35: now also 2D1.11, J49.2; no longer JA9.1, S9.SW2
- net N$36: now also J49.1, J50.2; no longer JA11.1, S11.SW2
- net N$37: now also 2D1.10, J51.2; no longer JA12.1, S12.SW2
- net N$39: now also J52.1, J53.2; no longer JB13.2, S13.SW1
- net N$4: now also J24.1, SV1.3; no longer JA4.1, S4.SW2
- net N$5: now also J24.2, J25.1; no longer JB14.2, S14.SW1
- net N$55: now also J2.1, J7.2; no longer D10.A, JB10.1
- net N$6: now also J26.2, J27.1; no longer JB20.2, S20.SW1
- net N$7: now also J26.1, SV1.2; no longer JB32.2, S32.SW1
- net N$70: now also S74.SW2; no longer S74.SW1
- net N$8: now also J27.2, J28.1; no longer JB38.2, S38.SW1
- net N$89: now also S73.SW2; no longer S73.SW1
- net N$94: now also S74B.SW1; no longer U$88.SW1
- net N$97: now also S74B.SW2; no longer U$88.SW2
Routing:
- net G6: track 0.00 -> 213.0 mm
- net 7: track 0.00 -> 210.2 mm
- net G1: track 0.00 -> 199.0 mm
- net N$407: track 188.7 -> 0.00 mm
- net SCK: track 185.4 -> 0.00 mm
- net N$410: track 178.5 -> 0.00 mm
- net G5: track 0.00 -> 173.2 mm
- net G4: track 0.00 -> 168.9 mm
- net 2I: track 0.00 -> 165.0 mm
- net G2: track 0.00 -> 138.3 mm
- net 1: track 0.00 -> 135.7 mm
- net 8J: track 0.00 -> 133.5 mm
- net N$414: track 132.8 -> 0.00 mm
- net N$416: track 130.9 -> 0.00 mm
- net 8: track 0.00 -> 119.8 mm
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- removed copper zone on layer 1, net GND
- removed copper zone on layer 1, net N$442
Other:
- board size 485.8 x 150.5 mm -> 169.5 x 134.6 mm
- board text added: "1177-16"
- board text removed: "1"
- board text removed: "1176-16"
- board text removed: "9"

Commit message: fix b
Parts:
- added R1, R2, R4, R6, R7: 10k, rcl:R0805
- added R5: 10k, rcl:R1206W
- moved J16 7.65 mm to (58.7, 95.2), turned to 180 degrees
- moved D53 5.85 mm to (34.9, 74.9)
- moved D54 4.55 mm to (38.4, 94.6), turned to 270 degrees
- moved J17 2.86 mm to (135.3, 134.3)
- moved J21 2.86 mm to (133.0, 130.5)
- moved J7 2.86 mm to (135.3, 130.5)
- moved JB54 2.54 mm to (41.3, 97.5), turned to 180 degrees
- moved J18 2.48 mm to (48.6, 134.9)
- moved JB57 2.46 mm to (89.2, 100.5)
- moved J22 1.91 mm to (45.1, 108.6)
- moved D61 1.42 mm to (41.6, 75.9), turned to 270 degrees
- moved D52 1.31 mm to (130.2, 130.5)
- moved D48 1.27 mm to (45.4, 136.2)
- moved JB77 1.14 mm to (57.8, 41.0)
- moved J3 1.00 mm to (98.4, 95.2)
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- renumbered S67C1 to S87
Connections:
- net N$293 renamed PG5
- removed net N$17: 2D2.5, J34.1
- removed net N$289: 2D2.3, J16.1
- removed net N$290: 2D2.13, J18.1
- removed net N$294: 2D2.11, J19.1
- new net GG5: 2D2.11, J19.1, R6.2
- new net PG3: 2D2.3, J16.1, R4.2
- new net PG4: 2D2.5, J34.1, R5.2
- new net PG6: 2D2.13, J18.1, R7.2
- net +5V: now also R1.1, R2.1, R4.1, R5.1, R6.1, R7.1
- net G1: now also R1.2
- net G2: now also R2.2
Routing:
- net PG4: track 0.00 -> 34.3 mm
- net N$17: track 24.2 -> 0.00 mm
- net PG3: track 0.00 -> 23.8 mm
- net N$289: track 17.1 -> 0.00 mm
- net PG6: track 0.00 -> 15.8 mm
- net +5V: track 184.4 -> 197.8 mm, vias 0 -> 2
- net N$290: track 12.9 -> 0.00 mm
- net N$294: track 12.5 -> 0.00 mm
- net GG5: track 0.00 -> 12.5 mm
- net N$285: track 17.9 -> 9.47 mm
- net 4J2: track 35.6 -> 27.3 mm
- net 2I: track 165.0 -> 170.8 mm
- net N$188: track 19.9 -> 25.4 mm
- net 6J2: track 71.0 -> 65.8 mm
- net G2: track 138.3 -> 142.3 mm
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Other:
- outline, holes or cut-outs redrawn

Commit message: pcb b
Parts:
- removed U$112: (no value), kbmx:18X37
- removed U$14: (no value), kbmx:18X28
- added U$2: (no value), kbmx:18X23
- moved U$90 24.1 mm to (94.9, 28.3)
- moved U$86 19.0 mm to (74.6, 27.0)
- moved D83 14.2 mm to (87.3, 22.9)
- moved JB83 5.99 mm to (90.5, 24.1), turned to 180 degrees
- moved JA54 3.18 mm to (31.9, 100.3), turned to 0 degrees
- moved JB80 3.14 mm to (110.5, 37.5), turned to 315 degrees
- moved J9 3.00 mm to (82.9, 29.2)
- moved JB81 2.54 mm to (147.6, 42.2)
- moved JA87 2.54 mm to (82.2, 24.4)
- moved S83 2.54 mm to (96.2, 27.0)
- moved JB87 2.54 mm to (75.9, 21.0)
- moved S81 2.54 mm to (154.6, 46.0)
- moved S87 2.54 mm to (74.6, 27.0)
- moved D87 2.25 mm to (80.3, 21.0)
- moved JA83 2.01 mm to (103.8, 24.4)
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Routing:
- net G2: track 142.3 -> 146.4 mm
- net 7J: track 68.5 -> 72.1 mm
- net N$221: track 7.09 -> 4.20 mm
- net 6: track 46.6 -> 43.8 mm
- net N$198: track 5.07 -> 2.45 mm
- net N$226: track 33.5 -> 31.0 mm
- net G5: track 170.4 -> 167.9 mm
- net N$33: track 39.4 -> 41.5 mm
- net 8J: track 134.2 -> 136.2 mm
- net N$204: track 5.68 -> 3.79 mm
- net G4: track 168.7 -> 167.5 mm
- net 6J2: track 65.8 -> 66.8 mm
- net N$263: track 3.05 -> 3.97 mm
- net N$187: track 52.1 -> 53.0 mm
- net G3: track 35.0 -> 34.2 mm
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Other:
- outline, holes or cut-outs redrawn

Commit message: .
Parts:
- added J13: (no value), detali2:R1206W
- added U$3: (no value), kbmx:18X18
- moved J8 0.63 mm to (151.4, 20.6)
- moved JA67B1 0.32 mm to (151.8, 75.9)
- renumbered JB67B1 to JB67B
Connections:
- new net N$17: J13.2, JB67B.2
- net N$271: now also J13.1; no longer JB67B.2
Routing:
- net N$17: track 0.00 -> 14.2 mm
- net N$271: track 12.9 -> 5.80 mm
- net N$37: track 61.6 -> 59.9 mm
- net 8J: track 136.2 -> 134.9 mm
- net 2I: track 170.8 -> 169.8 mm
- net +5V: track 197.8 -> 196.8 mm, vias 2 -> 3
- net 7: track 209.5 -> 208.9 mm
- net G6: track 213.5 -> 214.1 mm
- net N$27: track 20.0 -> 20.6 mm
