File: PCB/keyBoard_B/keyBoard_B.brd (EAGLE design)
At the start: 169.5 x 134.6 mm, 281 parts

Commit message: fix b
Other:
- outline, holes or cut-outs redrawn
Changed lines of the file:
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@@
 <setting verticaltext="up"/>
 </settings>
-<grid distance="25" unitdist="mil" unit="mil" style="lines" multiple="1" display="yes" altdistance="0.025" altunitdist="inch" altunit="inch"/>
+<grid distance="6.25" unitdist="mil" unit="mil" style="lines" multiple="1" display="yes" altdistance="0.025" altunitdist="inch" altunit="inch"/>
 <layers>
 <layer number="1" name="Top" color="4" fill="1" visible="yes" active="yes"/>
@@
 <circle x="107.15625" y="117.95125" radius="2.5" width="0.254" layer="20"/>
 <circle x="126.52375" y="116.99875" radius="2.5" width="0.254" layer="20"/>
+<wire x1="34.13125" y1="15.875" x2="28.41625" y2="15.875" width="0.2" layer="20"/>
 <wire x1="191.77" y1="150.495" x2="34.13125" y2="150.495" width="0.2" layer="20"/>
 <wire x1="30.95625" y1="147.32" x2="34.13125" y2="150.495" width="0.2" layer="20" curve="-90"/>
 <dimension x1="25.4" y1="21.74875" x2="194.945" y2="16.66875" x3="110.1725" y3="10.31875" layer="21" dtype="horizontal"/>
 <wire x1="194.945" y1="147.32" x2="194.945" y2="19.05" width="0.2" layer="20"/>
-<wire x1="30.95625" y1="19.05" x2="34.13125" y2="15.875" width="0.2" layer="20" curve="90"/>
 <wire x1="30.95625" y1="40.9575" x2="25.4" y2="40.9575" width="0.2" layer="20"/>
 <wire x1="25.4" y1="40.9575" x2="25.4" y2="22.38375" width="0.2" layer="20"/>
@@
 <dimension x1="31.115" y1="150.495" x2="30.95625" y2="15.875" x3="24.844375" y3="83.185" layer="21" dtype="vertical"/>
 <circle x="169.38625" y="41.275" radius="2.5" width="0.254" layer="20"/>
+<dimension x1="25.4" y1="7.77875" x2="30.95625" y2="15.08125" x3="28.178125" y3="7.46125" layer="21" dtype="horizontal"/>
+<dimension x1="24.13" y1="40.9575" x2="22.06625" y2="15.875" x3="15.954375" y3="28.41625" layer="21" dtype="vertical"/>
+<wire x1="25.4" y1="22.38375" x2="25.4" y2="19.05" width="0.2" layer="20"/>
+<wire x1="25.4" y1="19.05" x2="28.575" y2="15.875" width="0.2" layer="20" curve="90"/>
+<wire x1="30.95625" y1="19.05" x2="34.13125" y2="15.875" width="0.2" layer="20" curve="90"/>
+<dimension x1="30.95625" y1="150.97125" x2="194.945" y2="149.86" x3="112.950625" y3="153.67" layer="21" dtype="horizontal"/>
 </plain>
 <attributes>
@@
 <wire x1="172.67375" y1="136.955" x2="172.99125" y2="138.1125" width="0.6096" layer="16"/>
 </signal>
+<signal name="N$11">
+<via x="28.41625" y="19.05" extent="1-16" drill="3" diameter="5"/>
+</signal>
 <signal name="N$407">

Commit message: fw
Connections:
- net BD1: now also J72.2, SV4.8; no longer J70.2, SV4.10
- net BD3: now also J70.2, SV4.10; no longer J72.2, SV4.8
Routing:
- net BD3: track 53.8 -> 44.2 mm
- net BD1: track 44.2 -> 53.8 mm
Changed lines of the file:
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@@
 <wire x1="161.99525" y1="142.875" x2="163.35375" y2="141.5165" width="0.6096" layer="16"/>
 </signal>
-<signal name="BD1">
+<signal name="BD3">
 <contactref element="SV4" pad="10"/>
 <contactref element="J70" pad="2"/>
@@
 <wire x1="93.345" y1="120.3325" x2="89.2175" y2="123.66625" width="0.6096" layer="16"/>
 </signal>
-<signal name="BD3">
+<signal name="BD1">
 <contactref element="SV4" pad="8"/>
 <contactref element="J72" pad="2"/>

Commit message: add1
Parts:
- added STAB_RSP: STAB, kbmxco:ZEALIOS-PCB_2U
- moved D68 8.77 mm to (162.2, 86.8), turned to 90 degrees
- moved D67B 2.22 mm to (164.3, 90.5)
- moved JB66 1.59 mm to (158.0, 82.9), turned to 0 degrees
Routing:
- net B3J: track 46.2 -> 36.8 mm
- net N$399: track 46.3 -> 52.1 mm
- net N$331: track 2.31 -> 4.41 mm
- net N$288: track 2.71 -> 4.19 mm
- net N$393: track 153.2 -> 152.1 mm

Commit message: add22
Parts:
- added STAB_BS: STAB, kbmxco:ZEALIOS-PCB_2U
- moved J90 7.05 mm to (175.9, 106.5), turned to 270 degrees
- moved JA59 4.26 mm to (173.0, 106.5)
- moved JB59 1.59 mm to (158.0, 102.9)
- renumbered STAB_RSP to STAB_EN
Routing:
- net N$323: track 35.4 -> 15.7 mm
- net N$287: track 19.3 -> 17.1 mm
- net N$399: track 52.1 -> 53.7 mm
- net N$117: track 28.6 -> 27.3 mm
- net N$393: track 152.1 -> 150.9 mm
- net N$318: track 3.52 -> 4.31 mm
- removed copper zone on layer 16, net N$7

Commit message: add b
Parts:
- added STAB_RSP: STAB, kbmxco:ZEALIOS-PCB_2U
- moved D78 16.7 mm to (48.1, 47.3)
- moved D70 11.4 mm to (50.8, 48.7), turned to 270 degrees
- moved JB76 7.38 mm to (54.5, 47.9), turned to 180 degrees
- moved D84 3.62 mm to (66.5, 27.9)
- moved D89 2.31 mm to (76.7, 26.8)
- moved JB87 1.93 mm to (81.1, 26.7)
- moved JA82 0.63 mm to (44.6, 26.7)
Routing:
- net N$252: track 27.6 -> 14.9 mm
- net B6J3: track 16.7 -> 29.2 mm
- net N$296: track 27.0 -> 36.2 mm
- net 8J: track 123.6 -> 120.2 mm
- net N$259: track 2.42 -> 5.84 mm
- net N$254: track 2.94 -> 6.20 mm
- net B7J: track 69.8 -> 71.6 mm
- net G1: track 194.6 -> 193.3 mm
- net N$361: track 3.50 -> 2.85 mm
- removed copper zone on layer 16, net N$8
- removed copper zone on layer 16, net N$9

Commit message: .
Parts:
- moved J83 1.99 mm to (148.0, 107.3), turned to 270 degrees
- moved JA74 1.92 mm to (160.3, 64.9), turned to 0 degrees
- moved JB67B 1.62 mm to (167.5, 84.6)
- moved JB66 0.32 mm to (157.6, 82.9)
Routing:
- net B5J5: track 91.7 -> 84.8 mm
- net N$312: track 22.7 -> 17.1 mm
- net N$310: track 116.5 -> 113.3 mm
- net N$117: track 27.3 -> 24.3 mm
- net B8: track 139.8 -> 137.1 mm
- net N$399: track 53.7 -> 56.4 mm
- net B7: track 236.5 -> 234.3 mm
- net N$331: track 4.41 -> 6.17 mm
- net GND2: track 159.2 -> 157.7 mm
- net N$287: track 17.1 -> 15.7 mm
- net N$288: track 4.19 -> 4.78 mm
- removed copper zone on layer 16, net N$10
- removed copper zone on layer 16, net N$5
- removed copper zone on layer 16, net N$6
