File: PCB/keyBoard_B/keyBoard_B.sch (EAGLE design)
At the start: 239 parts, among them J1 J, J10 J, J11 J, J12 J, J13 J, J14 J, J15 J, J16 J, J17 J, J18 J, J19 J, J2 J, J21 J, J22 J, J23 J, J24 J, J25 J, J26 J, J27 J, J28 J, J29 J, J3 J, J30 J, J31 J, J32 J, J33 J, J34 J, J35 J, J36 J, J37 J, J38 J, J39 J, J4 J, J40 J, J41 J, J42 J, J43 J, J44 J, J46 J, J48 J, J49 J, J5 J, J50 J, J51 J, J52 J, J53 J, J6 J, J7 J, J8 J, J9 J

Commit message: pcb b ok
Parts:
- removed C1: 100n, rcl:C-EUC0805
- removed C2: 100n, rcl:C-EUC1206
- removed D1, D2, D47, D48: LL4148, detali:LL4148
- removed J10, J13, J2, J29, J3, J30, J31, J4, J44, J5, J6, J9: J, detali2:J
- removed JA67B1: (no value), detali:SJ
- removed R3: 1k, rcl:R-EU_R0805
- removed S67B: |u, cherrymx:CHERRY-MX
- removed S81A: R Shift, cherrymx:CHERRY-MX-4P
- added 2C1: 100n, rcl:C-EUC1206
- added 2C2: 100n, rcl:C-EUC1206K
- added D88, D89, D92, D93: LL4148, detali:LL4148
- added J83, J84, J85, J86, J88, J89, J90, J91, J92, J93, J94: J, detali2:J
- added R16: 1k, rcl:R-EU_R1206W
- added S82A: space, cherrymx:CHERRY-MX
- S67C: value | -> |u
- renumbered J1 to J70, J11 to J54, J12 to J55, J14 to J56, J15 to J57, J16 to J58, J17 to J59, J18 to J60, J19 to J61, J21 to J62, J22 to J63, J23 to J64, J24 to J65, J25 to J66, J26 to J67, J27 to J68, J28 to J69, J32 to J71, J33 to J72, J34 to J76, J35 to J73, J36 to J74, J37 to J75, J38 to J79, J39 to J77, J40 to J78, J41 to J80, J42 to J82, J43 to J81, J7 to J95, J8 to J87, R1 to 2R1, R2 to 2R2, R4 to 2R3, R5 to 2R4, R6 to 2R5, R7 to 2R6, SV1 to SV4
Connections:
- removed net +5V_B: 2D1P.VCC, 2R1.1, 2R2.1, 2R3.1, 2R4.1, 2R5.1, 2R6.1, C1.1, D2.A, R3.1, SV4.11
- removed net GND_B: 2D1A.G2A, 2D1A.G2B, 2D1P.GND, 2D2P.GND, C1.2, C2.2, SV4.1
- removed net N$10: D1.A, D2.C
- removed net N$11: J29.P$1, J70.P$2
- removed net N$12: J30.P$1, J71.P$2
- removed net N$13: J31.P$1, J72.P$2
- removed net N$156: JB82.2, S82G$1.PIN-1
- removed net N$17: J13.P$2, JB67B.2
- removed net N$186: JB81.2, S81AG$1.PIN-2, S81G$1.PIN-2
- removed net N$187: D47.A, JB47.1
- removed net N$188: D53.A, JB53.1
- removed net N$189: D60.A, JB60.1
- removed net N$190: D68.A, JB68.1
- removed net N$191: D75.A, JB75.1
- removed net N$192: D82.A, JB82.1
- removed net N$193: D48.A, JB48.1
- removed net N$194: D54.A, JB54.1
- removed net N$195: D61.A, JB61.1
- removed net N$196: D69.A, JB69.1
- removed net N$198: D83.A, JB83.1
- removed net N$199: D49.A, JB49.1
- removed net N$200: D55.A, JB55.1
- removed net N$201: D62.A, JB62.1
- removed net N$202: D70.A, JB70.1
- removed net N$203: D77.A, JB77.1
- removed net N$204: D84.A, JB84.1
- removed net N$205: D50.A, JB50.1
- removed net N$206: D56.A, JB56.1
- removed net N$207: D63.A, JB63.1
- removed net N$208: D71.A, JB71.1
- removed net N$209: D78.A, JB78.1
- removed net N$210: D85.A, JB85.1
- removed net N$211: D51.A, JB51.1
- removed net N$212: D57.A, JB57.1
- removed net N$213: D64.A, JB64.1
- removed net N$214: D72.A, JB72.1
- removed net N$215: D79.A, JB79.1
- removed net N$216: D86.A, JB86.1
- removed net N$217: D52.A, JB52.1
- removed net N$218: D58.A, JB58.1
- removed net N$219: D65.A, JB65.1
- removed net N$220: D73.A, JB73.1
- removed net N$221: D80.A, JB80.1
- removed net N$222: D59.A, JB59.1
- removed net N$223: D66.A, JB66.1
- removed net N$224: D67.A, JB67.1
- removed net N$226: D81.A, JB81.1
- removed net N$233 (its old number): JA82.1, S82G$1.PIN-2
- removed net N$27: 2D1A.Y0, J44.P$2
- removed net N$32: 2D1A.Y7, J46.P$2
- removed net N$33: J48.P$2, J51.P$1
- removed net N$34: 2D1A.Y6, J52.P$2
- removed net N$35: 2D1A.Y4, J49.P$2
- removed net N$36: J49.P$1, J50.P$2
- removed net N$37: 2D1A.Y5, J51.P$2
- removed net N$39: J52.P$1, J53.P$2
- removed net N$55: J2.P$1, J95.P$2
- removed net N$60: JA67B1.1, S67B.PIN-2
- new net +5V/2: 2D1P.VCC, 2R1.1, 2R2.1, 2R3.1, 2R4.1, 2R5.1, 2R6.1, D93.A, J86.P$2, SV4.11
- new net B5J4: J89.P$2, J92.P$1
- new net B5J5: 2D1A.Y5, D69.C, J92.P$2
- new net B6J4: D83.C, J93.P$1, J94.P$2
- new net GND2: 2C1.2, 2C2.2, 2D1A.G2A, 2D1A.G2B, 2D1P.GND, 2D2P.GND, SV4.1
- new net N$117: 2D1A.Y7, J83.P$2
- new net N$238: JB82.2, S82A.PIN-2, S82G$1.PIN-1
- new net N$249: D49.A, JB47.1
- new net N$250: D55.A, JB53.1
- new net N$251: D62.A, JB60.1
- new net N$252: D70.A, JB68.1
- new net N$253: D77.A, JB75.1
- new net N$254: D84.A, JB82.1
- new net N$255: D50.A, JB48.1
- new net N$256: D56.A, JB54.1
- new net N$257: D63.A, JB61.1
- new net N$258: D71.A, JB69.1
- new net N$259: D78.A, JB76.1
- new net N$260: D85.A, JB83.1
- new net N$261: D51.A, JB49.1
- new net N$262: D57.A, JB55.1
- new net N$264: D72.A, JB70.1
- new net N$265: D79.A, JB77.1
- new net N$266: D86.A, JB84.1
- new net N$267: D52.A, JB50.1
- new net N$268: D58.A, JB56.1
- new net N$270: D73.A, JB71.1
- new net N$272: D87.A, JB85.1
- new net N$274: D53.A, JB51.1
- new net N$275: D59.A, JB57.1
- new net N$278: D74.A, JB72.1
- new net N$279: D81.A, JB79.1
- new net N$280: D88.A, JB86.1
- new net N$281: D54.A, JB52.1
- new net N$282: D60.A, JB58.1
- new net N$283: D67.A, JB65.1
- new net N$285: D75.A, JB73.1
- new net N$286: D82.A, JB80.1
- new net N$287: D61.A, JB59.1
- new net N$289: D69.A, JB67.1
- new net N$290: D83.A, JB81.1
- new net N$296: JA82.1, S82A.PIN-1, S82G$1.PIN-2
- new net N$310: 2D1A.Y4, J93.P$2
- new net N$312: D76.A, JA74.2
- new net N$315: JB81.2, S81G$1.PIN-2
- new net N$316: JA81.1, S81G$1.PIN-1
- new net N$323: 2D1A.Y6, J90.P$2
- new net N$326: D89.A, JB87.1
- new net N$355: J48.P$1, J49.P$2
- new net N$360: 2D1A.G1, R16.2
- new net N$378: D92.A, D93.C
- new net N$393: J85.P$1, JA59.2, JA67.2, JA67B.2, JA81.2, JA85.2, JA86.2, JB74.1
- new net N$394: J84.P$1, J85.P$2
- new net N$399: J90.P$1, J91.P$2
- new net N$405: J46.P$1, J95.P$2
- new net N$406: JB67B.2, S67CG$1.PIN-2
- net +3VD: now also 2C1.1, D92.C; no longer C2.1, D1.C
- net 2I: now also D50.C; no longer D48.C
- net 8J: now also D79.C, D84.C, D85.C, D89.C; no longer D77.C, D82.C, D83.C, D87.C
- net B1: now also 2D1A.Y0, D51.C, D54.C, D58.C; no longer D49.C, D50.C, D56.C, J44.P$1
- net B2: now also D53.C, D60.C, D61.C, J46.P$2, J53.P$2; no longer D51.C, D58.C, D59.C, J10.P$2, J2.P$2
- net B2J: now also D57.C, J53.P$1; no longer D55.C, J10.P$1
- net B3: now also D49.C, D56.C, D59.C, D65.C, J48.P$2; no longer D47.C, D54.C, D57.C, D63.C, J3.P$2
- net B3J: now also D68.C, J49.P$1, J88.P$1; no longer D66.C, J4.P$1, J46.P$1
- net B4: now also D67.C, D76.C, J91.P$1; no longer D65.C, D74.C, J5.P$1
- net B4J: now also D66.C, D73.C, J50.P$2; no longer D64.C, D71.C, J5.P$2
- net B4J2: now also D55.C, D63.C; no longer D53.C, D61.C
- net B5: now also D75.C, J51.P$1, J89.P$1; no longer D67.C, D73.C, J48.P$1, J6.P$1
- net B5J: now also D64.C, D71.C, D74.C, J51.P$2; no longer D60.C, D69.C, D72.C, J6.P$2
- net B6: now also D82.C, J94.P$1; no longer D79.C, D80.C, J53.P$1
- net B6J2: now also D72.C; no longer D70.C
- net B6J3: now also D70.C; no longer D68.C
- net B7: now also D86.C, D87.C, J52.P$1; no longer D84.C, D85.C, J9.P$1
- net B7J: now also D77.C, D80.C, J52.P$2; no longer D75.C, D76.C, J9.P$2
- net B8: now also D88.C; no longer D86.C
- net BD1: now also J70.P$2; no longer J29.P$2
- net BD2: now also J71.P$2; no longer J30.P$2
- net BD3: now also J72.P$2; no longer J31.P$2
- net G6: now also J84.P$2; no longer JA59.2, JA67.2, JA67B.2, JA67B1.2, JA81.2, JA85.2, JA86.2, JB74.1
- net N$197: now also J83.P$1, J88.P$2; no longer D76.A, JB76.1
- net N$225: now also 2C2.1, J86.P$1, R16.1; no longer D74.A, JA74.2
- net N$263: now also D64.A, JB62.1; no longer JA81.1, S81AG$1.PIN-1, S81G$1.PIN-1
- net N$269: now also D65.A, JB63.1; no longer J3.P$1, J4.P$2
- net N$271: now also D80.A, JB78.1; no longer J13.P$1, S67B.PIN-1, S67CG$1.PIN-2
- net N$277: now also D66.A, JB64.1; no longer 2D1A.G1, R3.2
- net N$288: now also D68.A, JB66.1; no longer D87.A, JB87.1
Other:
- moved on the sheet: 2D1P, 2D2P, D49, D50, D51, D52, D53, D54, D55, D56, D57, D58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

Commit message: b pl mod
Parts:
- added S83B, S87B: CHERRY-MX, cherrymx:CHERRY-MX
Connections:
- removed net N$324: JA87.1, S87G$1.PIN-1
- removed net N$325: JB87.2, S87G$1.PIN-2
- removed net N$340: JB83.2, S83G$1.PIN-2
- removed net N$341: JA83.1, S83G$1.PIN-1
- new net FN2A: JB87.2, S87B.PIN-2, S87G$1.PIN-2
- new net FN2B: JA87.1, S87B.PIN-1, S87G$1.PIN-1
- new net FN3A: JB83.2, S83B.PIN-2, S83G$1.PIN-2
- new net FN3B: JA83.1, S83B.PIN-1, S83G$1.PIN-1
Other:
- moved on the sheet: 2C1, 2C2, 2D1, 2D1P, 2D2A, 2D2B, 2D2C, 2D2D, 2D2E, 2D2F, 2D2P, 2R1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

Commit message: new pcb b
Parts:
- removed J88: J, detali2:J
Connections:
- removed net N$197: J83.P$1, J88.P$2
- net B3J: now also J83.P$1; no longer J88.P$1
Other:
- moved on the sheet: D67B, JB67B, S67C
Changed lines of the file:
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@@
 <part name="J82" library="detali2" deviceset="J" device="" value=""/>
 <part name="J87" library="detali2" deviceset="J" device="" value=""/>
-<part name="J88" library="detali2" deviceset="J" device="" value=""/>
 <part name="J89" library="detali2" deviceset="J" device="" value=""/>
 <part name="J90" library="detali2" deviceset="J" device="" value=""/>
@@
 <instance part="JA74B" gate="1" x="198.12" y="104.14"/>
 <instance part="D64B" gate="G$1" x="157.48" y="104.14"/>
-<instance part="S67C" gate="G$1" x="180.34" y="60.96" rot="MR0"/>
+<instance part="S67C" gate="G$1" x="185.42" y="60.96" rot="MR0"/>
 <instance part="2D1" gate="A" x="76.2" y="213.36" smashed="yes">
 <attribute name="NAME" x="66.04" y="224.155" size="1.778" layer="95"/>
@@
 <attribute name="NAME" x="189.23" y="219.202" size="1.778" layer="95" rot="MR0"/>
 </instance>
-<instance part="JB67B" gate="1" x="167.64" y="60.96"/>
-<instance part="D67B" gate="G$1" x="154.94" y="60.96"/>
+<instance part="JB67B" gate="1" x="172.72" y="60.96"/>
+<instance part="D67B" gate="G$1" x="162.56" y="60.96"/>
 <instance part="JA87" gate="1" x="60.96" y="20.32"/>
 <instance part="JB87" gate="1" x="35.56" y="20.32"/>
@@
 <instance part="J87" gate="G$1" x="190.5" y="127" smashed="yes">
 <attribute name="NAME" x="188.595" y="127.635" size="1.27" layer="95"/>
-</instance>
-<instance part="J88" gate="G$1" x="104.14" y="203.2" smashed="yes">
-<attribute name="NAME" x="102.235" y="203.835" size="1.27" layer="95"/>
 </instance>
 <instance part="J89" gate="G$1" x="104.14" y="208.28" smashed="yes">
@@
 <pinref part="JA67B" gate="1" pin="1"/>
 <pinref part="S67C" gate="G$1" pin="PIN-1"/>
-<wire x1="185.42" y1="60.96" x2="193.04" y2="60.96" width="0.1524" layer="91"/>
+<wire x1="190.5" y1="60.96" x2="193.04" y2="60.96" width="0.1524" layer="91"/>
 </segment>
 </net>
@@
 <pinref part="D67B" gate="G$1" pin="A"/>
 <pinref part="JB67B" gate="1" pin="1"/>
-<wire x1="157.48" y1="60.96" x2="162.56" y2="60.96" width="0.1524" layer="91"/>
+<wire x1="165.1" y1="60.96" x2="167.64" y2="60.96" width="0.1524" layer="91"/>
 </segment>
 </net>
@@
 <pinref part="JB67B" gate="1" pin="2"/>
 <pinref part="S67C" gate="G$1" pin="PIN-2"/>
-<wire x1="175.26" y1="60.96" x2="172.72" y2="60.96" width="0.1524" layer="91"/>
+<wire x1="180.34" y1="60.96" x2="177.8" y2="60.96" width="0.1524" layer="91"/>
 </segment>
 </net>
@@
 <segment>
 <pinref part="D67B" gate="G$1" pin="C"/>
-<wire x1="152.4" y1="60.96" x2="144.78" y2="60.96" width="0.1524" layer="91"/>
+<wire x1="160.02" y1="60.96" x2="144.78" y2="60.96" width="0.1524" layer="91"/>
 <label x="147.32" y="60.96" size="1.778" layer="95"/>
 </segment>
 <segment>
-<pinref part="J88" gate="G$1" pin="P$1"/>
-<wire x1="109.22" y1="203.2" x2="114.3" y2="203.2" width="0.1524" layer="91"/>
 <label x="109.22" y="203.2" size="1.778" layer="95"/>
+<pinref part="J83" gate="G$1" pin="P$1"/>
+<wire x1="99.06" y1="203.2" x2="114.3" y2="203.2" width="0.1524" layer="91"/>
 </segment>
 </net>
@@
 </segment>
 </net>
-<net name="N$197" class="0">
-<segment>
-<pinref part="J83" gate="G$1" pin="P$1"/>
-<pinref part="J88" gate="G$1" pin="P$2"/>
-<wire x1="99.06" y1="203.2" x2="101.6" y2="203.2" width="0.1524" layer="91"/>
-</segment>
-</net>
