File: PCB/keyBoard_B/keyBoard_B.sch (EAGLE design)
At the start: 237 parts, among them J46 J, J48 J, J49 J, J50 J, J51 J, J52 J, J53 J, J54 J, J55 J, J56 J, J57 J, J58 J, J59 J, J60 J, J61 J, J62 J, J63 J, J64 J, J65 J, J66 J, J67 J, J68 J, J69 J, J70 J, J71 J, J72 J, J73 J, J74 J, J75 J, J76 J, J77 J, J78 J, J79 J, J80 J, J81 J, J82 J, J83 J, J84 J, J85 J, J86 J, J87 J, J89 J, J90 J, J91 J, J92 J, J93 J, J94 J, J95 J

Commit message: fix b
Other:
- moved on the sheet: D67B, J46, J48, J49, J50, J84, J85, J95, JA59, JA67, JA67B, JA74B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

Commit message: fw
Connections:
- net BD1: now also J72.P$2, SV4.8; no longer J70.P$2, SV4.10
- net BD3: now also J70.P$2, SV4.10; no longer J72.P$2, SV4.8
Changed lines of the file:
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@@
 <text x="190.5" y="231.14" size="1.778" layer="91">gnd</text>
 <text x="190.5" y="256.54" size="1.778" layer="91">vcc</text>
-<text x="190.5" y="254" size="1.778" layer="91">d1</text>
+<text x="190.5" y="248.92" size="1.778" layer="91">d1</text>
 <text x="190.5" y="251.46" size="1.778" layer="91">d2</text>
-<text x="190.5" y="248.92" size="1.778" layer="91">d3</text>
+<text x="190.5" y="254" size="1.778" layer="91">d3</text>
 </plain>
 <instances>
@@
 </segment>
 </net>
-<net name="BD1" class="0">
+<net name="BD3" class="0">
 <segment>
 <label x="12.7" y="215.9" size="1.778" layer="95"/>
@@
 </segment>
 </net>
-<net name="BD3" class="0">
+<net name="BD1" class="0">
 <segment>
 <label x="12.7" y="220.98" size="1.778" layer="95"/>

Commit message: b d1 d1 sw
Parts:
- added J1, J2, J3: J, detali2:J
Connections:
- net N$389 renamed BD2A
- removed net N$388: 2D1A.A, J80.P$1
- removed net N$391: 2D1A.C, J81.P$1
- new net BD1A: 2D1A.A, J1.P$1
- new net BD3A: 2D1A.C, J2.P$1
- new net N$12: J3.P$2, J80.P$1
- new net N$13: J1.P$2, J81.P$1
- new net N$14: J2.P$2, J3.P$1
- net BD1: now also J70.P$2, SV4.10; no longer J72.P$2, SV4.8
- net BD3: now also J72.P$2, SV4.8; no longer J70.P$2, SV4.10
Other:
- moved on the sheet: 2C1, 2D1P, 2D2P, D92, D93, J70, J71, J72, J73, J74, J75, J77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
