File: PCB/keyBoard_B/keyBoard_B - копия.brd (EAGLE design)
At the start: 169.5 x 134.6 mm, 281 parts

Commit message: pcb b old. pcb a ver txt
Connections:
- removed net N$388: 2D1.1, J80.1
- removed net N$391: 2D1.3, J81.1
- new net N$12: 2D1.1, J81.1
- new net N$14: 2D1.3, J80.1
- net BD1: now also J70.2, SV4.10; no longer J72.2, SV4.8
- net BD3: now also J72.2, SV4.8; no longer J70.2, SV4.10
Routing:
- net N$388: track 21.2 -> 0.00 mm
- net N$13: track 20.2 -> 0.00 mm
- net N$391: track 19.4 -> 0.00 mm
- net BD1: track 53.8 -> 42.9 mm
- net BD3: track 44.2 -> 51.9 mm
- net GND2: track 159.2 -> 158.3 mm
