File: PCB/keyBoard_B/keyBoard_B - копия.sch (EAGLE design)
At the start: 237 parts, among them J46 J, J48 J, J49 J, J50 J, J51 J, J52 J, J53 J, J54 J, J55 J, J56 J, J57 J, J58 J, J59 J, J60 J, J61 J, J62 J, J63 J, J64 J, J65 J, J66 J, J67 J, J68 J, J69 J, J70 J, J71 J, J72 J, J73 J, J74 J, J75 J, J76 J, J77 J, J78 J, J79 J, J80 J, J81 J, J82 J, J83 J, J84 J, J85 J, J86 J, J87 J, J89 J, J90 J, J91 J, J92 J, J93 J, J94 J, J95 J

Commit message: pcb b old. pcb a ver txt
Connections:
- removed net N$388: 2D1A.A, J80.P$1
- removed net N$391: 2D1A.C, J81.P$1
- new net N$12: 2D1A.A, J81.P$1
- new net N$14: 2D1A.C, J80.P$1
- net BD1: now also J70.P$2, SV4.10; no longer J72.P$2, SV4.8
- net BD3: now also J72.P$2, SV4.8; no longer J70.P$2, SV4.10
Other:
- moved on the sheet: 2C1, 2D1P, 2D2P, D92, D93, J70, J72, J73, J75, J77, J79, J80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
