File: PCB/~keyBoard_B/keyBoard_B.brd (EAGLE design)
At the start: 169.5 x 134.6 mm, 291 parts

Commit message: new pcb >
Connections:
- net +5V renamed +5V_B
- net 1 renamed B1
- net 2 renamed B2
- net 2J renamed B2J
- net 3 renamed B3
- net 3J renamed B3J
- net 4 renamed B4
- net 4J renamed B4J
- net 4J2 renamed B4J2
- net 5 renamed B5
- net 5J renamed B5J
- net 6 renamed B6
- net 6J2 renamed B6J2
- net 6J3 renamed B6J3
- net 7 renamed B7
- net 7J renamed B7J
- net 8 renamed B8
- net D1 renamed BD1
- net D2 renamed BD2
- net D3 renamed BD3
- net GND renamed GND_B
Changed lines of the file:
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@@
 <wire x1="144.4625" y1="124.9045" x2="143.1925" y2="127.5225" width="0.6096" layer="16"/>
 </signal>
-<signal name="GND">
+<signal name="GND_B">
 <contactref element="2D1" pad="4"/>
 <contactref element="2D1" pad="5"/>
@@
 <wire x1="152.0825" y1="40.9575" x2="148.3995" y2="42.2275" width="1.27" layer="16"/>
 <contactref element="S81A" pad="SW2"/>
-<wire x1="199.7075" y1="58.7375" x2="148.3995" y2="42.2275" width="0" layer="19" extent="16-16"/>
+<wire x1="199.7075" y1="58.7375" x2="152.0825" y2="40.9575" width="0" layer="19" extent="1-1"/>
 </signal>
 <signal name="N$263">
@@
 <wire x1="158.4325" y1="43.4975" x2="160.9725" y2="40.4495" width="1.27" layer="16"/>
 <contactref element="S81A" pad="SW1"/>
-<wire x1="206.0575" y1="61.2775" x2="158.4325" y2="43.4975" width="0" layer="19" extent="1-1"/>
+<wire x1="206.0575" y1="61.2775" x2="160.9725" y2="40.4495" width="0" layer="19" extent="16-16"/>
 </signal>
 <signal name="N$183">
 <contactref element="JB59" pad="2"/>
 <contactref element="S59" pad="SW2"/>
-<wire x1="136.3345" y1="98.1075" x2="152.0825" y2="98.1075" width="0" layer="19" extent="1-16"/>
+<wire x1="136.3345" y1="98.1075" x2="152.0825" y2="98.1075" width="0" layer="19" extent="16-16"/>
 </signal>
 <signal name="N$265">
 <contactref element="S59" pad="SW1"/>
 <contactref element="JA59" pad="1"/>
-<wire x1="158.4325" y1="100.6475" x2="150.0505" y2="100.6475" width="0" layer="19" extent="1-16"/>
+<wire x1="158.4325" y1="100.6475" x2="150.0505" y2="100.6475" width="0" layer="19" extent="16-16"/>
 </signal>
 <signal name="N$173">
@@
 <wire x1="143.51" y1="84.3425" x2="144.018" y2="80.9625" width="1.016" layer="16"/>
 </signal>
-<signal name="1">
+<signal name="B1">
 <contactref element="D50" pad="C"/>
 <contactref element="D52" pad="C"/>
@@
 <wire x1="141.7175" y1="130.9225" x2="143.1925" y2="130.9225" width="0.6096" layer="16"/>
 </signal>
-<signal name="2">
+<signal name="B2">
 <contactref element="D51" pad="C"/>
 <contactref element="D58" pad="C"/>
@@
 <wire x1="98.7425" y1="62.5475" x2="101.7905" y2="62.5475" width="1.016" layer="16"/>
 </signal>
-<signal name="3J">
-<contactref element="D66" pad="C"/>
-<contactref element="D67B" pad="C"/>
-<contactref element="J4" pad="1"/>
-<wire x1="118.6565" y1="94.2975" x2="121.8315" y2="97.79" width="0.6096" layer="16"/>
-<wire x1="121.8315" y1="97.79" x2="125.095" y2="97.79" width="0.6096" layer="16"/>
-<wire x1="125.095" y1="97.79" x2="129.2225" y2="93.6625" width="0.6096" layer="16"/>
-<wire x1="129.2225" y1="93.6625" x2="136.8425" y2="93.6625" width="0.6096" layer="16"/>
-<contactref element="J46" pad="1"/>
-<wire x1="159.7025" y1="99.7835" x2="157.886" y2="99.1485" width="0.6096" layer="16"/>
-<wire x1="157.886" y1="99.1485" x2="154.94" y2="95.25" width="0.6096" layer="16"/>
-<wire x1="154.94" y1="95.25" x2="150.65375" y2="95.25" width="0.6096" layer="16"/>
-<wire x1="150.65375" y1="95.25" x2="144.4625" y2="88.74125" width="0.6096" layer="16"/>
-<wire x1="135.685" y1="75.565" x2="140.335" y2="80.85" width="0.6096" layer="16"/>
-<wire x1="140.335" y1="80.85" x2="140.335" y2="87.7425" width="0.6096" layer="16"/>
-<wire x1="140.335" y1="87.7425" x2="140.335" y2="89.23501875" width="0.6096" layer="16"/>
-<wire x1="143.51" y1="87.7425" x2="140.335" y2="87.7425" width="0.6096" layer="16"/>
-<wire x1="144.4625" y1="88.74125" x2="143.51" y2="87.7425" width="0.6096" layer="16"/>
-<wire x1="140.335" y1="89.23501875" x2="136.8425" y2="93.6625" width="0.6096" layer="16"/>
-</signal>
-<signal name="4">
+<signal name="B4">
 <contactref element="D74" pad="C"/>
 <contactref element="D65" pad="C"/>
@@
 <wire x1="116" y1="75.565" x2="117.5875" y2="74.295" width="0.8128" layer="16"/>
 </signal>
-<signal name="5">
+<signal name="B5">
 <contactref element="D67" pad="C"/>
 <contactref element="D73" pad="C"/>
@@
 <wire x1="116.2935" y1="54.381" x2="116.205" y2="54.2925" width="0.6096" layer="16"/>
 </signal>
-<signal name="6">
+<signal name="B6">
 <contactref element="D81" pad="C"/>
 <contactref element="D80" pad="C"/>
@@
 <wire x1="105.41" y1="32.0675" x2="100.6475" y2="32.0675" width="1.016" layer="16"/>
 </signal>
-<signal name="7">
+<signal name="B7">
 <contactref element="D85" pad="C"/>
 <contactref element="D84" pad="C"/>
@@
 <wire x1="86.36" y1="19.685" x2="91.235" y2="18.3025" width="0.6096" layer="16"/>
 </signal>
-<signal name="8">
+<signal name="B8">
 <contactref element="D86" pad="C"/>
 <wire x1="169.2275" y1="48.26" x2="170.4975" y2="54.61" width="0.6096" layer="16"/>
@@
 <wire x1="169.8625" y1="60.96" x2="170.4975" y2="59.69" width="0.6096" layer="16"/>
 </signal>
-<signal name="3">
+<signal name="B3">
 <contactref element="D57" pad="C"/>
 <contactref element="J3" pad="2"/>
@@
 <wire x1="101.2825" y1="96.2025" x2="99.924" y2="95.25" width="0.6096" layer="16"/>
 </signal>
-<signal name="4J">
+<signal name="B4J">
 <contactref element="D64" pad="C"/>
 <contactref element="J5" pad="2"/>
@@
 <wire x1="84.3425" y1="69.9625" x2="86.6775" y2="69.9625" width="0.6096" layer="16"/>
 </signal>
-<signal name="5J">
+<signal name="B5J">
 <contactref element="J6" pad="2"/>
 <contactref element="D72" pad="C"/>
@@
 <wire x1="87.3125" y1="19.3675" x2="84.1375" y2="21.16" width="0.6096" layer="16"/>
 </signal>
-<signal name="7J">
+<signal name="B7J">
 <contactref element="D78" pad="C"/>
 <contactref element="J9" pad="2"/>
@@
 <wire x1="70.2945" y1="61.9125" x2="73.3425" y2="60.0075" width="1.016" layer="16"/>
 </signal>
-<signal name="+5V">
+<signal name="+5V_B">
 <contactref element="R3" pad="1"/>
 <contactref element="2D1" pad="16"/>
@@
 <wire x1="162.56" y1="111.4425" x2="166.0525" y2="111.7625" width="1.016" layer="16"/>
 </signal>
-<signal name="2J">
+<signal name="B2J">
 <contactref element="J10" pad="1"/>
 <contactref element="D55" pad="C"/>
@@
 <wire x1="69.85" y1="97.4725" x2="66.675" y2="98.63" width="0.8128" layer="16"/>
 </signal>
-<signal name="4J2">
+<signal name="B4J2">
 <contactref element="J11" pad="1"/>
 <contactref element="D61" pad="C"/>
@@
 <wire x1="37.465" y1="74.295" x2="36.625" y2="74.93" width="0.6096" layer="16"/>
 </signal>
-<signal name="6J2">
+<signal name="B6J2">
 <contactref element="J12" pad="1"/>
 <wire x1="89.745046875" y1="38.0487" x2="83.82" y2="45.6315" width="0.6096" layer="16"/>
@@
 <wire x1="57.4675" y1="54.815" x2="61.5065" y2="54.6985" width="0.6096" layer="16"/>
 </signal>
-<signal name="6J3">
+<signal name="B6J3">
 <contactref element="J14" pad="1"/>
 <contactref element="D68" pad="C"/>
@@
 <wire x1="153.797" y1="70.612" x2="153.797" y2="69.342" width="0.6096" layer="16"/>
 </signal>
-<signal name="D1">
+<signal name="BD1">
 <contactref element="SV1" pad="10"/>
 <contactref element="J29" pad="2"/>
@@
 <wire x1="71.12" y1="114.3" x2="68.10375" y2="116.84" width="0.6096" layer="16"/>
 </signal>
-<signal name="D2">
+<signal name="BD2">
 <contactref element="SV1" pad="9"/>
 <contactref element="J30" pad="2"/>
@@
 <wire x1="41.91" y1="120.65" x2="42.545" y2="120.65" width="0.4064" layer="16"/>
 </signal>
-<signal name="D3">
+<signal name="BD3">
 <contactref element="SV1" pad="8"/>
 <contactref element="J31" pad="2"/>
@@
 <wire x1="145.542" y1="78.2955" x2="145.542" y2="80.9625" width="0.6096" layer="16"/>
 </signal>
+<signal name="B3J">
+<contactref element="J4" pad="1"/>
+<contactref element="D66" pad="C"/>
+<contactref element="D67B" pad="C"/>
+<wire x1="121.8315" y1="97.79" x2="125.095" y2="97.79" width="0.6096" layer="16"/>
+<wire x1="125.095" y1="97.79" x2="129.2225" y2="93.6625" width="0.6096" layer="16"/>
+<wire x1="129.2225" y1="93.6625" x2="136.8425" y2="93.6625" width="0.6096" layer="16"/>
+<contactref element="J46" pad="1"/>
+<wire x1="159.7025" y1="99.7835" x2="157.886" y2="99.1485" width="0.6096" layer="16"/>
+<wire x1="157.886" y1="99.1485" x2="154.94" y2="95.25" width="0.6096" layer="16"/>
+<wire x1="154.94" y1="95.25" x2="150.65375" y2="95.25" width="0.6096" layer="16"/>
+<wire x1="150.65375" y1="95.25" x2="144.4625" y2="88.74125" width="0.6096" layer="16"/>
+<wire x1="135.685" y1="75.565" x2="140.335" y2="80.85" width="0.6096" layer="16"/>
+<wire x1="140.335" y1="80.85" x2="140.335" y2="87.7425" width="0.6096" layer="16"/>
+<wire x1="140.335" y1="87.7425" x2="140.335" y2="89.23501875" width="0.6096" layer="16"/>
+<wire x1="143.51" y1="87.7425" x2="140.335" y2="87.7425" width="0.6096" layer="16"/>
+<wire x1="144.4625" y1="88.74125" x2="143.51" y2="87.7425" width="0.6096" layer="16"/>
+<wire x1="140.335" y1="89.23501875" x2="136.8425" y2="93.6625" width="0.6096" layer="16"/>
+<wire x1="121.8315" y1="97.79" x2="118.6565" y2="94.2975" width="0.6096" layer="16"/>
+</signal>
 </signals>
