File: PCB/~keyBoard_B/keyBoard_B.sch (EAGLE design)
At the start: 239 parts, among them J1 J, J10 J, J11 J, J12 J, J13 J, J14 J, J15 J, J16 J, J17 J, J18 J, J19 J, J2 J, J21 J, J22 J, J23 J, J24 J, J25 J, J26 J, J27 J, J28 J, J29 J, J3 J, J30 J, J31 J, J32 J, J33 J, J34 J, J35 J, J36 J, J37 J, J38 J, J39 J, J4 J, J40 J, J41 J, J42 J, J43 J, J44 J, J46 J, J48 J, J49 J, J5 J, J50 J, J51 J, J52 J, J53 J, J6 J, J7 J, J8 J, J9 J

Commit message: new pcb >
Connections:
- net +5V renamed +5V_B
- net 1 renamed B1
- net 2 renamed B2
- net 2J renamed B2J
- net 3 renamed B3
- net 3J renamed B3J
- net 4 renamed B4
- net 4J renamed B4J
- net 4J2 renamed B4J2
- net 5 renamed B5
- net 5J renamed B5J
- net 6 renamed B6
- net 6J2 renamed B6J2
- net 6J3 renamed B6J3
- net 7 renamed B7
- net 7J renamed B7J
- net 8 renamed B8
- net D1 renamed BD1
- net D2 renamed BD2
- net D3 renamed BD3
- net GND renamed GND_B
Other:
- moved on the sheet: J3, J4, J5
Changed lines of the file:
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@@
 <instance part="D87" gate="G$1" x="22.86" y="10.16"/>
 <instance part="J2" gate="G$1" x="182.88" y="132.08"/>
-<instance part="J3" gate="G$1" x="190.5" y="144.78" rot="MR0"/>
-<instance part="J4" gate="G$1" x="180.34" y="144.78" rot="MR0"/>
-<instance part="J5" gate="G$1" x="177.8" y="139.7"/>
+<instance part="J3" gate="G$1" x="193.04" y="144.78" rot="MR0"/>
+<instance part="J4" gate="G$1" x="182.88" y="144.78" rot="MR0"/>
+<instance part="J5" gate="G$1" x="182.88" y="139.7"/>
 <instance part="J6" gate="G$1" x="162.56" y="132.08"/>
 <instance part="J9" gate="G$1" x="162.56" y="116.84"/>
@@
 </segment>
 </net>
-<net name="1" class="0">
+<net name="B1" class="0">
 <segment>
 <pinref part="D50" gate="G$1" pin="C"/>
@@
 </segment>
 </net>
-<net name="2" class="0">
+<net name="B2" class="0">
 <segment>
 <pinref part="D51" gate="G$1" pin="C"/>
@@
 </segment>
 </net>
-<net name="3J" class="0">
-<segment>
-<pinref part="D66" gate="G$1" pin="C"/>
-<wire x1="83.82" y1="50.8" x2="93.98" y2="50.8" width="0.1524" layer="91"/>
-<label x="86.36" y="50.8" size="1.778" layer="95"/>
-</segment>
-<segment>
-<pinref part="D67B" gate="G$1" pin="C"/>
-<wire x1="157.48" y1="63.5" x2="149.86" y2="63.5" width="0.1524" layer="91"/>
-<label x="152.4" y="63.5" size="1.778" layer="95"/>
-</segment>
-<segment>
-<pinref part="J4" gate="G$1" pin="P$1"/>
-<wire x1="175.26" y1="144.78" x2="172.72" y2="144.78" width="0.1524" layer="91"/>
-<label x="175.26" y="144.78" size="1.778" layer="95" rot="MR0"/>
-</segment>
-<segment>
-<pinref part="J46" gate="G$1" pin="P$1"/>
-<wire x1="104.14" y1="193.04" x2="119.38" y2="193.04" width="0.1524" layer="91"/>
-<label x="116.84" y="193.04" size="1.778" layer="95"/>
-</segment>
-</net>
-<net name="4" class="0">
+<net name="B4" class="0">
 <segment>
 <pinref part="D74" gate="G$1" pin="C"/>
@@
 <segment>
 <pinref part="J5" gate="G$1" pin="P$1"/>
-<wire x1="182.88" y1="139.7" x2="185.42" y2="139.7" width="0.1524" layer="91"/>
+<wire x1="187.96" y1="139.7" x2="190.5" y2="139.7" width="0.1524" layer="91"/>
 <label x="182.88" y="139.7" size="1.778" layer="95"/>
 </segment>
@@
 </segment>
 </net>
-<net name="5" class="0">
+<net name="B5" class="0">
 <segment>
 <pinref part="D67" gate="G$1" pin="C"/>
@@
 </segment>
 </net>
-<net name="6" class="0">
+<net name="B6" class="0">
 <segment>
 <pinref part="D81" gate="G$1" pin="C"/>
@@
 </segment>
 </net>
-<net name="7" class="0">
+<net name="B7" class="0">
 <segment>
 <pinref part="D85" gate="G$1" pin="C"/>
@@
 </segment>
 </net>
-<net name="8" class="0">
+<net name="B8" class="0">
 <segment>
 <pinref part="D86" gate="G$1" pin="C"/>
@@
 </segment>
 </net>
-<net name="3" class="0">
+<net name="B3" class="0">
 <segment>
 <pinref part="D57" gate="G$1" pin="C"/>
@@
 <segment>
 <pinref part="J3" gate="G$1" pin="P$2"/>
-<wire x1="193.04" y1="144.78" x2="195.58" y2="144.78" width="0.1524" layer="91"/>
-<label x="195.58" y="144.78" size="1.778" layer="95" rot="MR0"/>
+<wire x1="195.58" y1="144.78" x2="198.12" y2="144.78" width="0.1524" layer="91"/>
+<label x="198.12" y="144.78" size="1.778" layer="95" rot="MR0"/>
 </segment>
 <segment>
@@
 <pinref part="J3" gate="G$1" pin="P$1"/>
 <pinref part="J4" gate="G$1" pin="P$2"/>
-<wire x1="185.42" y1="144.78" x2="182.88" y2="144.78" width="0.1524" layer="91"/>
-</segment>
-</net>
-<net name="4J" class="0">
+<wire x1="187.96" y1="144.78" x2="185.42" y2="144.78" width="0.1524" layer="91"/>
+</segment>
+</net>
+<net name="B4J" class="0">
 <segment>
 <pinref part="D64" gate="G$1" pin="C"/>
@@
 <segment>
 <pinref part="J5" gate="G$1" pin="P$2"/>
-<wire x1="172.72" y1="139.7" x2="175.26" y2="139.7" width="0.1524" layer="91"/>
-<label x="172.72" y="139.7" size="1.778" layer="95"/>
+<wire x1="175.26" y1="139.7" x2="180.34" y2="139.7" width="0.1524" layer="91"/>
+<label x="175.26" y="139.7" size="1.778" layer="95"/>
 </segment>
 <segment>
@@
 </segment>
 </net>
-<net name="5J" class="0">
+<net name="B5J" class="0">
 <segment>
 <pinref part="J6" gate="G$1" pin="P$2"/>
@@
 </segment>
 </net>
-<net name="7J" class="0">
+<net name="B7J" class="0">
 <segment>
 <pinref part="D78" gate="G$1" pin="C"/>
@@
 </segment>
 </net>
-<net name="GND" class="0">
+<net name="GND_B" class="0">
 <segment>
 <pinref part="2D1" gate="A" pin="G2A"/>
@@
 </segment>
 </net>
-<net name="+5V" class="0">
+<net name="+5V_B" class="0">
 <segment>
 <pinref part="P+1" gate="1" pin="+5V"/>
@@
 </segment>
 </net>
-<net name="2J" class="0">
+<net name="B2J" class="0">
 <segment>
 <pinref part="J10" gate="G$1" pin="P$1"/>
@@
 </segment>
 </net>
-<net name="4J2" class="0">
+<net name="B4J2" class="0">
 <segment>
 <pinref part="J11" gate="G$1" pin="P$1"/>
@@
 </segment>
 </net>
-<net name="6J2" class="0">
+<net name="B6J2" class="0">
 <segment>
 <pinref part="J12" gate="G$1" pin="P$1"/>
@@
 </segment>
 </net>
-<net name="6J3" class="0">
+<net name="B6J3" class="0">
 <segment>
 <pinref part="J14" gate="G$1" pin="P$1"/>
@@
 </segment>
 </net>
-<net name="D1" class="0">
+<net name="BD1" class="0">
 <segment>
 <label x="10.16" y="205.74" size="1.778" layer="95"/>
@@
 </segment>
 </net>
-<net name="D2" class="0">
+<net name="BD2" class="0">
 <segment>
 <label x="10.16" y="208.28" size="1.778" layer="95"/>
@@
 </segment>
 </net>
-<net name="D3" class="0">
+<net name="BD3" class="0">
 <segment>
 <label x="10.16" y="210.82" size="1.778" layer="95"/>
@@
 </segment>
 </net>
+<net name="B3J" class="0">
+<segment>
+<pinref part="J4" gate="G$1" pin="P$1"/>
+<wire x1="177.8" y1="144.78" x2="172.72" y2="144.78" width="0.1524" layer="91"/>
+<label x="177.8" y="144.78" size="1.778" layer="95" rot="MR0"/>
+</segment>
+<segment>
+<pinref part="D66" gate="G$1" pin="C"/>
+<wire x1="83.82" y1="50.8" x2="93.98" y2="50.8" width="0.1524" layer="91"/>
+<label x="86.36" y="50.8" size="1.778" layer="95"/>
+</segment>
+<segment>
+<pinref part="D67B" gate="G$1" pin="C"/>
+<wire x1="157.48" y1="63.5" x2="149.86" y2="63.5" width="0.1524" layer="91"/>
+<label x="152.4" y="63.5" size="1.778" layer="95"/>
+</segment>
+<segment>
+<pinref part="J46" gate="G$1" pin="P$1"/>
+<wire x1="104.14" y1="193.04" x2="119.38" y2="193.04" width="0.1524" layer="91"/>
+<label x="116.84" y="193.04" size="1.778" layer="95"/>
+</segment>
+</net>
