File: PCB/keyBoard_A_B/keyBoard_A.sch (EAGLE design)
At the start: 525 parts, among them IC1 74HC04N, IC2 LMV358IDGKR, J1 J, J10 J, J11 J, J12 J, J13 J, J14 J, J15 J, J16 J, J17 J, J18 J, J19 J, J2 J, J20 J, J21 J, J22 J, J23 J, J24 J, J25 J, J26 J, J27 J, J28 J, J29 J, J3 J, J30 J, J31 J, J32 J, J33 J, J34 J, J35 J, J36 J, J37 J, J38 J, J39 J, J4 J, J40 J, J41 J, J42 J, J43 J, J44 J, J45 J, J46 J, J47 USB MICRO, J48 J, J49 J, J5 J, J50 J, J51 J, J52 J, J53 J, J54 J, J55 J, J56 J, J57 J, J58 J, J59 J, J6 J, J60 J, J61 J, J62 J, J63 J, J64 J, J65 J, J66 J, J67 J, J68 J, J69 J, J7 J, J70 J, J71 J, J72 J, J73 J, J74 J, J75 J, J76 J, J77 J, J78 J, J79 J, J8 J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

Commit message: pcb new b ab
Parts:
- added J84, J85: J, detali2:J
- C19: device rcl:C-EUC0805 -> rcl:C-EUC1206K
- R16: device rcl:R-EU_R0805 -> rcl:R-EU_R1206W
Connections:
- removed net N$400: 2D1A.Y4, J90.P$2
- removed net N$402: J93.P$1, J94.P$2
- removed net N$403: 2D1A.Y6, J93.P$2
- new net B6J4: D83.C, J93.P$1, J94.P$2
- new net N$310: 2D1A.Y4, J93.P$2
- new net N$323: 2D1A.Y6, J90.P$2
- new net N$393: J85.P$1, JA59.2, JA67.2, JA67B.2, JA81.2, JA85.2, JA86.2, JB74.1
- new net N$394: J84.P$1, J85.P$2
- net B6: no longer D83.C
- net G6: now also J84.P$2; no longer JA59.2, JA67.2, JA67B.2, JA67B1.2, JA81.2, JA85.2, JA86.2, JB74.1
Other:
- moved on the sheet: D83

Commit message: pcb b
Parts:
- added J86: J, detali2:J
Connections:
- new net N$225: C19.1, J86.P$1, R16.1
- net +5V_B: now also J86.P$2; no longer C19.1, R16.1
Other:
- moved on the sheet: 2D1P, 2D2P, C19, C20, D52, D53, D59, D66, D74, D80, D81, D89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

Commit message: pcb b ok
Parts:
- removed JA67B1: (no value), detali:SJ
- removed S67B: |u, cherrymx:CHERRY-MX
Changed lines of the file:
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@@
 <part name="S87" library="cherrymx" deviceset="CHERRY-MX-4P" device="" value="FN2"/>
 <part name="2D2" library="detali2" deviceset="74*04" device="N" technology="ALS" value="74HC04N"/>
-<part name="S67B" library="cherrymx" deviceset="CHERRY-MX" device="" value="|u"/>
-<part name="JA67B1" library="detali" deviceset="SJ" device=""/>
 <part name="SV4" library="detali2" deviceset="FE12-1" device="" value="CON_KB_B"/>
 <part name="JB67B" library="detali" deviceset="SJ" device=""/>
@@
 <instance part="S87" gate="G$1" x="53.34" y="10.16" rot="MR0"/>
 <instance part="2D2" gate="C" x="154.94" y="254"/>
-<instance part="S67B" gate="G$1" x="190.5" y="63.5" smashed="yes">
-<attribute name="PART" x="185.42" y="60.96" size="1.27" layer="95"/>
-<attribute name="VALUE" x="185.42" y="58.42" size="1.27" layer="96"/>
-</instance>
-<instance part="JA67B1" gate="1" x="203.2" y="63.5"/>
 <instance part="SV4" gate="G$1" x="193.04" y="233.68" smashed="yes" rot="MR0">
 <attribute name="VALUE" x="194.31" y="205.74" size="1.778" layer="96" rot="MR0"/>

Commit message: b pl mod
Changed lines of the file:
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@@
 <instance part="P+14" gate="1" x="30.48" y="195.58" rot="R90"/>
 <instance part="C19" gate="G$1" x="50.8" y="193.04" smashed="yes" rot="MR270">
-<attribute name="NAME" x="49.276" y="190.881" size="1.778" layer="95" rot="MR0"/>
-<attribute name="VALUE" x="44.196" y="190.881" size="1.778" layer="96" rot="MR0"/>
+<attribute name="NAME" x="41.656" y="190.881" size="1.778" layer="95" rot="MR0"/>
+<attribute name="VALUE" x="49.276" y="190.881" size="1.778" layer="96" rot="MR0"/>
 </instance>
 <instance part="2D1" gate="P" x="45.72" y="236.22" smashed="yes" rot="MR90">

Commit message: new pcb b
Parts:
- added S88: ~Ё, cherrymx:CHERRY-MX-4P
Changed lines of the file:
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@@
 <part name="J85" library="detali2" deviceset="J" device="" value=""/>
 <part name="J86" library="detali2" deviceset="J" device="" value=""/>
+<part name="S88" library="cherrymx" deviceset="CHERRY-MX-4P" device="" value="~Ё"/>
 </parts>
 <sheets>
@@
 </instance>
 <instance part="S44A" gate="G$1" x="238.76" y="152.4"/>
+<instance part="S88" gate="G$1" x="127" y="205.74"/>
 </instances>
 <busses>
