File: PCB/keyBoard_A_B/keyBoard_A.brd (EAGLE design)
At the start: 358.8 x 253 mm, 622 parts, among them IC1 74HC04N, IC2 LMV358IDGKR, J1 J, J10 J, J11 J, J12 J, J13 J, J14 J, J15 J, J16 J, J17 J, J18 J, J19 J, J2 J, J20 J, J21 J, J22 J, J23 J, J24 J, J25 J, J26 J, J27 J, J28 J, J29 J, J3 J, J30 J, J31 J, J32 J, J33 J, J34 J, J35 J, J36 J, J37 J, J38 J, J39 J, J4 J, J40 J, J41 J, J42 J, J43 J, J44 J, J45 J, J47 USB MICRO, J5 J, J6 J, J7 J, J8 J, J9 J, Y1 16MHz KX-7, Y3 16MHz KX-7

Commit message: pcb new b ab
Parts:
- removed U$99: (no value), kbmx:18X18
- added J84, J85: (no value), detali2:R1206W
- C19: device rcl:C0805 -> rcl:C1206K
- R16: device rcl:R0805 -> rcl:R1206W
- moved U$96 85.4 mm to (419.1, -322.6)
- moved JA67B1 34.7 mm to (369.3, -302.6), turned to 0 degrees
- moved J90 8.09 mm to (339.7, -281.9), turned to 180 degrees
- moved S67 7.36 mm to (332.1, -292.7)
- moved C19 6.38 mm to (321.3, -254.3)
- moved D83 6.13 mm to (314.6, -337.2)
- moved JA67 4.93 mm to (336.9, -299.1)
- moved D69 3.31 mm to (334.3, -301.6)
- moved JB42 2.62 mm to (180.3, -336.6)
- moved J92 2.54 mm to (333.9, -317.2)
- moved J88 2.13 mm to (324.5, -276.2)
- moved J83 1.91 mm to (324.5, -271.1)
- moved JB59 1.90 mm to (328.3, -276.2)
- moved 2D1 1.62 mm to (321.6, -253.0), turned to 270 degrees
- moved D42 1.59 mm to (179.1, -340.7)
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Connections:
- removed net N$400: 2D1.11, J90.2
- removed net N$402: J93.1, J94.2
- removed net N$403: 2D1.9, J93.2
- new net B6J4: D83.C, J93.1, J94.2
- new net N$310: 2D1.11, J93.2
- new net N$323: 2D1.9, J90.2
- new net N$393: J85.1, JA59.2, JA67.2, JA67B.2, JA81.2, JA85.2, JA86.2, JB74.1
- new net N$394: J84.1, J85.2
- net B6: no longer D83.C
- net G6: now also J84.2; no longer JA59.2, JA67.2, JA67B.2, JA67B1.2, JA81.2, JA85.2, JA86.2, JB74.1
Routing:
- net N$393: track 0.00 -> 172.2 mm
- net G6: track 175.8 -> 48.8 mm
- net N$310: track 0.00 -> 106.6 mm
- net N$403: track 94.5 -> 0.00 mm
- net N$323: track 0.00 -> 35.9 mm
- net GND_B: track 140.4 -> 161.8 mm
- net +5V_B: track 134.7 -> 153.4 mm
- net B6J4: track 0.00 -> 17.3 mm
- net B7: track 217.1 -> 234.2 mm
- net N$402: track 16.5 -> 0.00 mm
- net B8: track 123.9 -> 139.7 mm
- net B5J5: track 64.5 -> 78.9 mm
- net N$400: track 11.6 -> 0.00 mm
- net N$388: track 15.3 -> 20.9 mm
- net N$290: track 7.38 -> 2.09 mm
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Other:
- board size 358.8 x 253 mm -> 383.5 x 254.6 mm

Commit message: pcb b
Parts:
- added J86: (no value), detali2:R1206W
- moved J85 0.32 mm to (321.3, -246.7)
Connections:
- new net N$225: C19.1, J86.1, R16.1
- net +5V_B: now also J86.2; no longer C19.1, R16.1
Routing:
- net N$225: track 0.00 -> 8.67 mm
- net N$391: track 14.2 -> 19.4 mm
- net N$389: track 19.7 -> 20.2 mm
Changed lines of the file:
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@@
 <element name="J83" library="detali2" package="R1206W" value="" x="324.485" y="-271.145" rot="R270"/>
 <element name="J84" library="detali2" package="R1206W" value="" x="321.6275" y="-241.6175" rot="R270"/>
-<element name="J85" library="detali2" package="R1206W" value="" x="321.6275" y="-246.6975" rot="R270"/>
+<element name="J85" library="detali2" package="R1206W" value="" x="321.31" y="-246.6975" rot="R270"/>
+<element name="J86" library="detali2" package="R1206W" value="" x="323.215" y="-246.6975" rot="R270"/>
 </elements>
 <signals>
@@
 <contactref element="2D1" pad="4"/>
 <contactref element="2D1" pad="5"/>
-<contactref element="C19" pad="2"/>
 <contactref element="2D1" pad="8"/>
 <wire x1="317.8175" y1="-251.7775" x2="317.8175" y2="-254.3175" width="1.016" layer="16"/>
@@
 <wire x1="310.515" y1="-260.985" x2="310.515" y2="-261.9375" width="0.6096" layer="1"/>
 <wire x1="310.515" y1="-261.9375" x2="317.8175" y2="-261.9375" width="0.6096" layer="1"/>
-<wire x1="319.81" y1="-254.3175" x2="317.8175" y2="-254.3175" width="1.016" layer="16"/>
 <wire x1="317.8175" y1="-254.3175" x2="314.96" y2="-255.5875" width="1.016" layer="16"/>
 <wire x1="317.8175" y1="-261.9375" x2="314.96" y2="-261.9375" width="1.016" layer="16"/>
 <wire x1="314.96" y1="-261.9375" x2="314.96" y2="-255.5875" width="1.016" layer="16"/>
+<contactref element="C19" pad="2"/>
+<wire x1="319.81" y1="-254.3175" x2="317.8175" y2="-254.3175" width="1.016" layer="16"/>
 </signal>
 <signal name="N$407">
@@
 <wire x1="309.88" y1="-242.57" x2="311.4675" y2="-242.57" width="0.6096" layer="16"/>
 <contactref element="2D1" pad="15"/>
-<wire x1="325.4375" y1="-246.6975" x2="320.04" y2="-246.6975" width="0.6096" layer="16"/>
-<wire x1="320.04" y1="-246.6975" x2="320.04" y2="-243.205" width="0.6096" layer="16"/>
+<wire x1="325.4375" y1="-246.6975" x2="319.7225" y2="-246.6975" width="0.6096" layer="16"/>
+<wire x1="319.7225" y1="-246.6975" x2="319.7225" y2="-243.205" width="0.6096" layer="16"/>
 <wire x1="327.865" y1="-243.5225" x2="327.3425" y2="-246.0625" width="0.6096" layer="16"/>
 <wire x1="327.3425" y1="-246.0625" x2="325.4375" y2="-246.6975" width="0.6096" layer="16"/>
 <wire x1="311.4675" y1="-242.57" x2="312.1025" y2="-242.2525" width="0.6096" layer="16"/>
 <wire x1="312.1025" y1="-242.2525" x2="319.0875" y2="-242.2525" width="0.6096" layer="16"/>
-<wire x1="319.0875" y1="-242.2525" x2="320.04" y2="-243.205" width="0.6096" layer="16"/>
+<wire x1="319.0875" y1="-242.2525" x2="319.7225" y2="-243.205" width="0.6096" layer="16"/>
 </signal>
 <signal name="B2">
@@
 </signal>
 <signal name="+5V_B">
-<contactref element="R16" pad="1"/>
 <contactref element="2D1" pad="16"/>
-<contactref element="C19" pad="1"/>
 <contactref element="D93" pad="A"/>
 <contactref element="SV4" pad="11"/>
@@
 <via x="325.4375" y="-241.935" extent="1-16" drill="0.8" diameter="2.3" shape="square"/>
 <wire x1="325.4375" y1="-241.935" x2="325.4375" y2="-244.1575" width="1.016" layer="16"/>
-<wire x1="322.81" y1="-254.3175" x2="325.4375" y2="-244.1575" width="0" layer="19" extent="16-16"/>
-<wire x1="227.4185" y1="-269.24" x2="222.035" y2="-262.298490625" width="0" layer="19" extent="16-16"/>
-<wire x1="322.809" y1="-256.8575" x2="322.81" y2="-254.3175" width="1.016" layer="16"/>
 <wire x1="325.4375" y1="-237.8075" x2="325.4375" y2="-241.935" width="0.6096" layer="1"/>
+<contactref element="J86" pad="2"/>
+<wire x1="227.4185" y1="-269.24" x2="222.035" y2="-262.298490625" width="0" layer="19" extent="16-16"/>
+<wire x1="325.4375" y1="-244.1575" x2="324.256" y2="-244.1575" width="1.016" layer="16"/>
+<wire x1="324.256" y1="-244.1575" x2="323.215" y2="-245.1985" width="1.016" layer="16"/>
 </signal>
 <signal name="N$360">
@@
 <wire x1="305.435" y1="-332.4225" x2="303.022" y2="-332.4225" width="0.6096" layer="16"/>
 <wire x1="303.657" y1="-252.73" x2="307.635603125" y2="-252.73" width="0.6096" layer="16"/>
-<wire x1="311.4675" y1="-248.898103125" x2="311.4675" y2="-245.4275" width="0.4064" layer="16"/>
-<wire x1="311.4675" y1="-245.4275" x2="310.8325" y2="-244.069" width="0.4064" layer="16"/>
 <wire x1="302.54575" y1="-272.6055" x2="302.895" y2="-272.25625" width="0.6096" layer="16"/>
 <wire x1="302.895" y1="-272.25625" x2="302.895" y2="-268.9225" width="0.6096" layer="16"/>
 <wire x1="303.2125" y1="-262.89" x2="303.2125" y2="-254.635" width="0.6096" layer="16"/>
 <wire x1="303.2125" y1="-254.635" x2="303.657" y2="-252.73" width="0.6096" layer="16"/>
-<wire x1="307.635603125" y1="-252.73" x2="311.4675" y2="-248.898103125" width="0.6096" layer="16"/>
+<wire x1="307.635603125" y1="-252.73" x2="311.30875" y2="-249.056853125" width="0.6096" layer="16"/>
 <wire x1="302.895" y1="-268.9225" x2="301.3075" y2="-266.7" width="0.6096" layer="16"/>
 <wire x1="301.3075" y1="-266.7" x2="301.3075" y2="-264.16" width="0.6096" layer="16"/>
 <wire x1="301.3075" y1="-264.16" x2="303.2125" y2="-262.89" width="0.6096" layer="16"/>
+<wire x1="310.8325" y1="-244.069" x2="311.30875" y2="-245.0215" width="0.6096" layer="16"/>
+<wire x1="311.30875" y1="-245.0215" x2="311.30875" y2="-249.056853125" width="0.4064" layer="16"/>
 </signal>
 <signal name="G6">
@@
 <contactref element="2D1" pad="1"/>
 <wire x1="304.7115" y1="-257.175" x2="306.705" y2="-257.175" width="0.6096" layer="16"/>
-<wire x1="306.705" y1="-257.175" x2="314.0075" y2="-250.19" width="0.6096" layer="16"/>
-<wire x1="314.0075" y1="-250.19" x2="314.0075" y2="-247.015" width="0.6096" layer="16"/>
-<wire x1="314.0075" y1="-247.015" x2="315.2775" y2="-244.1575" width="0.6096" layer="16"/>
-<wire x1="315.2775" y1="-244.1575" x2="317.8175" y2="-244.1575" width="0.6096" layer="16"/>
+<wire x1="306.705" y1="-257.175" x2="313.21375" y2="-250.98375" width="0.6096" layer="16"/>
+<wire x1="317.8175" y1="-244.1575" x2="315.43625" y2="-244.1575" width="0.6096" layer="16"/>
+<wire x1="313.21375" y1="-246.22125" x2="313.21375" y2="-250.98375" width="0.4064" layer="16"/>
+<wire x1="315.43625" y1="-244.1575" x2="313.21375" y2="-246.22125" width="0.6096" layer="16"/>
 </signal>
 <signal name="N$389">
@@
 <contactref element="2D1" pad="2"/>
 <wire x1="304.7115" y1="-259.3975" x2="306.3875" y2="-259.3975" width="0.6096" layer="16"/>
-<wire x1="306.3875" y1="-259.3975" x2="315.2775" y2="-250.825" width="0.6096" layer="16"/>
-<wire x1="315.2775" y1="-250.825" x2="315.2775" y2="-247.9675" width="0.6096" layer="16"/>
-<wire x1="315.2775" y1="-247.9675" x2="317.8175" y2="-246.6975" width="0.6096" layer="16"/>
+<wire x1="306.3875" y1="-259.3975" x2="314.16625" y2="-251.93625" width="0.6096" layer="16"/>
+<wire x1="317.8175" y1="-246.6975" x2="316.07125" y2="-246.6975" width="0.6096" layer="16"/>
+<wire x1="314.16625" y1="-248.6025" x2="314.16625" y2="-251.93625" width="0.4064" layer="16"/>
+<wire x1="316.07125" y1="-246.6975" x2="314.16625" y2="-248.6025" width="0.6096" layer="16"/>
 </signal>
 <signal name="N$391">
@@
 <wire x1="304.7115" y1="-261.62" x2="306.07" y2="-261.62" width="0.6096" layer="16"/>
 <wire x1="306.07" y1="-261.62" x2="315.2775" y2="-252.73" width="0.6096" layer="16"/>
-<wire x1="315.2775" y1="-252.73" x2="317.8175" y2="-249.2375" width="0" layer="19" extent="16-16"/>
+<wire x1="315.2775" y1="-250.66625" x2="315.2775" y2="-252.73" width="0.4064" layer="16"/>
+<wire x1="317.8175" y1="-249.2375" x2="316.70625" y2="-249.2375" width="0.6096" layer="16"/>
+<wire x1="316.70625" y1="-249.2375" x2="315.2775" y2="-250.66625" width="0.6096" layer="16"/>
 </signal>
 <signal name="N$396">
@@
 <contactref element="J46" pad="1"/>
 <contactref element="J95" pad="2"/>
-<wire x1="312.7375" y1="-249.555" x2="312.7375" y2="-245.4275" width="0.4064" layer="16"/>
-<wire x1="312.7375" y1="-245.4275" x2="313.055" y2="-243.7515" width="0.4064" layer="16"/>
 <wire x1="304.7115" y1="-254.9525" x2="307.0225" y2="-254.9525" width="0.6096" layer="16"/>
-<wire x1="307.0225" y1="-254.9525" x2="312.7375" y2="-249.555" width="0.6096" layer="16"/>
+<wire x1="307.0225" y1="-254.9525" x2="312.26125" y2="-250.03125" width="0.6096" layer="16"/>
+<wire x1="312.26125" y1="-245.4275" x2="312.26125" y2="-250.03125" width="0.4064" layer="16"/>
+<wire x1="313.055" y1="-243.7515" x2="312.26125" y2="-245.4275" width="0.6096" layer="16"/>
 </signal>
 <signal name="N$406">
@@
 <wire x1="339.725" y1="-283.21" x2="339.725" y2="-280.67" width="0.6096" layer="16"/>
 <wire x1="339.725" y1="-280.67" x2="339.852" y2="-279.4" width="0.6096" layer="16"/>
-<wire x1="321.31" y1="-259.08" x2="321.6275" y2="-248.1965" width="0.6096" layer="16"/>
+<wire x1="321.31" y1="-259.08" x2="321.31" y2="-248.1965" width="0.6096" layer="16"/>
 <contactref element="J85" pad="1"/>
 <wire x1="323.0245" y1="-271.272" x2="325.9455" y2="-271.272" width="0.6096" layer="16"/>
@@
 <contactref element="J84" pad="1"/>
 <contactref element="J85" pad="2"/>
-<wire x1="321.6275" y1="-245.1985" x2="321.6275" y2="-243.1165" width="1.016" layer="16"/>
+<wire x1="321.31" y1="-245.1985" x2="321.6275" y2="-243.1165" width="1.016" layer="16"/>
+</signal>
+<signal name="N$225">
+<contactref element="R16" pad="1"/>
+<contactref element="C19" pad="1"/>
+<contactref element="J86" pad="1"/>
+<wire x1="322.809" y1="-256.8575" x2="322.81" y2="-254.3175" width="1.016" layer="16"/>
+<wire x1="322.81" y1="-254.3175" x2="323.215" y2="-248.1965" width="1.016" layer="16"/>
 </signal>
 </signals>

Commit message: pcb b ok
Parts:
- removed JA67B1: (no value), detali:SJ
- removed S67B: |u, cherrymx:CHERRY-MX
- removed U$165: (no value), kbmxco:SIZE132
- removed U$88: (no value), kbmx:18X37
- removed U$96: (no value), kbmx:18X28
- U$15: device kbmx:18X23 -> kbmxco:SIZE132
- moved U$97 11.5 mm to (253.2, -367.8)
- moved U$15 11.3 mm to (124.4, -368.0), turned to 270 degrees
- moved J90 3.81 mm to (335.9, -281.9)
- moved JA59 3.19 mm to (335.9, -279.1), turned to 90 degrees
- moved D58 0.32 mm to (264.2, -271.5)
Routing:
- net N$399: track 60.1 -> 56.2 mm
- net N$323: track 35.9 -> 38.1 mm
- net BD1: track 45.1 -> 44.1 mm
- net N$310: track 106.6 -> 107.4 mm
- net B8: track 139.7 -> 140.4 mm
- net B5J5: track 78.9 -> 79.6 mm
- net B7: track 234.2 -> 234.9 mm
- added copper zone on layer 16, net +5V_B
- added copper zone on layer 1, net GND
- added copper zone on layer 1, net N$559
Other:
- board size 383.5 x 254.6 mm -> 352.1 x 253 mm

Commit message: new pcb b
Parts:
- added S88: ~Ё, cherrymx:CHERRY-MX-4P
- added U$88: (no value), kbmx:18X18
- moved SV3 13.1 mm to (66.0, -261.0), turned to 0 degrees
Other:
- board size 352.1 x 253 mm -> 352.1 x 249.9 mm
Changed lines of the file:
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@@
 <circle x="169.545" y="-340.36" radius="2.5" width="0.254" layer="21"/>
 <circle x="169.545" y="-256.54" radius="2.5" width="0.254" layer="20"/>
-<wire x1="57.785" y1="-227.965" x2="57.785" y2="-356.235" width="0.2" layer="20"/>
+<wire x1="53.34" y1="-236.22" x2="53.34" y2="-364.49" width="0.2" layer="20"/>
 <wire x1="189.23" y1="-234.315" x2="189.23" y2="-340.6775" width="0.2" layer="20"/>
 <wire x1="350.04375" y1="-365.76" x2="192.405" y2="-365.76" width="0.2" layer="20"/>
@@
 <element name="J44" library="detali_main" package="R1206W" value="J" x="10.795" y="-334.01"/>
 <element name="J45" library="detali_main" package="R1206W" value="J" x="14.605" y="-293.0525" rot="R180"/>
-<element name="SV3" library="detali_main" package="FE13" value="" x="57.785" y="-271.145" rot="R90">
-<attribute name="OC_NEWARK" value="unknown" x="57.785" y="-271.145" size="1.778" layer="27" rot="R90" display="off"/>
-<attribute name="MPN" value="" x="57.785" y="-271.145" size="1.778" layer="27" rot="R90" display="off"/>
-<attribute name="MF" value="" x="57.785" y="-271.145" size="1.778" layer="27" rot="R90" display="off"/>
-<attribute name="OC_FARNELL" value="unknown" x="57.785" y="-271.145" size="1.778" layer="27" rot="R90" display="off"/>
+<element name="SV3" library="detali_main" package="FE13" value="" x="66.04" y="-260.985">
+<attribute name="OC_NEWARK" value="unknown" x="66.04" y="-260.985" size="1.778" layer="27" display="off"/>
+<attribute name="MPN" value="" x="66.04" y="-260.985" size="1.778" layer="27" display="off"/>
+<attribute name="MF" value="" x="66.04" y="-260.985" size="1.778" layer="27" display="off"/>
+<attribute name="OC_FARNELL" value="unknown" x="66.04" y="-260.985" size="1.778" layer="27" display="off"/>
 </element>
 <element name="SCROLL" library="detali_main" package="LED5MM" value="" x="59.055" y="-242.8875" rot="R180"/>
@@
 <element name="J86" library="detali2" package="R1206W" value="" x="323.215" y="-246.6975" rot="R270"/>
 <element name="U$15" library="kbmxco" package="SIZE132" value="" x="124.42825" y="-368.04168125" rot="R270"/>
+<element name="S88" library="cherrymx" package="CHERRY-MX-4P" value="~Ё" x="64.77" y="-273.685" rot="R180"/>
+<element name="U$88" library="kbmx" package="18X18" value="" x="63.5" y="-272.415"/>
 </elements>
 <signals>
@@
 <vertex x="392.43" y="-227.33"/>
 </polygon>
-<wire x1="50.8" y1="-292.4175" x2="57.785" y2="-286.385" width="0" layer="19" extent="1-1"/>
+<wire x1="50.8" y1="-292.4175" x2="50.8" y2="-260.985" width="0" layer="19" extent="1-1"/>
 <wire x1="31.435" y1="-401.0025" x2="17.145" y2="-339.0875" width="0" layer="19" extent="1-16"/>
 <wire x1="83.5025" y1="-399.9625" x2="31.435" y2="-401.0025" width="0" layer="19" extent="1-1"/>
@@
 <contactref element="R25" pad="2"/>
 <contactref element="SV6" pad="11"/>
-<wire x1="57.785" y1="-249.8725" x2="57.785" y2="-255.905" width="0" layer="19" extent="1-1"/>
+<wire x1="57.785" y1="-249.8725" x2="81.28" y2="-260.985" width="0" layer="19" extent="1-1"/>
 <wire x1="57.785" y1="-242.8875" x2="57.785" y2="-249.8725" width="0" layer="19" extent="1-1"/>
-<wire x1="19.685" y1="-317.18" x2="57.785" y2="-255.905" width="0" layer="19" extent="16-16"/>
+<wire x1="19.685" y1="-317.18" x2="81.28" y2="-260.985" width="0" layer="19" extent="16-16"/>
 <wire x1="16.51" y1="-318.45" x2="19.685" y2="-317.18" width="0" layer="19" extent="16-16"/>
 <wire x1="4.765" y1="-323.215" x2="16.51" y2="-318.45" width="0" layer="19" extent="16-16"/>
@@
 <wire x1="4.1275" y1="-347.665" x2="3.495" y2="-335.915" width="0" layer="19" extent="16-16"/>
 <wire x1="33.335" y1="-401.0025" x2="4.1275" y2="-347.665" width="0" layer="19" extent="1-16"/>
-<wire x1="139.7" y1="-256.54" x2="57.785" y2="-255.905" width="0" layer="19" extent="1-1"/>
+<wire x1="139.7" y1="-256.54" x2="81.28" y2="-260.985" width="0" layer="19" extent="1-1"/>
 <wire x1="152.4" y1="-258.851" x2="139.7" y2="-256.54" width="0" layer="19" extent="16-16"/>
 <wire x1="93.345" y1="-462.915" x2="33.335" y2="-401.0025" width="0" layer="19" extent="1-1"/>
@@
 <contactref element="J38" pad="2"/>
 <contactref element="SV3" pad="12"/>
-<wire x1="91.211" y1="-265.7475" x2="57.785" y2="-258.445" width="0" layer="19" extent="16-16"/>
+<wire x1="91.211" y1="-265.7475" x2="78.74" y2="-260.985" width="0" layer="19" extent="16-16"/>
 </signal>
 <signal name="D2">
 <contactref element="J39" pad="2"/>
 <contactref element="SV3" pad="11"/>
-<wire x1="91.211" y1="-263.525" x2="57.785" y2="-260.985" width="0" layer="19" extent="16-16"/>
+<wire x1="91.211" y1="-263.525" x2="76.2" y2="-260.985" width="0" layer="19" extent="16-16"/>
 </signal>
 <signal name="D3">
 <contactref element="J40" pad="2"/>
 <contactref element="SV3" pad="10"/>
-<wire x1="91.211" y1="-261.3025" x2="57.785" y2="-263.525" width="0" layer="19" extent="16-16"/>
+<wire x1="91.211" y1="-261.3025" x2="73.66" y2="-260.985" width="0" layer="19" extent="16-16"/>
 </signal>
 <signal name="AREF" class="4">
