File: PCB/keyBoard_A_B/keyBoard_A.brd (EAGLE design)
At the start: 352.1 x 249.9 mm, 621 parts, among them IC1 74HC04N, IC2 LMV358IDGKR, J1 J, J10 J, J11 J, J12 J, J13 J, J14 J, J15 J, J16 J, J17 J, J18 J, J19 J, J2 J, J20 J, J21 J, J22 J, J23 J, J24 J, J25 J, J26 J, J27 J, J28 J, J29 J, J3 J, J30 J, J31 J, J32 J, J33 J, J34 J, J35 J, J36 J, J37 J, J38 J, J39 J, J4 J, J40 J, J41 J, J42 J, J43 J, J44 J, J45 J, J47 USB MICRO, J5 J, J6 J, J7 J, J8 J, J9 J, Y1 16MHz KX-7, Y3 16MHz KX-7

Commit message: fix b
Other:
- outline, holes or cut-outs redrawn
Changed lines of the file:
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@@
 <setting verticaltext="up"/>
 </settings>
-<grid distance="25" unitdist="mil" unit="mil" style="lines" multiple="1" display="yes" altdistance="0.025" altunitdist="inch" altunit="inch"/>
+<grid distance="6.25" unitdist="mil" unit="mil" style="lines" multiple="1" display="yes" altdistance="0.025" altunitdist="inch" altunit="inch"/>
 <layers>
 <layer number="1" name="Top" color="4" fill="1" visible="no" active="yes"/>
@@
 <wire x1="188.595" y1="-234.315" x2="188.595" y2="-340.0425" width="0.2" layer="20"/>
 <wire x1="185.42" y1="-231.14" x2="4.28625" y2="-231.14" width="0.2" layer="20"/>
-<wire x1="185.42" y1="-365.76" x2="4.28625" y2="-365.76" width="0.2" layer="20"/>
+<wire x1="179.86375" y1="-365.76" x2="4.28625" y2="-365.76" width="0.2" layer="20"/>
 <wire x1="-0.635" y1="-349.5675" x2="20.955" y2="-370.5225" width="0.4064" layer="25"/>
 <wire x1="184.8485" y1="-427.6725" x2="186.3725" y2="-429.1965" width="0.254" layer="20"/>
@@
 <wire x1="53.34" y1="-236.22" x2="53.34" y2="-364.49" width="0.2" layer="20"/>
 <wire x1="189.23" y1="-234.315" x2="189.23" y2="-340.6775" width="0.2" layer="20"/>
-<wire x1="350.04375" y1="-365.76" x2="192.405" y2="-365.76" width="0.2" layer="20"/>
+<wire x1="350.04375" y1="-365.76" x2="344.4875" y2="-365.76" width="0.2" layer="20"/>
 <text x="237.49" y="-363.5375" size="2.286" layer="16" font="vector" ratio="15" rot="MR0">1177-16</text>
 <circle x="227.33" y="-283.21" radius="2.5" width="0.254" layer="20"/>
@@
 <circle x="265.43" y="-263.68375" radius="2.5" width="0.254" layer="20"/>
 <circle x="284.7975" y="-264.63625" radius="2.5" width="0.254" layer="20"/>
+<wire x1="344.4875" y1="-365.76" x2="192.405" y2="-365.76" width="0.2" layer="20"/>
 <wire x1="350.04375" y1="-231.14" x2="192.405" y2="-231.14" width="0.2" layer="20"/>
 <wire x1="189.23" y1="-234.315" x2="192.405" y2="-231.14" width="0.2" layer="20" curve="-90"/>
@@
 <dimension x1="213.6775" y1="-201.6125" x2="221.615" y2="-180.6575" x3="219.86875" y3="-191.135" layer="21" dtype="vertical"/>
 <wire x1="353.21875" y1="-234.315" x2="353.21875" y2="-362.585" width="0.2" layer="20"/>
-<wire x1="185.42" y1="-365.76" x2="188.595" y2="-362.585" width="0.2" layer="20" curve="90"/>
-<wire x1="189.23" y1="-362.585" x2="192.405" y2="-365.76" width="0.2" layer="20" curve="90"/>
-<wire x1="188.595" y1="-362.585" x2="188.595" y2="-359.88625" width="0.2" layer="20"/>
-<wire x1="188.595" y1="-359.88625" x2="183.03875" y2="-359.88625" width="0.2" layer="20"/>
 <wire x1="183.03875" y1="-359.88625" x2="183.03875" y2="-340.0425" width="0.2" layer="20"/>
 <wire x1="183.03875" y1="-340.0425" x2="188.595" y2="-340.0425" width="0.2" layer="20"/>
 <wire x1="189.23" y1="-340.6775" x2="183.67375" y2="-340.6775" width="0.2" layer="20"/>
 <wire x1="183.67375" y1="-340.6775" x2="183.67375" y2="-359.25125" width="0.2" layer="20"/>
-<wire x1="183.67375" y1="-359.25125" x2="189.23" y2="-359.25125" width="0.2" layer="20"/>
-<wire x1="189.23" y1="-359.25125" x2="189.23" y2="-362.585" width="0.2" layer="20"/>
 <dimension x1="187.96" y1="-238.125" x2="189.70625" y2="-238.28375" x3="188.833125" y3="-218.91625" layer="20" dtype="horizontal"/>
 <dimension x1="169.06875" y1="-238.125" x2="170.33875" y2="-238.125" x3="169.70375" y3="-218.44" layer="20" dtype="horizontal"/>
@@
 <dimension x1="189.23" y1="-342.265" x2="208.28" y2="-369.2525" x3="198.755" y3="-379.4125" layer="21" dtype="horizontal"/>
 <dimension x1="188.595" y1="-354.965" x2="169.545" y2="-362.9025" x3="179.07" y3="-379.4125" layer="21" dtype="horizontal"/>
+<wire x1="183.03875" y1="-362.585" x2="183.03875" y2="-359.88625" width="0.2" layer="20"/>
+<wire x1="179.86375" y1="-365.76" x2="183.03875" y2="-362.585" width="0.2" layer="20" curve="90"/>
+<wire x1="183.67375" y1="-359.25125" x2="183.67375" y2="-362.585" width="0.2" layer="20"/>
+<wire x1="183.67375" y1="-362.585" x2="186.84875" y2="-365.76" width="0.2" layer="20" curve="90"/>
+<wire x1="344.4875" y1="-365.76" x2="186.84875" y2="-365.76" width="0.2" layer="20"/>
+<wire x1="179.86375" y1="-237.01375" x2="179.86375" y2="-355.75875" width="0.2" layer="108"/>
+<wire x1="179.86375" y1="-355.75875" x2="179.86375" y2="-365.28375" width="0.2" layer="108"/>
+<wire x1="179.86375" y1="-227.48875" x2="179.86375" y2="-355.75875" width="0.2" layer="108"/>
 </plain>
 <attributes>
@@
 <vertex x="392.43" y="-227.33"/>
 </polygon>
-<wire x1="50.8" y1="-292.4175" x2="50.8" y2="-260.985" width="0" layer="19" extent="1-1"/>
+<wire x1="73.9775" y1="-264.4775" x2="50.8" y2="-260.985" width="0" layer="19" extent="1-1"/>
 <wire x1="31.435" y1="-401.0025" x2="17.145" y2="-339.0875" width="0" layer="19" extent="1-16"/>
 <wire x1="83.5025" y1="-399.9625" x2="31.435" y2="-401.0025" width="0" layer="19" extent="1-1"/>
@@
 </signal>
 <signal name="N$71">
-<via x="185.42" y="-362.585" extent="1-16" drill="3" diameter="5"/>
+<via x="179.86375" y="-362.585" extent="1-16" drill="3" diameter="5"/>
 </signal>
 <signal name="N$89">
@@
 <via x="169.545" y="-234.315" extent="1-16" drill="3" diameter="5"/>
 </signal>
+<signal name="N$395">
+<via x="185.42" y="-234.315" extent="1-16" drill="3" diameter="5"/>
+</signal>
 <signal name="N$94">
-<via x="185.42" y="-234.315" extent="1-16" drill="3" diameter="5"/>
+<via x="179.86375" y="-234.315" extent="1-16" drill="3" diameter="5"/>
 </signal>
 <signal name="N$84">
@@
 <contactref element="R25" pad="2"/>
 <contactref element="SV6" pad="11"/>
-<wire x1="57.785" y1="-249.8725" x2="81.28" y2="-260.985" width="0" layer="19" extent="1-1"/>
 <wire x1="57.785" y1="-242.8875" x2="57.785" y2="-249.8725" width="0" layer="19" extent="1-1"/>
-<wire x1="19.685" y1="-317.18" x2="81.28" y2="-260.985" width="0" layer="19" extent="16-16"/>
+<wire x1="81.28" y1="-260.985" x2="57.785" y2="-249.8725" width="0" layer="19" extent="1-1"/>
+<wire x1="139.7" y1="-256.54" x2="81.28" y2="-260.985" width="0" layer="19" extent="1-1"/>
+<wire x1="152.4" y1="-258.851" x2="139.7" y2="-256.54" width="0" layer="19" extent="16-16"/>
+<wire x1="19.685" y1="-317.18" x2="57.785" y2="-249.8725" width="0" layer="19" extent="16-16"/>
 <wire x1="16.51" y1="-318.45" x2="19.685" y2="-317.18" width="0" layer="19" extent="16-16"/>
 <wire x1="4.765" y1="-323.215" x2="16.51" y2="-318.45" width="0" layer="19" extent="16-16"/>
@@
 <wire x1="4.1275" y1="-347.665" x2="3.495" y2="-335.915" width="0" layer="19" extent="16-16"/>
 <wire x1="33.335" y1="-401.0025" x2="4.1275" y2="-347.665" width="0" layer="19" extent="1-16"/>
-<wire x1="139.7" y1="-256.54" x2="81.28" y2="-260.985" width="0" layer="19" extent="1-1"/>
-<wire x1="152.4" y1="-258.851" x2="139.7" y2="-256.54" width="0" layer="19" extent="16-16"/>
 <wire x1="93.345" y1="-462.915" x2="33.335" y2="-401.0025" width="0" layer="19" extent="1-1"/>
 <wire x1="98.1075" y1="-476.25" x2="93.345" y2="-462.915" width="0" layer="19" extent="1-1"/>
 <wire x1="92.7075" y1="-481.6475" x2="98.1075" y2="-476.25" width="0" layer="19" extent="1-1"/>
 <wire x1="129.2225" y1="-467.6775" x2="98.1075" y2="-476.25" width="0" layer="19" extent="1-1"/>
-<wire x1="131.1275" y1="-467.6775" x2="129.2225" y2="-467.6775" width="0" layer="19" extent="1-1"/>
-<wire x1="133.0325" y1="-467.6775" x2="131.1275" y2="-467.6775" width="0" layer="19" extent="1-1"/>
-<wire x1="134.9375" y1="-467.6775" x2="133.0325" y2="-467.6775" width="0" layer="19" extent="1-1"/>
-<wire x1="136.2075" y1="-463.8675" x2="134.9375" y2="-467.6775" width="0" layer="19" extent="1-1"/>
 <wire x1="140.2613" y1="-463.5475" x2="136.2075" y2="-463.8675" width="0" layer="19" extent="1-1"/>
 <wire x1="143.7975" y1="-461.3425" x2="142.5575" y2="-462.9175" width="0" layer="19" extent="1-1"/>
 <wire x1="159.9565" y1="-471.4875" x2="158.4325" y2="-475.2975" width="0" layer="19" extent="1-1"/>
-<wire x1="134.9375" y1="-459.4225" x2="136.2075" y2="-463.8675" width="0" layer="19" extent="1-1"/>
-<wire x1="133.0325" y1="-459.4225" x2="133.7075" y2="-458.1925" width="0" layer="19" extent="1-1"/>
-<wire x1="131.1275" y1="-459.4225" x2="133.0325" y2="-459.4225" width="0" layer="19" extent="1-1"/>
-<wire x1="129.2225" y1="-459.4225" x2="131.1275" y2="-459.4225" width="0" layer="19" extent="1-1"/>
 <wire x1="170.4975" y1="-475.2975" x2="159.9565" y2="-471.4875" width="0" layer="19" extent="1-16"/>
 <wire x1="173.6725" y1="-455.2315" x2="175.5775" y2="-453.2425" width="0" layer="19" extent="1-1"/>
