File: PCB/Controller/Controller.sch (EAGLE design)
At the start: 41 parts, among them IC2 LMV358IDGKR, J1 USB MICRO, Y2 16MHz KX-7

Commit message: cont fe11s
Parts:
- removed Z3, Z4: CG0603MLC-05E, varistor:VARISTORCN0603
- added C5, C6: 100n, rcl:C-EUC0805
- added C7, C8: 10m, rcl:C-EUC0805
- added LED1, LED2: (no value), led:LEDSML0603
- added R10, R12, R9: 100k, rcl:R-EU_R0805
- added R11: 47k, rcl:R-EU_R0805
- added R4, R5: 10, rcl:R-EU_R0603
- added R6, R7, R8: 2k7, rcl:R-EU_R0805
- added RN3: 22R, resistor-dil:4R-NCAY16
- added RU1, RU2: CG0603MLC-05E, varistor:VARISTORCN0603
- added X1: USB-B_PN61729-S, detali_controller:USB-B_PN61729-S
- added ZQ1: 12MHz, crystal:CRYSTALHC49S
- Z1A: value (none) -> 16MHz
- renumbered Q1 to Z1A, Y2 to Z1
Connections:
- new net DMI: DD1.DMU, RN3B.1
- new net DPI: DD1.DPU, RN3A.1
- new net N$10: DD1.XRSTJ, R9.2
- new net N$11: DD1.LED1, LED1.A
- new net N$12: R5.1, X1.3
- new net N$13: R4.1, X1.2
- new net N$14: DD1.LED2, LED2.A
- new net N$15: DD1.BUSJ, R12.2
- new net N$16: DD1.VBUSM, R10.2, R11.1
- new net N$17: LED1.C, R7.1
- new net N$18: LED2.C, R8.1
- new net N$20: R7.2, R8.2
- new net N$21: DD1.REXT, R6.2
- new net N$5: R4.2, RN3B.2, RU2.1
- new net N$6: R5.2, RN3A.2, RU1.1
- new net N$7: F2.2, X1.1
- new net N$8: DD1.XOUT, ZQ1.2
- new net N$9: DD1.XIN, ZQ1.1
- new net VD1V8: C5.1, C7.1, DD1.VD18, DD1.VD18_O
- new net VD3V3: C6.1, C8.1, DD1.OVCJ, DD1.VD33, DD1.VD33_O, R12.1, R9.1
- net D+: no longer Z3.1
- net D-: no longer Z4.1
- net GND: now also C5.2, C6.2, C7.2, C8.2, DD1.VSS, R10.1, R6.1, RU1.2, RU2.2, X1.4, X1.S1, X1.S2; no longer Z3.2, Z4.2
- net VUSB: now also DD1.VDD5, R11.2
- net XUSB: no longer F2.2
Other:
- note added: "?"
- moved on the sheet: C3, C4, DD1, F2, L1, SV1, SV5, SV6

Commit message: .
Parts:
- removed F2: MF-MSMF050-2 500mA, rcl:L-EUL1812
- removed LED1, LED2: (no value), led:LEDSML0603
- removed RN3, RN4: 22R, resistor-dil:4R-NCAY16
- added 1D1: ATMEGA168-AU, atmega8:ATMEGA48/88/168-AU
- added 2C1, 2C2: 20, resistor:C-EUC0805
- added 2C3: 100n, resistor:C-EUC0805
- added 2C4: 10mf, rcl:C-EUC1210
- added 2C5: 1mf, rcl:C-EUC0805
- added 2D1: PL-2303XA, SparkFun-DigitalIC:PL-2303XA
- added 2R1, 2R8: 100, resistor:R-EU_R0603
- added 2R2, 2R6, 2R7: 220k, resistor:R-EU_R0603
- added 2R3, 2R5: 220k, resistor:R-EU_R1206W
- added 2R4: 1.5k, resistor:R-EU_R0603
- added 2Z1: 12MHz, crystal:CRYSTALHC49S
- added C15, C9: 22, rcl:C-EUC0603
- added C16, C21: (no value), rcl:C-TRIMMTZ03
- added C23, C25: (no value), keycopy:C-EUC0805
- added C26: 100n, SmartPrj:C-EUC0603
- added F1: MF-MSMF050-2 500mA, rcl:L-EUL1812
- added HL1, HL2, HL3, HL4: (no value), led:LEDSML0603
- added IC1: 24C02CP, microchip:24C02CP
- added IC3: 74HC244DW, 74xx-eu:74HC244DW
- added ICSP2: 3x2 M, SmartPrj:PINHD-2X3
- added ISP2: (no value), con-lstb:MA03-2
- added J2, JI2, JO2, JR2, JS2: (no value), jumper:SJ
- added Q2: 16M, keycopy:CRYSTALHC49S
- added R13: 100k, rcl:R-EU_R0805
- added R14, R15, R16: (no value), keycopy:R-EU_R0805
- added RJ1: (no value), rcl:R-EU_R0805
- added RJ4: 0, rcl:R-EU_R1206
- added RN: 22R, resistor-dil:4R-NCAY16
- C4: device SmartPrj:C-EUC0603 -> rcl:C-EUC0805
- C7, C8: device rcl:C-EUC0805 -> rcl:C-EUC1206
- J1: value USB MICRO -> (none); device SmartPrj:MYCON2_USB-MINI-B -> jumper:SJ
- R7, R8: value 2k7 -> 1k
Connections:
- removed net D+: J1.D+, RN4A.2
- removed net D-: J1.D-, RN4D.2
- removed net N$20: R7.2, R8.2
- removed net USBID: J1.ID
- removed net XUSB: J1.VBUS
- new net 3VUSB2: 2C3.1, 2D1.VO_33, 2R4.1, RJ4.2
- new net MISO: 1D1.PB4(MISO/PCINT4), ISP2.1
- new net MISO0: JI2.2
- new net MOSI: 1D1.PB3(MOSI/OC2A/PCINT3), ISP2.4
- new net MOSI0: JO2.2
- new net N$19: DD1.OVCJ, R13.2
- new net N$22: 1D1.PB7(XTAL2/TOSC2/PCINT7), C25.2, Q2.1
- new net N$23: DD1.TESTJ, RJ1.1
- new net N$24: 1D1.PB6(XTAL1/TOSC1/PCINT6), C23.2, Q2.2
- new net N$25: C21.A, DD1.DM3
- new net N$27: C21.E, DD1.DP3
- new net N$29: C16.E, DD1.DP4
- new net N$30: C16.A, DD1.DM4
- new net N$31: HL1.A, HL3.C, R7.1
- new net N$52: 2D1.DP, 2R8.2
- new net N$53: 2D1.DM, 2R1.2
- new net N$54: 2D1.GP1, 2R2.2
- new net N$55: 2D1.GP0, 2R3.2
- new net N$56: 2C1.2, 2D1.OSC2, 2Z1.2
- new net N$57: 2C2.2, 2D1.OSC1, 2Z1.1
- new net N$58: 2D1.RI_N, 2R5.1
- new net N$59: 2D1.DSR_N, 2R6.2
- new net N$60: 2D1.DCD_N, 2R7.2
- new net N$61: 2D1.CTS_N, JI2.1
- new net N$62: 2D1.RTS_N, JS2.1
- new net N$63: 2D1.DTR_N, JO2.1
- new net N$64: 2D1.VDD_325, RJ4.1
- new net N$66: 2D1.EE_DATA, IC1.SDA, R15.1
- new net N$67: IC1.VCC, R15.2, R16.2
- new net N$68: 2D1.EE_CLK, IC1.SCL, R16.1
- new net RESET0: JR2.2
- new net RX: J1.2
- new net RXM: 1D1.PD0(RXD/PCINT16)
- new net RX_USB: 2D1.RXD, J1.1
- new net SCK: ISP2.3
- new net SCK0: JS2.2
- new net TX: J2.2
- new net TXM: 1D1.PD1(TXD/PCINT17)
- new net TX_USB: 2D1.TXD, J2.1, JR2.1
- new net UU+: 2R4.2, 2R8.1, DD1.DP2
- new net UU-: 2R1.1, DD1.DM2
- net +5V: now also 1D1.AREF, 1D1.AVCC, 1D1.VCC@1, 1D1.VCC@2, 2C4.2, 2C5.2, 2D1.RESET_N, 2D1.VDD_33, 2D1.VDD_33A, 2D1.VDD_5, 2R3.1, 2R5.2, 2R6.1, 2R7.1, ISP2.2, R14.2
- net DMI: now also RNB.1; no longer RN3B.1
- net DPI: now also RNA.1; no longer RN3A.1
- net GND: now also 1D1.AGND, 1D1.GND@1, 1D1.GND@2, 2C1.1, 2C2.1, 2C3.2, 2C4.1, 2C5.1, 2D1.GND@18, 2D1.GND@21, 2D1.GND@7, 2D1.GND_A, 2D1.PLL_TEST, 2R2.1, C15.1, C23.1, C25.1, C26.1, C9.1, IC1.A0, IC1.A1, IC1.A2, IC1.GND, ISP2.6, RJ1.2; no longer J1.SH1, J1.SH2, J1.SH3, J1.SH4, J1.SH5, J1.SH6
- net N$11: now also DD1.DRV, R7.2, R8.2; no longer DD1.LED1, LED1.A
- net N$14: now also DD1.LED1, HL1.C, HL3.A; no longer DD1.LED2, LED2.A
- net N$17: now also DD1.LED2, HL2.C, HL4.A; no longer LED1.C, R7.1
- net N$18: now also HL2.A, HL4.C; no longer LED2.C
- net N$5: now also RNB.2; no longer RN3B.2
- net N$6: now also RNA.2; no longer RN3A.2
- net N$7: now also F1.2; no longer F2.2
- net N$8: now also C9.2, ZQ1.1; no longer ZQ1.2
- net N$9: now also C15.2, ZQ1.2; no longer ZQ1.1
- net RD+: now also DD1.DP1; no longer RN4A.1
- net RD-: now also DD1.DM1; no longer RN4D.1
- net RESET: now also 1D1.PC6(/RESET/PCINT14), ISP2.5, R14.1
- net UGND: no longer J1.GND
- net VD3V3: now also R13.1; no longer DD1.OVCJ
- net VUSB: now also C26.2, F1.1; no longer F2.1
Other:
- note added: "1R6 для J HW"
- note added: "J HW не нужен"
- note added: "R1, R2, R6-R10 not"
- note added: "USB-HUB"
- note added: "pin 4 to +5V"
- note added: "pin 6 to +5V"
- note removed: "USB"
- moved on the sheet: C1, C17, C18, C19, C2, C20, C24, C3, C4, C5, C6, C7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

Commit message: .
Parts:
- added J_U1, J_U2: (no value), jumper:SJ
- R11, R9: device rcl:R-EU_R0805 -> rcl:R-EU_R1206W
Connections:
- net N$12 renamed ID+
- net N$13 renamed ID-
- removed net N$5: R4.2, RNB.2, RU2.1
- removed net N$6: R5.2, RNA.2, RU1.1
- new net D+: J_U1.2, R5.2, RNA.2, RU1.1
- new net D-: J_U2.2, R4.2, RNB.2, RU2.1
- net RD+: now also J_U1.1
- net RD-: now also J_U2.1
Changed lines of the file:
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@@
 <part name="R7" library="rcl" deviceset="R-EU_" device="R0805" value="1k"/>
 <part name="R8" library="rcl" deviceset="R-EU_" device="R0805" value="1k"/>
-<part name="R9" library="rcl" deviceset="R-EU_" device="R0805" value="100k"/>
+<part name="R9" library="rcl" deviceset="R-EU_" device="R1206W" value="100k"/>
 <part name="R10" library="rcl" deviceset="R-EU_" device="R0805" value="100k"/>
-<part name="R11" library="rcl" deviceset="R-EU_" device="R0805" value="47k"/>
+<part name="R11" library="rcl" deviceset="R-EU_" device="R1206W" value="47k"/>
 <part name="R12" library="rcl" deviceset="R-EU_" device="R0805" value="100k"/>
 <part name="R13" library="rcl" deviceset="R-EU_" device="R0805" value="100k"/>
@@
 <part name="HL2" library="led" deviceset="LED" device="SML0603"/>
 <part name="HL4" library="led" deviceset="LED" device="SML0603"/>
+<part name="J_U2" library="jumper" deviceset="SJ" device=""/>
+<part name="J_U1" library="jumper" deviceset="SJ" device=""/>
 </parts>
 <sheets>
@@
 <attribute name="VALUE" x="489.712" y="328.295" size="1.778" layer="96" rot="R180"/>
 </instance>
+<instance part="J_U2" gate="1" x="497.84" y="350.52"/>
+<instance part="J_U1" gate="1" x="497.84" y="358.14"/>
 </instances>
 <busses>
@@
 <label x="472.44" y="304.8" size="1.778" layer="95"/>
 </segment>
+<segment>
+<pinref part="J_U2" gate="1" pin="1"/>
+<wire x1="492.76" y1="350.52" x2="487.68" y2="350.52" width="0.1524" layer="91"/>
+<label x="487.68" y="350.52" size="1.778" layer="95"/>
+</segment>
 </net>
 <net name="RD+" class="0">
@@
 <wire x1="469.9" y1="307.34" x2="477.52" y2="307.34" width="0.1524" layer="91"/>
 <label x="472.44" y="307.34" size="1.778" layer="95"/>
+</segment>
+<segment>
+<pinref part="J_U1" gate="1" pin="1"/>
+<wire x1="492.76" y1="358.14" x2="487.68" y2="358.14" width="0.1524" layer="91"/>
+<label x="487.68" y="358.14" size="1.778" layer="95"/>
 </segment>
 </net>
@@
 </segment>
 </net>
-<net name="N$5" class="0">
-<segment>
-<pinref part="RU2" gate="G$1" pin="1"/>
-<wire x1="424.18" y1="363.22" x2="424.18" y2="370.84" width="0.1524" layer="91"/>
-<pinref part="RN" gate="B" pin="2"/>
-<wire x1="424.18" y1="370.84" x2="429.26" y2="370.84" width="0.1524" layer="91"/>
-<pinref part="R4" gate="G$1" pin="2"/>
-<wire x1="424.18" y1="370.84" x2="416.56" y2="370.84" width="0.1524" layer="91"/>
-<junction x="424.18" y="370.84"/>
-</segment>
-</net>
-<net name="N$6" class="0">
-<segment>
-<pinref part="RU1" gate="G$1" pin="1"/>
-<wire x1="419.1" y1="363.22" x2="419.1" y2="365.76" width="0.1524" layer="91"/>
-<pinref part="RN" gate="A" pin="2"/>
-<wire x1="419.1" y1="365.76" x2="429.26" y2="365.76" width="0.1524" layer="91"/>
-<pinref part="R5" gate="G$1" pin="2"/>
-<wire x1="419.1" y1="365.76" x2="416.56" y2="365.76" width="0.1524" layer="91"/>
-<junction x="419.1" y="365.76"/>
-</segment>
-</net>
 <net name="N$7" class="0">
 <segment>
@@
 </segment>
 </net>
-<net name="N$12" class="0">
-<segment>
-<pinref part="X1" gate="G$1" pin="3"/>
-<pinref part="R5" gate="G$1" pin="1"/>
-<wire x1="398.78" y1="365.76" x2="406.4" y2="365.76" width="0.1524" layer="91"/>
-</segment>
-</net>
-<net name="N$13" class="0">
-<segment>
-<pinref part="R4" gate="G$1" pin="1"/>
-<wire x1="406.4" y1="370.84" x2="403.86" y2="370.84" width="0.1524" layer="91"/>
-<wire x1="403.86" y1="370.84" x2="403.86" y2="368.3" width="0.1524" layer="91"/>
-<pinref part="X1" gate="G$1" pin="2"/>
-<wire x1="403.86" y1="368.3" x2="398.78" y2="368.3" width="0.1524" layer="91"/>
+<net name="D+" class="0">
+<segment>
+<pinref part="J_U1" gate="1" pin="2"/>
+<wire x1="502.92" y1="358.14" x2="508" y2="358.14" width="0.1524" layer="91"/>
+<label x="502.92" y="358.14" size="1.778" layer="95"/>
+</segment>
+<segment>
+<pinref part="RU1" gate="G$1" pin="1"/>
+<wire x1="419.1" y1="363.22" x2="419.1" y2="365.76" width="0.1524" layer="91"/>
+<pinref part="RN" gate="A" pin="2"/>
+<wire x1="419.1" y1="365.76" x2="429.26" y2="365.76" width="0.1524" layer="91"/>
+<pinref part="R5" gate="G$1" pin="2"/>
+<wire x1="419.1" y1="365.76" x2="416.56" y2="365.76" width="0.1524" layer="91"/>
+<junction x="419.1" y="365.76"/>
+</segment>
+</net>
+<net name="D-" class="0">
+<segment>
+<pinref part="J_U2" gate="1" pin="2"/>
+<wire x1="502.92" y1="350.52" x2="508" y2="350.52" width="0.1524" layer="91"/>
+<label x="502.92" y="350.52" size="1.778" layer="95"/>
+</segment>
+<segment>
+<pinref part="RU2" gate="G$1" pin="1"/>
+<wire x1="424.18" y1="363.22" x2="424.18" y2="370.84" width="0.1524" layer="91"/>
+<pinref part="RN" gate="B" pin="2"/>
+<wire x1="424.18" y1="370.84" x2="429.26" y2="370.84" width="0.1524" layer="91"/>
+<pinref part="R4" gate="G$1" pin="2"/>
+<wire x1="424.18" y1="370.84" x2="416.56" y2="370.84" width="0.1524" layer="91"/>
+<junction x="424.18" y="370.84"/>
 </segment>
 </net>
@@
 </segment>
 </net>
+<net name="ID-" class="0">
+<segment>
+<pinref part="R4" gate="G$1" pin="1"/>
+<wire x1="406.4" y1="370.84" x2="403.86" y2="370.84" width="0.1524" layer="91"/>
+<wire x1="403.86" y1="370.84" x2="403.86" y2="368.3" width="0.1524" layer="91"/>
+<pinref part="X1" gate="G$1" pin="2"/>
+<wire x1="403.86" y1="368.3" x2="398.78" y2="368.3" width="0.1524" layer="91"/>
+</segment>
+</net>
+<net name="ID+" class="0">
+<segment>
+<pinref part="X1" gate="G$1" pin="3"/>
+<pinref part="R5" gate="G$1" pin="1"/>
+<wire x1="398.78" y1="365.76" x2="406.4" y2="365.76" width="0.1524" layer="91"/>
+</segment>
+</net>

Commit message: pcb b mov det
Parts:
- removed C21: (no value), rcl:C-TRIMMTZ03
- removed C26: 100n, SmartPrj:C-EUC0603
- removed DD1: FE1.1S, imcom:FE1.1S
- removed IC1: 24C02CP, microchip:24C02CP
- removed IC3: 74HC244DW, 74xx-eu:74HC244DW
- removed ICSP2: 3x2 M, SmartPrj:PINHD-2X3
- removed R1: 1M, SmartPrj:R-EU_R0603
- removed R15, R16: (no value), keycopy:R-EU_R0805
- added 1C10, 1C9: 100n, rcl:C-EUC0805
- added 1R11, 1R12: 10, rcl:R-EU_R0603
- added 1X2: USB_TYPE_A_FEMALE_TH, imcom:USB_TYPE_A_FEMALE_TH
- added 2D2: 24C02CP, microchip:24C02CP
- added 2D3: 74HC244DW, 74xx-eu:74HC244DW
- added 2R10, 2R9: (no value), keycopy:R-EU_R0805
- added 3D1: ATMEGA168-AU, atmega8:ATMEGA48/88/168-AU
- added R100: 1M, SmartPrj:R-EU_R0603
- added U_U1, U_U2: (no value), jumper:SJ
- 1D1: value ATMEGA168-AU -> FE1.1S; device atmega8:ATMEGA48/88/168-AU -> imcom:FE1.1S
- J_U2: value (none) -> J; device jumper:SJ -> detali_controller:J
- renumbered C15 to 1C2, C3 to 1C7, C4 to 1C8, C5 to 1C4, C6 to 1C5, C7 to 1C3, C8 to 1C6, C9 to 1C1, R10 to 1R7, R11 to 1R6, R12 to 1R4, R13 to 1R3, R4 to 1R1, R5 to 1R2, R6 to 1R8, R7 to 1R9, R8 to 1R10, R9 to 1R5, RJ1 to 1RJ, X1 to 1X1, ZQ1 to 1Z1
Connections:
- removed net N$27: C21.E, DD1.DP3
- removed net RXM: 1D1.PD0(RXD/PCINT16)
- removed net TXM: 1D1.PD1(TXD/PCINT17)
- new net N$12: 1R11.2, 1X2.3
- new net N$13: 1R12.2, 1X2.2
- new net N$20: DD3.D+, U_U2.2
- new net N$5: 1D1.DP2, 1R11.1
- new net N$6: 1D1.DM2, 1R12.1
- new net RXP: 3D1.PD0(RXD/PCINT16)
- new net TXP: 3D1.PD1(TXD/PCINT17)
- net +5V: now also 3D1.AREF, 3D1.AVCC, 3D1.VCC@1, 3D1.VCC@2; no longer 1D1.AREF, 1D1.AVCC, 1D1.VCC@1, 1D1.VCC@2
- net D+: now also RNB.2; no longer RNA.2
- net D-: now also J_U2.P$1, RNA.2; no longer J_U2.2, RNB.2
- net DMI: now also 1D1.DMU, RNA.1; no longer DD1.DMU, RNB.1
- net DPI: now also 1D1.DPU, RNB.1; no longer DD1.DPU, RNA.1
- net GND: now also 1C10.1, 1C9.1, 1D1.VSS, 1X2.4, 2D2.A0, 2D2.A1, 2D2.A2, 2D2.GND, 3D1.AGND, 3D1.GND@1, 3D1.GND@2; no longer 1D1.AGND, 1D1.GND@1, 1D1.GND@2, C26.1, DD1.VSS, IC1.A0, IC1.A1, IC1.A2, IC1.GND
- net MISO: no longer 1D1.PB4(MISO/PCINT4)
- net MISO0: now also 3D1.PB4(MISO/PCINT4)
- net MOSI: no longer 1D1.PB3(MOSI/OC2A/PCINT3)
- net MOSI0: now also 3D1.PB3(MOSI/OC2A/PCINT3)
- net N$10: now also 1D1.XRSTJ; no longer DD1.XRSTJ
- net N$11: now also 1D1.DRV; no longer DD1.DRV
- net N$14: now also 1D1.LED1; no longer DD1.LED1
- net N$15: now also 1D1.BUSJ; no longer DD1.BUSJ
- net N$16: now also 1D1.VBUSM; no longer DD1.VBUSM
- net N$17: now also 1D1.LED2; no longer DD1.LED2
- net N$19: now also 1D1.OVCJ; no longer DD1.OVCJ
- net N$21: now also 1D1.REXT; no longer DD1.REXT
- net N$22: now also 3D1.PB7(XTAL2/TOSC2/PCINT7); no longer 1D1.PB7(XTAL2/TOSC2/PCINT7)
- net N$23: now also 1D1.TESTJ; no longer DD1.TESTJ
- net N$24: now also 3D1.PB6(XTAL1/TOSC1/PCINT6); no longer 1D1.PB6(XTAL1/TOSC1/PCINT6)
- net N$25: now also DD3.D-, U_U1.2; no longer C21.A, DD1.DM3
- net N$29: now also 1D1.DP4; no longer DD1.DP4
- net N$30: now also 1D1.DM4; no longer DD1.DM4
- net N$66: now also 2D2.SDA, 2R9.1; no longer IC1.SDA, R15.1
- net N$67: now also 2D2.VCC, 2R10.2, 2R9.2; no longer IC1.VCC, R15.2, R16.2
- net N$68: now also 2D2.SCL, 2R10.1; no longer IC1.SCL, R16.1
- net N$8: now also 1D1.XOUT; no longer DD1.XOUT
- net N$9: now also 1D1.XIN; no longer DD1.XIN
- net RD+: now also 1D1.DP1, U_U2.1; no longer DD1.DP1, DD3.D+
- net RD-: now also 1D1.DM1, J_U2.P$2, U_U1.1; no longer DD1.DM1, DD3.D-, J_U2.1
- net RESET: no longer 1D1.PC6(/RESET/PCINT14), R14.1
- net RESET0: now also 3D1.PC6(/RESET/PCINT14), R14.1
- net SCK0: now also 3D1.PB5(SCK/PCINT5)
- net UU+: now also 1D1.DP3; no longer DD1.DP2
- net UU-: now also 1D1.DM3; no longer DD1.DM2
- net VD1V8: now also 1D1.VD18, 1D1.VD18_O; no longer DD1.VD18, DD1.VD18_O
- net VD3V3: now also 1D1.VD33, 1D1.VD33_O; no longer DD1.VD33, DD1.VD33_O
- net VUSB: now also 1C10.2, 1C9.2, 1D1.VDD5, 1X2.1; no longer C26.2, DD1.VDD5
- net XTAL1: now also R100.1; no longer R1.1
- net XTAL2: now also R100.2; no longer R1.2
Other:
- moved on the sheet: 2C1, 2C2, 2C3, 2C4, 2C5, 2D1, 2R1, 2R2, 2R3, 2R4, 2R5, 2R6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

Commit message: sm
Parts:
- added 1C11: 100n, rcl:C-EUC0805
Connections:
- new net N$26: 3D1.PB2(SS/OC1B/PCINT2)
- net +5V: now also 1C11.1
- net GND: now also 1C11.2
Other:
- note added: "-"
- note added: "17 февраля 2012"
- note added: "31.03.2009"
- note added: "?out reset"
- note added: "AvrUsb500v2"
- note added: "Bonio"
- note added: "FT232_MISO"
- note added: "FT232_MOSI"
- note added: "FT232_SCK"
- note added: "LED_TARGET"
- note added: "LED_active"
- note added: "LED_ready"
- note added: "RadioKot"
- note added: "cp2102 rx"
- note added: "cp2102 suspend"
- note added: "cp2102 tx"
- note added: "ft232 rx"
- note added: "ft232 tx"
- note added: "out 1Mhz"
- note added: "out mhz"
- note added: "out miso"
- note added: "out reset"
- note added: "out sck"
- note added: "out_MOSI"
- note added: "rst adc"
- note added: "s1 boot"
- note added: "vcc a out"
- note added: "vcc out"
- note added: "x"
Changed lines of the file:
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@@
 <part name="U_U1" library="jumper" deviceset="SJ" device=""/>
 <part name="U_U2" library="jumper" deviceset="SJ" device=""/>
+<part name="1C11" library="rcl" deviceset="C-EU" device="C0805" value="100n"/>
 </parts>
 <sheets>
@@
 <text x="469.9" y="254" size="1.27" layer="91" ratio="6">1R6 для J HW</text>
 <text x="421.64" y="386.08" size="5.08" layer="94">USB-HUB</text>
+<text x="800.1" y="261.62" size="1.778" layer="91">LED_TARGET</text>
+<text x="800.1" y="317.5" size="1.778" layer="91">RadioKot</text>
+<text x="800.1" y="259.08" size="1.778" layer="91">FT232_MOSI</text>
+<text x="800.1" y="256.54" size="1.778" layer="91">FT232_MISO</text>
+<text x="800.1" y="254" size="1.778" layer="91">FT232_SCK</text>
+<text x="800.1" y="312.42" size="1.778" layer="91">out 1Mhz</text>
+<text x="800.1" y="309.88" size="1.778" layer="91">out_MOSI</text>
+<text x="800.1" y="307.34" size="1.778" layer="91">rst adc</text>
+<text x="800.1" y="304.8" size="1.778" layer="91">out reset</text>
+<text x="800.1" y="302.26" size="1.778" layer="91">out sck</text>
+<text x="800.1" y="299.72" size="1.778" layer="91">out miso</text>
+<text x="800.1" y="297.18" size="1.778" layer="91">x</text>
+<text x="800.1" y="294.64" size="1.778" layer="91">x</text>
+<text x="800.1" y="281.94" size="1.778" layer="91">x</text>
+<text x="800.1" y="279.4" size="1.778" layer="91">x</text>
+<text x="800.1" y="276.86" size="1.778" layer="91">x</text>
+<text x="800.1" y="274.32" size="1.778" layer="91">x</text>
+<text x="800.1" y="271.78" size="1.778" layer="91">x</text>
+<text x="800.1" y="266.7" size="1.778" layer="91">x</text>
+<text x="800.1" y="264.16" size="1.778" layer="91">x</text>
+<text x="800.1" y="289.56" size="1.778" layer="91">ft232 tx</text>
+<text x="800.1" y="287.02" size="1.778" layer="91">ft232 rx</text>
+<text x="800.1" y="284.48" size="1.778" layer="91">x</text>
+<text x="820.42" y="284.48" size="1.778" layer="91">x</text>
+<text x="820.42" y="281.94" size="1.778" layer="91">x</text>
+<text x="820.42" y="274.32" size="1.778" layer="91">x</text>
+<text x="820.42" y="271.78" size="1.778" layer="91">x</text>
+<text x="820.42" y="297.18" size="1.778" layer="91">x</text>
+<text x="820.42" y="294.64" size="1.778" layer="91">x</text>
+<text x="820.42" y="317.5" size="1.778" layer="91">Bonio</text>
+<text x="820.42" y="266.7" size="1.778" layer="91">cp2102 suspend</text>
+<text x="820.42" y="289.56" size="1.778" layer="91">cp2102 tx</text>
+<text x="820.42" y="287.02" size="1.778" layer="91">cp2102 rx</text>
+<text x="820.42" y="299.72" size="1.778" layer="91">vcc out</text>
+<text x="820.42" y="307.34" size="1.778" layer="91">vcc a out</text>
+<text x="820.42" y="259.08" size="1.778" layer="91">out_MOSI</text>
+<text x="820.42" y="264.16" size="1.778" layer="91">out mhz</text>
+<text x="820.42" y="312.42" size="1.778" layer="91">out reset</text>
+<text x="820.42" y="254" size="1.778" layer="91">out sck</text>
+<text x="820.42" y="256.54" size="1.778" layer="91">out miso</text>
+<text x="820.42" y="276.86" size="1.778" layer="91">LED_ready</text>
+<text x="820.42" y="302.26" size="1.778" layer="91">LED_TARGET</text>
+<text x="820.42" y="261.62" size="1.778" layer="91">LED_active</text>
+<text x="820.42" y="279.4" size="1.778" layer="91">s1 boot</text>
+<text x="820.42" y="304.8" size="1.778" layer="91">x</text>
+<text x="820.42" y="322.58" size="1.778" layer="91">17 февраля 2012</text>
+<text x="800.1" y="322.58" size="1.778" layer="91">31.03.2009</text>
+<text x="843.28" y="317.5" size="1.778" layer="91">AvrUsb500v2</text>
+<text x="843.28" y="299.72" size="1.778" layer="91">x</text>
+<text x="843.28" y="302.26" size="1.778" layer="91">x</text>
+<text x="843.28" y="304.8" size="1.778" layer="91">x</text>
+<text x="843.28" y="309.88" size="1.778" layer="91">x</text>
+<text x="843.28" y="307.34" size="1.778" layer="91">x</text>
+<text x="843.28" y="312.42" size="1.778" layer="91">?out reset</text>
+<text x="843.28" y="254" size="1.778" layer="91">FT232_SCK</text>
+<text x="843.28" y="256.54" size="1.778" layer="91">FT232_MISO</text>
+<text x="843.28" y="259.08" size="1.778" layer="91">FT232_MOSI</text>
+<text x="843.28" y="261.62" size="1.778" layer="91">out mhz</text>
+<text x="843.28" y="264.16" size="1.778" layer="91">LED_TARGET</text>
+<text x="843.28" y="274.32" size="1.778" layer="91">x</text>
+<text x="843.28" y="271.78" size="1.778" layer="91">x</text>
+<text x="843.28" y="276.86" size="1.778" layer="91">x</text>
+<text x="843.28" y="279.4" size="1.778" layer="91">out_MOSI</text>
+<text x="843.28" y="281.94" size="1.778" layer="91">out miso</text>
+<text x="843.28" y="284.48" size="1.778" layer="91">out sck</text>
+<text x="843.28" y="287.02" size="1.778" layer="91">ft232 rx</text>
+<text x="843.28" y="289.56" size="1.778" layer="91">ft232 tx</text>
+<text x="843.28" y="297.18" size="1.778" layer="91">-</text>
+<text x="843.28" y="294.64" size="1.778" layer="91">-</text>
 </plain>
 <instances>
@@
 <attribute name="VALUE" x="793.75" y="5.08" size="1.778" layer="96" rot="R90"/>
 </instance>
+<instance part="1C11" gate="G$1" x="718.82" y="269.24" rot="MR0"/>
 </instances>
 <busses>
@@
 <pinref part="P+5" gate="1" pin="+5V"/>
 <wire x1="718.82" y1="281.94" x2="716.28" y2="281.94" width="0.1524" layer="91"/>
+<pinref part="1C11" gate="G$1" pin="1"/>
+<wire x1="718.82" y1="274.32" x2="718.82" y2="271.78" width="0.1524" layer="91"/>
+<junction x="718.82" y="274.32"/>
 </segment>
 <segment>
@@
 <wire x1="718.82" y1="254" x2="718.82" y2="251.46" width="0.1524" layer="91"/>
 <junction x="718.82" y="254"/>
+<pinref part="1C11" gate="G$1" pin="2"/>
+<wire x1="718.82" y1="264.16" x2="718.82" y2="261.62" width="0.1524" layer="91"/>
+<junction x="718.82" y="261.62"/>
 </segment>
 <segment>
@@
 </segment>
 </net>
+<net name="N$26" class="0">
+<segment>
+<pinref part="3D1" gate="1" pin="PB2(SS/OC1B/PCINT2)"/>
+<wire x1="782.32" y1="261.62" x2="789.94" y2="261.62" width="0.1524" layer="91"/>
+</segment>
+</net>
