File: PCB/Controller/Controller.sch (EAGLE design)
At the start: 106 parts, among them IC2 LMV358IDGKR, Q2 16M

Commit message: fw
Connections:
- new net MISO(D1): DD3.(PD0/MISO/PCINT3)PB3
- new net SCK(D3): DD3.(SCLK/PCINT1)PB1
- net CD1: no longer SV6.10
- net CD3: no longer SV6.8
- net MISO(D3): no longer DD3.(PD0/MISO/PCINT3)PB3
- net SCK(D1): no longer DD3.(SCLK/PCINT1)PB1
Changed lines of the file:
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@@
 <text x="447.04" y="35.56" size="1.778" layer="91">kbn2</text>
 <text x="447.04" y="40.64" size="1.778" layer="91">kbn3</text>
-<text x="894.08" y="60.96" size="1.778" layer="91">d3</text>
+<text x="894.08" y="55.88" size="1.778" layer="91">d3</text>
 <text x="894.08" y="58.42" size="1.778" layer="91">d2</text>
-<text x="894.08" y="55.88" size="1.778" layer="91">d1</text>
+<text x="894.08" y="60.96" size="1.778" layer="91">d1</text>
 <text x="876.3" y="20.32" size="1.778" layer="91">kbn2</text>
 <text x="876.3" y="17.78" size="1.778" layer="91">kbn3</text>
@@
 <text x="482.6" y="43.18" size="1.778" layer="91">kbb5</text>
 <text x="482.6" y="45.72" size="1.778" layer="91">kbb6</text>
-<text x="482.6" y="48.26" size="1.778" layer="91">d3</text>
+<text x="482.6" y="53.34" size="1.778" layer="91">d3</text>
 <text x="482.6" y="50.8" size="1.778" layer="91">d2</text>
-<text x="482.6" y="53.34" size="1.778" layer="91">d1</text>
+<text x="482.6" y="48.26" size="1.778" layer="91">d1</text>
 <text x="447.04" y="43.18" size="1.778" layer="91">d3</text>
 <text x="447.04" y="45.72" size="1.778" layer="91">d2</text>
@@
 <net name="CD3" class="0">
 <segment>
-<pinref part="SV6" gate="G$1" pin="8"/>
-<wire x1="472.44" y1="48.26" x2="462.28" y2="48.26" width="0.1524" layer="91"/>
-<label x="464.82" y="48.26" size="1.778" layer="95"/>
-</segment>
-<segment>
 <pinref part="SV5" gate="G$1" pin="6"/>
 <wire x1="436.88" y1="43.18" x2="424.18" y2="43.18" width="0.1524" layer="91"/>
@@
 </net>
 <net name="CD1" class="0">
-<segment>
-<pinref part="SV6" gate="G$1" pin="10"/>
-<wire x1="472.44" y1="53.34" x2="462.28" y2="53.34" width="0.1524" layer="91"/>
-<label x="464.82" y="53.34" size="1.778" layer="95"/>
-</segment>
 <segment>
 <pinref part="SV5" gate="G$1" pin="8"/>
@@
 <pinref part="ICSP1" gate="A" pin="3"/>
 </segment>
-<segment>
-<pinref part="DD3" gate="G$1" pin="(SCLK/PCINT1)PB1"/>
-<wire x1="873.76" y1="55.88" x2="883.92" y2="55.88" width="0.1524" layer="91"/>
-<label x="876.3" y="55.88" size="1.778" layer="95"/>
-</segment>
 </net>
 <net name="MISO(D3)" class="0">
@@
 <label x="825.5" y="86.36" size="1.778" layer="95"/>
 <pinref part="ICSP1" gate="A" pin="1"/>
-</segment>
-<segment>
-<pinref part="DD3" gate="G$1" pin="(PD0/MISO/PCINT3)PB3"/>
-<wire x1="873.76" y1="60.96" x2="883.92" y2="60.96" width="0.1524" layer="91"/>
-<label x="876.3" y="60.96" size="1.778" layer="95"/>
 </segment>
 </net>
@@
 </segment>
 </net>
+<net name="SCK(D3)" class="0">
+<segment>
+<pinref part="DD3" gate="G$1" pin="(SCLK/PCINT1)PB1"/>
+<wire x1="873.76" y1="55.88" x2="883.92" y2="55.88" width="0.1524" layer="91"/>
+<label x="876.3" y="55.88" size="1.778" layer="95"/>
+</segment>
+</net>
+<net name="MISO(D1)" class="0">
+<segment>
+<pinref part="DD3" gate="G$1" pin="(PD0/MISO/PCINT3)PB3"/>
+<wire x1="873.76" y1="60.96" x2="883.92" y2="60.96" width="0.1524" layer="91"/>
+<label x="876.3" y="60.96" size="1.778" layer="95"/>
+</segment>
+</net>

Commit message: b d1 d1 sw
Changed lines of the file:
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@@
 <text x="482.6" y="43.18" size="1.778" layer="91">kbb5</text>
 <text x="482.6" y="45.72" size="1.778" layer="91">kbb6</text>
-<text x="482.6" y="53.34" size="1.778" layer="91">d3</text>
+<text x="482.6" y="48.26" size="1.778" layer="91">d3</text>
 <text x="482.6" y="50.8" size="1.778" layer="91">d2</text>
-<text x="482.6" y="48.26" size="1.778" layer="91">d1</text>
+<text x="482.6" y="53.34" size="1.778" layer="91">d1</text>
 <text x="447.04" y="43.18" size="1.778" layer="91">d3</text>
 <text x="447.04" y="45.72" size="1.778" layer="91">d2</text>
