File: PCB/Controller/Controller.sch (EAGLE design)
At the start: 106 parts, among them IC2 LMV358IDGKR, Q2 16M

Commit message: sh c
Parts:
- added 1C12: 100n, rcl:C-EUC0805
Connections:
- new net N$27: 1C12.1, 3D1.AREF
- net +5V: no longer 3D1.AREF
- net GND: now also 1C12.2
Other:
- note added: "kbb19"
- note added: "led_caps"
- note added: "led_scroll"
- moved on the sheet: 1C11
Changed lines of the file:
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@@
 <part name="U_U2" library="jumper" deviceset="SJ" device=""/>
 <part name="1C11" library="rcl" deviceset="C-EU" device="C0805" value="100n"/>
+<part name="1C12" library="rcl" deviceset="C-EU" device="C0805" value="100n"/>
 </parts>
 <sheets>
@@
 <text x="447.04" y="35.56" size="1.778" layer="91">kbn2</text>
 <text x="447.04" y="40.64" size="1.778" layer="91">kbn3</text>
-<text x="894.08" y="55.88" size="1.778" layer="91">d3</text>
-<text x="894.08" y="58.42" size="1.778" layer="91">d2</text>
-<text x="894.08" y="60.96" size="1.778" layer="91">d1</text>
-<text x="876.3" y="20.32" size="1.778" layer="91">kbn2</text>
-<text x="876.3" y="17.78" size="1.778" layer="91">kbn3</text>
-<text x="876.3" y="15.24" size="1.778" layer="91">kbn1</text>
-<text x="889" y="71.12" size="1.778" layer="91">led_num</text>
+<text x="891.54" y="55.88" size="1.778" layer="91">d3</text>
+<text x="891.54" y="58.42" size="1.778" layer="91">d2</text>
+<text x="891.54" y="60.96" size="1.778" layer="91">d1</text>
+<text x="891.54" y="5.08" size="1.778" layer="91">kbn2</text>
+<text x="891.54" y="7.62" size="1.778" layer="91">kbn3</text>
+<text x="891.54" y="2.54" size="1.778" layer="91">kbn1</text>
+<text x="891.54" y="71.12" size="1.778" layer="91">led_num</text>
 <text x="482.6" y="33.02" size="1.778" layer="91">kbb1</text>
 <text x="482.6" y="35.56" size="1.778" layer="91">kbb2</text>
@@
 <text x="843.28" y="297.18" size="1.778" layer="91">-</text>
 <text x="843.28" y="294.64" size="1.778" layer="91">-</text>
+<text x="891.54" y="43.18" size="1.778" layer="91">kbb3</text>
+<text x="891.54" y="22.86" size="1.778" layer="91">kbb4</text>
+<text x="891.54" y="-7.62" size="1.778" layer="91">kbb1</text>
+<text x="891.54" y="30.48" size="1.778" layer="91">kbb2</text>
+<text x="891.54" y="-10.16" size="1.778" layer="91">kbb5</text>
+<text x="891.54" y="15.24" size="1.778" layer="91">kbb19</text>
+<text x="891.54" y="38.1" size="1.778" layer="91">x</text>
+<text x="891.54" y="53.34" size="1.778" layer="91">x</text>
+<text x="891.54" y="66.04" size="1.778" layer="91">led_caps</text>
+<text x="891.54" y="68.58" size="1.778" layer="91">led_scroll</text>
 </plain>
 <instances>
@@
 <attribute name="VALUE" x="793.75" y="5.08" size="1.778" layer="96" rot="R90"/>
 </instance>
-<instance part="1C11" gate="G$1" x="718.82" y="269.24" rot="MR0"/>
+<instance part="1C11" gate="G$1" x="708.66" y="269.24" rot="MR0"/>
+<instance part="1C12" gate="G$1" x="718.82" y="269.24" rot="MR0"/>
 </instances>
 <busses>
@@
 </segment>
 <segment>
-<pinref part="3D1" gate="1" pin="AREF"/>
-<wire x1="721.36" y1="274.32" x2="718.82" y2="274.32" width="0.1524" layer="91"/>
-<wire x1="718.82" y1="274.32" x2="718.82" y2="276.86" width="0.1524" layer="91"/>
-<pinref part="3D1" gate="1" pin="AVCC"/>
-<wire x1="718.82" y1="276.86" x2="721.36" y2="276.86" width="0.1524" layer="91"/>
-<wire x1="718.82" y1="276.86" x2="718.82" y2="281.94" width="0.1524" layer="91"/>
-<pinref part="3D1" gate="1" pin="VCC@2"/>
-<wire x1="718.82" y1="281.94" x2="721.36" y2="281.94" width="0.1524" layer="91"/>
-<wire x1="718.82" y1="281.94" x2="718.82" y2="284.48" width="0.1524" layer="91"/>
-<pinref part="3D1" gate="1" pin="VCC@1"/>
-<wire x1="718.82" y1="284.48" x2="721.36" y2="284.48" width="0.1524" layer="91"/>
-<junction x="718.82" y="281.94"/>
-<junction x="718.82" y="276.86"/>
-<pinref part="P+5" gate="1" pin="+5V"/>
-<wire x1="718.82" y1="281.94" x2="716.28" y2="281.94" width="0.1524" layer="91"/>
-<pinref part="1C11" gate="G$1" pin="1"/>
-<wire x1="718.82" y1="274.32" x2="718.82" y2="271.78" width="0.1524" layer="91"/>
-<junction x="718.82" y="274.32"/>
-</segment>
-<segment>
 <pinref part="R14" gate="G$1" pin="2"/>
 <pinref part="P+2" gate="1" pin="+5V"/>
@@
 <pinref part="P+9" gate="1" pin="+5V"/>
 <wire x1="787.4" y1="231.14" x2="787.4" y2="233.68" width="0.1524" layer="91"/>
+</segment>
+<segment>
+<pinref part="3D1" gate="1" pin="VCC@1"/>
+<wire x1="718.82" y1="284.48" x2="721.36" y2="284.48" width="0.1524" layer="91"/>
+<pinref part="3D1" gate="1" pin="VCC@2"/>
+<wire x1="718.82" y1="281.94" x2="721.36" y2="281.94" width="0.1524" layer="91"/>
+<wire x1="718.82" y1="281.94" x2="718.82" y2="284.48" width="0.1524" layer="91"/>
+<junction x="718.82" y="281.94"/>
+<pinref part="1C11" gate="G$1" pin="1"/>
+<wire x1="708.66" y1="279.4" x2="708.66" y2="271.78" width="0.1524" layer="91"/>
+<wire x1="708.66" y1="279.4" x2="718.82" y2="279.4" width="0.1524" layer="91"/>
+<wire x1="718.82" y1="279.4" x2="718.82" y2="281.94" width="0.1524" layer="91"/>
+<pinref part="P+5" gate="1" pin="+5V"/>
+<wire x1="716.28" y1="281.94" x2="718.82" y2="281.94" width="0.1524" layer="91"/>
+<pinref part="3D1" gate="1" pin="AVCC"/>
+<wire x1="721.36" y1="276.86" x2="718.82" y2="276.86" width="0.1524" layer="91"/>
+<wire x1="718.82" y1="276.86" x2="718.82" y2="279.4" width="0.1524" layer="91"/>
+<junction x="718.82" y="279.4"/>
 </segment>
 </net>
@@
 <junction x="718.82" y="254"/>
 <pinref part="1C11" gate="G$1" pin="2"/>
+<junction x="718.82" y="261.62"/>
+<wire x1="718.82" y1="261.62" x2="708.66" y2="261.62" width="0.1524" layer="91"/>
+<wire x1="708.66" y1="261.62" x2="708.66" y2="264.16" width="0.1524" layer="91"/>
+<pinref part="1C12" gate="G$1" pin="2"/>
 <wire x1="718.82" y1="264.16" x2="718.82" y2="261.62" width="0.1524" layer="91"/>
-<junction x="718.82" y="261.62"/>
 </segment>
 <segment>
@@
 </segment>
 </net>
+<net name="N$27" class="0">
+<segment>
+<pinref part="3D1" gate="1" pin="AREF"/>
+<wire x1="721.36" y1="274.32" x2="718.82" y2="274.32" width="0.1524" layer="91"/>
+<pinref part="1C12" gate="G$1" pin="1"/>
+<wire x1="718.82" y1="274.32" x2="718.82" y2="271.78" width="0.1524" layer="91"/>
+</segment>
+</net>

Commit message: sh c
Other:
- note added: "10"
- note added: "11"
- note added: "14"
- note added: "15"
- note added: "16"
- note added: "17"
- note added: "3"
- note added: "5"
- note added: "6"
- note added: "9"
Changed lines of the file:
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@@
 <text x="891.54" y="66.04" size="1.778" layer="91">led_caps</text>
 <text x="891.54" y="68.58" size="1.778" layer="91">led_scroll</text>
+<text x="909.32" y="12.7" size="1.778" layer="91">1</text>
+<text x="909.32" y="15.24" size="1.778" layer="91">2</text>
+<text x="909.32" y="17.78" size="1.778" layer="91">3</text>
+<text x="909.32" y="20.32" size="1.778" layer="91">4</text>
+<text x="909.32" y="25.4" size="1.778" layer="91">5</text>
+<text x="909.32" y="22.86" size="1.778" layer="91">6</text>
+<text x="904.24" y="20.32" size="1.778" layer="91"></text>
+<text x="909.32" y="27.94" size="1.778" layer="91">7</text>
+<text x="909.32" y="30.48" size="1.778" layer="91">8</text>
+<text x="909.32" y="63.5" size="1.778" layer="91">9</text>
+<text x="909.32" y="43.18" size="1.778" layer="91">10</text>
+<text x="909.32" y="45.72" size="1.778" layer="91">11</text>
+<text x="909.32" y="7.62" size="1.778" layer="91">12</text>
+<text x="909.32" y="5.08" size="1.778" layer="91">13</text>
+<text x="909.32" y="2.54" size="1.778" layer="91">14</text>
+<text x="909.32" y="0" size="1.778" layer="91">15</text>
+<text x="909.32" y="-7.62" size="1.778" layer="91">16</text>
+<text x="909.32" y="-10.16" size="1.778" layer="91">17</text>
 </plain>
 <instances>

Commit message: fw add
Parts:
- added U_U3, U_U4: (no value), jumper:SJ
- C23, C25: value (none) -> 22
Connections:
- net D+: now also U_U3.1
- net D-: now also U_U4.1
- net N$20: now also U_U3.2
- net N$25: now also U_U4.2
Other:
- note added: "USB-TTL"
- moved on the sheet: 1C11, 1C12, 3D1, C1, C17, C18, C19, C2, C20, C23, C24, C25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

Commit message: pcb c
Parts:
- added F2: MF-MSMF050-2 500mA, rcl:L-EUL1812
Connections:
- new net VUSBH: 1C10.1, 1X2.1, F2.1, F2.2
- net GND: now also 1C10.2; no longer 1C10.1
- net VUSB: no longer 1C10.2, 1X2.1
Other:
- moved on the sheet: 1C10, C16
Changed lines of the file:
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@@
 <part name="U_U3" library="jumper" deviceset="SJ" device=""/>
 <part name="U_U4" library="jumper" deviceset="SJ" device=""/>
+<part name="F2" library="rcl" deviceset="L-EU" device="L1812" value="MF-MSMF050-2 500mA"/>
+<part name="GND29" library="supply1" deviceset="GND" device=""/>
 </parts>
 <sheets>
@@
 <instance part="2D3" gate="A" x="548.64" y="246.38"/>
 <instance part="2D3" gate="B" x="543.56" y="215.9"/>
-<instance part="C16" gate="G$1" x="490.22" y="284.48"/>
+<instance part="C16" gate="G$1" x="482.6" y="266.7"/>
 <instance part="1C9" gate="G$1" x="482.6" y="365.76" smashed="yes" rot="MR180">
 <attribute name="NAME" x="484.124" y="370.459" size="1.778" layer="95" rot="MR180"/>
@@
 <instance part="1X2" gate="G$1" x="500.38" y="299.72" smashed="yes" rot="MR180">
 <attribute name="NAME" x="499.11" y="308.61" size="1.778" layer="95" rot="MR180"/>
-<attribute name="VALUE" x="505.46" y="285.75" size="1.778" layer="96" rot="MR90"/>
+<attribute name="VALUE" x="505.46" y="290.83" size="1.778" layer="96" rot="MR90"/>
 </instance>
 <instance part="GND28" gate="1" x="492.76" y="307.34" rot="MR180"/>
@@
 <attribute name="VALUE" x="546.1" y="298.45" size="1.778" layer="96"/>
 </instance>
-<instance part="1C10" gate="G$1" x="492.76" y="365.76" smashed="yes" rot="MR180">
-<attribute name="NAME" x="494.284" y="370.459" size="1.778" layer="95" rot="MR180"/>
-<attribute name="VALUE" x="494.284" y="365.379" size="1.778" layer="96" rot="MR180"/>
-</instance>
+<instance part="1C10" gate="G$1" x="502.92" y="284.48" rot="MR0"/>
 <instance part="1R11" gate="G$1" x="477.52" y="299.72" smashed="yes">
 <attribute name="NAME" x="478.79" y="306.2986" size="1.778" layer="95"/>
@@
 <attribute name="VALUE" x="694.69" y="63.5" size="1.778" layer="96" rot="R90"/>
 </instance>
+<instance part="F2" gate="G$1" x="515.62" y="304.8" smashed="yes">
+<attribute name="NAME" x="510.7686" y="293.37" size="1.778" layer="95" rot="R270"/>
+<attribute name="VALUE" x="512.572" y="295.91" size="1.778" layer="96" rot="R90"/>
+</instance>
+<instance part="GND29" gate="1" x="502.92" y="274.32" rot="MR0"/>
 </instances>
 <busses>
@@
 <wire x1="482.6" y1="363.22" x2="482.6" y2="358.14" width="0.1524" layer="91"/>
 <wire x1="482.6" y1="358.14" x2="472.44" y2="358.14" width="0.1524" layer="91"/>
-<pinref part="1C10" gate="G$1" pin="1"/>
-<wire x1="492.76" y1="363.22" x2="492.76" y2="358.14" width="0.1524" layer="91"/>
-<wire x1="492.76" y1="358.14" x2="482.6" y2="358.14" width="0.1524" layer="91"/>
-<junction x="482.6" y="358.14"/>
 </segment>
 <segment>
@@
 <wire x1="492.76" y1="302.26" x2="492.76" y2="304.8" width="0.1524" layer="91"/>
 </segment>
+<segment>
+<pinref part="1C10" gate="G$1" pin="2"/>
+<pinref part="GND29" gate="1" pin="GND"/>
+<wire x1="502.92" y1="279.4" x2="502.92" y2="276.86" width="0.1524" layer="91"/>
+</segment>
 </net>
 <net name="CD3" class="0">
@@
 <pinref part="1C9" gate="G$1" pin="2"/>
 <wire x1="482.6" y1="373.38" x2="482.6" y2="370.84" width="0.1524" layer="91"/>
-<wire x1="482.6" y1="373.38" x2="492.76" y2="373.38" width="0.1524" layer="91"/>
-<pinref part="1C10" gate="G$1" pin="2"/>
-<wire x1="492.76" y1="373.38" x2="492.76" y2="370.84" width="0.1524" layer="91"/>
-<junction x="482.6" y="373.38"/>
 </segment>
 <segment>
@@
 <wire x1="388.62" y1="309.88" x2="388.62" y2="314.96" width="0.1524" layer="91"/>
 <label x="386.08" y="317.5" size="1.778" layer="95"/>
-</segment>
-<segment>
-<pinref part="1X2" gate="G$1" pin="1"/>
-<wire x1="495.3" y1="294.64" x2="487.68" y2="294.64" width="0.1524" layer="91"/>
-<label x="487.68" y="292.1" size="1.778" layer="95"/>
 </segment>
 </net>
@@
 <segment>
 <pinref part="1D1" gate="G$1" pin="DP4"/>
-<wire x1="469.9" y1="284.48" x2="477.52" y2="284.48" width="0.1524" layer="91"/>
 <label x="472.44" y="284.48" size="1.778" layer="95"/>
 <pinref part="C16" gate="G$1" pin="E"/>
-<wire x1="477.52" y1="284.48" x2="490.22" y2="287.02" width="0.1524" layer="91"/>
+<wire x1="469.9" y1="284.48" x2="482.6" y2="269.24" width="0.1524" layer="91"/>
 </segment>
 </net>
@@
 <label x="472.44" y="281.94" size="1.778" layer="95"/>
 <pinref part="C16" gate="G$1" pin="A"/>
-<wire x1="490.22" y1="279.4" x2="477.52" y2="281.94" width="0.1524" layer="91"/>
+<wire x1="482.6" y1="261.62" x2="477.52" y2="281.94" width="0.1524" layer="91"/>
 </segment>
 </net>
@@
 </segment>
 </net>
+<net name="VUSBH" class="0">
+<segment>
+<pinref part="1X2" gate="G$1" pin="1"/>
+<wire x1="495.3" y1="294.64" x2="487.68" y2="294.64" width="0.1524" layer="91"/>
+<wire x1="487.68" y1="294.64" x2="487.68" y2="289.56" width="0.1524" layer="91"/>
+<wire x1="487.68" y1="289.56" x2="502.92" y2="289.56" width="0.1524" layer="91"/>
+<pinref part="F2" gate="G$1" pin="2"/>
+<wire x1="502.92" y1="289.56" x2="515.62" y2="289.56" width="0.1524" layer="91"/>
+<wire x1="515.62" y1="289.56" x2="515.62" y2="297.18" width="0.1524" layer="91"/>
+<pinref part="1C10" gate="G$1" pin="1"/>
+<wire x1="515.62" y1="297.18" x2="515.62" y2="299.72" width="0.1524" layer="91"/>
+<wire x1="502.92" y1="289.56" x2="502.92" y2="287.02" width="0.1524" layer="91"/>
+<junction x="502.92" y="289.56"/>
+<wire x1="515.62" y1="297.18" x2="520.7" y2="297.18" width="0.1524" layer="91"/>
+<wire x1="520.7" y1="297.18" x2="520.7" y2="312.42" width="0.1524" layer="91"/>
+<pinref part="F2" gate="G$1" pin="1"/>
+<wire x1="515.62" y1="309.88" x2="515.62" y2="312.42" width="0.1524" layer="91"/>
+<wire x1="515.62" y1="312.42" x2="515.62" y2="317.5" width="0.1524" layer="91"/>
+<wire x1="520.7" y1="312.42" x2="515.62" y2="312.42" width="0.1524" layer="91"/>
+<junction x="515.62" y="312.42"/>
+<junction x="515.62" y="297.18"/>
+</segment>
+</net>

Commit message: .
Changed lines of the file:
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@@
 <text x="469.9" y="254" size="1.27" layer="91" ratio="6">1R6 для J HW</text>
 <text x="421.64" y="386.08" size="5.08" layer="94">USB-HUB</text>
-<text x="741.68" y="320.04" size="1.778" layer="91">LED_TARGET</text>
-<text x="741.68" y="375.92" size="1.778" layer="91">RadioKot</text>
-<text x="741.68" y="317.5" size="1.778" layer="91">FT232_MOSI</text>
-<text x="741.68" y="314.96" size="1.778" layer="91">FT232_MISO</text>
-<text x="741.68" y="312.42" size="1.778" layer="91">FT232_SCK</text>
-<text x="741.68" y="370.84" size="1.778" layer="91">out 1Mhz</text>
-<text x="741.68" y="368.3" size="1.778" layer="91">out_MOSI</text>
-<text x="741.68" y="365.76" size="1.778" layer="91">rst adc</text>
-<text x="741.68" y="363.22" size="1.778" layer="91">out reset</text>
-<text x="741.68" y="360.68" size="1.778" layer="91">out sck</text>
-<text x="741.68" y="358.14" size="1.778" layer="91">out miso</text>
-<text x="741.68" y="355.6" size="1.778" layer="91">x</text>
-<text x="741.68" y="353.06" size="1.778" layer="91">x</text>
-<text x="741.68" y="340.36" size="1.778" layer="91">x</text>
-<text x="741.68" y="337.82" size="1.778" layer="91">x</text>
-<text x="741.68" y="335.28" size="1.778" layer="91">x</text>
-<text x="741.68" y="332.74" size="1.778" layer="91">x</text>
-<text x="741.68" y="330.2" size="1.778" layer="91">x</text>
-<text x="741.68" y="325.12" size="1.778" layer="91">x</text>
-<text x="741.68" y="322.58" size="1.778" layer="91">x</text>
-<text x="741.68" y="347.98" size="1.778" layer="91">ft232 tx</text>
-<text x="741.68" y="345.44" size="1.778" layer="91">ft232 rx</text>
-<text x="741.68" y="342.9" size="1.778" layer="91">x</text>
-<text x="759.46" y="342.9" size="1.778" layer="91">x</text>
-<text x="759.46" y="340.36" size="1.778" layer="91">x</text>
-<text x="759.46" y="332.74" size="1.778" layer="91">x</text>
-<text x="759.46" y="330.2" size="1.778" layer="91">x</text>
-<text x="759.46" y="355.6" size="1.778" layer="91">x</text>
-<text x="759.46" y="353.06" size="1.778" layer="91">x</text>
-<text x="759.46" y="375.92" size="1.778" layer="91">Bonio</text>
-<text x="759.46" y="325.12" size="1.778" layer="91">cp2102 suspend</text>
-<text x="759.46" y="347.98" size="1.778" layer="91">cp2102 tx</text>
-<text x="759.46" y="345.44" size="1.778" layer="91">cp2102 rx</text>
-<text x="759.46" y="358.14" size="1.778" layer="91">vcc out</text>
-<text x="759.46" y="365.76" size="1.778" layer="91">vcc a out</text>
-<text x="759.46" y="317.5" size="1.778" layer="91">out_MOSI</text>
-<text x="759.46" y="322.58" size="1.778" layer="91">out mhz</text>
-<text x="759.46" y="370.84" size="1.778" layer="91">out reset</text>
-<text x="759.46" y="312.42" size="1.778" layer="91">out sck</text>
-<text x="759.46" y="314.96" size="1.778" layer="91">out miso</text>
-<text x="759.46" y="335.28" size="1.778" layer="91">LED_ready</text>
-<text x="759.46" y="360.68" size="1.778" layer="91">LED_TARGET</text>
-<text x="759.46" y="320.04" size="1.778" layer="91">LED_active</text>
-<text x="759.46" y="337.82" size="1.778" layer="91">s1 boot</text>
-<text x="759.46" y="363.22" size="1.778" layer="91">x</text>
-<text x="759.46" y="381" size="1.778" layer="91">17 февраля 2012</text>
-<text x="741.68" y="381" size="1.778" layer="91">31.03.2009</text>
-<text x="723.9" y="375.92" size="1.778" layer="91">AvrUsb500v2</text>
-<text x="723.9" y="358.14" size="1.778" layer="91">x</text>
-<text x="723.9" y="360.68" size="1.778" layer="91">x</text>
-<text x="723.9" y="363.22" size="1.778" layer="91">x</text>
-<text x="723.9" y="368.3" size="1.778" layer="91">x</text>
-<text x="723.9" y="365.76" size="1.778" layer="91">x</text>
-<text x="723.9" y="370.84" size="1.778" layer="91">?out reset</text>
-<text x="723.9" y="312.42" size="1.778" layer="91">FT232_SCK</text>
-<text x="723.9" y="314.96" size="1.778" layer="91">FT232_MISO</text>
-<text x="723.9" y="317.5" size="1.778" layer="91">FT232_MOSI</text>
-<text x="723.9" y="320.04" size="1.778" layer="91">out mhz</text>
-<text x="723.9" y="322.58" size="1.778" layer="91">LED_TARGET</text>
-<text x="723.9" y="332.74" size="1.778" layer="91">x</text>
-<text x="723.9" y="330.2" size="1.778" layer="91">x</text>
-<text x="723.9" y="335.28" size="1.778" layer="91">x</text>
-<text x="723.9" y="337.82" size="1.778" layer="91">out_MOSI</text>
-<text x="723.9" y="340.36" size="1.778" layer="91">out miso</text>
-<text x="723.9" y="342.9" size="1.778" layer="91">out sck</text>
-<text x="723.9" y="345.44" size="1.778" layer="91">ft232 rx</text>
-<text x="723.9" y="347.98" size="1.778" layer="91">ft232 tx</text>
-<text x="723.9" y="355.6" size="1.778" layer="91">-</text>
-<text x="723.9" y="353.06" size="1.778" layer="91">-</text>
+<text x="787.4" y="320.04" size="1.778" layer="91">LED_TARGET</text>
+<text x="787.4" y="375.92" size="1.778" layer="91">RadioKot</text>
+<text x="787.4" y="317.5" size="1.778" layer="91">FT232_MOSI</text>
+<text x="787.4" y="314.96" size="1.778" layer="91">FT232_MISO</text>
+<text x="787.4" y="312.42" size="1.778" layer="91">FT232_SCK</text>
+<text x="787.4" y="370.84" size="1.778" layer="91">out 1Mhz</text>
+<text x="787.4" y="368.3" size="1.778" layer="91">out_MOSI</text>
+<text x="787.4" y="365.76" size="1.778" layer="91">rst adc</text>
+<text x="787.4" y="363.22" size="1.778" layer="91">out reset</text>
+<text x="787.4" y="360.68" size="1.778" layer="91">out sck</text>
+<text x="787.4" y="358.14" size="1.778" layer="91">out miso</text>
+<text x="787.4" y="355.6" size="1.778" layer="91">x</text>
+<text x="787.4" y="353.06" size="1.778" layer="91">x</text>
+<text x="787.4" y="340.36" size="1.778" layer="91">x</text>
+<text x="787.4" y="337.82" size="1.778" layer="91">x</text>
+<text x="787.4" y="335.28" size="1.778" layer="91">x</text>
+<text x="787.4" y="332.74" size="1.778" layer="91">x</text>
+<text x="787.4" y="330.2" size="1.778" layer="91">x</text>
+<text x="787.4" y="325.12" size="1.778" layer="91">x</text>
+<text x="787.4" y="322.58" size="1.778" layer="91">x</text>
+<text x="787.4" y="347.98" size="1.778" layer="91">ft232 tx</text>
+<text x="787.4" y="345.44" size="1.778" layer="91">ft232 rx</text>
+<text x="787.4" y="342.9" size="1.778" layer="91">x</text>
+<text x="805.18" y="342.9" size="1.778" layer="91">x</text>
+<text x="805.18" y="340.36" size="1.778" layer="91">x</text>
+<text x="805.18" y="332.74" size="1.778" layer="91">x</text>
+<text x="805.18" y="330.2" size="1.778" layer="91">x</text>
+<text x="805.18" y="355.6" size="1.778" layer="91">x</text>
+<text x="805.18" y="353.06" size="1.778" layer="91">x</text>
+<text x="805.18" y="375.92" size="1.778" layer="91">Bonio</text>
+<text x="805.18" y="325.12" size="1.778" layer="91">cp2102 suspend</text>
+<text x="805.18" y="347.98" size="1.778" layer="91">cp2102 tx</text>
+<text x="805.18" y="345.44" size="1.778" layer="91">cp2102 rx</text>
+<text x="805.18" y="358.14" size="1.778" layer="91">vcc out</text>
+<text x="805.18" y="365.76" size="1.778" layer="91">vcc a out</text>
+<text x="805.18" y="317.5" size="1.778" layer="91">out_MOSI</text>
+<text x="805.18" y="322.58" size="1.778" layer="91">out mhz</text>
+<text x="805.18" y="370.84" size="1.778" layer="91">out reset</text>
+<text x="805.18" y="312.42" size="1.778" layer="91">out sck</text>
+<text x="805.18" y="314.96" size="1.778" layer="91">out miso</text>
+<text x="805.18" y="335.28" size="1.778" layer="91">LED_ready</text>
+<text x="805.18" y="360.68" size="1.778" layer="91">LED_TARGET</text>
+<text x="805.18" y="320.04" size="1.778" layer="91">LED_active</text>
+<text x="805.18" y="337.82" size="1.778" layer="91">s1 boot</text>
+<text x="805.18" y="363.22" size="1.778" layer="91">x</text>
+<text x="805.18" y="381" size="1.778" layer="91">17 февраля 2012</text>
+<text x="787.4" y="381" size="1.778" layer="91">31.03.2009</text>
+<text x="769.62" y="375.92" size="1.778" layer="91">AvrUsb500v2</text>
+<text x="769.62" y="358.14" size="1.778" layer="91">x</text>
+<text x="769.62" y="360.68" size="1.778" layer="91">x</text>
+<text x="769.62" y="363.22" size="1.778" layer="91">x</text>
+<text x="769.62" y="368.3" size="1.778" layer="91">x</text>
+<text x="769.62" y="365.76" size="1.778" layer="91">x</text>
+<text x="769.62" y="370.84" size="1.778" layer="91">?out reset</text>
+<text x="769.62" y="312.42" size="1.778" layer="91">FT232_SCK</text>
+<text x="769.62" y="314.96" size="1.778" layer="91">FT232_MISO</text>
+<text x="769.62" y="317.5" size="1.778" layer="91">FT232_MOSI</text>
+<text x="769.62" y="320.04" size="1.778" layer="91">out mhz</text>
+<text x="769.62" y="322.58" size="1.778" layer="91">LED_TARGET</text>
+<text x="769.62" y="332.74" size="1.778" layer="91">x</text>
+<text x="769.62" y="330.2" size="1.778" layer="91">x</text>
+<text x="769.62" y="335.28" size="1.778" layer="91">x</text>
+<text x="769.62" y="337.82" size="1.778" layer="91">out_MOSI</text>
+<text x="769.62" y="340.36" size="1.778" layer="91">out miso</text>
+<text x="769.62" y="342.9" size="1.778" layer="91">out sck</text>
+<text x="769.62" y="345.44" size="1.778" layer="91">ft232 rx</text>
+<text x="769.62" y="347.98" size="1.778" layer="91">ft232 tx</text>
+<text x="769.62" y="355.6" size="1.778" layer="91">-</text>
+<text x="769.62" y="353.06" size="1.778" layer="91">-</text>
 <text x="815.34" y="101.6" size="1.778" layer="91">kbb3</text>
 <text x="815.34" y="81.28" size="1.778" layer="91">kbb4</text>
