File: PCB/Controller/Controller.sch (EAGLE design)
At the start: 206 parts

Commit message: vil_45
Other:
- moved on the sheet: 1C1, 1C10, 1C19, 1C2, 1C20, 1C21, 1C22, 1C23, 1C24, 1C3, 1C4, 1C5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

Commit message: vil_46
Parts:
- removed J1, J2, J5, J6: (no value), jumper:SJ
- removed RJ4: 0, rcl:R-EU_R1206
- added JR, JT: (no value), jumper:SJ
Connections:
- removed net MISO0: JI2.2
- removed net MOSI0: JO2.2
- removed net N$37: J6.1
- removed net N$41: J5.1
- removed net N$64: 2D1.VDD_325, RJ4.1
- removed net RESET0: JR2.2
- removed net RX: J1.2
- removed net RX_AVR: 5D1.(TXD)PD1, J5.2
- removed net SCK0: JS2.2
- removed net TX: J2.2
- removed net TX_AVR: 5D1.(RXD)PD0, J6.2
- new net N$22: 5D6A.Y2, JT.1
- net 3VUSB2: now also 2D1.VDD_325; no longer RJ4.2
- net MISO8535: now also JI2.2
- net MOSI8535: now also JO2.2
- net RESET8535: now also JR2.2
- net RX_STK500: now also 5D1.(TXD)PD1, JR.1; no longer 5D6A.A4
- net RX_USB: no longer J1.1
- net SCK8535: now also JS2.2
- net TX_STK500: now also 5D1.(RXD)PD0, JT.2; no longer 5D6A.Y2
- net TX_USB: now also JR.2; no longer J2.1
Other:
- moved on the sheet: 1C7, 1C8, 1C9, 2C1, 2C2, 2C3, 2C4, 2C5, 2D1, 2D2, 2R1, 2R10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

Commit message: vil_47
Connections:
- new net N$24: 5D6A.A4, JR.2
- new net N$26: 5D6A.A3, 5D6B.Y2
- net LED/!STK500: now also 5D6A.A1
- net N$22: now also 5D6B.A2, 5D6B.A3
- net TX_USB: no longer JR.2
Other:
- moved on the sheet: 5D5C, 5D6B, JR, JT

Commit message: vil_48
Parts:
- removed JI2, JO2, JR2, JS2: (no value), jumper:SJ
- removed RESET2: TS42, SmartPrj:TS42
- added JD, JI, JO, JRX, JS, JWP: (no value), jumper:SJ
- added RXTXLED: (no value), pinhead:PINHD-1X3
Connections:
- removed net N$67: 2D2.VCC, 2R10.2, 2R9.2
- new net N$27: 2D2.SDA, JD.1
- new net N$37: 2D2.WP, JWP.2
- net 3VUSB2: now also 2D2.VCC, 2R10.2, 2R9.2
- net GND: now also JWP.1, RXTXLED.2
- net MISO8535: now also JI.2; no longer JI2.2
- net MOSI8535: now also JO.2; no longer JO2.2
- net N$24: now also JRX.2; no longer JR.2
- net N$61: now also JI.1; no longer JI2.1
- net N$62: now also JS.1; no longer JS2.1
- net N$63: now also JO.1; no longer JO2.1
- net N$66: now also JD.2; no longer 2D2.SDA
- net RESET8535: now also JR.2; no longer JR2.2
- net RX_LED: now also RXTXLED.3
- net RX_STK500: now also JRX.1; no longer JR.1
- net SCK8535: now also JS.2; no longer JS2.2
- net TX_LED: now also RXTXLED.1
- net TX_USB: now also JR.1; no longer JR2.1
- net URESET: now also RESET1.5-GND
Other:
- note added: "AVR PROGRAMMER"
- note added: "JD disable usb eep"
- moved on the sheet: 1C1, 1C10, 1C19, 1C2, 1C20, 1C21, 1C22, 1C23, 1C24, 1C3, 1C4, 1C5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

Commit message: vil_49
Parts:
- added 1R13: 10k, rcl:R-EU_M0805
Connections:
- net !HVPP_EN: now also D3.C; no longer D2.A
- net !ISP_EN: now also D2.C; no longer D3.A
- net +5V: now also 1R13.2
- net LED/!STK500: now also 1R13.1, D2.A, D3.A; no longer D2.C, D3.C
Other:
- note added: "Keyboard Controller"
- moved on the sheet: 1R15, 1R16, D2, D3, JP2
