File: PCB/Controller/Controller.brd (EAGLE design)
At the start: 160 x 100 mm, 41 parts, among them IC2 LMV358IDGKR, J1 USB MICRO, Y2 16MHz KX-7

Commit message: cont fe11s
Parts:
- removed Z3, Z4: CG0603MLC-05E, varistor:CT/CN0603
- added C5, C6: 100n, rcl:C0805
- added C7, C8: 10m, rcl:C0805
- added LED1, LED2: (no value), led:SML0603
- added R10, R12, R9: 100k, rcl:R0805
- added R11: 47k, rcl:R0805
- added R4, R5: 10, rcl:R0603
- added R6, R7, R8: 2k7, rcl:R0805
- added RN3: 22R, resistor-dil:CAY16
- added RU1, RU2: CG0603MLC-05E, varistor:CT/CN0603
- added X1: USB-B_PN61729-S, detali_controller:USB-B_PN61729-S
- added ZQ1: 12MHz, crystal:HC49/S
- Z1A: value (none) -> 16MHz
- moved F2 129.4 mm to (87.9, -51.1)
- moved SV1 59.7 mm to (77.5, -17.5)
- moved C4 11.6 mm to (-30.5, -71.8), turned to 180 degrees
- moved L1 11.3 mm to (-21.6, -82.5), turned to 180 degrees
- moved DD1 10.9 mm to (65.4, -41.0), turned to 270 degrees
- moved C3 9.94 mm to (-29.5, -67.9)
- moved R2 9.10 mm to (8.26, -55.6)
- moved C18 5.41 mm to (11.1, -50.5)
- moved C1 5.02 mm to (4.76, -51.1)
- moved C2 4.85 mm to (3.49, -61.0), turned to 180 degrees
- moved RN2 4.32 mm to (6.03, -44.5)
- moved RESET1 3.19 mm to (8.26, -28.9), turned to 270 degrees
- renumbered Q1 to Z1A, Y2 to Z1
Connections:
- new net DMI: DD1.15, RN3.2
- new net DPI: DD1.16, RN3.1
- new net N$10: DD1.17, R9.2
- new net N$11: DD1.23, LED1.A
- new net N$12: R5.1, X1.3
- new net N$13: R4.1, X1.2
- new net N$14: DD1.24, LED2.A
- new net N$15: DD1.19, R12.2
- new net N$16: DD1.18, R10.2, R11.1
- new net N$17: LED1.C, R7.1
- new net N$18: LED2.C, R8.1
- new net N$20: R7.2, R8.2
- new net N$21: DD1.14, R6.2
- new net N$5: R4.2, RN3.7, RU2.1
- new net N$6: R5.2, RN3.8, RU1.1
- new net N$7: F2.2, X1.1
- new net N$8: DD1.2, ZQ1.2
- new net N$9: DD1.3, ZQ1.1
- new net VD1V8: C5.1, C7.1, DD1.12, DD1.28
- new net VD3V3: C6.1, C8.1, DD1.13, DD1.21, DD1.26, R12.1, R9.1
- net D+: no longer Z3.1
- net D-: no longer Z4.1
- net GND: now also C5.2, C6.2, C7.2, C8.2, DD1.1, R10.1, R6.1, RU1.2, RU2.2, X1.4, X1.S1, X1.S2; no longer Z3.2, Z4.2
- net VUSB: now also DD1.20, R11.2
- net XUSB: no longer F2.2
Routing:
- net VD3V3: track 0.00 -> 13.0 mm
- net VD1V8: track 0.00 -> 11.5 mm

Commit message: .
Parts:
- removed F2: MF-MSMF050-2 500mA, rcl:L1812
- removed LED1, LED2: (no value), led:SML0603
- removed RN3, RN4: 22R, resistor-dil:CAY16
- added 1D1: ATMEGA168-AU, atmega8:TQFP32-08
- added 2C1, 2C2: 20, resistor:C0805
- added 2C3: 100n, resistor:C0805
- added 2C4: 10mf, rcl:C1210
- added 2C5: 1mf, rcl:C0805
- added 2D1: PL-2303XA, SparkFun-DigitalIC:SSOP28DB
- added 2R1, 2R8: 100, resistor:R0603
- added 2R2, 2R6, 2R7: 220k, resistor:R0603
- added 2R3, 2R5: 220k, resistor:R1206W
- added 2R4: 1.5k, resistor:R0603
- added 2Z1: 12MHz, crystal:HC49/S
- added C15, C9: 22, rcl:C0603
- added C16, C21: (no value), rcl:CTRIMTZ03
- added C23, C25: (no value), keycopy:C0805
- added C26: 100n, SmartPrj:C0603-ROUND
- added F1: MF-MSMF050-2 500mA, rcl:L1812
- added HL1, HL2, HL3, HL4: (no value), led:SML0603
- added IC1: 24C02CP, microchip:DIL8
- added IC3: 74HC244DW, 74xx-eu:SO20W
- added ICSP2: 3x2 M, SmartPrj:2X03
- added ISP2: (no value), con-lstb:MA03-2
- added J2, JI2, JO2, JR2, JS2: (no value), jumper:SJ
- added Q2: 16M, keycopy:HC49/S
- added R13: 100k, rcl:R0805
- added R14, R15, R16: (no value), keycopy:R0805
- added RJ1: (no value), rcl:R0805
- added RJ4: 0, rcl:R1206
- added RN: 22R, resistor-dil:CAY16
- C4: device SmartPrj:C0603-ROUND -> rcl:C0805
- C7, C8: device rcl:C0805 -> rcl:C1206
- J1: value USB MICRO -> (none); device SmartPrj:CON2_USB_MICRO_B_AT -> jumper:SJ
- R7, R8: value 2k7 -> 1k
- moved C4 214.3 mm to (99.4, 98.7), flipped to the bottom, turned to 270 degrees
- moved C3 208.4 mm to (96.8, 97.8), flipped to the bottom, turned to 90 degrees
- moved J1 157.3 mm to (118.1, -33.7)
- moved R5 145.6 mm to (107.3, 99.4), flipped to the bottom
- moved R4 145.3 mm to (107.3, 96.8), flipped to the bottom
- moved RU1 144.1 mm to (112.7, 101.0), flipped to the bottom, turned to 90 degrees
- moved X1 143.6 mm to (103.2, 102.2), flipped to the top
- moved RU2 141.1 mm to (111.8, 93.7), flipped to the bottom, turned to 0 degrees
- moved L1 136.7 mm to (13.7, 49.5), turned to 0 degrees
- moved R10 134.3 mm to (71.1, 100.3)
- moved C6 129.7 mm to (75.9, 86.4)
- moved C7 128.5 mm to (61.6, 92.1), turned to 180 degrees
- moved C5 126.7 mm to (61.9, 89.9), turned to 180 degrees
- moved R6 125.9 mm to (52.4, 81.0)
- moved R12 125.7 mm to (72.4, 83.8)
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Connections:
- removed net D+: J1.P3, RN4.8
- removed net D-: J1.P2, RN4.5
- removed net N$20: R7.2, R8.2
- removed net USBID: J1.P4
- removed net XUSB: J1.P1
- new net 3VUSB2: 2C3.1, 2D1.17, 2R4.1, RJ4.2
- new net MISO: 1D1.16, ISP2.1
- new net MISO0: JI2.2
- new net MOSI: 1D1.15, ISP2.4
- new net MOSI0: JO2.2
- new net N$19: DD1.26, R13.2
- new net N$22: 1D1.8, C25.2, Q2.1
- new net N$23: DD1.27, RJ1.1
- new net N$24: 1D1.7, C23.2, Q2.2
- new net N$25: C21.2, DD1.6
- new net N$27: C21.1, DD1.7
- new net N$29: C16.1, DD1.5
- new net N$30: C16.2, DD1.4
- new net N$31: HL1.A, HL3.C, R7.1
- new net N$52: 2D1.15, 2R8.2
- new net N$53: 2D1.16, 2R1.2
- new net N$54: 2D1.23, 2R2.2
- new net N$55: 2D1.22, 2R3.2
- new net N$56: 2C1.2, 2D1.28, 2Z1.2
- new net N$57: 2C2.2, 2D1.27, 2Z1.1
- new net N$58: 2D1.6, 2R5.1
- new net N$59: 2D1.9, 2R6.2
- new net N$60: 2D1.10, 2R7.2
- new net N$61: 2D1.11, JI2.1
- new net N$62: 2D1.3, JS2.1
- new net N$63: 2D1.2, JO2.1
- new net N$64: 2D1.4, RJ4.1
- new net N$66: 2D1.14, IC1.5, R15.1
- new net N$67: IC1.8, R15.2, R16.2
- new net N$68: 2D1.13, IC1.6, R16.1
- new net RESET0: JR2.2
- new net RX: J1.2
- new net RXM: 1D1.30
- new net RX_USB: 2D1.5, J1.1
- new net SCK: ISP2.3
- new net SCK0: JS2.2
- new net TX: J2.2
- new net TXM: 1D1.31
- new net TX_USB: 2D1.1, J2.1, JR2.1
- new net UU+: 2R4.2, 2R8.1, DD1.9
- new net UU-: 2R1.1, DD1.8
- new net VCC: IC3.20
- net +5V: now also 1D1.18, 1D1.20, 1D1.4, 1D1.6, 2C4.2, 2C5.2, 2D1.19, 2D1.20, 2D1.24, 2D1.8, 2R3.1, 2R5.2, 2R6.1, 2R7.1, ISP2.2, R14.2
- net DMI: now also RN.2; no longer RN3.2
- net DPI: now also RN.1; no longer RN3.1
- net GND: now also 1D1.21, 1D1.3, 1D1.5, 2C1.1, 2C2.1, 2C3.2, 2C4.1, 2C5.1, 2D1.18, 2D1.21, 2D1.25, 2D1.26, 2D1.7, 2R2.1, C15.1, C23.1, C25.1, C26.1, C9.1, IC1.1, IC1.2, IC1.3, IC1.4, IC3.10, ISP2.6, RJ1.2; no longer J1.S1, J1.S2, J1.S3, J1.S4, J1.S5, J1.S6
- net N$11: now also DD1.22, R7.2, R8.2; no longer DD1.23, LED1.A
- net N$14: now also DD1.23, HL1.C, HL3.A; no longer DD1.24, LED2.A
- net N$17: now also DD1.24, HL2.C, HL4.A; no longer LED1.C, R7.1
- net N$18: now also HL2.A, HL4.C; no longer LED2.C
- net N$5: now also RN.7; no longer RN3.7
- net N$6: now also RN.8; no longer RN3.8
- net N$7: now also F1.2; no longer F2.2
- net N$8: now also C9.2, ZQ1.1; no longer ZQ1.2
- net N$9: now also C15.2, ZQ1.2; no longer ZQ1.1
- net RD+: now also DD1.11; no longer RN4.1
- net RD-: now also DD1.10; no longer RN4.4
- net RESET: now also 1D1.29, ISP2.5, R14.1
- net UGND: no longer J1.P5
- net VD3V3: now also R13.1; no longer DD1.26
- net VUSB: now also C26.2, F1.1; no longer F2.1
Routing:
- net GND: track 53.7 -> 101.7 mm
- net N$11: track 0.00 -> 18.1 mm, vias 0 -> 1
- net N$19: track 0.00 -> 15.8 mm
- net VD3V3: track 13.0 -> 26.0 mm
- net N$17: track 0.00 -> 12.6 mm, vias 0 -> 1
- net VUSB: track 0.00 -> 12.4 mm
- net N$14: track 0.00 -> 11.2 mm, vias 0 -> 1
- net N$10: track 0.00 -> 9.69 mm
- net N$15: track 0.00 -> 8.81 mm
- net N$8: track 0.00 -> 7.66 mm
- net N$16: track 0.00 -> 6.14 mm
- net N$9: track 0.00 -> 4.69 mm
- net VD1V8: track 11.5 -> 16.2 mm
- net N$23: track 0.00 -> 4.12 mm
- net N$7: track 0.00 -> 3.71 mm
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Other:
- board size 160 x 100 mm -> 149.9 x 50.8 mm

Commit message: .
Parts:
- added J_U1, J_U2: (no value), jumper:SJ
- R11, R9: device rcl:R0805 -> rcl:R1206W
- moved C21 75.1 mm to (127.0, 75.6), turned to 90 degrees
- moved C26 55.7 mm to (109.2, 68.3), turned to 90 degrees
- moved C1 55.4 mm to (37.5, 6.03)
- moved C17 55.4 mm to (54.3, -15.9)
- moved C18 55.4 mm to (31.1, 5.40)
- moved C2 55.4 mm to (38.7, 15.9)
- moved C20 55.4 mm to (45.1, 8.89)
- moved C24 55.4 mm to (52.1, 8.89)
- moved DD3 55.4 mm to (49.8, -6.35)
- moved R1 55.4 mm to (49.8, 4.45)
- moved R2 55.4 mm to (34.0, 10.5)
- moved R25 55.4 mm to (27.6, 2.86)
- moved RESET1 55.4 mm to (34.0, -16.2)
- moved RN2 55.4 mm to (36.2, -0.64)
- moved Z1 55.4 mm to (48.6, 8.89)
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Connections:
- net N$12 renamed ID+
- net N$13 renamed ID-
- removed net N$5: R4.2, RN.7, RU2.1
- removed net N$6: R5.2, RN.8, RU1.1
- new net D+: J_U1.2, R5.2, RN.8, RU1.1
- new net D-: J_U2.2, R4.2, RN.7, RU2.1
- net RD+: now also J_U1.1
- net RD-: now also J_U2.1
Routing:
- net GND: track 101.7 -> 247.4 mm
- net AVCC: track 1.88 -> 54.6 mm
- net +5V: track 26.4 -> 78.2 mm
- net D+: track 0.00 -> 18.0 mm
- net D-: track 0.00 -> 15.5 mm
- net VUSB: track 12.4 -> 24.2 mm, vias 0 -> 1
- net N$16: track 6.14 -> 15.7 mm
- net N$18: track 3.06 -> 10.2 mm
- net N$11: track 18.1 -> 11.8 mm
- net N$10: track 9.69 -> 14.7 mm
- net VD3V3: track 26.0 -> 30.3 mm
- net ID+: track 0.00 -> 3.94 mm
- net ID-: track 0.00 -> 2.88 mm
- net N$15: track 8.81 -> 11.3 mm
- net N$19: track 15.8 -> 18.1 mm
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
Commit message: pcb b mov det
Parts:
- removed C15, C9: 22, rcl:C0603
- removed C21: (no value), rcl:CTRIMTZ03
- removed C26: 100n, SmartPrj:C0603-ROUND
- removed C3: 10u, rcl:SMC_B
- removed C4, C5, C6: 100n, rcl:C0805
- removed C7, C8: 10m, rcl:C1206
- removed DD1: FE1.1S, imcom:FE1.1S_SSOP-28
- removed IC1: 24C02CP, microchip:DIL8
- removed ICSP2: 3x2 M, SmartPrj:2X03
- removed R1: 1M, SmartPrj:R0603-ROUND
- removed R10, R12, R13: 100k, rcl:R0805
- removed R11: 47k, rcl:R1206W
- removed R15, R16: (no value), keycopy:R0805
- removed R4, R5: 10, rcl:R0603
- removed R6: 2k7, rcl:R0805
- removed R7, R8: 1k, rcl:R0805
- removed R9: 100k, rcl:R1206W
- removed RJ1: (no value), rcl:R0805
- removed X1: USB-B_PN61729-S, detali_controller:USB-B_PN61729-S
- removed ZQ1: 12MHz, crystal:HC49/S
- added 1C1, 1C2: 22, rcl:C0603
- added 1C10, 1C4, 1C5, 1C8, 1C9: 100n, rcl:C0805
- added 1C3, 1C6: 10m, rcl:C1206
- added 1C7: 10u, rcl:SMC_B
- added 1R1, 1R11, 1R12, 1R2: 10, rcl:R0603
- added 1R10, 1R9: 1k, rcl:R0805
- added 1R3, 1R4, 1R7: 100k, rcl:R0805
- added 1R5: 100k, rcl:R1206W
- added 1R6: 47k, rcl:R1206W
- added 1R8: 2k7, rcl:R0805
- added 1RJ: (no value), rcl:R0805
- added 1X1: USB-B_PN61729-S, detali_controller:USB-B_PN61729-S
- added 1X2: USB_TYPE_A_FEMALE_TH, imcom:USB_TYPE_A_FEMALE_TH
- added 1Z1: 12MHz, crystal:HC49/S
- added 2D2: 24C02CP, microchip:DIL8
- added 2R10, 2R9: (no value), keycopy:R0805
- added 3D1: ATMEGA168-AU, atmega8:TQFP32-08
- added R100: 1M, SmartPrj:R0603-ROUND
- added U$10, U$36, U$37, U$38, U$39, U$40, U$41, U$42, U$43, U$44, U$45, U$46, U$47, U$48, U$7, U$8, U$88: (no value), kbmx:18X18
- added U_U1, U_U2: (no value), jumper:SJ@1
- 1D1: value ATMEGA168-AU -> FE1.1S; device atmega8:TQFP32-08 -> imcom:FE1.1S_SSOP-28
- J1, J2, JI2, JO2, JR2, JS2, J_U1: device jumper:SJ -> jumper:SJ@1
- J_U2: value (none) -> J; device jumper:SJ -> detali_controller:R1206W
- moved J2 143.2 mm to (149.2, 107.0), turned to 90 degrees
- moved JS2 136.6 mm to (150.2, 98.1), turned to 90 degrees
- moved JI2 136.0 mm to (145.4, 101.0), turned to 90 degrees
- moved JR2 133.3 mm to (148.9, 93.7), turned to 90 degrees
- moved JO2 131.3 mm to (145.1, 91.4), turned to 90 degrees
- moved 2C2 130.7 mm to (122.9, 108.3), turned to 180 degrees
- moved 2C1 130.7 mm to (118.4, 108.3), turned to 180 degrees
- moved 2R7 128.1 mm to (136.8, 96.8), turned to 90 degrees
- moved 2R8 125.2 mm to (118.7, 96.8)
- moved 2R5 122.7 mm to (133.7, 99.1), turned to 180 degrees
- moved 2R1 122.6 mm to (116.8, 94.3)
- moved J1 122.1 mm to (143.8, 85.7), turned to 90 degrees
- moved 2C3 120.4 mm to (138.1, 96.8), turned to 90 degrees
- moved 2R2 119.7 mm to (123.5, 88.9), turned to 270 degrees
- moved 2C5 118.6 mm to (138.7, 91.1), turned to 90 degrees
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- renumbered IC3 to 2D3
Connections:
- removed net N$27: C21.1, DD1.7
- removed net RXM: 1D1.30
- removed net TXM: 1D1.31
- new net N$12: 1R11.2, 1X2.3
- new net N$13: 1R12.2, 1X2.2
- new net N$20: DD3.4, U_U2.2
- new net N$5: 1D1.9, 1R11.1
- new net N$6: 1D1.8, 1R12.1
- new net RXP: 3D1.30
- new net TXP: 3D1.31
- net +5V: now also 3D1.18, 3D1.20, 3D1.4, 3D1.6; no longer 1D1.18, 1D1.20, 1D1.4, 1D1.6
- net D+: now also 1R2.2, RN.7; no longer R5.2, RN.8
- net D-: now also 1R1.2, J_U2.1, RN.8; no longer J_U2.2, R4.2, RN.7
- net DMI: now also 1D1.15, RN.1; no longer DD1.15, RN.2
- net DPI: now also 1D1.16, RN.2; no longer DD1.16, RN.1
- net GND: now also 1C1.1, 1C10.1, 1C2.1, 1C3.2, 1C4.2, 1C5.2, 1C6.2, 1C7.-, 1C8.1, 1C9.1, 1D1.1, 1R7.1, 1R8.1, 1RJ.2, 1X1.4, 1X1.S1, 1X1.S2, 1X2.4, 2D2.1, 2D2.2, 2D2.3, 2D2.4, 3D1.21, 3D1.3, 3D1.5; no longer 1D1.21, 1D1.3, 1D1.5, C15.1, C26.1, C3.-, C4.1, C5.2, C6.2, C7.2, C8.2, C9.1, DD1.1, IC1.1, IC1.2, IC1.3, IC1.4, R10.1, R6.1, RJ1.2, X1.4, X1.S1, X1.S2
- net ID+: now also 1R2.1, 1X1.3; no longer R5.1, X1.3
- net ID-: now also 1R1.1, 1X1.2; no longer R4.1, X1.2
- net MISO: no longer 1D1.16
- net MISO0: now also 3D1.16
- net MOSI: no longer 1D1.15
- net MOSI0: now also 3D1.15
- net N$10: now also 1D1.17, 1R5.2; no longer DD1.17, R9.2
- net N$11: now also 1D1.22, 1R10.2, 1R9.2; no longer DD1.22, R7.2, R8.2
- net N$14: now also 1D1.23; no longer DD1.23
- net N$15: now also 1D1.19, 1R4.2; no longer DD1.19, R12.2
- net N$16: now also 1D1.18, 1R6.1, 1R7.2; no longer DD1.18, R10.2, R11.1
- net N$17: now also 1D1.24; no longer DD1.24
- net N$18: now also 1R10.1; no longer R8.1
- net N$19: now also 1D1.26, 1R3.2; no longer DD1.26, R13.2
- net N$21: now also 1D1.14, 1R8.2; no longer DD1.14, R6.2
- net N$22: now also 3D1.8; no longer 1D1.8
- net N$23: now also 1D1.27, 1RJ.1; no longer DD1.27, RJ1.1
- net N$24: now also 3D1.7; no longer 1D1.7
- net N$25: now also DD3.3, U_U1.2; no longer C21.2, DD1.6
- net N$29: now also 1D1.5; no longer DD1.5
- net N$30: now also 1D1.4; no longer DD1.4
- net N$31: now also 1R9.1; no longer R7.1
- net N$66: now also 2D2.5, 2R9.1; no longer IC1.5, R15.1
- net N$67: now also 2D2.8, 2R10.2, 2R9.2; no longer IC1.8, R15.2, R16.2
- net N$68: now also 2D2.6, 2R10.1; no longer IC1.6, R16.1
- net N$7: now also 1X1.1; no longer X1.1
- net N$8: now also 1C1.2, 1D1.2, 1Z1.1; no longer C9.2, DD1.2, ZQ1.1
- net N$9: now also 1C2.2, 1D1.3, 1Z1.2; no longer C15.2, DD1.3, ZQ1.2
- net RD+: now also 1D1.11, U_U2.1; no longer DD1.11, DD3.4
- net RD-: now also 1D1.10, J_U2.2, U_U1.1; no longer DD1.10, DD3.3, J_U2.1
- net RESET: no longer 1D1.29, R14.1
- net RESET0: now also 3D1.29, R14.1
- net SCK0: now also 3D1.17
- net UU+: now also 1D1.7; no longer DD1.9
- net UU-: now also 1D1.6; no longer DD1.8
- net VD1V8: now also 1C3.1, 1C4.1, 1D1.12, 1D1.28; no longer C5.1, C7.1, DD1.12, DD1.28
- net VD3V3: now also 1C5.1, 1C6.1, 1D1.13, 1D1.21, 1R3.1, 1R4.1, 1R5.1; no longer C6.1, C8.1, DD1.13, DD1.21, R12.1, R13.1, R9.1
- net VUSB: now also 1C10.2, 1C7.+, 1C8.2, 1C9.2, 1D1.20, 1R6.2, 1X2.1; no longer C26.2, C3.+, C4.2, DD1.20, R11.2
- net XTAL1: now also R100.1; no longer R1.1
- net XTAL2: now also R100.2; no longer R1.2
Routing:
- net GND: track 247.4 -> 182.1 mm, vias 0 -> 1
- net AVCC: track 54.6 -> 3.21 mm
- net +5V: track 78.2 -> 27.6 mm
- net VUSB: track 24.2 -> 66.4 mm
- net N$5: track 0.00 -> 17.7 mm
- net RD-: track 0.00 -> 16.8 mm
- net N$6: track 0.00 -> 16.8 mm
- net D-: track 15.5 -> 6.98 mm, vias 0 -> 1
- net RD+: track 0.00 -> 6.98 mm
- net N$18: track 10.2 -> 16.1 mm
- net DPI: track 3.50 -> 8.99 mm
- net N$13: track 0.00 -> 5.31 mm
- net N$21: track 0.00 -> 5.03 mm, vias 0 -> 1
- net DMI: track 2.91 -> 7.52 mm
- net D+: track 18.0 -> 15.7 mm, vias 0 -> 1
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Other:
- board size 149.9 x 50.8 mm -> 184.3 x 132.7 mm

Commit message: sm
Parts:
- added 1C11: 100n, rcl:C0805
Connections:
- new net N$26: 3D1.14
- net +5V: now also 1C11.1
- net GND: now also 1C11.2
Changed lines of the file:
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@@
 <element name="U_U1" library="jumper" package="SJ@1" value="" x="85.725" y="93.98" rot="MR0"/>
 <element name="U_U2" library="jumper" package="SJ@1" value="" x="85.4075" y="96.52" rot="MR0"/>
+<element name="1C11" library="rcl" package="C0805" value="100n" x="1.5875" y="-36.195"/>
 </elements>
 <signals>
@@
 <wire x1="38.1" y1="14.9225" x2="34.9" y2="14.9225" width="0.4064" layer="1"/>
 <wire x1="86.6775" y1="90.4875" x2="85.7225" y2="89.535" width="0.4064" layer="1"/>
+<contactref element="1C11" pad="2"/>
 <wire x1="160.655" y1="82.2325" x2="163.195" y2="82.2325" width="0" layer="19" extent="1-1"/>
 <wire x1="158.115" y1="82.2325" x2="160.655" y2="82.2325" width="0" layer="19" extent="1-1"/>
@@
 <wire x1="57.8485" y1="3.81" x2="57.531" y2="17.78" width="0" layer="19" extent="1-1"/>
 <wire x1="64.1985" y1="5.08" x2="57.8485" y2="3.81" width="0" layer="19" extent="1-1"/>
+<wire x1="2.5375" y1="-36.195" x2="24.475" y2="0.88" width="0" layer="19" extent="1-1"/>
 <wire x1="167.5892" y1="-18.7325" x2="127.3175" y2="28.575" width="0" layer="19" extent="1-1"/>
 </signal>
@@
 <contactref element="R14" pad="2"/>
 <contactref element="ISP2" pad="2"/>
+<contactref element="1C11" pad="1"/>
 <wire x1="129.67" y1="99.3775" x2="132.1685" y2="99.06" width="0" layer="19" extent="1-1"/>
 <wire x1="136.8425" y1="95.9875" x2="132.1685" y2="99.06" width="0" layer="19" extent="1-1"/>
@@
 <wire x1="16.825" y1="24.13" x2="20.2565" y2="26.67" width="0" layer="19" extent="1-1"/>
 <wire x1="46.649" y1="44.657" x2="56.134" y2="30.48" width="0" layer="19" extent="1-1"/>
+<wire x1="0.6375" y1="-36.195" x2="34.1" y2="9.1225" width="0" layer="19" extent="1-1"/>
 </signal>
 <signal name="RESET">
@@
 <wire x1="43.9" y1="12.5225" x2="84.963" y2="93.98" width="0" layer="19" extent="1-16"/>
 </signal>
+<signal name="N$26">
+<contactref element="3D1" pad="14"/>
+</signal>
 </signals>

Commit message: fw
Connections:
- new net MISO(D1): DD3.11
- new net SCK(D3): DD3.9
- net CD1: no longer SV6.10
- net CD3: no longer SV6.8
- net MISO(D3): no longer DD3.11
- net SCK(D1): no longer DD3.9
Changed lines of the file:
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@@
 </signal>
 <signal name="CD3">
-<contactref element="SV6" pad="8"/>
 <contactref element="SV5" pad="6"/>
-<wire x1="115.2525" y1="67.6275" x2="113.665" y2="75.8825" width="0" layer="19" extent="1-1"/>
 </signal>
 <signal name="CD2">
@@
 </signal>
 <signal name="CD1">
-<contactref element="SV6" pad="10"/>
 <contactref element="SV5" pad="8"/>
-<wire x1="120.3325" y1="67.6275" x2="118.745" y2="75.8825" width="0" layer="19" extent="1-1"/>
 </signal>
 <signal name="KBN2">
@@
 <signal name="MISO(D3)">
 <contactref element="ICSP1" pad="1"/>
-<contactref element="DD3" pad="11"/>
-<wire x1="43.9" y1="18.9225" x2="51.435" y2="20.32" width="0" layer="19" extent="1-1"/>
 </signal>
 <signal name="MOSI(D2)">
@@
 <signal name="SCK(D1)">
 <contactref element="ICSP1" pad="3"/>
-<contactref element="DD3" pad="9"/>
-<wire x1="43.9" y1="17.3225" x2="53.975" y2="20.32" width="0" layer="19" extent="1-1"/>
 </signal>
 <signal name="N$7">
@@
 <contactref element="3D1" pad="14"/>
 </signal>
+<signal name="SCK(D3)">
+<contactref element="DD3" pad="9"/>
+</signal>
+<signal name="MISO(D1)">
+<contactref element="DD3" pad="11"/>
+</signal>
 </signals>

Commit message: sh c
Parts:
- added 1C12: 100n, rcl:C0805
- moved 2C1 29.9 mm to (120.3, 78.4), turned to 0 degrees
- moved JS2 29.0 mm to (137.5, 72.1)
- moved J2 28.3 mm to (149.5, 78.7), turned to 0 degrees
- moved 2C2 26.8 mm to (120.3, 81.6), turned to 0 degrees
- moved JI2 24.1 mm to (145.4, 76.8)
- moved SV1 24.1 mm to (61.9, 87.0)
- moved JR2 23.4 mm to (133.0, 76.5)
- moved JO2 15.9 mm to (137.5, 77.5)
- moved 2R6 15.4 mm to (124.1, 95.9)
- moved 2R4 14.9 mm to (129.5, 95.6), turned to 90 degrees
- moved SV6 13.4 mm to (98.1, 68.9)
- moved 2R10 13.3 mm to (155.6, 93.0), flipped to the bottom, turned to 0 degrees
- moved SV5 12.7 mm to (98.4, 75.9)
- moved 2R5 12.4 mm to (141.6, 89.5), turned to 90 degrees
- moved 2R3 11.9 mm to (120.7, 87.6), turned to 270 degrees
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Connections:
- new net N$27: 1C12.1, 3D1.20
- net +5V: no longer 3D1.20
- net GND: now also 1C12.2

Commit message: fw add
Parts:
- added U_U3, U_U4: (no value), jumper:SJ@1
- C23, C25: value (none) -> 22
- moved 1C12 131.1 mm to (113.3, 26.4), turned to 90 degrees
- moved 1C11 129.4 mm to (115.6, 25.1), turned to 90 degrees
- moved C16 7.10 mm to (100.3, 83.5)
- moved 2R3 4.58 mm to (116.8, 90.2)
- moved 2R2 2.54 mm to (120.0, 88.6)
- moved 2C4 0.64 mm to (123.5, 92.1)
Connections:
- net D+: now also U_U3.1
- net D-: now also U_U4.1
- net N$20: now also U_U3.2
- net N$25: now also U_U4.2
