File: PCB/Controller/Controller.brd (EAGLE design)
At the start: 184.3 x 132.7 mm, 126 parts, among them IC2 LMV358IDGKR, Q2 16M

Commit message: pcb c
Parts:
- moved 2D2 40.0 mm to (119.4, 107.0), turned to 180 degrees
- moved 2R9 39.4 mm to (117.2, 99.7), turned to 180 degrees
- moved 2R10 38.1 mm to (120.0, 106.7), turned to 180 degrees
- moved 2C3 29.6 mm to (108.9, 92.1), turned to 180 degrees
- moved JI2 25.2 mm to (128.6, 95.6), turned to 270 degrees
- moved 2R4 19.2 mm to (111.8, 102.9), turned to 180 degrees
- moved 2C4 18.1 mm to (105.7, 88.9), turned to 90 degrees
- moved 2C5 16.6 mm to (128.6, 87.9)
- moved 2R1 15.2 mm to (105.1, 99.1)
- moved 2R8 15.1 mm to (107.0, 100.3)
- moved 2D1 14.3 mm to (116.8, 88.6)
- moved J2 14.3 mm to (135.3, 78.1)
- moved JO2 14.3 mm to (123.2, 76.8)
- moved JR2 14.3 mm to (118.7, 75.9)
- moved JS2 14.3 mm to (123.2, 71.4)
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Routing:
- net GND: track 182.1 -> 221.1 mm
- net +5V: track 27.6 -> 50.3 mm
- net UU+: track 0.00 -> 16.7 mm
- net UU-: track 0.00 -> 16.5 mm
- net N$54: track 0.00 -> 5.57 mm
- net N$55: track 0.00 -> 5.32 mm

Commit message: pcb b
Parts:
- moved R14 54.2 mm to (168.0, 41.0)
- moved 1C11 54.2 mm to (165.4, 46.4)
- moved 1C12 54.2 mm to (163.2, 47.6)
- moved 3D1 54.2 mm to (155.3, 47.6)
- moved C23 54.2 mm to (143.2, 46.4)
- moved C25 54.2 mm to (142.9, 42.2)
- moved ISP2 54.2 mm to (174.6, 48.6)
- moved Q2 54.2 mm to (147.0, 44.5)
- moved 2C1 11.9 mm to (104.1, 88.3), turned to 270 degrees
- moved 2R6 6.29 mm to (120.7, 93.7)
- moved 2Z1 6.10 mm to (108.6, 86.4), turned to 180 degrees
- moved 2R2 5.99 mm to (106.7, 89.9), turned to 90 degrees
- moved 2C3 5.91 mm to (105.4, 96.8)
- moved 2D1 5.65 mm to (113.3, 93.0)
- moved 2C4 5.65 mm to (102.2, 93.3)
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Routing:
- net GND: track 221.1 -> 261.3 mm
- net N$67: track 0.00 -> 16.3 mm
- net N$29: track 0.00 -> 10.9 mm
- net N$68: track 0.00 -> 9.88 mm
- net 3VUSB2: track 0.00 -> 9.82 mm
- net N$30: track 0.00 -> 9.51 mm
- net N$66: track 0.00 -> 7.82 mm
- net UU+: track 16.7 -> 24.2 mm
- net N$57: track 0.00 -> 7.43 mm
- net N$56: track 0.00 -> 6.82 mm
- net N$53: track 0.00 -> 5.64 mm
- net N$52: track 0.00 -> 2.70 mm
- net N$54: track 5.57 -> 3.68 mm
- net N$9: track 4.99 -> 6.13 mm
- net UU-: track 16.5 -> 17.2 mm
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
Commit message: pcb c
Parts:
- added F2: MF-MSMF050-2 500mA, rcl:L1812
- moved 1C10 0.32 mm to (104.5, 108.9), turned to 0 degrees
Connections:
- new net VUSBH: 1C10.1, 1X2.1, F2.1, F2.2
- net GND: now also 1C10.2; no longer 1C10.1
- net VUSB: no longer 1C10.2, 1X2.1
Routing:
- net VUSB: track 66.0 -> 47.5 mm
- net VUSBH: track 0.00 -> 12.3 mm

Commit message: .
Parts:
- moved RJ4 2.56 mm to (130.5, 87.9)
- moved 2Z1 0.32 mm to (108.6, 86.0), flipped to the bottom, turned to 0 degrees
Changed lines of the file:
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@@
 <layer number="20" name="Dimension" color="15" fill="1" visible="yes" active="yes"/>
 <layer number="21" name="tPlace" color="7" fill="1" visible="yes" active="yes"/>
-<layer number="22" name="bPlace" color="7" fill="1" visible="yes" active="yes"/>
+<layer number="22" name="bPlace" color="6" fill="1" visible="yes" active="yes"/>
 <layer number="23" name="tOrigins" color="15" fill="1" visible="yes" active="yes"/>
 <layer number="24" name="bOrigins" color="15" fill="1" visible="yes" active="yes"/>
@@
 <attribute name="VALUE" x="102.362" y="94.361" size="1.27" layer="27" rot="R270"/>
 </element>
-<element name="2Z1" library="crystal" package="HC49/S" value="12MHz" x="108.585" y="86.36" smashed="yes" rot="R180">
-<attribute name="OC_NEWARK" value="unknown" x="136.525" y="93.0275" size="1.778" layer="27" rot="R180" display="off"/>
-<attribute name="MPN" value="" x="136.525" y="93.0275" size="1.778" layer="27" rot="R180" display="off"/>
-<attribute name="MF" value="" x="136.525" y="93.0275" size="1.778" layer="27" rot="R180" display="off"/>
-<attribute name="OC_FARNELL" value="1667008" x="136.525" y="93.0275" size="1.778" layer="27" rot="R180" display="off"/>
-<attribute name="NAME" x="113.665" y="83.693" size="1.27" layer="25" ratio="10" rot="R180"/>
-<attribute name="VALUE" x="113.665" y="90.297" size="1.27" layer="27" ratio="10" rot="R180"/>
+<element name="2Z1" library="crystal" package="HC49/S" value="12MHz" x="108.585" y="86.0425" smashed="yes" rot="MR0">
+<attribute name="OC_NEWARK" value="unknown" x="136.525" y="79.375" size="1.778" layer="28" rot="MR0" display="off"/>
+<attribute name="MPN" value="" x="136.525" y="79.375" size="1.778" layer="28" rot="MR0" display="off"/>
+<attribute name="MF" value="" x="136.525" y="79.375" size="1.778" layer="28" rot="MR0" display="off"/>
+<attribute name="OC_FARNELL" value="1667008" x="136.525" y="79.375" size="1.778" layer="28" rot="MR0" display="off"/>
+<attribute name="NAME" x="113.665" y="88.7095" size="1.27" layer="26" ratio="10" rot="MR0"/>
+<attribute name="VALUE" x="113.665" y="82.1055" size="1.27" layer="28" ratio="10" rot="MR0"/>
 </element>
 <element name="2C1" library="resistor" package="C0805" value="20" x="104.14" y="88.265" smashed="yes" rot="R270">
@@
 <element name="J1" library="jumper" package="SJ@1" value="" x="135.89" y="82.2325"/>
 <element name="J2" library="jumper" package="SJ@1" value="" x="135.255" y="78.105"/>
-<element name="RJ4" library="rcl" package="R1206" value="0" x="129.2225" y="85.725" rot="R90"/>
+<element name="RJ4" library="rcl" package="R1206" value="0" x="130.4925" y="87.9475" rot="R90"/>
 <element name="2C5" library="rcl" package="C0805" value="1mf" x="125.095" y="92.075" smashed="yes" rot="R90">
 <attribute name="NAME" x="123.825" y="90.805" size="1.27" layer="25" rot="R90"/>
@@
 <contactref element="2C1" pad="2"/>
 <wire x1="109.6915" y1="88.8025" x2="108.6145" y2="88.8025" width="0.3048" layer="1"/>
-<wire x1="108.6145" y1="88.8025" x2="106.172" y2="86.36" width="0.3048" layer="1"/>
-<wire x1="106.172" y1="86.36" x2="104.14" y2="87.415" width="0.6096" layer="1"/>
+<wire x1="106.172" y1="86.0425" x2="108.6145" y2="88.8025" width="0.3048" layer="1"/>
+<wire x1="106.172" y1="86.0425" x2="104.14" y2="87.415" width="0.6096" layer="1"/>
 </signal>
 <signal name="N$57">
@@
 <wire x1="111.2075" y1="89.4525" x2="111.76" y2="88.9" width="0.3048" layer="1"/>
 <wire x1="111.76" y1="88.9" x2="111.76" y2="87.122" width="0.3048" layer="1"/>
-<wire x1="111.76" y1="87.122" x2="110.998" y2="86.36" width="0.3048" layer="1"/>
-<wire x1="109.7525" y1="84.455" x2="110.998" y2="86.36" width="0.6096" layer="1"/>
+<wire x1="111.76" y1="87.122" x2="110.998" y2="86.0425" width="0.3048" layer="1"/>
+<wire x1="110.998" y1="86.0425" x2="109.7525" y2="84.455" width="0.6096" layer="1"/>
 </signal>
 <signal name="3VUSB2">
@@
 <wire x1="110.875" y1="95.9525" x2="112.2925" y2="97.37" width="0.3048" layer="1"/>
 <wire x1="112.2925" y1="97.37" x2="112.2925" y2="100.33" width="0.3048" layer="1"/>
-<wire x1="112.2925" y1="97.37" x2="129.2225" y2="87.147" width="0" layer="19" extent="1-1"/>
+<wire x1="112.2925" y1="97.37" x2="130.4925" y2="89.3695" width="0" layer="19" extent="1-1"/>
 </signal>
 <signal name="N$58">
@@
 <contactref element="2D1" pad="4"/>
 <contactref element="RJ4" pad="1"/>
-<wire x1="117.0035" y1="90.7525" x2="129.2225" y2="84.303" width="0" layer="19" extent="1-1"/>
+<wire x1="117.0035" y1="90.7525" x2="130.4925" y2="86.5255" width="0" layer="19" extent="1-1"/>
 </signal>
 <signal name="N$66">

Commit message: pcb a
Parts:
- moved SV1 4.86 mm to (62.9, 82.2)
Changed lines of the file:
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@@
 <setting verticaltext="up"/>
 </settings>
-<grid distance="12.5" unitdist="mil" unit="mil" style="lines" multiple="1" display="yes" altdistance="0.025" altunitdist="inch" altunit="inch"/>
+<grid distance="50" unitdist="mil" unit="mil" style="lines" multiple="1" display="yes" altdistance="0.025" altunitdist="inch" altunit="inch"/>
 <layers>
 <layer number="1" name="Top" color="4" fill="1" visible="yes" active="yes"/>
@@
 <plain>
 <wire x1="20.32" y1="112.395" x2="170.18" y2="112.395" width="0.3048" layer="20"/>
-<dimension x1="57.15" y1="112.395" x2="173.0375" y2="61.595" x3="44.45" y3="86.995" layer="20" dtype="vertical"/>
+<dimension x1="181.61" y1="118.745" x2="181.2925" y2="65.7225" x3="44.45" y3="92.23375" layer="20" dtype="vertical"/>
 <wire x1="20.32" y1="112.395" x2="20.32" y2="61.595" width="0.3048" layer="20"/>
 <wire x1="170.18" y1="112.395" x2="170.18" y2="61.595" width="0.3048" layer="20"/>
@@
 <attribute name="OC_FARNELL" value="unknown" x="124.7775" y="16.8275" size="1.778" layer="27" display="off"/>
 </element>
-<element name="SV1" library="detali_controller" package="FE13" value="" x="61.9125" y="86.995" rot="R90">
-<attribute name="OC_NEWARK" value="unknown" x="107.6325" y="132.715" size="1.778" layer="27" rot="R90" display="off"/>
-<attribute name="MPN" value="" x="107.6325" y="132.715" size="1.778" layer="27" rot="R90" display="off"/>
-<attribute name="MF" value="" x="107.6325" y="132.715" size="1.778" layer="27" rot="R90" display="off"/>
-<attribute name="OC_FARNELL" value="unknown" x="107.6325" y="132.715" size="1.778" layer="27" rot="R90" display="off"/>
+<element name="SV1" library="detali_controller" package="FE13" value="" x="62.865" y="82.2325" rot="R90">
+<attribute name="OC_NEWARK" value="unknown" x="108.585" y="127.9525" size="1.778" layer="27" rot="R90" display="off"/>
+<attribute name="MPN" value="" x="108.585" y="127.9525" size="1.778" layer="27" rot="R90" display="off"/>
+<attribute name="MF" value="" x="108.585" y="127.9525" size="1.778" layer="27" rot="R90" display="off"/>
+<attribute name="OC_FARNELL" value="unknown" x="108.585" y="127.9525" size="1.778" layer="27" rot="R90" display="off"/>
 </element>
 <element name="ICSP1" library="SmartPrj" package="2X03" value="ICSP" x="53.975" y="21.59"/>

Commit message: .
Parts:
- removed U$10, U$36, U$37, U$38, U$39, U$40, U$41, U$42, U$43, U$44, U$45, U$46, U$47, U$48, U$7, U$8, U$88: (no value), kbmx:18X18
- added 1C19, 1C22, 1C23, 1C24: 100n, rcl:C0805
- added 1C20, 1C21: 33p, rcl:C0805
- added 1D2, 1D5: MEGA8535-A, atmel:TQFP44
- added 1D4: 74HC165D, 74xx-eu:SO16
- added 1R28: 10k, rcl:R0805
- added 1R29, 1R30, 1R31, 1R37, 1R38, 1R41, 4R7: 10k, rcl:M0805
- added 1R32, 4R10: 1k, rcl:M0805
- added 1R33, 1R34: 1k5, rcl:M0805
- added 1R35: 36k, rcl:M0805
- added 1R36: 150k, rcl:R1206
- added 1R39: 47k, rcl:M0805
- added 1R40: 2k, rcl:R1206W
- added 1R42: 22k, rcl:M1206
- added 1VD3: SB130, diode:SMB
- added 1VD4, 3VD2: SS12, diode:SMB
- added 1VT4, 1VT6: BC847, transistor:SOT23
- added 1VT5: BC857, transistor:SOT23-BEC
- added 3C10: 100n, rcl:C025-025X050
- added 3C6: 100n, rc-elektronik:C025-024X044
- added 3C7: 1n, rcl:C025-025X050
- added 3C8: 470µ / 10V, HWProgUSB:RCL_E3,5-8
- added 3C9: 100µ 16V, HWProgUSB:RCL_E3,5-8
- added 3D2, 3D4: ATMEGA168-AU, atmega8:TQFP32-08
- added 3D3: MC34063AD, mc34063:SOIC8
- added 3L2: 100uh, rcl:0207/10
- added 3R5: 220, rcl:R1206
- added 3R6: 0.5-1, rcl:M1206
- added 3R7: 20k, rcl:M0805
- added 3R8, 4R9: 2k2, rcl:M0805
- added 4C2: 10n, rcl:C1206
- added 4R6: 1.5k, rcl:M0805
- added 4R8: 2k2, rcl:M1206
- added 4VT4: BC847, transistor-neu-to92:SOT23
- added 4VT5: IRML6402, transistor-power:SUPER-SOT3
- added 4VT6: IRML2502, transistor-small-signal:SOT23
- added HW: yellow, led:SML0603
- added HW1: High Voltage Enable, HWProgUSB:PINHEAD_1X02
- added IC1, IC3: MEGA16-A, atmel:TQFP44
- added ISP1: (no value), con-lstb:MA03-2
- added J5, J6, JV1, JX1: (no value), jumper:SJ
- added JP1: Selfprogramming, HWProgUSB:JUMPER_JP2
- added LED: red, led:SML0603
- added READY: green, led:SML0603
- added RES1: 0R-JUMPA, jump-0r-smd:A0R-JMP
- added RESET2, RESET3: TS42, SmartPrj:TS42
- added RJ11, RJ12, RJ13, RJ14, RJ15, RJ9: 0, rcl:R1206
- added Z3: 7,3728MHz, crystal:HC49U-V
- J1, J2, JI2, JO2, JR2, JS2, J_U1, U_U1, U_U2, U_U3, U_U4: device jumper:SJ@1 -> jumper:SJ
- moved 3D1 61.3 mm to (108.3, 8.26)
Connections:
- new net +12V: 1R31.2, 1VT5.E, 3C10.2, 3C9.+, 3R7.2, 3VD2.C
- new net D0: 1D5.40
- new net D1: 1D5.41
- new net D2: 1D5.42
- new net D3: 1D5.43
- new net D4: 1D5.44
- new net GND2: 1D2.39, IC1.39, IC3.39
- new net MISO8535: 1D5.2, RJ11.2
- new net MOSI8535: 1D5.1, ISP1.4
- new net N$100: 1D2.23, 3D4.27
- new net N$101: 1D2.24, 3D4.28
- new net N$102: 1D2.25, 3D4.29
- new net N$103: 1D2.2, 3D4.7
- new net N$104: 1D2.40, 3D4.12
- new net N$105: 1D2.41, 3D4.13
- new net N$106: 1D2.42, 3D4.14
- new net N$107: 1D2.43, 3D4.15
- new net N$108: 1D2.44, 3D4.16
- new net N$109: 1D2.1, 3D4.17
- new net N$110: 1D2.3, 3D4.8
- new net N$28: 1R34.1, READY.A
- new net N$32: 1D5.30, 1D5.31, 1R35.1, 1R36.2
- new net N$33: 1D4.2, 1D5.32, READY.C
- new net N$34: 1D4.6, 1R39.2, RESET3.3, RESET3.4
- new net N$35: 1D5.12, HW1.1
- new net N$36: 1R29.2, 1R42.2, HW1.2
- new net N$37: 3D2.20, IC3.29
- new net N$38: IC1.30, IC1.31
- new net N$39: 1R32.2, 1VD3.C, 1VT5.C, HW.A
- new net N$40: 1R29.1, 1VT4.1
- new net N$41: 3D2.8, IC3.8
- new net N$42: 3D2.7, IC3.7
- new net N$43: 3D2.29, IC3.4
- new net N$44: 3D2.30, IC3.9
- new net N$45: 1R30.1, 1VT4.3
- new net N$46: 1R30.2, 1R31.1, 1VT5.B
- new net N$47: 1D4.9, 1D5.15
- new net N$48: 1R33.1, LED.A
- new net N$49: 1D4.11, 1D4.13, 1D4.14, 1R38.2
- new net N$50: 3D2.31, IC3.10
- new net N$51: 1D2.19, 3D4.23
- new net N$65: 1D4.12, 1D4.3, 1D4.4, 1D4.5, 1R37.2
- new net N$69: 1R28.2, 1VT6.1
- new net N$70: 3D3.8, 3R5.1
- new net N$71: 1D2.20, 3D4.24
- new net N$72: 1D2.21, 3D4.25
- new net N$73: 1D2.9, 3D4.30
- new net N$74: 1D2.10, 3D4.31
- new net N$75: 3D3.7, 3L2.1, 3R5.2, 3R6.2
- new net N$76: 1D2.11, 3D4.32
- new net N$77: 1D2.12, 3D4.1
- new net N$78: 1D2.13, 3D4.2
- new net N$79: 3D3.5, 3R7.1, 3R8.2
- new net N$80: 3D3.1, 3L2.2, 3VD2.A
- new net N$81: 3C7.1, 3D3.3
- new net N$82: 1C20.2, 1D5.7, Z3.2
- new net N$83: 1C21.2, 1D5.8, Z3.1
- new net N$84: 4R6.2, 4VT4.3, 4VT5.1
- new net N$85: 4R7.2, 4R8.2, 4VT4.1
- new net N$86: 4C2.2, 4R8.1, 4R9.2
- new net N$87: 1D2.14, 3D4.9
- new net N$88: 1D5.4, RJ9.2
- new net N$89: ISP1.1, RJ11.1
- new net N$90: 1VT4.2, RJ12.2
- new net N$91: 1VD4.C, ISP1.2
- new net N$92: 1VD4.A, RJ13.1
- new net N$93: RJ13.2, RJ14.1
- new net N$94: 1C22.1, 1C23.1, RESET2.1, RESET2.2, RJ15.2
- new net N$95: 1R40.1, HW.C
- new net N$96: 4R10.2, 4VT6.1
- new net N$97: 1D2.15, 3D4.10
- new net N$98: 1D2.16, 3D4.11
- new net N$99: 1D2.22, 3D4.26
- new net N1: 1D4.1, 1D5.33, LED.C
- new net PD2: 1D5.11, 1R28.1
- new net PD5: 1D5.14, 4R9.1
- new net PD7: 1D5.16, 4VT6.3, JX1.1
- new net PPC0(BS2): 1D5.19
- new net PPC1(RB): 1D5.20
- new net PPC2(OE): 1D5.21
- new net PPC3(WR): 1D5.22
- new net PPC4(BS1): 1D5.23
- new net PPC5(XA0): 1D5.24
- new net PPC6(XA1): 1D5.25
- new net PPC7(PAGEL): 1D5.26
- new net RESET(P): ISP1.5, JP1.2, RES1.2
- new net RESET8535: 1C22.2, 1R41.1, JP1.1, RES1.3, RESET2.3, RESET2.4, RJ9.1
- new net RX_AVR: 1D5.10, J5.2
- new net SCK8535: 1D5.3, ISP1.3
- new net SWCLK(XTAL1): 4VT6.2, JX1.2
- new net TRST(RESET): 1R32.1, 1VT6.3, JP1.3, RES1.1
- new net TX_AVR: 1D5.9, J6.2
- new net VCC1: 1D2.17, IC1.17, IC3.17
- new net VCC2: 1D2.38, IC1.38, IC3.38
- new net VTG: 4R10.1, 4VT5.3, JV1.2, RJ14.2
- net +5V: now also 1C19.1, 1C23.2, 1C24.2, 1D4.16, 1D5.17, 1D5.27, 1D5.29, 1D5.38, 1D5.5, 1R33.2, 1R34.2, 1R35.2, 1R37.1, 1R39.1, 1R40.2, 1R41.2, 1VD3.A, 3C6.1, 3C8.+, 3D3.6, 3R6.1, 4R6.1, 4VT5.2, JV1.1
- net 5-GND: now also RESET2.5
- net AGND: now also 3D2.21, 3D4.21
- net AVCC: now also 1D2.27, IC1.27, IC3.27
- net GND: now also 1C19.2, 1C20.1, 1C21.1, 1C24.1, 1D2.28, 1D2.6, 1D4.10, 1D4.15, 1D4.8, 1D5.18, 1D5.28, 1D5.39, 1D5.6, 1R36.1, 1R38.1, 1R42.1, 1VT6.2, 3C10.1, 3C6.2, 3C7.2, 3C8.-, 3C9.-, 3D2.3, 3D2.5, 3D3.2, 3D3.4, 3D4.3, 3D4.5, 3R8.1, 4C2.1, 4R7.1, 4VT4.2, IC1.28, IC1.6, IC3.28, IC3.6, ISP1.6, RESET3.1, RESET3.2, RESET3.5, RJ12.1, RJ15.1
- net UGND: now also 1D2.18, IC1.18, IC3.18
- net VCC: now also 1D2.5, 3D2.4, 3D2.6, 3D4.4, 3D4.6, IC1.5, IC3.5
Other:
- board size 184.3 x 132.7 mm -> 149.9 x 50.8 mm

Commit message: pcb c
Parts:
- removed IC2: LMV358IDGKR, linear:MSOP08
- removed R23: (no value), rcl:M0805
- removed RN2: 10K, resistor-dil:CAY16
- removed SV1: (no value), detali_controller:FE13
- added !OE, !WR, BS1, BS2, DATA0, DATA1, DATA2, DATA3, DATA4, DATA5, DATA6, DATA7, PAG, R/!B, RES, XA0, XA1, XTAL1: (no value), pinhead:1X01
- added R1: 10k, rcl:M0805
- added SV2: (no value), detali_main:FE03-1
- added SV3: (no value), detali_main:FE08
- J1, J2, J5, J6, JI2, JO2, JR2, JS2, JV1, JX1, J_U1, U_U1, U_U2, U_U3, U_U4: device jumper:SJ -> jumper:SJ@1
- moved 2D3 361.3 mm to (-46.0, 270.5), turned to 0 degrees
- moved C19 278.2 mm to (-59.7, 283.8)
- moved R3 275.6 mm to (-62.2, 286.7)
- moved L1 273.6 mm to (-67.9, 285.1)
- moved D1 273.5 mm to (-66.0, 274.3), turned to 0 degrees
- moved C11 272.3 mm to (-56.5, 250.5), turned to 270 degrees
- moved C10 271.0 mm to (-46.0, 286.1)
- moved C13 271.0 mm to (-39.4, 273.7)
- moved C20 271.0 mm to (-81.0, 275.9)
- moved C24 271.0 mm to (-74.0, 275.9)
- moved DD3 271.0 mm to (-76.2, 260.7)
- moved L3 271.0 mm to (-67.9, 254.3)
- moved Z1 271.0 mm to (-77.5, 275.9)
- moved Z1A 271.0 mm to (-76.2, 273.1)
- moved C12 271.0 mm to (-42.5, 287.7)
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Connections:
- removed net MISO(D1): DD3.11
- removed net N$2: DD3.12, R23.1
- removed net SCK(D3): DD3.9
- new net UMISO(D1): DATA3.1, DD3.11
- new net UMOSI(D2): DATA2.1, DD3.10
- new net UPB0: DATA0.1, DD3.8
- new net UPB4: DATA4.1, DD3.28
- new net UPB5: DATA5.1, DD3.29
- new net UPB6: DATA6.1, DD3.30
- new net UPB7: DATA7.1, DD3.12
- new net UPD1: DD3.19, R/!B.1
- new net UPD2: !OE.1, DD3.20
- new net UPD3: !WR.1, DD3.21
- new net UPD4: BS1.1, DD3.25
- new net UPD5: DD3.22, XA0.1
- new net UPD6: DD3.26, XA1.1
- new net UPD7: DD3.27, PAG.1
- new net UPE6: BS2.1, DD3.1
- new net URESET: D1.A, DD3.13, R1.1, RES.1, RESET1.1, RESET1.2
- new net USCK(D3): DATA1.1, DD3.9
- net +5V: now also R1.2; no longer IC2.8, RN2.5
- net GND: no longer IC2.4
- net MOSI(D2): no longer DD3.10
- net RESET: no longer D1.A, DD3.13, RESET1.1, RESET1.2, RN2.4
- net XTAL1: now also C20.2, DD3.17, R100.2, XTAL1.1, Z1.3, Z1A.2; no longer C24.1, DD3.16, R100.1, Z1.1, Z1A.1
- net XTAL2: now also C24.1, DD3.16, R100.1, Z1.1, Z1A.1; no longer C20.2, DD3.17, R100.2, Z1.3, Z1A.2
Routing:
- net VUSBH: track 12.3 -> 24.3 mm
- net XTAL1: track 15.6 -> 7.50 mm
- net N$5: track 17.7 -> 13.9 mm
- net GND: track 261.6 -> 265.2 mm
- net N$6: track 16.8 -> 13.6 mm
- net N$13: track 5.31 -> 4.49 mm
- net XTAL2: track 11.6 -> 12.4 mm
Other:
- board size 149.9 x 50.8 mm -> 425.8 x 149.2 mm
- board text added: "1179-16"

Commit message: pcb c
Parts:
- removed 1D2: MEGA8535-A, atmel:TQFP44
- removed 3D4: ATMEGA168-AU, atmega8:TQFP32-08
- removed C16: (no value), rcl:CTRIMTZ03
- removed IC3: MEGA16-A, atmel:TQFP44
- removed R2, R3: NM, SmartPrj:R0402
- removed R25: (no value), rcl:M0805
- added IC10, IC6, IC8, IC9: 74HC595D, 74xx-eu:SO16
- added IOL10, IOL7, IOL8, IOL9: 8x1F-H8.5, SmartPrj:1X08
- added PINS: 1k, rcl:R0805
- added R10, R11, R12, R13, R15, R16, R17, R18, R19, R20, R21, R4, R5, R6, R7, R8, R9: 10k, rcl:M0805
- J1, J2, J5, J6, JI2, JO2, JR2, JS2, JV1, JX1, J_U1, U_U1, U_U2, U_U3, U_U4: device jumper:SJ@1 -> jumper:SJ
- moved 3D2 388.9 mm to (148.0, 257.2)
- moved ICSP1 20.7 mm to (-57.8, 271.8)
- moved J2 12.9 mm to (132.7, 249.7)
- moved J1 11.4 mm to (134.6, 253.2)
- moved 2R4 7.03 mm to (114.3, 269.7)
- moved 2R10 5.78 mm to (119.2, 272.6)
- moved 2R9 4.69 mm to (117.3, 270.7)
- moved F2 4.61 mm to (110.6, 269.7)
- moved 2D2 4.52 mm to (123.7, 273.1)
- moved 2R8 4.27 mm to (114.3, 268.0), turned to 0 degrees
- moved 1R11 0.64 mm to (107.3, 271.0)
- moved 1R12 0.48 mm to (108.1, 269.4)
- moved 1C10 0.32 mm to (110.5, 276.1)
Connections:
- removed net MISO(D3): ICSP1.1
- removed net MOSI(D2): ICSP1.4
- removed net N$100: 1D2.23, 3D4.27
- removed net N$101: 1D2.24, 3D4.28
- removed net N$102: 1D2.25, 3D4.29
- removed net N$103: 1D2.2, 3D4.7
- removed net N$104: 1D2.40, 3D4.12
- removed net N$105: 1D2.41, 3D4.13
- removed net N$106: 1D2.42, 3D4.14
- removed net N$107: 1D2.43, 3D4.15
- removed net N$108: 1D2.44, 3D4.16
- removed net N$109: 1D2.1, 3D4.17
- removed net N$110: 1D2.3, 3D4.8
- removed net N$29: 1D1.5, C16.1
- removed net N$3: DD3.33, R25.1
- removed net N$4: ICSP1.5
- removed net N$51: 1D2.19, 3D4.23
- removed net N$71: 1D2.20, 3D4.24
- removed net N$72: 1D2.21, 3D4.25
- removed net N$73: 1D2.9, 3D4.30
- removed net N$74: 1D2.10, 3D4.31
- removed net N$76: 1D2.11, 3D4.32
- removed net N$77: 1D2.12, 3D4.1
- removed net N$78: 1D2.13, 3D4.2
- removed net N$87: 1D2.14, 3D4.9
- removed net N$97: 1D2.15, 3D4.10
- removed net N$98: 1D2.16, 3D4.11
- removed net N$99: 1D2.22, 3D4.26
- removed net SCK(D1): ICSP1.3
- new net CR+: 1D1.5, PINS.2
- new net CR-: 1D1.4, PINS.1
- new net GND1: R16.2, R17.2, R18.2, R19.2, R20.2, R21.2
- new net N$139: IC10.11, IC6.11, IC8.11, IC9.11
- new net N$140: IC10.12, IC6.12, IC8.12, IC9.12
- new net N$141: IC8.9, IC9.14
- new net N$142: IC10.14, IC9.9
- new net REG1: IC6.14
- new net UPC6: DD3.31, R6.1
- new net UPC7: DD3.32, R4.1
- new net UPD0: DD3.18, R15.1
- new net UPF0: DD3.41, R21.1
- new net UPF1: DD3.40, R20.1
- new net UPF4: DD3.39, R19.1
- new net UPF5: DD3.38, R18.1
- new net UPF6: DD3.37, R17.1
- new net UPF7: DD3.36, R16.1
- net +5V: now also IC10.10, IC6.10, IC8.10, IC9.10, R5.2; no longer R25.2
- net AGND: no longer 3D4.21, C1.1, R2.1
- net AVCC: no longer 1D2.27, IC3.27
- net GND: now also C1.1, IC10.13, IC10.8, IC6.13, IC6.8, IC8.13, IC8.8, IC9.13, IC9.8, R10.2, R11.2, R12.2, R13.2, R15.2, R4.2, R6.2, R7.2, R8.2, R9.2; no longer 1D2.28, 1D2.6, 3D4.3, 3D4.5, IC3.28, IC3.6, R2.2, R3.1
- net GND2: no longer 1D2.39, IC3.39
- net HWB: now also DD3.33, R5.1
- net N$30: now also IC6.9, IC8.14; no longer 1D1.4, C16.2
- net N$37: no longer IC3.29
- net N$41: no longer IC3.8
- net N$42: no longer IC3.7
- net N$43: no longer IC3.4
- net N$44: no longer IC3.9
- net N$50: no longer IC3.10
- net UGND: no longer 1D2.18, IC3.18, R3.2
- net UMISO(D1): now also ICSP1.1
- net UMOSI(D2): now also ICSP1.4
- net UPD1: now also R13.1
- net UPD2: now also R12.1
- net UPD3: now also R11.1
- net UPD4: now also R10.1
- net UPD5: now also R9.1
- net UPD6: now also R8.1
- net UPD7: now also R7.1
- net URESET: now also ICSP1.5
- net USCK(D3): now also ICSP1.3
- net VCC: now also IC10.16, IC6.16, IC8.16, IC9.16; no longer 1D2.5, 3D4.4, 3D4.6, IC3.5
- net VCC1: no longer 1D2.17, IC3.17
- net VCC2: no longer 1D2.38, IC3.38
Routing:
- net N$29: track 10.9 -> 0.00 mm
- net N$30: track 9.51 -> 0.00 mm
- net GND: track 265.2 -> 256.9 mm
- net VUSBH: track 24.3 -> 16.8 mm
- net N$68: track 9.88 -> 17.3 mm
- net UU+: track 24.2 -> 19.4 mm
- net 3VUSB2: track 9.82 -> 14.4 mm
- net N$66: track 7.82 -> 12.3 mm
- net N$52: track 2.70 -> 6.19 mm
- net N$67: track 16.3 -> 15.6 mm
