File: PCB/Controller/Controller.brd (EAGLE design)
At the start: 425.8 x 149.2 mm, 206 parts

Commit message: vil_46
Parts:
- removed J5, J6: (no value), jumper:SJ
- removed RJ4: 0, rcl:R1206
- renumbered J1 to JR, J2 to JT
Connections:
- removed net MISO0: JI2.2
- removed net MOSI0: JO2.2
- removed net N$37: J6.1
- removed net N$41: J5.1
- removed net N$64: 2D1.4, RJ4.1
- removed net RESET0: JR2.2
- removed net RX: JR.2
- removed net RX_AVR: 5D1.10, J5.2
- removed net SCK0: JS2.2
- removed net TX: JT.2
- removed net TX_AVR: 5D1.9, J6.2
- new net N$22: 5D6.16, JT.1
- net 3VUSB2: now also 2D1.4; no longer RJ4.2
- net MISO8535: now also JI2.2
- net MOSI8535: now also JO2.2
- net RESET8535: now also JR2.2
- net RX_STK500: now also 5D1.10, JR.1; no longer 5D6.8
- net RX_USB: no longer JR.1
- net SCK8535: now also JS2.2
- net TX_STK500: now also 5D1.9, JT.2; no longer 5D6.16
- net TX_USB: now also JR.2; no longer JT.1
Routing:
- net GND: track 268.9 -> 264.5 mm

Commit message: vil_47
Connections:
- new net N$24: 5D6.8, JR.2
- new net N$26: 5D6.6, 5D6.7
- net LED/!STK500: now also 5D6.2
- net N$22: now also 5D6.13, 5D6.15
- net TX_USB: no longer JR.2
Changed lines of the file:
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@@
 <contactref element="5D6" pad="17"/>
 <contactref element="5D6" pad="4"/>
-<contactref element="JR" pad="2"/>
-<wire x1="126.5285" y1="255.96625" x2="135.382" y2="253.20625" width="0" layer="19" extent="1-1"/>
 <wire x1="124.7775" y1="246.41175" x2="126.5285" y2="255.96625" width="0" layer="19" extent="1-1"/>
 <wire x1="114.45875" y1="202.03795" x2="124.7775" y2="246.41175" width="0" layer="19" extent="1-1"/>
@@
 <contactref element="5D5" pad="9"/>
 <contactref element="5D5" pad="8"/>
+<contactref element="5D6" pad="2"/>
 <wire x1="80.44" y1="177.4825" x2="80.44" y2="171.45" width="0" layer="19" extent="16-16"/>
 <wire x1="105.3084" y1="193.04" x2="80.44" y2="177.4825" width="0" layer="19" extent="1-16"/>
 <wire x1="105.3084" y1="194.31" x2="105.3084" y2="193.04" width="0" layer="19" extent="1-1"/>
 <wire x1="110.64875" y1="191.97955" x2="105.3084" y2="193.04" width="0" layer="19" extent="1-1"/>
+<wire x1="111.91875" y1="191.97955" x2="110.64875" y2="191.97955" width="0" layer="19" extent="1-1"/>
 </signal>
 <signal name="!OE741">
@@
 <wire x1="133.858" y1="253.20625" x2="-22.67625" y2="209.3175" width="0" layer="19" extent="1-16"/>
 </signal>
+<signal name="N$24">
+<contactref element="JR" pad="2"/>
+<contactref element="5D6" pad="8"/>
+<wire x1="119.53875" y1="191.97955" x2="135.382" y2="253.20625" width="0" layer="19" extent="1-1"/>
+</signal>
 <signal name="N$22">
+<contactref element="5D6" pad="15"/>
+<contactref element="5D6" pad="13"/>
 <contactref element="5D6" pad="16"/>
 <contactref element="JT" pad="1"/>
-<wire x1="115.72875" y1="202.03795" x2="131.953" y2="249.71375" width="0" layer="19" extent="1-1"/>
+<wire x1="119.53875" y1="202.03795" x2="131.953" y2="249.71375" width="0" layer="19" extent="1-1"/>
+<wire x1="116.99875" y1="202.03795" x2="119.53875" y2="202.03795" width="0" layer="19" extent="1-1"/>
+<wire x1="115.72875" y1="202.03795" x2="116.99875" y2="202.03795" width="0" layer="19" extent="1-1"/>
+</signal>
+<signal name="N$26">
+<contactref element="5D6" pad="7"/>
+<contactref element="5D6" pad="6"/>
+<wire x1="116.99875" y1="191.97955" x2="118.26875" y2="191.97955" width="0" layer="19" extent="1-1"/>
 </signal>
 </signals>

Commit message: vil_48
Parts:
- removed JR2: (no value), jumper:SJ
- removed RESET2: TS42, SmartPrj:TS42
- added JD, JRX, JWP: (no value), jumper:SJ
- added RXTXLED: (no value), pinhead:1X03
- moved JR 11.5 mm to (124.8, 247.2), turned to 90 degrees
- moved 5D5 5.75 mm to (102.9, 202.6)
- moved 5D6 5.08 mm to (116.4, 202.1)
- moved 2R9 1.42 mm to (116.0, 271.3)
- renumbered JI2 to JI, JO2 to JO, JS2 to JS
Connections:
- removed net 5-GND: RESET1.5, RESET2.5
- removed net N$67: 2D2.8, 2R10.2, 2R9.2
- new net N$27: 2D2.5, JD.1
- new net N$37: 2D2.7, JWP.2
- net 3VUSB2: now also 2D2.8, 2R10.2, 2R9.2
- net GND: now also JWP.1, RXTXLED.2
- net N$24: now also JRX.2; no longer JR.2
- net N$66: now also JD.2; no longer 2D2.5
- net RESET8535: now also JR.2; no longer JR2.2
- net RX_LED: now also RXTXLED.3
- net RX_STK500: now also JRX.1; no longer JR.1
- net TX_LED: now also RXTXLED.1
- net TX_USB: now also JR.1; no longer JR2.1
- net URESET: now also RESET1.5
Routing:
- net 3VUSB2: track 14.4 -> 30.6 mm
- net N$67: track 15.6 -> 0.00 mm
- net N$37: track 0.00 -> 14.1 mm
- net N$66: track 12.3 -> 8.01 mm
- net GND: track 264.5 -> 268.2 mm

Commit message: vil_49
Parts:
- added 1R13: 10k, rcl:M0805
- moved D3 5.72 mm to (78.7, 177.2), turned to 180 degrees
- moved D2 5.08 mm to (78.7, 172.4), turned to 180 degrees
- moved D6 2.01 mm to (68.6, 172.1)
- moved D9 1.27 mm to (68.6, 177.2)
- moved D7 0.90 mm to (63.5, 170.2)
- moved 1R14 0.90 mm to (67.9, 181.6)
- moved 1R15 0.90 mm to (78.1, 169.5), flipped to the bottom, turned to 180 degrees
- moved 1R16 0.90 mm to (78.1, 179.7), flipped to the bottom, turned to 180 degrees
Connections:
- net !HVPP_EN: now also D3.C; no longer D2.A
- net !ISP_EN: now also D2.C; no longer D3.A
- net +5V: now also 1R13.2
- net LED/!STK500: now also 1R13.1, D2.A, D3.A; no longer D2.C, D3.C

Commit message: vil_50
Parts:
- renumbered JP2 to JP, JT to JTX
Changed lines of the file:
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@@
 <element name="JR" library="jumper" package="SJ" value="" x="124.7775" y="247.17375" rot="R90"/>
 <element name="JRX" library="jumper" package="SJ" value="" x="134.62" y="253.20625"/>
-<element name="JT" library="jumper" package="SJ" value="" x="132.715" y="249.71375"/>
+<element name="JTX" library="jumper" package="SJ" value="" x="132.715" y="249.71375"/>
 <element name="2C5" library="rcl" package="C0805" value="1mf" x="134.62" y="259.23875" smashed="yes" rot="R90">
 <attribute name="NAME" x="133.35" y="257.96875" size="1.27" layer="25" rot="R90"/>
@@
 <element name="T_RESET" library="jumper" package="JP1" value="" x="-33.9725" y="193.83375"/>
 <element name="5D6" library="74xx-eu" package="SO20W" value="74HC244DW" x="116.36375" y="202.08875"/>
-<element name="JP2" library="jumper" package="JP2" value="" x="73.66" y="174.625" rot="R90"/>
+<element name="JP" library="jumper" package="JP2" value="" x="73.66" y="174.625" rot="R90"/>
 <element name="1R15" library="rcl" package="M0805" value="10k" x="78.105" y="169.545" rot="MR180"/>
 <element name="1R16" library="rcl" package="M0805" value="10k" x="78.105" y="179.705" rot="MR180"/>
@@
 <contactref element="5D6" pad="10"/>
 <contactref element="5D6" pad="10"/>
-<contactref element="JP2" pad="2"/>
+<contactref element="JP" pad="2"/>
 <contactref element="1R14" pad="1"/>
 <contactref element="1R17" pad="1"/>
@@
 </signal>
 <signal name="!HVPP_EN">
-<contactref element="JP2" pad="3"/>
+<contactref element="JP" pad="3"/>
 <contactref element="1R16" pad="1"/>
 <contactref element="D9" pad="A"/>
@@
 </signal>
 <signal name="!ISP_EN">
-<contactref element="JP2" pad="1"/>
+<contactref element="JP" pad="1"/>
 <contactref element="1R15" pad="1"/>
 <contactref element="D6" pad="A"/>
@@
 </signal>
 <signal name="TX_STK500">
-<contactref element="JT" pad="2"/>
+<contactref element="JTX" pad="2"/>
 <contactref element="5D1" pad="9"/>
 <wire x1="133.477" y1="249.71375" x2="-23.47625" y2="209.3175" width="0" layer="19" extent="1-16"/>
@@
 <contactref element="5D6" pad="13"/>
 <contactref element="5D6" pad="16"/>
-<contactref element="JT" pad="1"/>
+<contactref element="JTX" pad="1"/>
 <wire x1="119.53875" y1="207.11795" x2="131.953" y2="249.71375" width="0" layer="19" extent="1-1"/>
 <wire x1="116.99875" y1="207.11795" x2="119.53875" y2="207.11795" width="0" layer="19" extent="1-1"/>

Commit message: копейки
Parts:
- added SV1: (no value), detali_main:FE12
Other:
- outline, holes or cut-outs redrawn
Changed lines of the file:
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@@
 <board>
 <plain>
-<wire x1="7.3025" y1="279.55875" x2="175.26" y2="279.55875" width="0.3048" layer="20"/>
+<wire x1="7.3025" y1="279.55875" x2="161.29" y2="279.55875" width="0.3048" layer="20"/>
+<wire x1="161.29" y1="279.55875" x2="175.26" y2="279.55875" width="0.3048" layer="20"/>
 <wire x1="7.3025" y1="279.55875" x2="7.3025" y2="228.75875" width="0.3048" layer="20"/>
 <wire x1="175.26" y1="279.55875" x2="175.26" y2="228.75875" width="0.3048" layer="20"/>
-<wire x1="175.26" y1="228.75875" x2="7.3025" y2="228.75875" width="0.3048" layer="20"/>
+<wire x1="175.26" y1="228.75875" x2="161.29" y2="228.75875" width="0.3048" layer="20"/>
+<wire x1="161.29" y1="228.75875" x2="7.3025" y2="228.75875" width="0.3048" layer="20"/>
 <wire x1="180.34" y1="286.385" x2="2.38125" y2="286.385" width="0.2" layer="20"/>
 <wire x1="183.515" y1="283.21" x2="180.34" y2="286.385" width="0.2" layer="20" curve="90"/>
@@
 <wire x1="50.00625" y1="254.15875" x2="50.00625" y2="236.37875" width="0.4064" layer="21"/>
 <wire x1="47.625" y1="236.37875" x2="52.3875" y2="236.37875" width="0.4064" layer="21"/>
-<wire x1="47.625" y1="254.15875" x2="52.3875" y2="254.15875" width="0.4064" layer="21"/>
+<wire x1="47.625" y1="254.15875" x2="203.5175" y2="254.15875" width="0.4064" layer="21"/>
 <wire x1="47.625" y1="251.61875" x2="52.3875" y2="251.61875" width="0.4064" layer="21"/>
 <wire x1="47.625" y1="249.07875" x2="52.3875" y2="249.07875" width="0.4064" layer="21"/>
@@
 <dimension x1="-0.79375" y1="305.1175" x2="48.895" y2="296.70375" x3="24.050625" y3="313.3725" layer="21" dtype="horizontal"/>
 <dimension x1="-89.69375" y1="292.4175" x2="-40.005" y2="284.00375" x3="-64.849375" y3="300.6725" layer="21" dtype="horizontal"/>
+<wire x1="65.0875" y1="259.23875" x2="217.4875" y2="259.23875" width="0.4064" layer="21"/>
+<wire x1="161.29" y1="279.55875" x2="161.29" y2="228.75875" width="0.3048" layer="20"/>
 </plain>
 <attributes>
@@
 </element>
 <element name="1R13" library="rcl" package="M0805" value="10k" x="104.775" y="193.675" rot="R180"/>
+<element name="SV1" library="detali_main" package="FE12" value="" x="72.86625" y="270.66875" rot="R270">
+<attribute name="OC_NEWARK" value="unknown" x="72.86625" y="270.66875" size="1.778" layer="27" rot="R270" display="off"/>
+<attribute name="MPN" value="" x="72.86625" y="270.66875" size="1.778" layer="27" rot="R270" display="off"/>
+<attribute name="MF" value="" x="72.86625" y="270.66875" size="1.778" layer="27" rot="R270" display="off"/>
+<attribute name="OC_FARNELL" value="unknown" x="72.86625" y="270.66875" size="1.778" layer="27" rot="R270" display="off"/>
+</element>
 </elements>
 <signals>

Commit message: .
Parts:
- added U$3: (no value), detali_controller:U235
- moved JI 5.34 mm to (139.5, 261.9), turned to 270 degrees
- moved JD 2.01 mm to (117.5, 272.4)
- moved JWP 1.27 mm to (128.9, 273.7)
- moved 2R7 0.63 mm to (132.4, 261.8)
- moved U_U3 0.63 mm to (108.6, 266.5)
Routing:
- net GND: track 268.2 -> 272.8 mm
