File: PCB/Controller/Controller-b.brd (EAGLE design)
At the start: 425.8 x 149.2 mm, 206 parts

Commit message: vil_44
Parts:
- added 1C13, 1C14: 100n, rcl:C0805
- added 3D2: ATMEGA168-AU, atmega8:TQFP32-08
- added C10, C12: 10u, rcl:SMC_B
- added C11, C14: 1u, SmartPrj:C0603-ROUND
- added C13, C22: 100n, SmartPrj:C0603-ROUND
- added C3, C4: 22, keycopy:C0805
- added D90: M7, diode:SMB
- added IC2, IC3, IC4, IC5: 74HC595D, 74xx-eu:SO16
- added IC6: MEGA16-A, atmel:TQFP44
- added IOL1, IOL2, IOL3, IOL4: 8x1F-H8.5, SmartPrj:1X08
- added ISP3: (no value), con-lstb:MA03-2
- added Q1: 16M, keycopy:HC49/S
- added R3: (no value), keycopy:R0805
- added RN1: 10K, resistor-dil:CAY16
Connections:
- new net +3V3: C14.2
- new net CMP: C22.2, RN1.7, RN1.8
- new net GND1: IC6.18
- new net GND2: IC6.39
- new net MISO: ISP3.1
- new net MOSI: ISP3.4
- new net N$30: 3D2.8, C4.2, Q1.1
- new net N$42: IC2.9, IC3.14
- new net N$44: IC2.11, IC3.11, IC4.11, IC5.11
- new net N$51: IC2.12, IC3.12, IC4.12, IC5.12
- new net N$71: IC3.9, IC4.14
- new net N$72: IC4.9, IC5.14
- new net N$73: 3D2.7, C3.2, Q1.2
- new net N$77: 3D2.14
- new net N$78: 1C14.1, 3D2.20
- new net N$87: IC6.30, IC6.31
- new net REG1: IC2.14
- new net RESET: ISP3.5
- new net RXP: 3D2.30
- new net SCK: ISP3.3
- new net TXP: 3D2.31
- new net VCC: IC2.16, IC3.16, IC4.16, IC5.16, IC6.5
- new net VCC1: IC6.17
- new net VCC2: IC6.38
- new net VIN: D90.C, RN1.1
- net +5V: now also 1C13.1, 3D2.18, 3D2.4, 3D2.6, C11.2, C12.+, C13.1, IC2.10, IC3.10, IC4.10, IC5.10, ISP3.2, R3.2
- net AVCC: now also IC6.27
- net GND: now also 1C13.2, 1C14.2, 3D2.21, 3D2.3, 3D2.5, C10.-, C11.1, C12.-, C13.2, C14.1, C22.1, C3.1, C4.1, D90.A, IC2.13, IC2.8, IC3.13, IC3.8, IC4.13, IC4.8, IC5.13, IC5.8, IC6.28, IC6.6, ISP3.6, RN1.2, RN1.3
- net HWB: now also RN1.6
- net MISO0: now also 3D2.16
- net MOSI0: now also 3D2.15
- net RESET0: now also 3D2.29, R3.1
- net SCK0: now also 3D2.17
