File: PCB/Controller/Controller-b.sch (EAGLE design)
At the start: 206 parts

Commit message: vil_44
Parts:
- added 1C13, 1C14: 100n, rcl:C-EUC0805
- added 3D2: ATMEGA168-AU, atmega8:ATMEGA48/88/168-AU
- added C10, C12: 10u, rcl:CPOL-EUSMCB
- added C11, C14: 1u, SmartPrj:C-EUC0603
- added C13, C22: 100n, SmartPrj:C-EUC0603
- added C3, C4: 22, keycopy:C-EUC0805
- added D90: M7, diode:DIODE-SMB
- added IC2, IC3, IC4, IC5: 74HC595D, 74xx-eu:74HC595D
- added IC6: MEGA16-A, atmel:MEGA16-A
- added IOL1, IOL2, IOL3, IOL4: 8x1F-H8.5, SmartPrj:PINHD-1X8
- added ISP3: (no value), con-lstb:MA03-2
- added Q1: 16M, keycopy:CRYSTALHC49S
- added R3: (no value), keycopy:R-EU_R0805
- added RN1: 10K, resistor-dil:4R-NCAY16
Connections:
- new net +3V3: C14.2
- new net CMP: C22.2, RN1A.2, RN1B.2
- new net MISO: ISP3.1
- new net MOSI: ISP3.4
- new net N$30: 3D2.PB7(XTAL2/TOSC2/PCINT7), C4.2, Q1.1
- new net N$42: IC2A.QH*, IC3A.SER
- new net N$44: IC2A.SCK, IC3A.SCK, IC4A.SCK, IC5A.SCK
- new net N$51: IC2A.RCK, IC3A.RCK, IC4A.RCK, IC5A.RCK
- new net N$71: IC3A.QH*, IC4A.SER
- new net N$72: IC4A.QH*, IC5A.SER
- new net N$73: 3D2.PB6(XTAL1/TOSC1/PCINT6), C3.2, Q1.2
- new net N$77: 3D2.PB2(SS/OC1B/PCINT2)
- new net N$78: 1C14.1, 3D2.AREF
- new net N$87: IC6.(ADC6)PA6, IC6.(ADC7)PA7
- new net REG1: IC2A.SER
- new net RESET: ISP3.5
- new net RXP: 3D2.PD0(RXD/PCINT16)
- new net SCK: ISP3.3
- new net TXP: 3D2.PD1(TXD/PCINT17)
- new net VIN: D90.C, RN1A.1
- net +5V: now also 1C13.1, 3D2.AVCC, 3D2.VCC@1, 3D2.VCC@2, C11.2, C12.+, C13.1, IC2A.SCL, IC3A.SCL, IC4A.SCL, IC5A.SCL, ISP3.2, R3.2
- net GND: now also 1C13.2, 1C14.2, 3D2.AGND, 3D2.GND@1, 3D2.GND@2, C10.-, C11.1, C12.-, C13.2, C14.1, C22.1, C3.1, C4.1, D90.A, IC2A.G, IC3A.G, IC4A.G, IC5A.G, ISP3.6, RN1B.1, RN1C.1
- net HWB: now also RN1C.2
- net MISO0: now also 3D2.PB4(MISO/PCINT4)
- net MOSI0: now also 3D2.PB3(MOSI/OC2A/PCINT3)
- net RESET0: now also 3D2.PC6(/RESET/PCINT14), R3.1
- net SCK0: now also 3D2.PB5(SCK/PCINT5)
Other:
- note added: "#PWM 10bit"
- note added: "#PWM 16bit"
- note added: "#PWM 8/16bit"
- note added: "#PWM 8bit"
- note added: "#PWM Hi-Speed"
- note added: "+A10"
- note added: "+A11"
- note added: "+A6"
- note added: "+A7"
- note added: "+A8"
- note added: "+A9"
- note added: "+AIN0"
- note added: "+PWM COMPL IO10"
- note added: "-"
- note added: "0"
- note added: "10#"
- note added: "11#"
- note added: "17 февраля 2012"
- note added: "3#"
- note added: "31.03.2009"
- note added: "5#"
- note added: "6#"
- note added: "74hc165"
- note added: "9#"
- note added: "?out reset"
- note added: "ALT1"
- note added: "ALT2"
- note added: "ALT3"
- note added: "AvrUsb500v2"
- note added: "Bonio"
- note added: "FT232_MISO"
- note added: "FT232_MOSI"
- note added: "FT232_SCK"
- note added: "HVPP"
- note added: "IO"
- note added: "LED_TARGET"
- note added: "LED_active"
- note added: "LED_ready"
- note added: "PWM 16bit COMPL D6"
- note added: "Petka"
- note added: "RadioKot"
- note added: "TO ICSP"
- note added: "USB boot En"
- note added: "ano"
- note added: "blue"
- note added: "bs1"
- note added: "bs2"
- note added: "cp2102 rx"
- note added: "cp2102 suspend"
- note added: "cp2102 tx"
- note added: "d0"
- note added: "d4"
- note added: "d5 & isp"
- note added: "d6 & isp"
- note added: "d7 & isp"
- note added: "ft232 rx"
- note added: "ft232 tx"
- note added: "green"
- note added: "hw on"
- note added: "led green ready &"
- note added: "led red &"
- note added: "oe"
- note added: "out 1Mhz"
- note added: "out mhz"
- note added: "out miso"
- note added: "out reset"
- note added: "out sck"
- note added: "out_MOSI"
- note added: "pagel"
- note added: "rb"
- note added: "red"
- note added: "rst adc"
- note added: "rx"
- note added: "s1 boot"
- note added: "sw clk"
- note added: "sw trst"
- note added: "sw vtg"
- note added: "tx"
- note added: "vcc a out"
- note added: "vcc out"
- note added: "wr"
- note added: "xa0"
- note added: "xa1"
- note added: "делитель"
