File: PCB/keyBoard_A/keyBoard_A.sch (EAGLE design)
At the start: 252 parts, among them IC1 74HC04N, J1 J, J10 J, J11 J, J12 J, J13 J, J14 J, J15 J, J16 J, J17 J, J18 J, J19 J, J2 J, J20 J, J21 J, J22 J, J23 J, J24 J, J25 J, J26 J, J27 J, J28 J, J29 J, J3 J, J30 J, J31 J, J32 J, J33 J, J34 J, J35 J, J36 J, J37 J, J38 J, J39 J, J4 J, J40 J, J41 J, J42 J, J43 J, J44 J, J45 J, J5 J, J6 J, J7 J, J8 J, J9 J

Commit message: pcb a n>
Connections:
- removed net N$111: JA41.1, S41G$1.PIN-2
- removed net N$225: JA88.2
- new net N$65: JB41.2, S41G$1.PIN-2
- net 3: now also D88.C; no longer D19.C
- net 4: now also D19.C; no longer D20.C
- net 5: now also D20.C; no longer D21.C
- net 6: now also D21.C; no longer D22.C
- net 7: no longer D42.C
- net 7J: now also D22.C; no longer D23.C
- net 7J3: now also D42.C
- net 8: now also D23.C
- net L2: now also JA88.2; no longer JA24.2
- net L3: now also JA24.2; no longer JA30.2
- net L4: now also JA30.2
- net N$108: now also S38G$1.PIN-1; no longer S38G$1.PIN-2
- net N$109: now also S39G$1.PIN-1; no longer S39G$1.PIN-2
- net N$110: now also S40G$1.PIN-1; no longer S40G$1.PIN-2
- net N$42: now also S42G$1.PIN-2; no longer S42G$1.PIN-1
- net N$43: now also S42G$1.PIN-1; no longer S42G$1.PIN-2
- net N$75: now also JA41.1; no longer JB41.2
- net N$8: now also S38G$1.PIN-2; no longer S38G$1.PIN-1
- net N$80: now also S40G$1.PIN-2; no longer S40G$1.PIN-1
- net N$86: now also S39G$1.PIN-2; no longer S39G$1.PIN-1
Other:
- moved on the sheet: D19, D20, D21, D22, D23, D24, D30, D36, D37, D38, D39, D40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

Commit message: pcb a 2
Parts:
- added SV1: (no value), detali_main:FE03-1
Connections:
- removed net N$197: JA88.1, S88G$1.PIN-1
- new net N$111: JB88.2, S88G$1.PIN-1
- net 7: now also D22.C
- net 7J: no longer D22.C
- net D1: now also SV1.1; no longer SV3.10
- net D2: now also SV1.2; no longer SV3.11
- net D3: now also SV1.3; no longer SV3.12
- net N$117: now also JA88.1; no longer JB88.2
Changed lines of the file:
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@@
 <part name="JB88" library="detali" deviceset="SJ" device=""/>
 <part name="D88" library="detali" deviceset="LL4148" device=""/>
+<part name="SV1" library="detali_main" deviceset="FE03-1" device=""/>
 </parts>
 <sheets>
@@
 </instance>
 <instance part="S44A" gate="G$1" x="238.76" y="152.4"/>
-<instance part="S88" gate="G$1" x="127" y="269.24" rot="MR0"/>
+<instance part="S88" gate="G$1" x="127" y="269.24"/>
 <instance part="JA88" gate="1" x="139.7" y="269.24"/>
 <instance part="JB88" gate="1" x="114.3" y="269.24"/>
 <instance part="D88" gate="G$1" x="104.14" y="269.24"/>
+<instance part="SV1" gate="G$1" x="396.24" y="322.58" rot="MR0"/>
 </instances>
 <busses>
@@
 </segment>
 <segment>
-<pinref part="SV3" gate="G$1" pin="12"/>
-<wire x1="358.14" y1="322.58" x2="347.98" y2="322.58" width="0.1524" layer="91"/>
-<label x="353.06" y="322.58" size="1.778" layer="95"/>
+<pinref part="SV1" gate="G$1" pin="3"/>
+<wire x1="388.62" y1="322.58" x2="381" y2="322.58" width="0.1524" layer="91"/>
+<label x="383.54" y="322.58" size="1.778" layer="95"/>
 </segment>
 </net>
@@
 </segment>
 <segment>
-<pinref part="SV3" gate="G$1" pin="11"/>
-<wire x1="358.14" y1="320.04" x2="347.98" y2="320.04" width="0.1524" layer="91"/>
-<label x="353.06" y="320.04" size="1.778" layer="95"/>
+<pinref part="SV1" gate="G$1" pin="2"/>
+<wire x1="381" y1="320.04" x2="388.62" y2="320.04" width="0.1524" layer="91"/>
+<label x="383.54" y="320.04" size="1.778" layer="95"/>
 </segment>
 </net>
@@
 </segment>
 <segment>
-<pinref part="SV3" gate="G$1" pin="10"/>
-<wire x1="358.14" y1="317.5" x2="347.98" y2="317.5" width="0.1524" layer="91"/>
-<label x="353.06" y="317.5" size="1.778" layer="95"/>
+<pinref part="SV1" gate="G$1" pin="1"/>
+<wire x1="388.62" y1="317.5" x2="381" y2="317.5" width="0.1524" layer="91"/>
+<label x="383.54" y="317.5" size="1.778" layer="95"/>
 </segment>
 </net>
@@
 <label x="53.34" y="114.3" size="1.778" layer="95"/>
 </segment>
+<segment>
+<pinref part="D22" gate="G$1" pin="C"/>
+<wire x1="96.52" y1="228.6" x2="104.14" y2="228.6" width="0.1524" layer="91"/>
+<label x="99.06" y="228.6" size="1.778" layer="95"/>
+</segment>
 </net>
 <net name="7J" class="0">
@@
 <wire x1="114.3" y1="314.96" x2="149.86" y2="314.96" width="0.1524" layer="91"/>
 <label x="147.32" y="314.96" size="1.778" layer="95"/>
-</segment>
-<segment>
-<pinref part="D22" gate="G$1" pin="C"/>
-<wire x1="96.52" y1="228.6" x2="104.14" y2="228.6" width="0.1524" layer="91"/>
-<label x="99.06" y="228.6" size="1.778" layer="95"/>
 </segment>
 </net>
@@
 </segment>
 </net>
-<net name="N$117" class="0">
-<segment>
-<pinref part="JB88" gate="1" pin="2"/>
-<pinref part="S88" gate="G$1" pin="PIN-2"/>
-<wire x1="119.38" y1="269.24" x2="121.92" y2="269.24" width="0.1524" layer="91"/>
-</segment>
-</net>
-<net name="N$197" class="0">
-<segment>
-<pinref part="S88" gate="G$1" pin="PIN-1"/>
-<pinref part="JA88" gate="1" pin="1"/>
-<wire x1="132.08" y1="269.24" x2="134.62" y2="269.24" width="0.1524" layer="91"/>
-</segment>
-</net>
 <net name="N$196" class="0">
 <segment>
@@
 </segment>
 </net>
+<net name="N$111" class="0">
+<segment>
+<pinref part="JB88" gate="1" pin="2"/>
+<pinref part="S88" gate="G$1" pin="PIN-1"/>
+<wire x1="119.38" y1="269.24" x2="121.92" y2="269.24" width="0.1524" layer="91"/>
+</segment>
+</net>
+<net name="N$117" class="0">
+<segment>
+<pinref part="S88" gate="G$1" pin="PIN-2"/>
+<pinref part="JA88" gate="1" pin="1"/>
+<wire x1="132.08" y1="269.24" x2="134.62" y2="269.24" width="0.1524" layer="91"/>
+</segment>
+</net>

Commit message: pcb a 3
Parts:
- added J47, J48, J49: J, detali_main:J
- added SCROLL1: (no value), detali_main:LED5MM
- SV3: device detali_main:FE13-1 -> detali_main:FE08-1
Connections:
- new net L3J: J45.P$2, J49.P$1, JA5.2, JA6.2
- new net N$223: J47.P$1, J48.P$2
- new net N$224: J48.P$1, J49.P$2
- net +5V: now also SV3.8; no longer SV3.13
- net L3: now also J47.P$2; no longer J45.P$2, JA5.2, JA6.2
- net LED_CAPS: no longer SV3.8
- net LED_SCROLL: no longer SV3.9
- net N$195: now also SV3.5; no longer SV3.6
- net N$196: now also SV3.6; no longer SV3.5
Other:
- moved on the sheet: J45

Commit message: pcb a 4
Parts:
- removed CAPS, SCROLL, SCROLL1: (no value), detali_main:LED5MM
- removed J23: J, detali_main:J
- removed R3, R9: (no value), rcl:R-EU_R1206W
Connections:
- removed net LED_CAPS: R9.2
- removed net LED_SCROLL: R3.2
- removed net N$231: R3.1, SCROLL.A
- removed net N$232: CAPS.A, R9.1
- removed net N$60: 1D1A.Y6, J23.P$2
- net +5V: no longer CAPS.C, SCROLL.C
- net 8: now also 1D1A.Y6; no longer J23.P$1
- net N$49: now also S24G$1.PIN-2; no longer S24G$1.PIN-1
- net N$50: now also S24G$1.PIN-1; no longer S24G$1.PIN-2
Changed lines of the file:
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@@
 <part name="J20" library="detali_main" deviceset="J" device=""/>
 <part name="J21" library="detali_main" deviceset="J" device=""/>
-<part name="J23" library="detali_main" deviceset="J" device=""/>
 <part name="J24" library="detali_main" deviceset="J" device=""/>
 <part name="J25" library="detali_main" deviceset="J" device=""/>
@@
 <part name="GND19" library="supply1" deviceset="GND" device=""/>
 <part name="P+11" library="supply1" deviceset="+5V" device=""/>
-<part name="SCROLL" library="detali_main" deviceset="LED" device="5MM"/>
-<part name="CAPS" library="detali_main" deviceset="LED" device="5MM"/>
-<part name="P+12" library="supply1" deviceset="+5V" device=""/>
-<part name="R3" library="rcl" deviceset="R-EU_" device="R1206W"/>
-<part name="R9" library="rcl" deviceset="R-EU_" device="R1206W"/>
 <part name="R10" library="rcl" deviceset="R-EU_" device="M0805"/>
 <part name="R11" library="rcl" deviceset="R-EU_" device="M0805"/>
@@
 <part name="D88" library="detali" deviceset="LL4148" device=""/>
 <part name="SV1" library="detali_main" deviceset="FE03-1" device=""/>
-<part name="SCROLL1" library="detali_main" deviceset="LED" device="5MM"/>
 <part name="SV3" library="detali_main" deviceset="FE08-1" device=""/>
 <part name="J47" library="detali_main" deviceset="J" device=""/>
@@
 <instance part="S22" gate="G$1" x="129.54" y="228.6"/>
 <instance part="S23" gate="G$1" x="129.54" y="218.44"/>
-<instance part="S24" gate="G$1" x="187.96" y="218.44"/>
+<instance part="S24" gate="G$1" x="187.96" y="218.44" smashed="yes" rot="MR0">
+<attribute name="PART" x="193.04" y="215.9" size="1.27" layer="95" rot="MR0"/>
+<attribute name="VALUE" x="187.96" y="215.9" size="1.27" layer="96" rot="MR0"/>
+</instance>
 <instance part="S25" gate="G$1" x="187.96" y="269.24"/>
 <instance part="S26" gate="G$1" x="187.96" y="259.08"/>
@@
 <attribute name="NAME" x="195.58" y="111.76" size="1.27" layer="95"/>
 </instance>
-<instance part="J23" gate="G$1" x="129.54" y="312.42" smashed="yes">
-<attribute name="NAME" x="132.08" y="312.42" size="1.27" layer="95"/>
-</instance>
 <instance part="J24" gate="G$1" x="129.54" y="322.58" smashed="yes">
 <attribute name="NAME" x="132.08" y="322.58" size="1.27" layer="95"/>
@@
 <attribute name="VALUE" x="358.14" y="322.58" size="1.778" layer="96" rot="R180"/>
 </instance>
-<instance part="SCROLL" gate="G$1" x="287.02" y="198.12" rot="R270"/>
-<instance part="CAPS" gate="G$1" x="287.02" y="187.96" rot="R270"/>
-<instance part="P+12" gate="1" x="279.4" y="203.2" smashed="yes">
-<attribute name="VALUE" x="281.94" y="205.74" size="1.778" layer="96" rot="R180"/>
-</instance>
-<instance part="R3" gate="G$1" x="297.18" y="198.12"/>
-<instance part="R9" gate="G$1" x="297.18" y="187.96"/>
 <instance part="R10" gate="G$1" x="254" y="332.74"/>
 <instance part="R11" gate="G$1" x="254" y="322.58"/>
@@
 <instance part="D88" gate="G$1" x="104.14" y="269.24"/>
 <instance part="SV1" gate="G$1" x="396.24" y="322.58" rot="MR0"/>
-<instance part="SCROLL1" gate="G$1" x="294.64" y="210.82" rot="R270"/>
 <instance part="SV3" gate="G$1" x="365.76" y="302.26" rot="MR0"/>
 <instance part="J47" gate="G$1" x="55.88" y="101.6"/>
@@
 <wire x1="96.52" y1="297.18" x2="154.94" y2="297.18" width="0.762" layer="92"/>
 <wire x1="154.94" y1="297.18" x2="154.94" y2="132.08" width="0.762" layer="92"/>
-<wire x1="238.76" y1="335.28" x2="238.76" y2="271.78" width="0.762" layer="92"/>
 </segment>
 </bus>
@@
 <wire x1="355.6" y1="312.42" x2="355.6" y2="317.5" width="0.1524" layer="91"/>
 <pinref part="SV3" gate="G$1" pin="8"/>
-</segment>
-<segment>
-<pinref part="SCROLL" gate="G$1" pin="C"/>
-<wire x1="281.94" y1="198.12" x2="279.4" y2="198.12" width="0.1524" layer="91"/>
-<pinref part="P+12" gate="1" pin="+5V"/>
-<wire x1="279.4" y1="198.12" x2="279.4" y2="200.66" width="0.1524" layer="91"/>
-<pinref part="CAPS" gate="G$1" pin="C"/>
-<wire x1="281.94" y1="187.96" x2="279.4" y2="187.96" width="0.1524" layer="91"/>
-<wire x1="279.4" y1="187.96" x2="279.4" y2="198.12" width="0.1524" layer="91"/>
-<junction x="279.4" y="198.12"/>
 </segment>
 <segment>
@@
 </segment>
 </net>
-<net name="N$49" class="0">
-<segment>
-<pinref part="JB24" gate="1" pin="2"/>
-<pinref part="S24" gate="G$1" pin="PIN-1"/>
-<wire x1="180.34" y1="218.44" x2="182.88" y2="218.44" width="0.1524" layer="91"/>
-</segment>
-</net>
-<net name="N$50" class="0">
-<segment>
-<pinref part="S24" gate="G$1" pin="PIN-2"/>
-<pinref part="JA24" gate="1" pin="1"/>
-<wire x1="193.04" y1="218.44" x2="195.58" y2="218.44" width="0.1524" layer="91"/>
-</segment>
-</net>
 <net name="N$46" class="0">
 <segment>
@@
 </segment>
 <segment>
-<pinref part="J23" gate="G$1" pin="P$1"/>
-<wire x1="134.62" y1="312.42" x2="149.86" y2="312.42" width="0.1524" layer="91"/>
 <label x="147.32" y="312.42" size="1.778" layer="95"/>
+<pinref part="1D1" gate="A" pin="Y6"/>
+<wire x1="114.3" y1="312.42" x2="149.86" y2="312.42" width="0.1524" layer="91"/>
 </segment>
 <segment>
@@
 </segment>
 <segment>
-<wire x1="43.18" y1="101.6" x2="38.1" y2="101.6" width="0.1524" layer="91"/>
-<label x="38.1" y="101.6" size="1.778" layer="95"/>
-<wire x1="43.18" y1="101.6" x2="45.72" y2="99.06" width="0.1524" layer="91"/>
+<wire x1="53.34" y1="101.6" x2="48.26" y2="101.6" width="0.1524" layer="91"/>
+<label x="48.26" y="101.6" size="1.778" layer="95"/>
 <pinref part="J47" gate="G$1" pin="P$2"/>
-<wire x1="50.8" y1="101.6" x2="53.34" y2="101.6" width="0.1524" layer="91"/>
-<wire x1="45.72" y1="99.06" x2="50.8" y2="101.6" width="0.1524" layer="91"/>
 </segment>
 </net>
@@
 </segment>
 </net>
-<net name="N$60" class="0">
-<segment>
-<pinref part="1D1" gate="A" pin="Y6"/>
-<pinref part="J23" gate="G$1" pin="P$2"/>
-<wire x1="114.3" y1="312.42" x2="127" y2="312.42" width="0.1524" layer="91"/>
-</segment>
-</net>
 <net name="N$67" class="0">
 <segment>
@@
 <segment>
 <pinref part="R11" gate="G$1" pin="2"/>
-<wire x1="266.7" y1="322.58" x2="259.08" y2="322.58" width="0.1524" layer="91"/>
-<label x="261.62" y="322.58" size="1.778" layer="95"/>
+<wire x1="264.16" y1="322.58" x2="259.08" y2="322.58" width="0.1524" layer="91"/>
+<label x="264.16" y="322.58" size="1.778" layer="95" rot="R90"/>
 </segment>
 </net>
@@
 <segment>
 <pinref part="R12" gate="G$1" pin="2"/>
-<wire x1="266.7" y1="309.88" x2="259.08" y2="309.88" width="0.1524" layer="91"/>
-<label x="261.62" y="309.88" size="1.778" layer="95"/>
+<wire x1="264.16" y1="309.88" x2="259.08" y2="309.88" width="0.1524" layer="91"/>
+<label x="264.16" y="309.88" size="1.778" layer="95" rot="R90"/>
 </segment>
 </net>
@@
 </segment>
 </net>
-<net name="N$231" class="0">
-<segment>
-<pinref part="SCROLL" gate="G$1" pin="A"/>
-<pinref part="R3" gate="G$1" pin="1"/>
-<wire x1="289.56" y1="198.12" x2="292.1" y2="198.12" width="0.1524" layer="91"/>
-</segment>
-</net>
-<net name="N$232" class="0">
-<segment>
-<pinref part="CAPS" gate="G$1" pin="A"/>
-<pinref part="R9" gate="G$1" pin="1"/>
-<wire x1="289.56" y1="187.96" x2="292.1" y2="187.96" width="0.1524" layer="91"/>
-</segment>
-</net>
 <net name="LED_SCROLL" class="0">
-<segment>
-<pinref part="R3" gate="G$1" pin="2"/>
-<wire x1="302.26" y1="198.12" x2="309.88" y2="198.12" width="0.1524" layer="91"/>
-<label x="302.26" y="198.12" size="1.778" layer="95"/>
-</segment>
 <segment>
 <label x="383.54" y="342.9" size="1.778" layer="95"/>
@@
 </net>
 <net name="LED_CAPS" class="0">
-<segment>
-<pinref part="R9" gate="G$1" pin="2"/>
-<wire x1="302.26" y1="187.96" x2="309.88" y2="187.96" width="0.1524" layer="91"/>
-<label x="302.26" y="187.96" size="1.778" layer="95"/>
-</segment>
 <segment>
 <label x="383.54" y="340.36" size="1.778" layer="95"/>
@@
 </segment>
 <segment>
-<wire x1="269.24" y1="304.8" x2="276.86" y2="309.88" width="0.1524" layer="91"/>
-<label x="269.24" y="307.34" size="1.778" layer="95"/>
+<wire x1="269.24" y1="309.88" x2="276.86" y2="309.88" width="0.1524" layer="91"/>
+<label x="269.24" y="309.88" size="1.778" layer="95"/>
 <pinref part="J45" gate="G$1" pin="P$2"/>
 </segment>
@@
 </segment>
 </net>
+<net name="N$49" class="0">
+<segment>
+<pinref part="S24" gate="G$1" pin="PIN-2"/>
+<pinref part="JB24" gate="1" pin="2"/>
+<wire x1="182.88" y1="218.44" x2="180.34" y2="218.44" width="0.1524" layer="91"/>
+</segment>
+</net>
+<net name="N$50" class="0">
+<segment>
+<pinref part="S24" gate="G$1" pin="PIN-1"/>
+<pinref part="JA24" gate="1" pin="1"/>
+<wire x1="193.04" y1="218.44" x2="195.58" y2="218.44" width="0.1524" layer="91"/>
+</segment>
+</net>
