File: PCB/keyBoard_A/keyBoard_A.sch (EAGLE design)
At the start: 251 parts, among them IC1 74HC04N, J1 J, J10 J, J11 J, J12 J, J13 J, J14 J, J15 J, J16 J, J17 J, J18 J, J19 J, J2 J, J20 J, J21 J, J22 J, J24 J, J25 J, J26 J, J27 J, J28 J, J29 J, J3 J, J30 J, J31 J, J32 J, J33 J, J34 J, J35 J, J36 J, J37 J, J38 J, J39 J, J4 J, J40 J, J41 J, J42 J, J43 J, J44 J, J45 J, J47 J, J48 J, J49 J, J5 J, J6 J, J7 J, J8 J, J9 J

Commit message: sw ls
Parts:
- R10, R12: value (none) -> 10k; device rcl:R-EU_M0805 -> rd:RD
Connections:
- net +5V: now also R10.T, R12.T; no longer R10.1, R12.1
- net L1: now also IC1E.I, R10.B; no longer IC1D.I, R10.2
- net L4: now also IC1D.I; no longer IC1C.I
- net N$193: now also IC1C.I, R12.B; no longer IC1E.I, R12.2
- net N$196: now also IC1C.O; no longer IC1E.O
- net N$200: now also IC1D.O; no longer IC1C.O
- net N$203: now also IC1E.O; no longer IC1D.O
Other:
- moved on the sheet: IC1C, IC1D, IC1E, J47, J48, J49, S44A
Changed lines of the file:
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@@
 <part name="GND19" library="supply1" deviceset="GND" device=""/>
 <part name="P+11" library="supply1" deviceset="+5V" device=""/>
-<part name="R10" library="rcl" deviceset="R-EU_" device="M0805"/>
 <part name="R11" library="rcl" deviceset="R-EU_" device="M0805"/>
-<part name="R12" library="rcl" deviceset="R-EU_" device="M0805"/>
 <part name="R13" library="rcl" deviceset="R-EU_" device="M0805"/>
 <part name="R14" library="rcl" deviceset="R-EU_" device="M0805"/>
@@
 <part name="J48" library="detali_main" deviceset="J" device=""/>
 <part name="J49" library="detali_main" deviceset="J" device=""/>
+<part name="R10" library="rd" deviceset="RD" device="" value="10k"/>
+<part name="R12" library="rd" deviceset="RD" device="" value="10k"/>
 </parts>
 <sheets>
@@
 </instance>
 <instance part="C17" gate="G$1" x="185.42" y="314.96" rot="MR180"/>
-<instance part="IC1" gate="D" x="302.26" y="335.28"/>
+<instance part="IC1" gate="E" x="302.26" y="335.28"/>
 <instance part="IC1" gate="F" x="302.26" y="322.58"/>
-<instance part="IC1" gate="E" x="302.26" y="309.88"/>
-<instance part="IC1" gate="C" x="302.26" y="297.18"/>
+<instance part="IC1" gate="C" x="302.26" y="309.88"/>
+<instance part="IC1" gate="D" x="302.26" y="297.18"/>
 <instance part="IC1" gate="B" x="302.26" y="284.48"/>
 <instance part="IC1" gate="A" x="302.26" y="271.78"/>
@@
 <attribute name="VALUE" x="358.14" y="322.58" size="1.778" layer="96" rot="R180"/>
 </instance>
-<instance part="R10" gate="G$1" x="254" y="332.74"/>
 <instance part="R11" gate="G$1" x="254" y="322.58"/>
-<instance part="R12" gate="G$1" x="254" y="309.88"/>
 <instance part="R13" gate="G$1" x="254" y="297.18"/>
 <instance part="R14" gate="G$1" x="254" y="284.48"/>
@@
 <attribute name="VALUE" x="248.92" y="340.36" size="1.778" layer="96" rot="R180"/>
 </instance>
-<instance part="S44A" gate="G$1" x="238.76" y="152.4"/>
+<instance part="S44A" gate="G$1" x="129.54" y="203.2"/>
 <instance part="S88" gate="G$1" x="127" y="269.24"/>
 <instance part="JA88" gate="1" x="139.7" y="269.24"/>
@@
 <instance part="SV1" gate="G$1" x="396.24" y="322.58" rot="MR0"/>
 <instance part="SV3" gate="G$1" x="365.76" y="302.26" rot="MR0"/>
-<instance part="J47" gate="G$1" x="55.88" y="101.6"/>
-<instance part="J48" gate="G$1" x="66.04" y="101.6"/>
-<instance part="J49" gate="G$1" x="76.2" y="101.6"/>
+<instance part="J47" gate="G$1" x="45.72" y="104.14"/>
+<instance part="J48" gate="G$1" x="55.88" y="104.14"/>
+<instance part="J49" gate="G$1" x="66.04" y="104.14"/>
+<instance part="R10" gate="G$1" x="254" y="332.74" smashed="yes">
+<attribute name="NAME" x="250.19" y="336.55" size="1.778" layer="95"/>
+<attribute name="VALUE" x="252.73" y="327.66" size="1.778" layer="95"/>
+</instance>
+<instance part="R12" gate="G$1" x="254" y="309.88" smashed="yes">
+<attribute name="NAME" x="250.19" y="313.69" size="1.778" layer="95"/>
+<attribute name="VALUE" x="252.73" y="304.8" size="1.778" layer="95"/>
+</instance>
 </instances>
 <busses>
@@
 <segment>
 <pinref part="S44A" gate="G$1" pin="PIN-1"/>
-<wire x1="233.68" y1="152.4" x2="228.6" y2="152.4" width="0.1524" layer="91"/>
-<label x="231.14" y="152.4" size="1.778" layer="95" rot="R90"/>
+<wire x1="124.46" y1="203.2" x2="119.38" y2="203.2" width="0.1524" layer="91"/>
+<label x="121.92" y="203.2" size="1.778" layer="95" rot="R90"/>
 </segment>
 </net>
@@
 <segment>
 <pinref part="S44A" gate="G$1" pin="PIN-2"/>
-<wire x1="243.84" y1="152.4" x2="248.92" y2="152.4" width="0.1524" layer="91"/>
-<label x="246.38" y="152.4" size="1.778" layer="95" rot="R90"/>
+<wire x1="134.62" y1="203.2" x2="139.7" y2="203.2" width="0.1524" layer="91"/>
+<label x="137.16" y="203.2" size="1.778" layer="95" rot="R90"/>
 </segment>
 </net>
@@
 </segment>
 <segment>
-<pinref part="R10" gate="G$1" pin="1"/>
 <wire x1="248.92" y1="332.74" x2="246.38" y2="332.74" width="0.1524" layer="91"/>
 <wire x1="246.38" y1="332.74" x2="246.38" y2="322.58" width="0.1524" layer="91"/>
@@
 <wire x1="246.38" y1="322.58" x2="248.92" y2="322.58" width="0.1524" layer="91"/>
 <wire x1="246.38" y1="322.58" x2="246.38" y2="309.88" width="0.1524" layer="91"/>
-<pinref part="R12" gate="G$1" pin="1"/>
 <wire x1="246.38" y1="309.88" x2="248.92" y2="309.88" width="0.1524" layer="91"/>
 <wire x1="246.38" y1="309.88" x2="246.38" y2="297.18" width="0.1524" layer="91"/>
@@
 <junction x="246.38" y="297.18"/>
 <junction x="246.38" y="284.48"/>
+<pinref part="R10" gate="G$1" pin="T"/>
+<pinref part="R12" gate="G$1" pin="T"/>
 </segment>
 </net>
@@
 </segment>
 <segment>
-<pinref part="IC1" gate="D" pin="I"/>
+<pinref part="IC1" gate="E" pin="I"/>
 <wire x1="266.7" y1="335.28" x2="292.1" y2="335.28" width="0.1524" layer="91"/>
 <label x="266.7" y="335.28" size="1.778" layer="95"/>
 </segment>
 <segment>
-<pinref part="R10" gate="G$1" pin="2"/>
 <wire x1="266.7" y1="332.74" x2="259.08" y2="332.74" width="0.1524" layer="91"/>
 <label x="261.62" y="332.74" size="1.778" layer="95"/>
+<pinref part="R10" gate="G$1" pin="B"/>
 </segment>
 </net>
@@
 </segment>
 <segment>
-<wire x1="53.34" y1="101.6" x2="48.26" y2="101.6" width="0.1524" layer="91"/>
-<label x="48.26" y="101.6" size="1.778" layer="95"/>
+<wire x1="43.18" y1="104.14" x2="38.1" y2="104.14" width="0.1524" layer="91"/>
+<label x="38.1" y="104.14" size="1.778" layer="95"/>
 <pinref part="J47" gate="G$1" pin="P$2"/>
 </segment>
@@
 </segment>
 <segment>
-<pinref part="IC1" gate="C" pin="I"/>
+<pinref part="IC1" gate="D" pin="I"/>
 <wire x1="266.7" y1="297.18" x2="292.1" y2="297.18" width="0.1524" layer="91"/>
 <label x="269.24" y="297.18" size="1.778" layer="95"/>
@@
 <net name="N$200" class="0">
 <segment>
-<pinref part="IC1" gate="C" pin="O"/>
+<pinref part="IC1" gate="D" pin="O"/>
 <wire x1="337.82" y1="302.26" x2="337.82" y2="297.18" width="0.1524" layer="91"/>
 <wire x1="337.82" y1="297.18" x2="312.42" y2="297.18" width="0.1524" layer="91"/>
@@
 <net name="N$203" class="0">
 <segment>
-<pinref part="IC1" gate="D" pin="O"/>
+<pinref part="IC1" gate="E" pin="O"/>
 <wire x1="340.36" y1="309.88" x2="340.36" y2="335.28" width="0.1524" layer="91"/>
 <wire x1="340.36" y1="335.28" x2="312.42" y2="335.28" width="0.1524" layer="91"/>
@@
 <segment>
 <pinref part="J45" gate="G$1" pin="P$1"/>
-<pinref part="IC1" gate="E" pin="I"/>
+<pinref part="IC1" gate="C" pin="I"/>
 <wire x1="284.48" y1="309.88" x2="292.1" y2="309.88" width="0.1524" layer="91"/>
 <label x="287.02" y="309.88" size="1.778" layer="95" rot="R90"/>
 </segment>
 <segment>
-<pinref part="R12" gate="G$1" pin="2"/>
 <wire x1="264.16" y1="309.88" x2="259.08" y2="309.88" width="0.1524" layer="91"/>
 <label x="264.16" y="309.88" size="1.778" layer="95" rot="R90"/>
+<pinref part="R12" gate="G$1" pin="B"/>
 </segment>
 </net>
@@
 <net name="N$196" class="0">
 <segment>
-<pinref part="IC1" gate="E" pin="O"/>
+<pinref part="IC1" gate="C" pin="O"/>
 <wire x1="312.42" y1="309.88" x2="332.74" y2="309.88" width="0.1524" layer="91"/>
 <wire x1="332.74" y1="309.88" x2="332.74" y2="304.8" width="0.1524" layer="91"/>
@@
 <segment>
 <pinref part="J49" gate="G$1" pin="P$1"/>
-<wire x1="81.28" y1="101.6" x2="86.36" y2="101.6" width="0.1524" layer="91"/>
-<label x="81.28" y="101.6" size="1.778" layer="95"/>
+<wire x1="71.12" y1="104.14" x2="76.2" y2="104.14" width="0.1524" layer="91"/>
+<label x="71.12" y="104.14" size="1.778" layer="95"/>
 </segment>
 </net>
@@
 <pinref part="J47" gate="G$1" pin="P$1"/>
 <pinref part="J48" gate="G$1" pin="P$2"/>
-<wire x1="60.96" y1="101.6" x2="63.5" y2="101.6" width="0.1524" layer="91"/>
+<wire x1="50.8" y1="104.14" x2="53.34" y2="104.14" width="0.1524" layer="91"/>
 </segment>
 </net>
@@
 <pinref part="J49" gate="G$1" pin="P$2"/>
 <pinref part="J48" gate="G$1" pin="P$1"/>
-<wire x1="73.66" y1="101.6" x2="71.12" y2="101.6" width="0.1524" layer="91"/>
-</segment>
-</net>
+<wire x1="63.5" y1="104.14" x2="60.96" y2="104.14" width="0.1524" layer="91"/>
+</segment>
+</net>

Commit message: sw ls
Connections:
- removed net N$196 (its old number): IC1C.O, SV3.6
- removed net N$198 (its old number): IC1A.O, SV3.2
- new net N$195: IC1A.O, SV3.4
- new net N$199: IC1C.O, SV3.2
- net L5: now also IC1C.I; no longer IC1B.I
- net L6: now also IC1B.I; no longer IC1A.I
- net N$193: now also IC1F.I; no longer IC1C.I
- net N$194: now also IC1A.I; no longer IC1F.I
- net N$200: now also SV3.7; no longer SV3.4
- net N$203: now also SV3.6; no longer SV3.7
Other:
- moved on the sheet: IC1A, IC1B, IC1C, IC1F, SV3
Changed lines of the file:
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@@
 <plain>
 <text x="398.78" y="317.5" size="1.778" layer="91">d1</text>
-<text x="368.3" y="312.42" size="1.778" layer="91">vcc</text>
+<text x="378.46" y="312.42" size="1.778" layer="91">vcc</text>
 <text x="398.78" y="320.04" size="1.778" layer="91">d2</text>
 <text x="398.78" y="322.58" size="1.778" layer="91">d3</text>
-<text x="368.3" y="294.64" size="1.778" layer="91">gnd</text>
+<text x="378.46" y="294.64" size="1.778" layer="91">gnd</text>
 <text x="40.64" y="304.8" size="5.08" layer="91">LEFT KB</text>
 </plain>
@@
 <instance part="C17" gate="G$1" x="185.42" y="314.96" rot="MR180"/>
 <instance part="IC1" gate="E" x="302.26" y="335.28"/>
-<instance part="IC1" gate="F" x="302.26" y="322.58"/>
-<instance part="IC1" gate="C" x="302.26" y="309.88"/>
+<instance part="IC1" gate="A" x="302.26" y="322.58"/>
+<instance part="IC1" gate="F" x="302.26" y="309.88"/>
 <instance part="IC1" gate="D" x="302.26" y="297.18"/>
-<instance part="IC1" gate="B" x="302.26" y="284.48"/>
-<instance part="IC1" gate="A" x="302.26" y="271.78"/>
+<instance part="IC1" gate="C" x="302.26" y="284.48"/>
+<instance part="IC1" gate="B" x="302.26" y="271.78"/>
 <instance part="IC1" gate="P" x="274.32" y="226.06"/>
 <instance part="J1" gate="G$1" x="45.72" y="119.38"/>
@@
 <instance part="D88" gate="G$1" x="104.14" y="269.24"/>
 <instance part="SV1" gate="G$1" x="396.24" y="322.58" rot="MR0"/>
-<instance part="SV3" gate="G$1" x="365.76" y="302.26" rot="MR0"/>
+<instance part="SV3" gate="G$1" x="370.84" y="302.26" rot="MR0"/>
 <instance part="J47" gate="G$1" x="45.72" y="104.14"/>
 <instance part="J48" gate="G$1" x="55.88" y="104.14"/>
@@
 <segment>
 <pinref part="P+11" gate="1" pin="+5V"/>
-<wire x1="358.14" y1="312.42" x2="355.6" y2="312.42" width="0.1524" layer="91"/>
+<wire x1="363.22" y1="312.42" x2="355.6" y2="312.42" width="0.1524" layer="91"/>
 <wire x1="355.6" y1="312.42" x2="355.6" y2="317.5" width="0.1524" layer="91"/>
 <pinref part="SV3" gate="G$1" pin="8"/>
@@
 <pinref part="GND19" gate="1" pin="GND"/>
 <wire x1="355.6" y1="292.1" x2="355.6" y2="294.64" width="0.1524" layer="91"/>
-<wire x1="355.6" y1="294.64" x2="358.14" y2="294.64" width="0.1524" layer="91"/>
+<wire x1="355.6" y1="294.64" x2="363.22" y2="294.64" width="0.1524" layer="91"/>
 <pinref part="SV3" gate="G$1" pin="1"/>
 </segment>
@@
 </segment>
 <segment>
-<pinref part="IC1" gate="B" pin="I"/>
+<pinref part="IC1" gate="C" pin="I"/>
 <wire x1="266.7" y1="284.48" x2="292.1" y2="284.48" width="0.1524" layer="91"/>
 <label x="269.24" y="284.48" size="1.778" layer="95"/>
@@
 </segment>
 <segment>
-<pinref part="IC1" gate="A" pin="I"/>
+<pinref part="IC1" gate="B" pin="I"/>
 <wire x1="266.7" y1="271.78" x2="292.1" y2="271.78" width="0.1524" layer="91"/>
 <label x="269.24" y="271.78" size="1.778" layer="95"/>
@@
 <net name="N$198" class="0">
 <segment>
-<pinref part="IC1" gate="A" pin="O"/>
+<pinref part="IC1" gate="B" pin="O"/>
 <wire x1="342.9" y1="297.18" x2="342.9" y2="271.78" width="0.1524" layer="91"/>
 <wire x1="342.9" y1="271.78" x2="312.42" y2="271.78" width="0.1524" layer="91"/>
-<wire x1="358.14" y1="297.18" x2="342.9" y2="297.18" width="0.1524" layer="91"/>
-<pinref part="SV3" gate="G$1" pin="2"/>
 <label x="342.9" y="297.18" size="1.778" layer="95"/>
+<wire x1="355.6" y1="297.18" x2="342.9" y2="297.18" width="0.1524" layer="91"/>
+<pinref part="SV3" gate="G$1" pin="3"/>
+<wire x1="355.6" y1="297.18" x2="363.22" y2="299.72" width="0.1524" layer="91"/>
 </segment>
 </net>
 <net name="N$199" class="0">
 <segment>
-<pinref part="IC1" gate="B" pin="O"/>
+<pinref part="IC1" gate="C" pin="O"/>
 <wire x1="340.36" y1="299.72" x2="340.36" y2="284.48" width="0.1524" layer="91"/>
 <wire x1="340.36" y1="284.48" x2="312.42" y2="284.48" width="0.1524" layer="91"/>
-<wire x1="358.14" y1="299.72" x2="340.36" y2="299.72" width="0.1524" layer="91"/>
-<pinref part="SV3" gate="G$1" pin="3"/>
 <label x="342.9" y="299.72" size="1.778" layer="95"/>
+<wire x1="355.6" y1="299.72" x2="340.36" y2="299.72" width="0.1524" layer="91"/>
+<pinref part="SV3" gate="G$1" pin="2"/>
+<wire x1="363.22" y1="297.18" x2="355.6" y2="299.72" width="0.1524" layer="91"/>
 </segment>
 </net>
@@
 <wire x1="337.82" y1="302.26" x2="337.82" y2="297.18" width="0.1524" layer="91"/>
 <wire x1="337.82" y1="297.18" x2="312.42" y2="297.18" width="0.1524" layer="91"/>
-<wire x1="358.14" y1="302.26" x2="337.82" y2="302.26" width="0.1524" layer="91"/>
-<pinref part="SV3" gate="G$1" pin="4"/>
 <label x="342.9" y="302.26" size="1.778" layer="95"/>
+<wire x1="355.6" y1="302.26" x2="337.82" y2="302.26" width="0.1524" layer="91"/>
+<pinref part="SV3" gate="G$1" pin="7"/>
+<wire x1="355.6" y1="302.26" x2="363.22" y2="309.88" width="0.1524" layer="91"/>
 </segment>
 </net>
@@
 <wire x1="340.36" y1="309.88" x2="340.36" y2="335.28" width="0.1524" layer="91"/>
 <wire x1="340.36" y1="335.28" x2="312.42" y2="335.28" width="0.1524" layer="91"/>
-<wire x1="340.36" y1="309.88" x2="358.14" y2="309.88" width="0.1524" layer="91"/>
-<pinref part="SV3" gate="G$1" pin="7"/>
+<wire x1="340.36" y1="309.88" x2="355.6" y2="309.88" width="0.1524" layer="91"/>
 <label x="342.9" y="309.88" size="1.778" layer="95"/>
+<pinref part="SV3" gate="G$1" pin="6"/>
+<wire x1="363.22" y1="307.34" x2="355.6" y2="309.88" width="0.1524" layer="91"/>
 </segment>
 </net>
@@
 <segment>
 <pinref part="J45" gate="G$1" pin="P$1"/>
-<pinref part="IC1" gate="C" pin="I"/>
+<pinref part="IC1" gate="F" pin="I"/>
 <wire x1="284.48" y1="309.88" x2="292.1" y2="309.88" width="0.1524" layer="91"/>
 <label x="287.02" y="309.88" size="1.778" layer="95" rot="R90"/>
@@
 <segment>
 <pinref part="J44" gate="G$1" pin="P$1"/>
-<pinref part="IC1" gate="F" pin="I"/>
+<pinref part="IC1" gate="A" pin="I"/>
 <wire x1="289.56" y1="322.58" x2="292.1" y2="322.58" width="0.1524" layer="91"/>
 </segment>
@@
 <net name="N$195" class="0">
 <segment>
-<pinref part="IC1" gate="F" pin="O"/>
+<pinref part="IC1" gate="A" pin="O"/>
 <wire x1="337.82" y1="307.34" x2="337.82" y2="322.58" width="0.1524" layer="91"/>
 <wire x1="337.82" y1="322.58" x2="312.42" y2="322.58" width="0.1524" layer="91"/>
 <wire x1="337.82" y1="307.34" x2="353.06" y2="307.34" width="0.1524" layer="91"/>
 <label x="342.9" y="307.34" size="1.778" layer="95"/>
-<pinref part="SV3" gate="G$1" pin="5"/>
-<wire x1="358.14" y1="304.8" x2="355.6" y2="304.8" width="0.1524" layer="91"/>
-<wire x1="355.6" y1="304.8" x2="353.06" y2="307.34" width="0.1524" layer="91"/>
+<pinref part="SV3" gate="G$1" pin="4"/>
+<wire x1="363.22" y1="302.26" x2="353.06" y2="307.34" width="0.1524" layer="91"/>
 </segment>
 </net>
@@
 <net name="N$196" class="0">
 <segment>
-<pinref part="IC1" gate="C" pin="O"/>
+<pinref part="IC1" gate="F" pin="O"/>
 <wire x1="312.42" y1="309.88" x2="332.74" y2="309.88" width="0.1524" layer="91"/>
 <wire x1="332.74" y1="309.88" x2="332.74" y2="304.8" width="0.1524" layer="91"/>
-<wire x1="332.74" y1="304.8" x2="353.06" y2="304.8" width="0.1524" layer="91"/>
+<wire x1="332.74" y1="304.8" x2="363.22" y2="304.8" width="0.1524" layer="91"/>
 <label x="342.9" y="304.8" size="1.778" layer="95"/>
-<pinref part="SV3" gate="G$1" pin="6"/>
-<wire x1="358.14" y1="307.34" x2="355.6" y2="307.34" width="0.1524" layer="91"/>
-<wire x1="355.6" y1="307.34" x2="353.06" y2="304.8" width="0.1524" layer="91"/>
-</segment>
-</net>
+<pinref part="SV3" gate="G$1" pin="5"/>
+</segment>
+</net>

Commit message: sw s10
Parts:
- removed J18: J, detali_main:J
Connections:
- removed net 2J3: D37.C, D9.C, J18.P$2
- net 2J2: now also D37.C, D9.C; no longer J18.P$1
- net N$13: now also S10G$1.PIN-2; no longer S10G$1.PIN-1
- net N$28: now also S10G$1.PIN-1; no longer S10G$1.PIN-2
Changed lines of the file:
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@@
 <part name="J16" library="detali_main" deviceset="J" device=""/>
 <part name="J17" library="detali_main" deviceset="J" device=""/>
-<part name="J18" library="detali_main" deviceset="J" device=""/>
 <part name="J19" library="detali_main" deviceset="J" device=""/>
 <part name="J20" library="detali_main" deviceset="J" device=""/>
@@
 <instance part="S8" gate="G$1" x="71.12" y="193.04"/>
 <instance part="S9" gate="G$1" x="187.96" y="193.04"/>
-<instance part="S10" gate="G$1" x="187.96" y="203.2"/>
+<instance part="S10" gate="G$1" x="187.96" y="203.2" rot="MR0"/>
 <instance part="S11" gate="G$1" x="187.96" y="182.88"/>
 <instance part="S12" gate="G$1" x="187.96" y="172.72"/>
@@
 <attribute name="NAME" x="170.18" y="116.84" size="1.27" layer="95"/>
 </instance>
-<instance part="J18" gate="G$1" x="172.72" y="109.22" smashed="yes">
-<attribute name="NAME" x="170.18" y="111.76" size="1.27" layer="95"/>
-</instance>
 <instance part="J19" gate="G$1" x="198.12" y="119.38" smashed="yes">
 <attribute name="NAME" x="195.58" y="121.92" size="1.27" layer="95"/>
@@
 </segment>
 </net>
-<net name="N$13" class="0">
-<segment>
-<pinref part="JB10" gate="1" pin="2"/>
-<pinref part="S10" gate="G$1" pin="PIN-1"/>
-<wire x1="180.34" y1="203.2" x2="182.88" y2="203.2" width="0.1524" layer="91"/>
-</segment>
-</net>
 <net name="N$25" class="0">
 <segment>
@@
 <wire x1="180.34" y1="172.72" x2="182.88" y2="172.72" width="0.1524" layer="91"/>
 <pinref part="JB12" gate="1" pin="2"/>
-</segment>
-</net>
-<net name="N$28" class="0">
-<segment>
-<pinref part="S10" gate="G$1" pin="PIN-2"/>
-<pinref part="JA10" gate="1" pin="1"/>
-<wire x1="193.04" y1="203.2" x2="195.58" y2="203.2" width="0.1524" layer="91"/>
 </segment>
 </net>
@@
 </segment>
 <segment>
-<pinref part="J18" gate="G$1" pin="P$1"/>
-<wire x1="177.8" y1="109.22" x2="182.88" y2="109.22" width="0.1524" layer="91"/>
-<label x="180.34" y="109.22" size="1.778" layer="95"/>
-</segment>
-<segment>
 <pinref part="D8" gate="G$1" pin="C"/>
 <wire x1="38.1" y1="193.04" x2="45.72" y2="193.04" width="0.1524" layer="91"/>
 <label x="40.64" y="193.04" size="1.778" layer="95"/>
 </segment>
-</net>
-<net name="2J3" class="0">
-<segment>
-<pinref part="J18" gate="G$1" pin="P$2"/>
-<wire x1="170.18" y1="109.22" x2="165.1" y2="109.22" width="0.1524" layer="91"/>
-<label x="165.1" y="109.22" size="1.778" layer="95"/>
+<segment>
+<pinref part="D37" gate="G$1" pin="C"/>
+<wire x1="96.52" y1="193.04" x2="104.14" y2="193.04" width="0.1524" layer="91"/>
+<label x="99.06" y="193.04" size="1.778" layer="95"/>
 </segment>
 <segment>
@@
 <wire x1="154.94" y1="193.04" x2="162.56" y2="193.04" width="0.1524" layer="91"/>
 <label x="157.48" y="193.04" size="1.778" layer="95"/>
-</segment>
-<segment>
-<pinref part="D37" gate="G$1" pin="C"/>
-<wire x1="96.52" y1="193.04" x2="104.14" y2="193.04" width="0.1524" layer="91"/>
-<label x="99.06" y="193.04" size="1.778" layer="95"/>
 </segment>
 </net>
@@
 </segment>
 </net>
+<net name="N$13" class="0">
+<segment>
+<pinref part="JB10" gate="1" pin="2"/>
+<pinref part="S10" gate="G$1" pin="PIN-2"/>
+<wire x1="180.34" y1="203.2" x2="182.88" y2="203.2" width="0.1524" layer="91"/>
+</segment>
+</net>
+<net name="N$28" class="0">
+<segment>
+<pinref part="S10" gate="G$1" pin="PIN-1"/>
+<pinref part="JA10" gate="1" pin="1"/>
+<wire x1="193.04" y1="203.2" x2="195.58" y2="203.2" width="0.1524" layer="91"/>
+</segment>
+</net>
