File: PCB/keyBoard_A/keyBoard_A.sch (EAGLE design)
At the start: 250 parts, among them IC1 74HC04N, J1 J, J10 J, J11 J, J12 J, J13 J, J14 J, J15 J, J16 J, J17 J, J19 J, J2 J, J20 J, J21 J, J22 J, J24 J, J25 J, J26 J, J27 J, J28 J, J29 J, J3 J, J30 J, J31 J, J32 J, J33 J, J34 J, J35 J, J36 J, J37 J, J38 J, J39 J, J4 J, J40 J, J41 J, J42 J, J43 J, J44 J, J45 J, J47 J, J48 J, J49 J, J5 J, J6 J, J7 J, J8 J, J9 J

Commit message: .
Parts:
- added J18: J, detali_main:J
- added R4: (no value), rcl:R-EU_R0603
- added SV2: (no value), detali_main:FE03-1
Connections:
- new net N$60: IC1D.O, J18.P$2
- net N$19: now also S3G$1.PIN-2; no longer S3G$1.PIN-1
- net N$2: now also S4G$1.PIN-2; no longer S4G$1.PIN-1
- net N$200: now also J18.P$1; no longer IC1D.O
- net N$32: now also S3G$1.PIN-1; no longer S3G$1.PIN-2
- net N$4: now also S4G$1.PIN-1; no longer S4G$1.PIN-2
Changed lines of the file:
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@@
 <clearance class="1" value="0.254"/>
 </class>
-<class number="2" name="gnd" width="0.254" drill="0.6096">
+<class number="2" name="gnd" width="0.3048" drill="0.5588">
 <clearance class="2" value="0.254"/>
 </class>
@@
 <part name="R10" library="rd" deviceset="RD" device="" value="10k"/>
 <part name="R12" library="rd" deviceset="RD" device="" value="10k"/>
+<part name="SV2" library="detali_main" deviceset="FE03-1" device="">
+<attribute name="MF" value=""/>
+<attribute name="MPN" value=""/>
+<attribute name="OC_FARNELL" value="unknown"/>
+<attribute name="OC_NEWARK" value="unknown"/>
+</part>
+<part name="R4" library="rcl" deviceset="R-EU_" device="R0603"/>
+<part name="J18" library="detali_main" deviceset="J" device=""/>
 </parts>
 <sheets>
@@
 <instances>
 <instance part="S2" gate="G$1" x="71.12" y="279.4"/>
-<instance part="S3" gate="G$1" x="129.54" y="289.56"/>
-<instance part="S4" gate="G$1" x="129.54" y="279.4"/>
+<instance part="S3" gate="G$1" x="129.54" y="289.56" rot="MR0"/>
+<instance part="S4" gate="G$1" x="129.54" y="279.4" rot="MR0"/>
 <instance part="S5" gate="G$1" x="187.96" y="289.56"/>
 <instance part="S6" gate="G$1" x="187.96" y="279.4"/>
@@
 <attribute name="VALUE" x="252.73" y="304.8" size="1.778" layer="95"/>
 </instance>
+<instance part="SV2" gate="G$1" x="419.1" y="322.58" rot="MR0"/>
+<instance part="R4" gate="G$1" x="276.86" y="355.6"/>
+<instance part="J18" gate="G$1" x="320.04" y="297.18" smashed="yes">
+<attribute name="NAME" x="322.58" y="297.18" size="1.27" layer="95"/>
+</instance>
 </instances>
 <busses>
@@
 </segment>
 </net>
-<net name="N$19" class="0">
-<segment>
-<pinref part="S3" gate="G$1" pin="PIN-1"/>
-<pinref part="JB3" gate="1" pin="2"/>
-<wire x1="124.46" y1="289.56" x2="121.92" y2="289.56" width="0.1524" layer="91"/>
-</segment>
-</net>
 <net name="N$20" class="0">
 <segment>
@@
 </segment>
 </net>
-<net name="N$32" class="0">
-<segment>
-<pinref part="S3" gate="G$1" pin="PIN-2"/>
-<pinref part="JA3" gate="1" pin="1"/>
-<wire x1="134.62" y1="289.56" x2="137.16" y2="289.56" width="0.1524" layer="91"/>
-</segment>
-</net>
 <net name="N$33" class="0">
 <segment>
@@
 <pinref part="D12" gate="G$1" pin="A"/>
 <pinref part="JB12" gate="1" pin="1"/>
-</segment>
-</net>
-<net name="N$2" class="0">
-<segment>
-<pinref part="JB4" gate="1" pin="2"/>
-<pinref part="S4" gate="G$1" pin="PIN-1"/>
-<wire x1="121.92" y1="279.4" x2="124.46" y2="279.4" width="0.1524" layer="91"/>
-</segment>
-</net>
-<net name="N$4" class="0">
-<segment>
-<pinref part="S4" gate="G$1" pin="PIN-2"/>
-<pinref part="JA4" gate="1" pin="1"/>
-<wire x1="134.62" y1="279.4" x2="137.16" y2="279.4" width="0.1524" layer="91"/>
 </segment>
 </net>
@@
 <net name="N$200" class="0">
 <segment>
-<pinref part="IC1" gate="D" pin="O"/>
 <wire x1="337.82" y1="302.26" x2="337.82" y2="297.18" width="0.1524" layer="91"/>
-<wire x1="337.82" y1="297.18" x2="312.42" y2="297.18" width="0.1524" layer="91"/>
+<wire x1="337.82" y1="297.18" x2="325.12" y2="297.18" width="0.1524" layer="91"/>
 <label x="342.9" y="302.26" size="1.778" layer="95"/>
 <wire x1="355.6" y1="302.26" x2="337.82" y2="302.26" width="0.1524" layer="91"/>
 <pinref part="SV3" gate="G$1" pin="7"/>
 <wire x1="355.6" y1="302.26" x2="363.22" y2="309.88" width="0.1524" layer="91"/>
+<pinref part="J18" gate="G$1" pin="P$1"/>
 </segment>
 </net>
@@
 </segment>
 </net>
+<net name="N$19" class="0">
+<segment>
+<pinref part="JB3" gate="1" pin="2"/>
+<pinref part="S3" gate="G$1" pin="PIN-2"/>
+<wire x1="121.92" y1="289.56" x2="124.46" y2="289.56" width="0.1524" layer="91"/>
+</segment>
+</net>
+<net name="N$32" class="0">
+<segment>
+<pinref part="S3" gate="G$1" pin="PIN-1"/>
+<pinref part="JA3" gate="1" pin="1"/>
+<wire x1="134.62" y1="289.56" x2="137.16" y2="289.56" width="0.1524" layer="91"/>
+</segment>
+</net>
+<net name="N$2" class="0">
+<segment>
+<pinref part="JB4" gate="1" pin="2"/>
+<pinref part="S4" gate="G$1" pin="PIN-2"/>
+<wire x1="121.92" y1="279.4" x2="124.46" y2="279.4" width="0.1524" layer="91"/>
+</segment>
+</net>
+<net name="N$4" class="0">
+<segment>
+<pinref part="S4" gate="G$1" pin="PIN-1"/>
+<pinref part="JA4" gate="1" pin="1"/>
+<wire x1="134.62" y1="279.4" x2="137.16" y2="279.4" width="0.1524" layer="91"/>
+</segment>
+</net>
+<net name="N$60" class="0">
+<segment>
+<pinref part="IC1" gate="D" pin="O"/>
+<pinref part="J18" gate="G$1" pin="P$2"/>
+<wire x1="312.42" y1="297.18" x2="317.5" y2="297.18" width="0.1524" layer="91"/>
+</segment>
+</net>
