File: PCB/keyBoard_A/keyBoard_A.sch (EAGLE design)
At the start: 253 parts, among them IC1 74HC04N, J1 J, J10 J, J11 J, J12 J, J13 J, J14 J, J15 J, J16 J, J17 J, J18 J, J19 J, J2 J, J20 J, J21 J, J22 J, J24 J, J25 J, J26 J, J27 J, J28 J, J29 J, J3 J, J30 J, J31 J, J32 J, J33 J, J34 J, J35 J, J36 J, J37 J, J38 J, J39 J, J4 J, J40 J, J41 J, J42 J, J43 J, J44 J, J45 J, J47 J, J48 J, J49 J, J5 J, J6 J, J7 J, J8 J, J9 J

Commit message: .
Parts:
- removed R11, R13, R14, R15: (no value), rcl:R-EU_M0805
- added J23, J46, J50, J51, J52, J53, J54, J55, J56, J57: J, detali_main:J
- added R1, R2, R3, R5: 10k, rd:RD
Connections:
- new net N$197: IC1E.O, J23.P$2
- new net N$225: J23.P$1, J46.P$2
- new net N$229: IC1F.O, J50.P$2
- new net N$230: J50.P$1, J51.P$2
- new net N$231: IC1A.O, J52.P$2
- new net N$232: J52.P$1, J53.P$2
- new net N$233: IC1B.O, J54.P$2
- new net N$235: J54.P$1, J55.P$2
- new net N$236: IC1C.O, J56.P$2
- new net N$237: J56.P$1, J57.P$2
- net +5V: now also R1.T, R2.T, R3.T, R5.T; no longer R11.1, R13.1, R14.1, R15.1
- net L4: now also R1.B; no longer R13.2
- net L5: now also R3.B; no longer R14.2
- net L6: now also R5.B; no longer R15.2
- net N$150: now also R2.B; no longer R11.2
- net N$195: now also J53.P$1; no longer IC1A.O
- net N$196: now also J51.P$1; no longer IC1F.O
- net N$198: now also J55.P$1; no longer IC1B.O
- net N$199: now also J57.P$1; no longer IC1C.O
- net N$203: now also J46.P$1; no longer IC1E.O

Commit message: pcb a r
Parts:
- removed R12: 10k, rd:RD
- removed R8: (no value), rcl:R-EU_R1206W
- added R100: 10k, rd:RD
- R1: value 10k -> (none); device rd:RD -> rcl:R-EU_R1206W
- R2, R5: device rd:RD -> rcl:R-EU_R1206W
- R4: value (none) -> 10k; device rcl:R-EU_R0603 -> rcl:R-EU_R0805
- renumbered IC1 to 1D2
Connections:
- removed net N$181: 1D2P.VCC, C18.2, D47.C
- new net VCCD2: 1D2P.VCC, C18.2, D47.C, R4.1, R5.1
- net +5V: now also R1.1, R100.T, R2.2; no longer R1.T, R12.T, R2.T, R5.T, R8.1
- net L4: now also R100.B; no longer R1.B
- net L6: now also R5.2; no longer R5.B
- net N$150: no longer R2.B
- net N$193: no longer R12.B
- net N$194: now also R4.2
- net N$223: now also R2.1
- net N$390: now also R1.2; no longer R8.2
Other:
- moved on the sheet: J42, J44, J48, J49, R4

Commit message: pcb a r
Parts:
- removed SV2: (no value), detali_main:FE03-1
Other:
- moved on the sheet: SV1
Changed lines of the file:
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@@
 <part name="J49" library="detali_main" deviceset="J" device=""/>
 <part name="R10" library="rd" deviceset="RD" device="" value="10k"/>
-<part name="SV2" library="detali_main" deviceset="FE03-1" device="">
-<attribute name="MF" value=""/>
-<attribute name="MPN" value=""/>
-<attribute name="OC_FARNELL" value="unknown"/>
-<attribute name="OC_NEWARK" value="unknown"/>
-</part>
 <part name="J18" library="detali_main" deviceset="J" device=""/>
 <part name="R100" library="rd" deviceset="RD" device="" value="10k"/>
@@
 <description>KB_A</description>
 <plain>
-<text x="398.78" y="317.5" size="1.778" layer="91">d1</text>
+<text x="322.58" y="228.6" size="1.778" layer="91">d1</text>
 <text x="378.46" y="312.42" size="1.778" layer="91">vcc</text>
-<text x="398.78" y="320.04" size="1.778" layer="91">d2</text>
-<text x="398.78" y="322.58" size="1.778" layer="91">d3</text>
+<text x="322.58" y="231.14" size="1.778" layer="91">d2</text>
+<text x="322.58" y="233.68" size="1.778" layer="91">d3</text>
 <text x="378.46" y="294.64" size="1.778" layer="91">gnd</text>
 <text x="40.64" y="304.8" size="5.08" layer="91">LEFT KB</text>
@@
 <instance part="JB88" gate="1" x="114.3" y="269.24"/>
 <instance part="D88" gate="G$1" x="104.14" y="269.24"/>
-<instance part="SV1" gate="G$1" x="396.24" y="322.58" rot="MR0"/>
+<instance part="SV1" gate="G$1" x="320.04" y="233.68" rot="MR0"/>
 <instance part="SV3" gate="G$1" x="370.84" y="302.26" rot="MR0"/>
 <instance part="J47" gate="G$1" x="45.72" y="104.14"/>
@@
 <attribute name="VALUE" x="252.73" y="327.66" size="1.778" layer="95"/>
 </instance>
-<instance part="SV2" gate="G$1" x="419.1" y="322.58" rot="MR0"/>
 <instance part="J18" gate="G$1" x="320.04" y="297.18" smashed="yes">
 <attribute name="NAME" x="322.58" y="297.18" size="1.27" layer="95"/>
@@
 <segment>
 <pinref part="SV1" gate="G$1" pin="3"/>
-<wire x1="388.62" y1="322.58" x2="381" y2="322.58" width="0.1524" layer="91"/>
-<label x="383.54" y="322.58" size="1.778" layer="95"/>
+<wire x1="312.42" y1="233.68" x2="304.8" y2="233.68" width="0.1524" layer="91"/>
+<label x="307.34" y="233.68" size="1.778" layer="95"/>
 </segment>
 </net>
@@
 <segment>
 <pinref part="SV1" gate="G$1" pin="2"/>
-<wire x1="381" y1="320.04" x2="388.62" y2="320.04" width="0.1524" layer="91"/>
-<label x="383.54" y="320.04" size="1.778" layer="95"/>
+<wire x1="304.8" y1="231.14" x2="312.42" y2="231.14" width="0.1524" layer="91"/>
+<label x="307.34" y="231.14" size="1.778" layer="95"/>
 </segment>
 </net>
@@
 <segment>
 <pinref part="SV1" gate="G$1" pin="1"/>
-<wire x1="388.62" y1="317.5" x2="381" y2="317.5" width="0.1524" layer="91"/>
-<label x="383.54" y="317.5" size="1.778" layer="95"/>
-</segment>
-</net>
+<wire x1="312.42" y1="228.6" x2="304.8" y2="228.6" width="0.1524" layer="91"/>
+<label x="307.34" y="228.6" size="1.778" layer="95"/>
+</segment>
+</net>

Commit message: pcb a
Parts:
- removed R10, R100: 10k, rd:RD
- added R6, R7: 10k, rcl:R-EU_R1206W
- added R8: 10k, rcl:R-EU_R0805
- R3: device rd:RD -> rcl:R-EU_R1206W
Connections:
- new net N$238: R3.2, R6.1
- net +5V: now also R7.1, R8.2; no longer R10.T, R100.T, R3.T
- net L1: now also R7.2; no longer R10.B
- net L4: now also R8.1; no longer R100.B
- net L5: now also R6.2; no longer R3.B
- net VCCD2: now also R3.1
Other:
- note added: "kba1"
- note added: "kba2"
- note added: "kba3"
- note added: "kba4"
- note added: "kba5"
- note added: "kba6"
- moved on the sheet: 1D1, 1D1P, 1D2A, 1D2B, 1D2C, 1D2D, 1D2E, 1D2F, 1D2P, C17, C18, D1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

Commit message: .
Parts:
- added S44A1: Caps Lock, cherrymx:CHERRY-MX
Connections:
- net N$113: now also S44A1.PIN-2
- net N$63: now also S44A1.PIN-1
Other:
- moved on the sheet: S44A
Changed lines of the file:
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@@
 <part name="R7" library="rcl" deviceset="R-EU_" device="R1206W" value="10k"/>
 <part name="R8" library="rcl" deviceset="R-EU_" device="R0805" value="10k"/>
+<part name="S44A1" library="cherrymx" deviceset="CHERRY-MX" device="" value="Caps Lock"/>
 </parts>
 <sheets>
@@
 <attribute name="VALUE" x="256.54" y="251.46" size="1.778" layer="96" rot="R180"/>
 </instance>
-<instance part="S44A" gate="G$1" x="111.76" y="121.92"/>
+<instance part="S44A" gate="G$1" x="96.52" y="119.38"/>
 <instance part="S88" gate="G$1" x="109.22" y="187.96"/>
 <instance part="JA88" gate="1" x="121.92" y="187.96"/>
@@
 <instance part="R7" gate="G$1" x="261.62" y="228.6"/>
 <instance part="R8" gate="G$1" x="261.62" y="241.3" rot="R180"/>
+<instance part="S44A1" gate="G$1" x="223.52" y="76.2"/>
 </instances>
 <busses>
@@
 <pinref part="JB43" gate="1" pin="2"/>
 <wire x1="162.56" y1="81.28" x2="165.1" y2="81.28" width="0.1524" layer="91"/>
+<label x="165.1" y="81.28" size="1.778" layer="95" rot="R90"/>
+</segment>
+<segment>
+<pinref part="S44A1" gate="G$1" pin="PIN-1"/>
+<wire x1="218.44" y1="76.2" x2="213.36" y2="76.2" width="0.1524" layer="91"/>
+<label x="213.36" y="76.2" size="1.778" layer="95"/>
 </segment>
 </net>
@@
 <segment>
 <pinref part="S44A" gate="G$1" pin="PIN-1"/>
-<wire x1="106.68" y1="121.92" x2="101.6" y2="121.92" width="0.1524" layer="91"/>
-<label x="104.14" y="121.92" size="1.778" layer="95" rot="R90"/>
+<wire x1="91.44" y1="119.38" x2="86.36" y2="119.38" width="0.1524" layer="91"/>
+<label x="83.82" y="119.38" size="1.778" layer="95"/>
 </segment>
 </net>
@@
 <pinref part="JA43" gate="1" pin="1"/>
 <wire x1="177.8" y1="81.28" x2="175.26" y2="81.28" width="0.1524" layer="91"/>
+<label x="177.8" y="81.28" size="1.778" layer="95" rot="R90"/>
+</segment>
+<segment>
+<pinref part="S44A1" gate="G$1" pin="PIN-2"/>
+<wire x1="228.6" y1="76.2" x2="233.68" y2="76.2" width="0.1524" layer="91"/>
+<label x="228.6" y="76.2" size="1.778" layer="95"/>
 </segment>
 </net>
@@
 <segment>
 <pinref part="S44A" gate="G$1" pin="PIN-2"/>
-<wire x1="116.84" y1="121.92" x2="121.92" y2="121.92" width="0.1524" layer="91"/>
-<label x="119.38" y="121.92" size="1.778" layer="95" rot="R90"/>
-</segment>
-</net>
+<wire x1="101.6" y1="119.38" x2="106.68" y2="119.38" width="0.1524" layer="91"/>
+<label x="101.6" y="119.38" size="1.778" layer="95"/>
+</segment>
+</net>

Commit message: add stab pcb a
Parts:
- added STAB_LSH, STAB_LSP: STAB, kbmxco:STAB
Other:
- moved on the sheet: S44A1
Changed lines of the file:
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@@
 <layer number="131" name="tAdjust" color="7" fill="1" visible="yes" active="yes"/>
 <layer number="132" name="bAdjust" color="7" fill="1" visible="yes" active="yes"/>
+<layer number="133" name="Frame" color="13" fill="1" visible="yes" active="yes"/>
 <layer number="144" name="Drill_legend" color="7" fill="1" visible="yes" active="yes"/>
 <layer number="150" name="Notes" color="7" fill="1" visible="yes" active="yes"/>
@@
 <part name="R8" library="rcl" deviceset="R-EU_" device="R0805" value="10k"/>
 <part name="S44A1" library="cherrymx" deviceset="CHERRY-MX" device="" value="Caps Lock"/>
+<part name="STAB_LSP" library="kbmxco" deviceset="STAB" device=""/>
+<part name="STAB_LSH" library="kbmxco" deviceset="STAB" device=""/>
 </parts>
 <sheets>
@@
 <instance part="R7" gate="G$1" x="261.62" y="228.6"/>
 <instance part="R8" gate="G$1" x="261.62" y="241.3" rot="R180"/>
-<instance part="S44A1" gate="G$1" x="223.52" y="76.2"/>
+<instance part="S44A1" gate="G$1" x="279.4" y="104.14"/>
+<instance part="STAB_LSP" gate="STAB" x="304.8" y="106.68"/>
+<instance part="STAB_LSH" gate="STAB" x="320.04" y="106.68"/>
 </instances>
 <busses>
@@
 <segment>
 <pinref part="S44A1" gate="G$1" pin="PIN-1"/>
-<wire x1="218.44" y1="76.2" x2="213.36" y2="76.2" width="0.1524" layer="91"/>
-<label x="213.36" y="76.2" size="1.778" layer="95"/>
+<wire x1="274.32" y1="104.14" x2="269.24" y2="104.14" width="0.1524" layer="91"/>
+<label x="269.24" y="104.14" size="1.778" layer="95"/>
 </segment>
 </net>
@@
 <segment>
 <pinref part="S44A1" gate="G$1" pin="PIN-2"/>
-<wire x1="228.6" y1="76.2" x2="233.68" y2="76.2" width="0.1524" layer="91"/>
-<label x="228.6" y="76.2" size="1.778" layer="95"/>
-</segment>
-</net>
+<wire x1="284.48" y1="104.14" x2="289.56" y2="104.14" width="0.1524" layer="91"/>
+<label x="284.48" y="104.14" size="1.778" layer="95"/>
+</segment>
+</net>
