File: PCB/keyBoard_A/keyBoard_A.brd (EAGLE design)
At the start: 184.3 x 134.6 mm, 305 parts, among them IC1 74HC04N, J1 J, J10 J, J11 J, J12 J, J13 J, J14 J, J15 J, J16 J, J17 J, J18 J, J19 J, J2 J, J20 J, J21 J, J22 J, J23 J, J24 J, J25 J, J26 J, J27 J, J28 J, J29 J, J3 J, J30 J, J31 J, J32 J, J33 J, J34 J, J35 J, J36 J, J37 J, J38 J, J39 J, J4 J, J40 J, J41 J, J42 J, J43 J, J44 J, J45 J, J47 J, J48 J, J49 J, J5 J, J6 J, J7 J, J8 J, J9 J

Commit message: pcb a 4
Parts:
- removed CAPS, SCROLL, SCROLL1: (no value), detali_main:LED5MM
- removed J23: J, detali_main:R1206W
- removed R3, R9: (no value), rcl:R1206W
- moved D24 16.9 mm to (190.2, 121.0), turned to 180 degrees
- moved JA24 8.47 mm to (201.9, 110.8)
- moved D37 8.26 mm to (76.5, 67.9)
- moved JB24 7.85 mm to (192.1, 113.3), turned to 90 degrees
- moved D18 4.76 mm to (195.3, 134.0), turned to 180 degrees
- moved C18 3.81 mm to (40.0, 53.0)
- moved R15 3.17 mm to (43.8, 54.6)
- moved D11 1.93 mm to (73.0, 68.6)
- moved IC1 1.90 mm to (41.9, 62.2)
- moved D23 1.62 mm to (185.7, 121.0)
- moved R14 1.59 mm to (42.2, 59.4)
- moved R13 1.27 mm to (42.5, 62.9)
- moved J1 0.95 mm to (195.3, 130.8)
- moved SV1 0.93 mm to (86.8, 130.3)
- moved JB23 0.45 mm to (187.0, 115.9)
Connections:
- removed net LED_CAPS: R9.2
- removed net LED_SCROLL: R3.2
- removed net N$231: R3.1, SCROLL.A
- removed net N$232: CAPS.A, R9.1
- removed net N$60: 1D1.9, J23.2
- net +5V: no longer CAPS.K, SCROLL.K
- net 8: now also 1D1.9; no longer J23.1
- net N$49: now also S24.SW2; no longer S24.SW1
- net N$50: now also S24.SW1; no longer S24.SW2
Routing:
- net GND: track 281.7 -> 166.5 mm
- net N$200: track 75.3 -> 56.4 mm
- net 8: track 138.2 -> 150.4 mm
- net L3: track 145.4 -> 154.3 mm
- net N$199: track 79.1 -> 72.0 mm
- net N$60: track 6.91 -> 0.00 mm
- net 7J: track 37.4 -> 31.6 mm
- net N$48: track 2.76 -> 7.56 mm
- net N$198: track 81.9 -> 78.7 mm
- net N$121: track 1.67 -> 4.55 mm
- net N$203: track 83.5 -> 81.6 mm
- net 3J3: track 46.6 -> 44.7 mm
- net N$196: track 86.6 -> 85.5 mm
- net L4: track 208.8 -> 209.5 mm
- net N$195: track 88.5 -> 87.9 mm
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
Commit message: pcb c new progr >
Routing:
- net L4: track 209.5 -> 211.2 mm
Changed lines of the file:
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@@
 <wire x1="57.912" y1="78.105" x2="58.42" y2="78.613" width="0.6096" layer="16"/>
 <contactref element="IC1" pad="5"/>
-<wire x1="43.4975" y1="64.77" x2="46.355" y2="66.675" width="0.6096" layer="16"/>
-<wire x1="46.355" y1="66.675" x2="46.355" y2="68.8975" width="0.6096" layer="16"/>
-<wire x1="46.355" y1="68.8975" x2="46.355" y2="74.3585" width="0.6096" layer="16"/>
-<wire x1="46.355" y1="74.3585" x2="43.053" y2="77.6605" width="0.6096" layer="16"/>
+<wire x1="43.4975" y1="64.77" x2="47.9425" y2="65.7225" width="0.6096" layer="16"/>
+<wire x1="47.9425" y1="65.7225" x2="47.9425" y2="68.8975" width="0.6096" layer="16"/>
+<wire x1="47.9425" y1="68.8975" x2="47.9425" y2="74.3585" width="0.6096" layer="16"/>
+<wire x1="47.9425" y1="74.3585" x2="43.053" y2="77.6605" width="0.6096" layer="16"/>
 <contactref element="R13" pad="2"/>
 <wire x1="95.885" y1="71.628" x2="108.458" y2="71.628" width="0.6096" layer="16"/>
@@
 <wire x1="68.2625" y1="70.485" x2="68.2625" y2="69.85" width="0.6096" layer="16"/>
 <wire x1="68.2625" y1="69.85" x2="67.31" y2="68.8975" width="0.6096" layer="16"/>
-<wire x1="67.31" y1="68.8975" x2="46.355" y2="68.8975" width="0.6096" layer="16"/>
+<wire x1="67.31" y1="68.8975" x2="47.9425" y2="68.8975" width="0.6096" layer="16"/>
 <wire x1="40.005" y1="79.248" x2="41.4655" y2="79.248" width="0.6096" layer="16"/>
 <wire x1="41.4655" y1="79.248" x2="43.053" y2="77.6605" width="0.6096" layer="16"/>
-<wire x1="46.355" y1="66.675" x2="45.72" y2="64.77" width="0" layer="19" extent="16-16"/>
+<wire x1="47.9425" y1="65.7225" x2="45.72" y2="64.77" width="0" layer="19" extent="16-16"/>
 <wire x1="42.545" y1="63.815" x2="43.4975" y2="64.77" width="0" layer="19" extent="16-16"/>
 </signal>

Commit message: sw ls
Parts:
- R10, R12: value (none) -> 10k; device rcl:M0805 -> rd:0603R
- moved C17 155.0 mm to (168.9, 129.9), flipped to the bottom, turned to 90 degrees
- moved D48 10.6 mm to (30.5, 57.1), turned to 270 degrees
- moved D11 8.86 mm to (70.8, 60.0), turned to 0 degrees
- moved R14 6.68 mm to (48.9, 59.7), turned to 0 degrees
- moved R8 5.17 mm to (176.5, 129.9), turned to 0 degrees
- moved D10 5.12 mm to (33.0, 62.2), turned to 90 degrees
- moved R15 5.08 mm to (48.9, 54.6), turned to 0 degrees
- moved R10 4.55 mm to (34.3, 65.1), flipped to the top, turned to 90 degrees
- moved D47 4.46 mm to (34.3, 54.6)
- moved J44 4.45 mm to (34.3, 57.1)
- moved R12 2.71 mm to (35.6, 59.7), flipped to the top, turned to 90 degrees
- moved R11 2.56 mm to (29.8, 60.6)
- moved C18 0.32 mm to (40.3, 53.0)
Connections:
- net +5V: now also R10.PT, R12.PT; no longer R10.1, R12.1
- net L1: now also IC1.11, R10.PB; no longer IC1.9, R10.2
- net L4: now also IC1.9; no longer IC1.5
- net N$193: now also IC1.5, R12.PB; no longer IC1.11, R12.2
- net N$196: now also IC1.6; no longer IC1.10
- net N$200: now also IC1.8; no longer IC1.6
- net N$203: now also IC1.10; no longer IC1.8
Routing:
- net +5V: track 0.00 -> 126.7 mm, vias 0 -> 1
- net GND: track 166.5 -> 153.2 mm
- net L5: track 171.9 -> 184.3 mm
- net N$55: track 44.6 -> 33.9 mm
- net N$31: track 33.0 -> 25.2 mm
- net L4: track 211.2 -> 203.5 mm
- net L1: track 306.9 -> 313.8 mm
- net N$193: track 36.6 -> 43.4 mm
- net 3J3: track 44.7 -> 51.2 mm
- net N$203: track 81.6 -> 86.7 mm
- net N$181: track 0.00 -> 4.42 mm
- net N$196: track 85.5 -> 89.1 mm
- net N$390: track 2.31 -> 5.65 mm
- net N$194: track 0.00 -> 2.31 mm
- net N$192: track 0.00 -> 2.27 mm
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
Commit message: sw ls
Parts:
- moved R14 14.6 mm to (58.4, 70.8)
- moved R13 7.36 mm to (49.8, 63.8)
- moved J44 7.05 mm to (35.2, 50.2)
- moved R15 5.83 mm to (54.0, 57.5)
- moved R10 2.73 mm to (35.9, 62.9)
- moved R12 1.91 mm to (35.6, 57.8)
Connections:
- removed net N$196 (its old number): IC1.6, SV3.6
- removed net N$198 (its old number): IC1.2, SV3.2
- new net N$195: IC1.2, SV3.4
- new net N$199: IC1.6, SV3.2
- net L5: now also IC1.5; no longer IC1.3
- net L6: now also IC1.3; no longer IC1.1
- net N$193: now also IC1.13; no longer IC1.5
- net N$194: now also IC1.1; no longer IC1.13
- net N$200: now also SV3.7; no longer SV3.4
- net N$203: now also SV3.6; no longer SV3.7
Routing:
- net N$196 (its old number): track 89.1 -> 0.00 mm
- net N$195: track 0.00 -> 88.7 mm
- net N$198 (its old number): track 78.7 -> 0.00 mm
- net N$199: track 0.00 -> 63.2 mm
- net N$200: track 56.4 -> 77.3 mm
- net GND: track 153.2 -> 132.4 mm
- net L4: track 203.5 -> 218.8 mm
- net N$198: track 72.0 -> 81.4 mm
- net N$150: track 66.0 -> 70.5 mm
- net N$193: track 43.4 -> 39.3 mm
- net L1: track 313.8 -> 309.7 mm
- net L6: track 156.8 -> 161.0 mm
- net N$203: track 86.7 -> 84.1 mm
- net N$194: track 2.31 -> 0.00 mm
- net +5V: track 126.7 -> 124.8 mm
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
Commit message: sw s10
Parts:
- removed J18: J, detali_main:R1206W
- moved JB10 14.2 mm to (33.0, 36.2), turned to 180 degrees
- moved R14 8.67 mm to (50.8, 66.7)
- moved JA10 6.03 mm to (46.4, 34.3)
- moved D37 3.86 mm to (72.7, 68.6)
- moved R15 3.18 mm to (51.4, 59.4), turned to 270 degrees
- moved C18 2.03 mm to (41.6, 54.6), turned to 0 degrees
- moved J44 1.85 mm to (34.3, 51.8)
- moved R13 0.90 mm to (50.5, 64.5)
Connections:
- removed net 2J3: D37.C, D9.C, J18.2
- net 2J2: now also D37.C, D9.C; no longer J18.1
- net N$13: now also S10.SW2; no longer S10.SW1
- net N$28: now also S10.SW1; no longer S10.SW2
Routing:
- net 2J2: track 21.9 -> 31.7 mm
- net N$55: track 33.9 -> 26.1 mm
- net L6: track 161.0 -> 153.3 mm
- net GND: track 132.4 -> 125.1 mm
- net 2J3: track 6.40 -> 0.00 mm
- net 3J3: track 51.2 -> 54.2 mm
- net N$150: track 70.5 -> 68.7 mm
- net L5: track 184.3 -> 182.7 mm
- net N$28: track 3.67 -> 4.86 mm

Commit message: .
Parts:
- added J18: J, detali_main:R1206W
- added R4: (no value), rcl:R0603
- added SV2: (no value), detali_main:FE03-1
- moved D4 15.6 mm to (50.5, 128.3), turned to 0 degrees
- moved JB4 14.0 mm to (52.4, 122.2), turned to 135 degrees
- moved D3 14.0 mm to (32.7, 129.2)
- moved JB3 13.8 mm to (33.3, 122.2), turned to 180 degrees
- moved J42 13.0 mm to (32.1, 102.6)
- moved D6 12.9 mm to (61.0, 98.4), turned to 0 degrees
- moved JB6 7.84 mm to (60.0, 100.6), turned to 180 degrees
- moved JA6 7.57 mm to (52.7, 103.2), turned to 0 degrees
- moved JA4 4.26 mm to (62.2, 118.7)
- moved JA9 4.13 mm to (52.4, 57.1), turned to 0 degrees
- moved J16 3.49 mm to (59.1, 116.2)
- moved JA7 3.43 mm to (37.1, 78.1)
- moved JA3 3.24 mm to (43.2, 118.7)
- moved J49 3.18 mm to (48.3, 121.6)
- moved J48 2.73 mm to (63.8, 135.3), turned to 135 degrees
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Connections:
- new net N$60: IC1.8, J18.2
- net N$19: now also S3.SW2; no longer S3.SW1
- net N$2: now also S4.SW2; no longer S4.SW1
- net N$200: now also J18.1; no longer IC1.8
- net N$32: now also S3.SW1; no longer S3.SW2
- net N$4: now also S4.SW1; no longer S4.SW2
Routing:
- net L4: track 218.8 -> 205.1 mm
- net L2: track 182.8 -> 196.3 mm
- net 1: track 30.9 -> 43.9 mm
- net N$150: track 68.7 -> 56.5 mm
- net 2: track 26.3 -> 36.0 mm
- net L3J: track 47.0 -> 40.4 mm
- net N$60: track 0.00 -> 6.46 mm
- net 2J: track 21.0 -> 25.9 mm
- net N$224: track 22.2 -> 26.8 mm
- net N$203: track 84.1 -> 88.4 mm
- net N$196: track 87.1 -> 82.9 mm
- net N$24: track 2.01 -> 5.94 mm
- net N$200: track 77.3 -> 73.5 mm
- net 2J2: track 31.7 -> 28.1 mm
- net N$195: track 88.8 -> 86.1 mm
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Other:
- outline, holes or cut-outs redrawn

Commit message: .
Parts:
- removed R11, R13, R14, R15: (no value), rcl:M0805
- added J23, J46, J50, J51, J52, J53, J54, J55, J56, J57: J, detali_main:R1206W
- added R1, R2, R3, R5: 10k, rd:0603R
- moved D37 12.0 mm to (84.5, 69.5), turned to 90 degrees
- moved JA8 7.41 mm to (52.1, 83.2), turned to 0 degrees
- moved D9 6.36 mm to (71.8, 68.6)
- moved JB37 1.62 mm to (87.3, 53.7)
- moved D48 0.90 mm to (29.8, 57.8)
- moved J44 0.32 mm to (34.3, 52.1)
- moved R12 0.32 mm to (35.9, 57.1)
Connections:
- new net N$197: IC1.10, J23.2
- new net N$225: J23.1, J46.2
- new net N$229: IC1.12, J50.2
- new net N$230: J50.1, J51.2
- new net N$231: IC1.2, J52.2
- new net N$232: J52.1, J53.2
- new net N$233: IC1.4, J54.2
- new net N$235: J54.1, J55.2
- new net N$236: IC1.6, J56.2
- new net N$237: J56.1, J57.2
- net +5V: now also R1.PT, R2.PT, R3.PT, R5.PT; no longer R11.1, R13.1, R14.1, R15.1
- net L4: now also R1.PB; no longer R13.2
- net L5: now also R3.PB; no longer R14.2
- net L6: now also R5.PB; no longer R15.2
- net N$150: now also R2.PB; no longer R11.2
- net N$195: now also J53.1; no longer IC1.2
- net N$196: now also J51.1; no longer IC1.12
- net N$198: now also J55.1; no longer IC1.4
- net N$199: now also J57.1; no longer IC1.6
- net N$203: now also J46.1; no longer IC1.10
Routing:
- net N$198: track 80.4 -> 13.1 mm
- net N$195: track 86.1 -> 36.0 mm
- net N$203: track 88.4 -> 42.9 mm
- net N$196: track 82.9 -> 39.8 mm
- net N$197: track 0.00 -> 37.0 mm
- net N$231: track 0.00 -> 36.3 mm
- net N$229: track 0.00 -> 36.0 mm
- net N$199: track 63.2 -> 31.0 mm
- net L5: track 182.7 -> 213.8 mm
- net N$140: track 0.00 -> 28.8 mm
- net N$233: track 0.00 -> 26.7 mm
- net N$236: track 0.00 -> 16.4 mm
- net N$194: track 0.00 -> 15.6 mm
- net 2J2: track 28.1 -> 40.7 mm
- net N$150: track 56.5 -> 50.2 mm
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
Commit message: .
Parts:
- moved J57 0.95 mm to (67.6, 69.8)
- moved J56 0.63 mm to (61.9, 69.8)
- moved JA38 0.32 mm to (123.2, 54.9)
Routing:
- net GND: track 127.7 -> 216.9 mm
- net N$198: track 13.1 -> 34.0 mm
- net N$199: track 31.0 -> 15.4 mm
- net N$195: track 36.0 -> 37.0 mm
- net N$196: track 39.8 -> 40.6 mm
- net N$236: track 16.4 -> 15.7 mm
- net N$203: track 42.9 -> 43.4 mm
Other:
- outline, holes or cut-outs redrawn
