File: PCB/keyBoard_A/keyBoard_A.brd (EAGLE design)
At the start: 184.3 x 134.6 mm, 311 parts, among them IC1 74HC04N, J1 J, J10 J, J11 J, J12 J, J13 J, J14 J, J15 J, J16 J, J17 J, J18 J, J19 J, J2 J, J20 J, J21 J, J22 J, J23 J, J24 J, J25 J, J26 J, J27 J, J28 J, J29 J, J3 J, J30 J, J31 J, J32 J, J33 J, J34 J, J35 J, J36 J, J37 J, J38 J, J39 J, J4 J, J40 J, J41 J, J42 J, J43 J, J44 J, J45 J, J46 J, J47 J, J48 J, J49 J, J5 J, J50 J, J51 J, J52 J, J53 J, J54 J, J55 J, J56 J, J57 J, J6 J, J7 J, J8 J, J9 J

Commit message: pcb a r
Parts:
- removed R12: 10k, rd:0603R
- removed R8: (no value), rcl:R1206W
- added R100: 10k, rd:0603R
- R1: value 10k -> (none); device rd:0603R -> rcl:R1206W
- R2, R5: device rd:0603R -> rcl:R1206W
- R4: value (none) -> 10k; device rcl:R0603 -> rcl:R0805
- moved R1 154.5 mm to (176.5, 129.9), flipped to the bottom
- moved R2 81.8 mm to (69.5, 129.9), flipped to the bottom, turned to 270 degrees
- moved R4 9.53 mm to (42.9, 54.3), flipped to the bottom, turned to 90 degrees
- moved R5 9.47 mm to (47.9, 52.1), flipped to the bottom, turned to 180 degrees
- moved D37 5.72 mm to (78.7, 69.7)
- moved D48 5.21 mm to (34.0, 54.6), turned to 180 degrees
- moved D9 2.84 mm to (69.2, 67.3)
- moved D10 2.56 mm to (32.7, 59.7)
- moved J57 2.25 mm to (69.2, 71.4)
- moved D47 2.25 mm to (34.0, 52.4)
- moved JB10 2.25 mm to (33.3, 38.4)
- moved J46 2.13 mm to (69.2, 81.6)
- moved J51 2.13 mm to (69.2, 79.1)
- moved J53 2.13 mm to (69.2, 76.5)
- moved J44 1.93 mm to (34.0, 50.2)
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- renumbered IC1 to 1D2
Connections:
- removed net N$181: 1D2.14, C18.2, D47.C
- new net VCCD2: 1D2.14, C18.2, D47.C, R4.1, R5.1
- net +5V: now also R1.1, R100.PT, R2.2; no longer R1.PT, R12.PT, R2.PT, R5.PT, R8.1
- net L4: now also R100.PB; no longer R1.PB
- net L6: now also R5.2; no longer R5.PB
- net N$150: no longer R2.PB
- net N$193: no longer R12.PB
- net N$194: now also R4.2
- net N$223: now also R2.1
- net N$390: now also R1.2; no longer R8.2
Routing:
- net +5V: track 122.9 -> 266.9 mm
- net N$199: track 15.4 -> 49.2 mm
- net GND: track 216.9 -> 233.7 mm
- net N$198: track 34.0 -> 49.4 mm
- net VCCD2: track 0.00 -> 13.1 mm
- net N$195: track 37.0 -> 49.2 mm
- net N$193: track 38.2 -> 49.5 mm
- net L1: track 308.1 -> 316.5 mm
- net N$196: track 40.6 -> 48.8 mm
- net N$194: track 15.6 -> 21.3 mm
- net N$150: track 50.2 -> 55.8 mm
- net N$55: track 25.8 -> 21.0 mm
- net N$181: track 4.65 -> 0.00 mm
- net N$203: track 43.4 -> 47.3 mm
- net L5: track 213.9 -> 210.0 mm
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
Commit message: pcb a r
Parts:
- removed SV2: (no value), detali_main:FE03-1
Routing:
- net +5V: track 266.9 -> 248.9 mm, vias 1 -> 2
- net GND: track 233.7 -> 234.4 mm
- net N$193: track 49.5 -> 48.8 mm

Commit message: pcb a
Parts:
- removed R10, R100: 10k, rd:0603R
- added R6, R7: 10k, rcl:R1206W
- added R8: 10k, rcl:R0805
- R3: device rd:0603R -> rcl:R1206W
- moved J44 32.6 mm to (51.8, 22.9), turned to 90 degrees
- moved R3 30.7 mm to (52.1, 34.3), flipped to the bottom
- moved D48 24.3 mm to (40.3, 31.1), turned to 0 degrees
- moved D47 24.3 mm to (45.7, 31.1)
- moved R5 24.1 mm to (51.8, 28.3), turned to 225 degrees
- moved D10 22.9 mm to (36.5, 37.1)
- moved JA88 22.2 mm to (85.4, 88.3)
- moved JB37 21.1 mm to (89.9, 32.7)
- moved 1D1 20.6 mm to (170.8, 110.5)
- moved D15 20.6 mm to (140.0, 116.2)
- moved D18 20.6 mm to (198.4, 113.7)
- moved D19 20.6 mm to (114.6, 101.6)
- moved D20 20.6 mm to (133.0, 101.3)
- moved D21 20.6 mm to (154.3, 100.3)
- moved D22 20.6 mm to (174.0, 100.6)
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Connections:
- new net N$238: R3.2, R6.1
- net +5V: now also R7.1, R8.2; no longer R10.PT, R100.PT, R3.PT
- net L1: now also R7.2; no longer R10.PB
- net L4: now also R8.1; no longer R100.PB
- net L5: now also R6.2; no longer R3.PB
- net VCCD2: now also R3.1
Routing:
- net +5V: track 248.9 -> 314.7 mm
- net N$150: track 55.8 -> 97.1 mm
- net L6: track 156.9 -> 166.6 mm
- net L5: track 210.0 -> 216.8 mm
- net L1: track 316.5 -> 319.3 mm
- net N$55: track 21.0 -> 18.3 mm
- net 1J3: track 36.3 -> 38.6 mm
- net N$238: track 0.00 -> 2.08 mm
- net N$194: track 21.3 -> 19.3 mm
- net VCCD2: track 13.1 -> 15.0 mm
- net N$28: track 4.86 -> 3.49 mm
- net N$140: track 27.7 -> 28.9 mm
- net N$193: track 48.8 -> 50.0 mm
- net L2: track 197.2 -> 198.4 mm
- net L4: track 210.5 -> 211.6 mm
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- added copper zone on layer 16, net N$181
- added copper zone on layer 16, net N$239
- added copper zone on layer 16, net N$240
- added copper zone on layer 16, net N$241
Other:
- outline, holes or cut-outs redrawn

Commit message: pcb a +
Parts:
- moved D46 0.79 mm to (187.0, 23.0)
- moved D23 0.65 mm to (189.1, 101.3)
- moved JB46 0.64 mm to (187.0, 18.7)
- moved JA45 0.48 mm to (141.6, 13.8)
- moved D48 0.48 mm to (40.3, 30.6)
- moved J27 0.45 mm to (157.8, 106.7)
- moved D18 0.32 mm to (198.4, 114.0)
- moved JA44 0.16 mm to (110.5, 13.8)
Routing:
- net L2: track 198.4 -> 204.2 mm
- net N$223: track 44.1 -> 45.1 mm
- net +5V: track 314.7 -> 313.7 mm, vias 2 -> 3
- net 8: track 150.1 -> 149.4 mm
- net N$126: track 2.91 -> 3.44 mm

Commit message: pcb a
Parts:
- removed U$98: (no value), kbmx:18X18
- moved U$9 34.9 mm to (84.1, -12.1)
- moved D37 5.40 mm to (77.2, 46.8)
- moved R8 3.49 mm to (84.6, 58.1)
- moved JB37 2.54 mm to (89.9, 35.2)
- moved D9 1.59 mm to (70.8, 47.0)
Routing:
- net 3J3: track 50.0 -> 59.5 mm
- net L4: track 211.6 -> 216.6 mm
- net 2J2: track 38.0 -> 34.1 mm
- net +5V: track 313.7 -> 310.2 mm
- net N$140: track 28.9 -> 25.9 mm
- net L2: track 204.2 -> 205.6 mm
- net N$56: track 34.6 -> 35.5 mm
- net L5: track 216.8 -> 217.6 mm
- net N$62: track 4.03 -> 3.38 mm
- net N$30: track 5.75 -> 5.25 mm
Other:
- outline, holes or cut-outs redrawn

Commit message: .
Parts:
- added S44A1: Caps Lock, cherrymx:CHERRY-MX
- added U$14: (no value), kbmx:18X18
- added U$15: (no value), kbmx:18X23
- moved U$9 49.9 mm to (120.3, 22.2), turned to 270 degrees
- moved JA44 9.84 mm to (120.3, 13.8)
- moved JA43 7.63 mm to (93.0, 13.7)
- moved JB43 3.31 mm to (108.6, 15.2)
- moved S44 2.86 mm to (116.5, 21.0)
- moved S44A 2.54 mm to (119.1, 21.0)
- moved S43 2.54 mm to (102.6, 21.0)
- moved JA37 2.25 mm to (98.1, 34.3)
- moved J34 1.91 mm to (90.5, 128.9)
- moved D12 0.71 mm to (114.6, 35.6)
- moved JA11 0.32 mm to (62.2, 13.7)
- moved JA12 0.32 mm to (81.3, 13.7)
Connections:
- net N$113: now also S44A1.SW2
- net N$63: now also S44A1.SW1
Routing:
- net GND: track 234.4 -> 240.7 mm
- net N$146: track 34.6 -> 38.8 mm
- net N$113: track 3.37 -> 7.22 mm
- net N$63: track 3.05 -> 6.03 mm
- net L1: track 318.9 -> 321.5 mm
- net AFN1A: track 5.91 -> 8.45 mm
- net N$191: track 90.3 -> 88.5 mm
- net +5V: track 310.2 -> 311.5 mm
- net L5: track 217.6 -> 218.6 mm
- net 4J3: track 32.8 -> 32.1 mm
- net N$56: track 35.5 -> 34.9 mm
- net N$234: track 2.73 -> 3.28 mm
Other:
- outline, holes or cut-outs redrawn

Commit message: pcb c
Changed lines of the file:
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@@
 <grid distance="12.5" unitdist="mil" unit="mil" style="lines" multiple="1" display="yes" altdistance="0.025" altunitdist="inch" altunit="inch"/>
 <layers>
-<layer number="1" name="Top" color="4" fill="1" visible="yes" active="yes"/>
+<layer number="1" name="Top" color="4" fill="1" visible="no" active="yes"/>
 <layer number="2" name="Route2" color="1" fill="3" visible="no" active="no"/>
 <layer number="3" name="Route3" color="4" fill="3" visible="no" active="no"/>
@@
 <contactref element="SV3" pad="6"/>
 <contactref element="J46" pad="1"/>
-<wire x1="73.9775" y1="61.366" x2="73.9775" y2="80.01" width="0.6096" layer="16"/>
-<wire x1="73.9775" y1="80.01" x2="71.12" y2="82.8675" width="0.6096" layer="16"/>
+<wire x1="73.9775" y1="61.366" x2="73.9775" y2="72.39" width="0.6096" layer="16"/>
 <wire x1="71.4375" y1="100.6475" x2="73.18375" y2="102.39375" width="0.6096" layer="16"/>
 <wire x1="73.18375" y1="102.39375" x2="77.31125" y2="102.39375" width="0.6096" layer="16"/>
@@
 <wire x1="71.12" y1="100.33" x2="71.4375" y2="100.6475" width="0.4064" layer="16"/>
 <wire x1="73.9775" y1="61.366" x2="73.889" y2="61.2775" width="0.6096" layer="16"/>
+<wire x1="73.9775" y1="72.39" x2="72.39" y2="73.9775" width="0.6096" layer="16"/>
+<wire x1="72.39" y1="73.9775" x2="72.39" y2="81.5975" width="0.6096" layer="16"/>
+<wire x1="72.39" y1="81.5975" x2="71.12" y2="82.8675" width="0.6096" layer="16"/>
 </signal>
 <signal name="N$150">
@@
 <contactref element="SV3" pad="4"/>
 <contactref element="J53" pad="1"/>
-<wire x1="77.1525" y1="64.135" x2="77.1525" y2="82.8675" width="0.6096" layer="16"/>
-<wire x1="77.1525" y1="82.8675" x2="73.025" y2="86.995" width="0.6096" layer="16"/>
+<wire x1="77.1525" y1="64.135" x2="77.1525" y2="74.6125" width="0.6096" layer="16"/>
 <wire x1="75.08875" y1="97.31375" x2="73.3425" y2="95.5675" width="0.6096" layer="16"/>
 <wire x1="75.08875" y1="97.31375" x2="77.31125" y2="97.31375" width="0.6096" layer="16"/>
@@
 <wire x1="78.105" y1="58.42" x2="75.8825" y2="56.1975" width="0.6096" layer="16"/>
 <wire x1="75.8825" y1="56.1975" x2="73.889" y2="56.1975" width="0.6096" layer="16"/>
+<wire x1="77.1525" y1="74.6125" x2="76.835" y2="74.93" width="0.6096" layer="16"/>
+<wire x1="76.835" y1="74.93" x2="76.835" y2="83.185" width="0.6096" layer="16"/>
+<wire x1="76.835" y1="83.185" x2="73.025" y2="86.995" width="0.6096" layer="16"/>
 </signal>
 <signal name="N$151">
@@
 <contactref element="SV3" pad="5"/>
 <contactref element="J51" pad="1"/>
-<wire x1="75.565" y1="63.1825" x2="75.565" y2="81.5975" width="0.6096" layer="16"/>
-<wire x1="75.565" y1="81.5975" x2="72.0725" y2="85.09" width="0.6096" layer="16"/>
+<wire x1="75.565" y1="63.1825" x2="75.565" y2="73.9775" width="0.6096" layer="16"/>
 <wire x1="72.39" y1="98.1075" x2="74.13625" y2="99.85375" width="0.6096" layer="16"/>
 <wire x1="74.13625" y1="99.85375" x2="77.31125" y2="99.85375" width="0.6096" layer="16"/>
@@
 <wire x1="76.2" y1="59.3725" x2="75.565" y2="58.7375" width="0.6096" layer="16"/>
 <wire x1="75.565" y1="58.7375" x2="73.889" y2="58.7375" width="0.6096" layer="16"/>
+<wire x1="75.565" y1="73.9775" x2="74.6125" y2="74.93" width="0.6096" layer="16"/>
+<wire x1="74.6125" y1="74.93" x2="74.6125" y2="82.55" width="0.6096" layer="16"/>
+<wire x1="74.6125" y1="82.55" x2="72.0725" y2="85.09" width="0.6096" layer="16"/>
 </signal>
 <signal name="N$62">
