File: PCB/RGB/rgb.brd (EAGLE design)
At the start: 88.9 x 196.2 mm, 82 parts

Commit message: vil_26
Parts:
- moved JP1 1.80 mm to (239.9, 214.3)
- moved DD1 1.42 mm to (231.8, 215.6)
- moved R7 0.32 mm to (224.2, 211.5)
- moved R2 0.32 mm to (224.5, 223.8)
- moved R6 0.32 mm to (224.2, 214.0)
Routing:
- net VCC: track 7.89 -> 68.2 mm, vias 3 -> 4
- net N$140: track 36.0 -> 84.3 mm, vias 0 -> 2
- net GND: track 66.3 -> 110.4 mm
- net N$141: track 0.00 -> 22.1 mm
- net N$142: track 0.00 -> 17.3 mm, vias 0 -> 2
- net +5V: track 48.9 -> 57.7 mm
- net N$139: track 57.5 -> 63.6 mm
- net N$35: track 2.32 -> 6.65 mm
- net N$17: track 13.3 -> 17.0 mm
- net N$2: track 6.71 -> 4.96 mm
- net N$4: track 5.66 -> 4.12 mm
- net N$5: track 5.13 -> 3.60 mm
- net N$3: track 6.18 -> 4.87 mm
- net N$6: track 5.13 -> 3.82 mm
- net N$7: track 5.66 -> 4.62 mm
Other:
- board size 88.9 x 196.2 mm -> 88.9 x 142.9 mm

Commit message: vil_27
Parts:
- removed U$1, U$100, U$101, U$102, U$103, U$104, U$105, U$106, U$107, U$108, U$109, U$110, U$88, U$89, U$90, U$91, U$92, U$93, U$94, U$95, U$96, U$97, U$98, U$99: (no value), kbmx:18X18
- removed U$10, U$11, U$12, U$13, U$14, U$15, U$16, U$17, U$18, U$19, U$20, U$21, U$22, U$23, U$24, U$3, U$4, U$5, U$6, U$7, U$8, U$9: (no value), kbmxco:KEY
- removed U$111: (no value), kbmx:37X18
- removed U$2: (no value), kbmxco:NUMENTER
- removed U$26: (no value), kbmxco:SIZE132
- moved JP1 17.2 mm to (238.6, 197.2)
- moved DD3 1.27 mm to (253.0, 199.7)
- moved DD2 0.64 mm to (228.6, 194.6)
Routing:
- net N$139: track 63.6 -> 99.3 mm
- net +5V: track 57.7 -> 89.9 mm
- net REG1: track 6.33 -> 27.8 mm, vias 0 -> 2
- net N$59: track 20.6 -> 41.5 mm
- net N$140: track 84.3 -> 102.8 mm, vias 2 -> 0
- net VCC: track 68.2 -> 83.9 mm, vias 4 -> 5
- net GND: track 110.4 -> 118.0 mm
- net N$142: track 17.3 -> 15.8 mm
- net N$1: track 14.8 -> 13.5 mm
- net N$17: track 17.0 -> 15.7 mm
- net N$9: track 14.4 -> 15.7 mm
- net N$16: track 6.18 -> 7.45 mm
- net N$15: track 5.66 -> 6.93 mm
- net N$14: track 5.13 -> 6.40 mm
- net N$13: track 5.13 -> 6.40 mm
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- removed copper zone on layer 1, net GND
- removed copper zone on layer 1, net N$96
Other:
- board size 88.9 x 142.9 mm -> 51.8 x 42.5 mm
- board text removed: "1"
- board text removed: "1176-16"
- board text removed: "9"

Commit message: vil_28
Parts:
- moved R2 0.32 mm to (224.2, 223.8)
