File: PCB/keyBoard_NumPad/NumPad.sch (EAGLE design)
At the start: 125 parts, among them J1 J, J10 J, J11 J, J12 J, J13 J, J14 J, J15 J, J16 J, J17 J, J2 J, J3 J, J4 J, J5 J, J6 J, J7 J, J8 J, J9 J

Commit message: add1
Parts:
- added STAB_NEN: STAB, kbmxco:STAB
Changed lines of the file:
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@@
 <?xml version="1.0" encoding="utf-8"?>
 <!DOCTYPE eagle SYSTEM "eagle.dtd">
-<eagle version="6.3">
+<eagle version="6.4">
 <drawing>
 <settings>
@@
 <setting verticaltext="up"/>
 </settings>
-<grid distance="100" unitdist="mil" unit="mil" style="lines" multiple="1" display="yes" altdistance="0.01" altunitdist="inch" altunit="inch"/>
+<grid distance="0.1" unitdist="inch" unit="inch" style="lines" multiple="1" display="no" altdistance="0.01" altunitdist="inch" altunit="inch"/>
 <layers>
 <layer number="1" name="Top" color="4" fill="1" visible="no" active="no"/>
@@
 <layer number="131" name="tAdjust" color="7" fill="1" visible="yes" active="yes"/>
 <layer number="132" name="bAdjust" color="7" fill="1" visible="yes" active="yes"/>
+<layer number="133" name="Frame" color="13" fill="1" visible="yes" active="yes"/>
 <layer number="144" name="Drill_legend" color="7" fill="1" visible="yes" active="yes"/>
 <layer number="150" name="Notes" color="7" fill="1" visible="yes" active="yes"/>
@@
 <part name="C2" library="rcl" deviceset="C-EU" device="C1206"/>
 <part name="P+4" library="supply1" deviceset="+5V" device=""/>
+<part name="STAB_NEN" library="kbmxco" deviceset="STAB" device=""/>
 </parts>
 <sheets>
@@
 <attribute name="VALUE" x="40.64" y="121.92" size="1.778" layer="96" rot="R180"/>
 </instance>
+<instance part="STAB_NEN" gate="STAB" x="30.48" y="73.66" smashed="yes">
+<attribute name="NAME" x="25.4" y="76.2" size="1.27" layer="95"/>
+</instance>
 </instances>
